File: HW/CC_Debug/CC_Debug/mech.kicad_sch (KiCad schematic)
At the start: 4 parts

Commit message: .
Parts:
- added H4001, H4002, H4003, H4004: MountingHole, MountingHole:MountingHole_3.2mm_M3, symbol Mechanical:MountingHole
