File: HW/CC_Debug/CC_Debug/CC_Debug.kicad_sch (KiCad schematic)
At the start: 0 parts

Commit message: .
Other:
- added sheet USB2UART2 (USB2UART2.kicad_sch)
- sheet USB2UART1 ports: added UART_A_1{UART}, UART_A_2{UART}, UART_A_3{UART}, UART_A_4{UART}; removed none
Changed lines of the file:
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@@
+	(bus
+		(pts
+			(xy 91.44 93.98) (xy 101.6 93.98)
+		)
+		(stroke
+			(width 0)
+			(type default)
+		)
+	)
+	(bus
+		(pts
+			(xy 101.6 118.11) (xy 110.49 118.11)
+		)
+		(stroke
+			(width 0)
+			(type default)
+		)
+	)
 	(bus
 		(pts
@@
 		(pts
 			(xy 100.33 88.9) (xy 100.33 59.69)
+		)
+		(stroke
+			(width 0)
+			(type default)
+		)
+	)
+	(bus
+		(pts
+			(xy 101.6 93.98) (xy 101.6 118.11)
 		)
 		(stroke
@@
 			)
 			(justify right bottom)
+		)
+	)
+	(label "USB2{USB}"
+		(at 101.6 109.22 90)
+		(fields_autoplaced yes)
+		(effects
+			(font
+				(size 1.27 1.27)
+			)
+			(justify left bottom)
+		)
+	)
+	(sheet
+		(at 110.49 106.68)
+		(size 39.37 25.4)
+		(fields_autoplaced yes)
+		(stroke
+			(width 0.1524)
+			(type solid)
+		)
+		(fill
+			(color 0 0 0 0.0000)
+		)
+		(property "Sheetname" "USB2UART2"
+			(at 110.49 105.9684 0)
+			(effects
+				(font
+					(size 1.27 1.27)
+				)
+				(justify left bottom)
+			)
+		)
+		(property "Sheetfile" "USB2UART2.kicad_sch"
+			(at 110.49 132.6646 0)
+			(effects
+				(font
+					(size 1.27 1.27)
+				)
+				(justify left top)
+			)
+		)
+		(pin "USB2{USB}" input
+			(at 110.49 118.11 180)
+			(effects
+				(font
+					(size 1.27 1.27)
+				)
+				(justify left)
+			)
+		)
+		(pin "UART_B_3{UART}" bidirectional
+			(at 149.86 124.46 0)
+			(effects
+				(font
+					(size 1.27 1.27)
+				)
+				(justify right)
+			)
+		)
+		(pin "UART_B_4{UART}" bidirectional
+			(at 149.86 128.27 0)
+			(effects
+				(font
+					(size 1.27 1.27)
+				)
+				(justify right)
+			)
+		)
+		(pin "UART_B_1{UART}" bidirectional
+			(at 149.86 116.84 0)
+			(effects
+				(font
+					(size 1.27 1.27)
+				)
+				(justify right)
+			)
+		)
+		(pin "UART_B_2{UART}" bidirectional
+			(at 149.86 120.65 0)
+			(effects
+				(font
+					(size 1.27 1.27)
+				)
+				(justify right)
+			)
+		)
+		(instances
+			(project "CC_Debug"
+				(path "/333523da-fbe0-4b62-b707-15c1b23f3b41"
+					(page "6")
+				)
+			)
 		)
 	)
@@
 			)
 		)
+		(pin "UART_A_4{UART}" bidirectional
+			(at 149.86 68.58 0)
+			(effects
+				(font
+					(size 1.27 1.27)
+				)
+				(justify right)
+			)
+		)
+		(pin "UART_A_1{UART}" bidirectional
+			(at 149.86 52.07 0)
+			(effects
+				(font
+					(size 1.27 1.27)
+				)
+				(justify right)
+			)
+		)
+		(pin "UART_A_2{UART}" bidirectional
+			(at 149.86 55.88 0)
+			(effects
+				(font
+					(size 1.27 1.27)
+				)
+				(justify right)
+			)
+		)
+		(pin "UART_A_3{UART}" bidirectional
+			(at 149.86 60.96 0)
+			(effects
+				(font
+					(size 1.27 1.27)
+				)
+				(justify right)
+			)
+		)

Commit message: .
Other:
- added sheet Isolation_output (Isolation_output.kicad_sch)
- sheet USB2UART2 ports: added I2C_B_1{I2C}, I2C_B_2{I2C}; removed UART_B_1{UART}, UART_B_2{UART}
