File: HW/CC_Debug/CC_Debug/USB_CON.kicad_sch (KiCad schematic)
At the start: 2 parts, among them J3001 USB_B

Commit message: .
Changed lines of the file:
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@@
+	)
+	(bus_entry
+		(at 204.47 90.17)
+		(size -2.54 2.54)
+		(stroke
+			(width 0)
+			(type default)
+		)
 	)
 	(bus_entry
@@
 	)
 	(bus_entry
-		(at 204.47 90.17)
-		(size -2.54 2.54)
-		(stroke
-			(width 0)
-			(type default)
-		)
-	)
-	(bus_entry
 		(at 204.47 85.09)
 		(size -2.54 2.54)
@@
 	(bus
 		(pts
-			(xy 204.47 85.09) (xy 204.47 81.28)
+			(xy 204.47 78.74) (xy 217.17 78.74)
 		)
 		(stroke
@@
 	(bus
 		(pts
+			(xy 204.47 78.74) (xy 204.47 81.28)
+		)
+		(stroke
+			(width 0)
+			(type default)
+		)
+	)
+	(wire
+		(pts
+			(xy 128.27 83.82) (xy 201.93 83.82)
+		)
+		(stroke
+			(width 0)
+			(type default)
+		)
+	)
+	(bus
+		(pts
 			(xy 204.47 96.52) (xy 204.47 90.17)
 		)
@@
 	(wire
 		(pts
-			(xy 128.27 83.82) (xy 201.93 83.82)
-		)
-		(stroke
-			(width 0)
-			(type default)
-		)
-	)
-	(bus
-		(pts
-			(xy 204.47 81.28) (xy 217.17 81.28)
-		)
-		(stroke
-			(width 0)
-			(type default)
-		)
-	)
-	(wire
-		(pts
 			(xy 171.45 87.63) (xy 201.93 87.63)
 		)
@@
 			(width 0)
 			(type default)
+		)
+	)
+	(bus
+		(pts
+			(xy 204.47 81.28) (xy 204.47 85.09)
+		)
+		(stroke
+			(width 0)
+			(type default)
+		)
+	)
+	(label "USB_IN.VBUS"
+		(at 163.83 83.82 0)
+		(fields_autoplaced yes)
+		(effects
+			(font
+				(size 1.27 1.27)
+			)
+			(justify left bottom)
 		)
 	)
@@
 		)
 	)
-	(label "USB_IN.VBUS"
-		(at 128.27 83.82 0)
+	(label "VBUS"
+		(at 135.89 83.82 0)
 		(fields_autoplaced yes)
 		(effects
@@
 	(hierarchical_label "USB_IN{USB_EXT}"
 		(shape bidirectional)
-		(at 217.17 81.28 0)
-		(fields_autoplaced yes)
-		(effects
+		(at 217.17 78.74 0)
+		(fields_autoplaced yes)
+		(effects
