File: HW/CC_Debug/CC_Debug/CC USB hub.kicad_sch (KiCad schematic)
At the start: 27 parts, among them U2001 USB2514B/M2, U2002 24Mhz,50ppm

Commit message: .
Parts:
- added C2011, C2012, C2013, C2014: 10u 10V, Capacitor_SMD:C_0603_1608Metric, symbol bt_capacitor:C;M;10u;10p;10V;S;0603
- added L2001: 1uH, Inductor_SMD:L_0805_2012Metric, symbol bt_Inductors:L;1uH;3.1A;55m;S;0805
- added R2016: 22K, Resistor_SMD:R_0603_1608Metric, symbol bt_resistors:R;G;22K;10P0;S;0603
- added R2017: 430K, Resistor_SMD:R_0603_1608Metric, symbol bt_resistors:R;G;430K;10P0;S;0603
- added R2018: 100K, Resistor_SMD:R_0603_1608Metric, symbol bt_resistors:R;G;100K;10P0;S;0603
- added U2003: TPS62A01, Package_TO_SOT_SMD:SOT-23-6, symbol bt_power:TPS62A01_SOT23
Connections:
- net +3.3V: now also C2012.1, C2013.1, C2014.1, L2001.2, R2016.1
- net GND: now also C2011.2, C2012.2, C2013.2, C2014.2, R2018.2, U2003.2 (GND)
- net USB_IN.VBUS: now also C2011.1, U2003.1 (EN), U2003.4 (VIN)
- new net: R2016.2, R2017.1
- new net FB: R2017.2, R2018.1, U2003.6 (FB)
- new net SW: L2001.1, U2003.3 (SW)
Other:
- moved on the sheet: C2001, C2002, C2003, C2004, R2003, R2004, R2005, R2006, R2008, R2010, R2011, R2012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

Commit message: .
Parts:
- added TP2001: TestPoint, TestPoint:TestPoint_THTPad_D1.0mm_Drill0.5mm, symbol bt_misc:TestPoint_THD
- added TP2002: TestPoint, TestPoint:TestPoint_THTPad_1.0x1.0mm_Drill0.5mm, symbol bt_misc:TestPoint_SQU
Connections:
- net +3.3V: now also TP2001.1
- net GND: now also TP2002.1
- no-connect marks 7 -> 8
Changed lines of the file:
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@@
 	)
 	(junction
+		(at 171.45 45.72)
+		(diameter 0)
+		(color 0 0 0 0)
+	)
+	(junction
 		(at 156.21 64.77)
 		(diameter 0)
@@
 	)
 	(no_connect
+		(at 85.09 54.61)
+	)
+	(no_connect
 		(at 161.29 185.42)
 	)
@@
 		)
 	)
+	(wire
+		(pts
+			(xy 179.07 73.66) (xy 179.07 78.74)
+		)
+		(stroke
+			(width 0)
+			(type default)
+		)
+	)
 	(bus
 		(pts
@@
 	)
 	(symbol
+		(lib_id "bt_misc:TestPoint_SQU")
+		(at 179.07 73.66 0)
+		(unit 1)
+		(exclude_from_sim no)
+		(in_bom yes)
+		(on_board yes)
+		(dnp no)
+		(fields_autoplaced yes)
+		(property "Reference" "TP2002"
+			(at 181.61 73.6599 0)
+			(effects
+				(font
+					(size 1.27 1.27)
+				)
+				(justify left)
+			)
+		)
+		(property "Value" "TestPoint"
+			(at 179.07 71.628 0)
+			(effects
+				(font
+					(size 1.27 1.27)
+				)
+				(hide yes)
+			)
+		)
+		(property "Footprint" "TestPoint:TestPoint_THTPad_1.0x1.0mm_Drill0.5mm"
+			(at 184.404 77.724 0)
+			(effects
+				(font
+					(size 1.27 1.27)
+				)
+				(hide yes)
+			)
+		)
+		(property "Datasheet" "~"
+			(at 184.15 73.66 0)
+			(effects
+				(font
+					(size 1.27 1.27)
+				)
+				(hide yes)
+			)
+		)
+		(property "Description" "test point"
+			(at 172.466 75.184 0)
+			(effects
+				(font
+					(size 1.27 1.27)
+				)
+				(hide yes)
+			)
+		)
+		(pin "1"
+		)
+		(instances
+			(project "CC_Debug"
+				(path "/333523da-fbe0-4b62-b707-15c1b23f3b41/31542dab-9c61-4595-8293-40a7ee8bdc51"
+					(reference "TP2002")
+					(unit 1)
+				)
+			)
+		)
+	)
+	(symbol
 		(lib_id "bt_resistors:R;G;100K;10P0;S;0603")
 		(at 123.19 140.97 90)
@@
 	)
 	(symbol
+		(lib_id "bt_misc:TestPoint_THD")
+		(at 171.45 45.72 0)
+		(unit 1)
+		(exclude_from_sim no)
+		(in_bom yes)
+		(on_board yes)
+		(dnp no)
+		(fields_autoplaced yes)
+		(property "Reference" "TP2001"
+			(at 173.99 45.7199 0)
+			(effects
+				(font
+					(size 1.27 1.27)
+				)
+				(justify left)
+			)
+		)
+		(property "Value" "TestPoint"
+			(at 171.45 43.688 0)
+			(effects
+				(font
+					(size 1.27 1.27)
+				)
+				(hide yes)
+			)
+		)
+		(property "Footprint" "TestPoint:TestPoint_THTPad_D1.0mm_Drill0.5mm"
+			(at 176.784 49.784 0)
+			(effects
+				(font
+					(size 1.27 1.27)
+				)
+				(hide yes)
+			)
+		)
+		(property "Datasheet" "~"
+			(at 176.53 45.72 0)
+			(effects
+				(font
+					(size 1.27 1.27)
+				)
+				(hide yes)
+			)
+		)
+		(property "Description" "test point"
+			(at 164.846 47.244 0)
+			(effects
+				(font
+					(size 1.27 1.27)
+				)
+				(hide yes)
+			)
+		)
+		(pin "1"
+		)
+		(instances
+			(project "CC_Debug"
+				(path "/333523da-fbe0-4b62-b707-15c1b23f3b41/31542dab-9c61-4595-8293-40a7ee8bdc51"
+					(reference "TP2001")
+					(unit 1)
+				)
+			)
+		)
+	)
+	(symbol
 		(lib_id "bt_resistors:R;G;100K;10P0;S;0603")
 		(at 38.1 264.16 0)
@@
 					(unit 1)
 				)
+			)
+		)
+	)
+	(symbol
+		(lib_id "power:GND")
+		(at 179.07 78.74 0)
+		(unit 1)
+		(exclude_from_sim no)
+		(in_bom yes)
+		(on_board yes)
+		(dnp no)
+		(fields_autoplaced yes)
+		(property "Reference" "#PWR02025"
+			(at 179.07 85.09 0)
+			(effects
+				(font
+					(size 1.27 1.27)
+				)
+				(hide yes)
+			)
+		)
+		(property "Value" "GND"
+			(at 179.07 83.82 0)
+			(effects
+				(font
+					(size 1.27 1.27)
+				)
+			)
+		)
+		(property "Footprint" ""
+			(at 179.07 78.74 0)
+			(effects
+				(font
+					(size 1.27 1.27)
+				)
+				(hide yes)
+			)
+		)
+		(property "Datasheet" ""
+			(at 179.07 78.74 0)
+			(effects
+				(font
+					(size 1.27 1.27)
+				)
+				(hide yes)
+			)
+		)
+		(property "Description" "Power symbol creates a global label with name \"GND\" , ground"
+			(at 179.07 78.74 0)
+			(effects
+				(font
+					(size 1.27 1.27)
+				)
+				(hide yes)
+			)
+		)
+		(pin "1"
+		)
+		(instances
+			(project "CC_Debug"
+				(path "/333523da-fbe0-4b62-b707-15c1b23f3b41/31542dab-9c61-4595-8293-40a7ee8bdc51"
+					(reference "#PWR02025")
+					(unit 1)
+				)
