File: HW/CC_Debug/CC_Debug/Debug_connector.kicad_sch (KiCad schematic)
At the start: 1 part, among them J8001 62684-401100ALF

Commit message: .
Parts:
- added D8001, D8002, D8003, D8004, D8005: LED, LED_SMD:LED_0603_1608Metric, symbol Device:LED
- added J8002, J8003, J8004, J8005, J8006: Conn_02x10_Odd_Even, Connector_IDC:IDC-Header_2x10_P2.54mm_Vertical, symbol Connector_Generic:Conn_02x10_Odd_Even
- added J8007, J8008: Conn_02x05_Odd_Even, Connector_IDC:IDC-Header_2x05_P2.54mm_Vertical, symbol Connector_Generic:Conn_02x05_Odd_Even
- added Q8001, Q8002, Q8003, Q8004, Q8005: BSS138, Package_TO_SOT_SMD:SOT-23, symbol bt_transistor:T;Mn;BSS138;SOT23
- added R8001, R8002, R8003, R8004, R8005, R8006, R8007, R8008, R8009, R8010, R8011, R8012, R8013, R8014, R8015, R8016, R8017, R8018, R8019, R8020, R8021, R8022, R8023, R8024, R8025, R8026, R8027, R8028, R8029, R8030, R8034, R8035: 10K, Resistor_SMD:R_0603_1608Metric, symbol bt_resistors:R;G;10K;10P0;S;0603
- added R8031, R8032, R8033, R8036, R8037: 510R, Resistor_SMD:R_0603_1608Metric, symbol bt_resistors:R;G;510R;10P0;S;0603
- added SW8001, SW8002, SW8003, SW8004, SW8005, SW8006, SW8007, SW8008, SW8009: M;SW;3;SPST, bt_footprints:SW_DS04-254-2-03BK-SMT, symbol bt_misc:M;SW;3;SPST;S
Connections:
- net FORCE#: now reaches J8001.01
- net FORCE#: now also SW8002.4
- net E_RESET#: now reaches J8001.02
- net E_RESET#: now also J8006.15 (Pin_15)
- net E_TRST#: now reaches J8001.03
- net E_TRST#: now also J8006.3 (Pin_3)
- net E_TCK: now reaches J8001.04
- net E_TCK: now also J8006.9 (Pin_9)
- net E_TMS: now reaches J8001.05
- net E_TMS: now also J8006.7 (Pin_7)
- net E_TDO: now reaches J8001.06
- net E_TDO: now also J8006.13 (Pin_13)
- net E_TDI: now reaches J8001.07
- net E_TDI: now also J8006.5 (Pin_5)
- net GND2: now reaches J8001.08
- net GND2: now also J8001.16, J8001.23, J8001.30, J8001.37, J8001.S1, J8001.S2, J8002.10 (Pin_10), J8002.12 (Pin_12), J8002.14 (Pin_14), J8002.16 (Pin_16), J8002.18 (Pin_18), J8002.20 (Pin_20), J8002.4 (Pin_4), J8002.6 (Pin_6), J8002.8 (Pin_8), J8003.10 (Pin_10), J8003.12 (Pin_12), J8003.14 (Pin_14), J8003.16 (Pin_16), J8003.18 (Pin_18), J8003.20 (Pin_20), J8003.4 (Pin_4), J8003.6 (Pin_6), J8003.8 (Pin_8), J8004.10 (Pin_10), J8004.12 (Pin_12), J8004.14 (Pin_14), J8004.16 (Pin_16), J8004.18 (Pin_18), J8004.20 (Pin_20), J8004.4 (Pin_4), J8004.6 (Pin_6), J8004.8 (Pin_8), J8005.10 (Pin_10), J8005.12 (Pin_12), J8005.14 (Pin_14), J8005.16 (Pin_16), J8005.18 (Pin_18), J8005.20 (Pin_20), J8005.4 (Pin_4), J8005.6 (Pin_6), J8005.8 (Pin_8), J8006.10 (Pin_10), J8006.12 (Pin_12), J8006.14 (Pin_14), J8006.16 (Pin_16), J8006.18 (Pin_18), J8006.20 (Pin_20), J8006.4 (Pin_4), J8006.6 (Pin_6), J8006.8 (Pin_8), J8007.10 (Pin_10), J8007.2 (Pin_2), J8008.10 (Pin_10), J8008.2 (Pin_2), Q8001.2 (S), Q8002.2 (S), Q8003.2 (S), Q8004.2 (S), Q8005.2 (S), R8001.1, R8002.1, R8003.1, R8004.1, R8005.1, R8006.1, R8007.1, R8008.1, R8009.1, R8010.1, R8011.1, R8012.1, R8013.1, R8014.1, R8015.1, R8016.1, R8017.1, R8018.1, R8019.1, R8020.1, R8021.1, R8022.1, R8023.1, R8024.1, R8025.1, R8026.1, R8027.1, R8028.1, R8029.1, R8030.1, R8034.1, R8035.1, SW8002.3
- net E_VCC: now reaches J8001.09
- net E_VCC: now also J8006.1 (Pin_1), J8006.2 (Pin_2), Q8003.1 (G), R8030.2, SW8003.6
- net E_RX: now reaches J8001.10
- net E_RX: now also SW8003.5
- net E_TX: now reaches J8001.11
- net E_TX: now also SW8003.4
- net D_IO/F_VCC: now reaches J8001.12
- net D_IO/F_VCC: now also J8007.3 (Pin_3), SW8001.6, SW8008.6
- net D_RESET#: now reaches J8001.13
- net D_RESET#: now also J8005.15 (Pin_15), J8007.1 (Pin_1), SW8008.5
- net D_SWCLK: now reaches J8001.14
- net D_SWCLK: now also J8005.9 (Pin_9), J8008.1 (Pin_1), SW8001.5, SW8009.5
- net D_SWDIO: now reaches J8001.15
- net D_SWDIO: now also J8005.7 (Pin_7), J8008.3 (Pin_3), SW8001.4, SW8009.4
- net D_VCC: now reaches J8001.17
- net D_VCC: now also J8005.1 (Pin_1), J8005.2 (Pin_2), Q8005.1 (G), R8035.2, SW8004.6, SW8008.4, SW8009.6
- net D_RX: now reaches J8001.18
- net D_RX: now also SW8004.5
- net D_TX: now reaches J8001.19
- net D_TX: now also SW8004.4
- net C_RESET#: now reaches J8001.20
- net C_RESET#: now also J8004.15 (Pin_15)
- net C_SWCLK: now reaches J8001.21
- net C_SWCLK: now also J8004.9 (Pin_9)
- net C_SWDIO: now reaches J8001.22
- net C_SWDIO: now also J8004.7 (Pin_7)
- net C_VCC: now reaches J8001.24
- net C_VCC: now also J8004.1 (Pin_1), J8004.2 (Pin_2), Q8002.1 (G), R8029.2, SW8005.6
- net C_RX: now reaches J8001.25
- net C_RX: now also SW8005.5
- net C_TX: now reaches J8001.26
- net C_TX: now also SW8005.4
- net B_RESET#: now reaches J8001.27
- net B_RESET#: now also J8003.15 (Pin_15)
- net B_SWCLK: now reaches J8001.28
- net B_SWCLK: now also J8003.9 (Pin_9)
- net B_SWDIO: now reaches J8001.29
- net B_SWDIO: now also J8003.7 (Pin_7)
- net B_VCC: now reaches J8001.31
- net B_VCC: now also J8003.1 (Pin_1), J8003.2 (Pin_2), Q8004.1 (G), R8034.2, SW8006.6
- net B_RX: now reaches J8001.32
- net B_RX: now also SW8006.5
- net B_TX: now reaches J8001.33
- net B_TX: now also SW8006.4
- net A_RESET#: now reaches J8001.34
- net A_RESET#: now also J8002.15 (Pin_15)
- net A_SWCLK: now reaches J8001.35
- net A_SWCLK: now also J8002.9 (Pin_9)
- net A_SWDIO: now reaches J8001.36
- net A_SWDIO: now also J8002.7 (Pin_7)
- net A_VCC: now reaches J8001.38
- net A_VCC: now also J8002.1 (Pin_1), J8002.2 (Pin_2), Q8001.1 (G), R8028.2, SW8007.6
- net A_RX: now reaches J8001.39
- net A_RX: now also SW8007.5
- net A_TX: now reaches J8001.40
- net A_TX: now also SW8007.4
- new net: D8003.2 (A), R8033.2
- new net: D8003.1 (K), Q8003.3 (D)
- new net: D8005.1 (K), Q8005.3 (D)
- new net: D8005.2 (A), R8037.2
- new net: D8001.2 (A), R8031.2
- new net: D8004.2 (A), R8036.2
- new net: D8002.2 (A), R8032.2
- new net: D8002.1 (K), Q8002.3 (D)
- new net: D8001.1 (K), Q8001.3 (D)
- new net: D8004.1 (K), Q8004.3 (D)
- new net A_DBACK: J8002.19 (Pin_19), R8003.2
- new net A_DBRQ: J8002.17 (Pin_17), R8017.2
- new net A_RTCK: J8002.11 (Pin_11), R8016.2
- new net A_TDI: J8002.5 (Pin_5), R8001.2
- new net A_TDO: J8002.13 (Pin_13), R8002.2
- new net A_TRST#: J8002.3 (Pin_3), R8015.2
- new net B_DBACK: J8003.19 (Pin_19), R8006.2
- new net B_DBRQ: J8003.17 (Pin_17), R8020.2
- new net B_RTCK: J8003.11 (Pin_11), R8019.2
- new net B_TDI: J8003.5 (Pin_5), R8004.2
- new net B_TDO: J8003.13 (Pin_13), R8005.2
- new net B_TRST#: J8003.3 (Pin_3), R8018.2
- new net C_DBACK: J8004.19 (Pin_19), R8009.2
- new net C_DBRQ: J8004.17 (Pin_17), R8023.2
- new net C_RTCK: J8004.11 (Pin_11), R8022.2
- new net C_TDI: J8004.5 (Pin_5), R8007.2
- new net C_TDO: J8004.13 (Pin_13), R8008.2
- new net C_TRST#: J8004.3 (Pin_3), R8021.2
- new net D_DBACK: J8005.19 (Pin_19), R8012.2
- new net D_DBRQ: J8005.17 (Pin_17), R8026.2
- new net D_RTCK: J8005.11 (Pin_11), R8025.2
- new net D_TDI: J8005.5 (Pin_5), R8010.2
- new net D_TDO: J8005.13 (Pin_13), R8011.2
- new net D_TRST#: J8005.3 (Pin_3), R8024.2
- new net E_DBACK: J8006.19 (Pin_19), R8014.2
- new net E_DBRQ: J8006.17 (Pin_17), R8027.2
- new net E_RTCK: J8006.11 (Pin_11), R8013.2
- new net I2C1.SCL: SW8009.2
- new net I2C1.SDA: SW8009.3
- new net I2C2.SCL: SW8008.2
- new net I2C2.SDA: SW8008.1
- new net SW_A.RX: SW8007.2
- new net SW_A.TX: SW8007.3
- new net SW_A_VCC: SW8007.1
- new net SW_B.RX: SW8006.2
- new net SW_B.TX: SW8006.3
- new net SW_B_VCC: SW8006.1
- new net SW_C.RX: SW8005.2
- new net SW_C.TX: SW8005.3
- new net SW_C_VCC: SW8005.1
- new net SW_D.RX: SW8004.2
- new net SW_D.TX: SW8004.3
- new net SW_D_I2C1_VCC: SW8009.1
- new net SW_D_I2C2_VCC: SW8008.3
- new net SW_D_VCC: SW8004.1
- new net SW_E.RX: SW8003.2
- new net SW_E.TX: SW8003.3
- new net SW_E_VCC: SW8003.1
- new net SW_F.RX: SW8001.2
- new net SW_F.TX: SW8001.3
- new net SW_F_VCC: SW8001.1
- new net VCC_LED: R8031.1, R8032.1, R8033.1, R8036.1, R8037.1
- no-connect marks 0 -> 16
Other:
- moved on the sheet: J8001
