File: HW/CC_Debug/CC_Debug/USB2UART2.kicad_sch (KiCad schematic)
At the start: 31 parts, among them U5001 12Mhz,50ppm, U5002 FT4232H_QFN, U5003 93AA46BT-I/OT

Commit message: .
Parts:
- removed C5001, C5002, C5003, C5004, C5005, C5006, C5007, C5008, C5009, C5011, C5012: 100n 25V, Capacitor_SMD:C_0603_1608Metric, symbol bt_capacitor:C;M;100n;10p;25V;S;0603
- removed C5010, C5013, C5014: 10u 10V, Capacitor_SMD:C_0603_1608Metric, symbol bt_capacitor:C;M;10u;10p;10V;S;0603
- removed D5001: LED, LED_SMD:LED_0603_1608Metric, symbol Device:LED
- removed R5001, R5003, R5004: 10K, Resistor_SMD:R_0603_1608Metric, symbol bt_resistors:R;G;10K;10P0;S;0603
- removed R5002: 12K, Resistor_SMD:R_0603_1608Metric, symbol bt_resistors:R;G;12K;10P0;S;0603
- removed R5005: 2K2, Resistor_SMD:R_0603_1608Metric, symbol bt_resistors:R;G;2K2;10P0;S;0603
- removed R5006: 510R, Resistor_SMD:R_0603_1608Metric, symbol bt_resistors:R;G;510R;10P0;S;0603
- removed TP5001, TP5002, TP5004, TP5005, TP5007: TestPoint, TestPoint:TestPoint_THTPad_D1.0mm_Drill0.5mm, symbol bt_misc:TestPoint_THD
- removed TP5003, TP5006: TestPoint, TestPoint:TestPoint_THTPad_1.0x1.0mm_Drill0.5mm, symbol bt_misc:TestPoint_SQU
- removed U5001: 12Mhz,50ppm, Oscillator:Oscillator_SMD_SeikoEpson_SG8002CE-4Pin_3.2x2.5mm, symbol bt_oscillator:OSC;12Mhz;50ppm;3v3;SG3225CAN
- removed U5002: FT4232H_QFN, Package_DFN_QFN:QFN-64-1EP_9x9mm_P0.5mm_EP4.35x4.35mm, symbol bt_communication:FT4232H_QFN
- removed U5003: 93AA46BT-I/OT, Package_TO_SOT_SMD:SOT-23-6, symbol bt_memory:93AA46BT-I/OT
- added C6001, C6002, C6003, C6004, C6005, C6007, C6008, C6010, C6011, C6012, C6013: 100n 25V, Capacitor_SMD:C_0603_1608Metric, symbol bt_capacitor:C;M;100n;10p;25V;S;0603
- added C6006, C6009, C6014: 10u 10V, Capacitor_SMD:C_0603_1608Metric, symbol bt_capacitor:C;M;10u;10p;10V;S;0603
- added D6001: LED, LED_SMD:LED_0201_0603Metric, symbol Device:LED
- added R6001, R6002, R6005: 10K, Resistor_SMD:R_0603_1608Metric, symbol bt_resistors:R;G;10K;10P0;S;0603
- added R6003: 2K2, Resistor_SMD:R_0603_1608Metric, symbol bt_resistors:R;G;2K2;10P0;S;0603
- added R6004: 12K, Resistor_SMD:R_0603_1608Metric, symbol bt_resistors:R;G;12K;10P0;S;0603
- added R6006: 510R, Resistor_SMD:R_0603_1608Metric, symbol bt_resistors:R;G;510R;10P0;S;0603
- added U6001: 93AA46BT-I/OT, Package_TO_SOT_SMD:SOT-23-6, symbol bt_memory:93AA46BT-I/OT
- added U6002: 12Mhz,50ppm, Oscillator:Oscillator_SMD_SeikoEpson_SG8002CE-4Pin_3.2x2.5mm, symbol bt_oscillator:OSC;12Mhz;50ppm;3v3;SG3225CAN
- added U6003: FT4232H_QFN, Package_DFN_QFN:QFN-64-1EP_9x9mm_P0.5mm_EP4.35x4.35mm, symbol bt_communication:FT4232H_QFN
Connections:
- net +1V8A: now also C6002.1, C6003.1, C6005.1, C6014.1, U6003.12 (VCORE), U6003.37 (VCORE), U6003.49 (VREGOUT), U6003.64 (VCORE)
- net +3.3V: now also C6001.1, C6004.1, C6006.1, C6007.1, C6008.1, C6009.1, C6010.1, C6011.1, C6012.1, C6013.1, D6001.2 (A), R6001.2, R6002.1, R6005.2, U6001.6 (VCC), U6002.4 (Vcc), U6003.20 (VCCIO), U6003.31 (VCCIO), U6003.4 (VPHY), U6003.42 (VCCIO), U6003.50 (VREGIN), U6003.56 (VCCIO), U6003.9 (VPLL)
- net 12Mhz: now also U6002.3 (OUT), U6003.2 (OSCI)
- net EECLK: now also U6001.4 (CLK), U6003.62 (EECLK)
- net EECS: now also U6001.5 (CS), U6003.63 (EECS)
- net EEDATA: now also R6003.2, U6001.3 (DI), U6003.61 (EEDATA)
- net EEDATA_OUT: now also R6001.1, R6003.1, U6001.1 (DO)
- net GND: now also C6001.2, C6002.2, C6003.2, C6004.2, C6005.2, C6006.2, C6007.2, C6008.2, C6009.2, C6010.2, C6011.2, C6012.2, C6013.2, C6014.2, R6004.2, U6001.2 (GND), U6002.2 (GND), U6003.1 (GND), U6003.10 (AGND), U6003.11 (GND), U6003.13 (TEST), U6003.15 (GND), U6003.25 (GND), U6003.35 (GND), U6003.47 (GND), U6003.5 (GND), U6003.51 (GND)
- net USB1.D+: now also U6003.8 (DP)
- net USB1.D-: now also U6003.7 (DM)
- new net: R6005.1, U6003.14 (~{RESET})
- new net: D6001.1 (K), R6006.2
- new net: R6004.1, U6003.6 (REF)
- new net: R6006.1, U6003.60 (~{PWREN})
- new net: R6002.2, U6002.1 (ST#)
- new net UART_B_1.RX: U6003.17 (ADBUS1), U6003.18 (ADBUS2)
- new net UART_B_1.TX: U6003.16 (ADBUS0), U6003.26 (BDBUS0), U6003.38 (CDBUS0)
- new net UART_B_2.RX: U6003.27 (BDBUS1), U6003.28 (BDBUS2)
- new net UART_B_3.RX: U6003.39 (CDBUS1)
- new net UART_B_4.RX: U6003.52 (DDBUS1)
- new net UART_B_4.TX: U6003.48 (DDBUS0)

Commit message: .
Parts:
- added C6015: 100n 25V, Capacitor_SMD:C_0603_1608Metric, symbol bt_capacitor:C;M;100n;10p;25V;S;0603
- added TP6001, TP6002, TP6003, TP6004, TP6005: TestPoint, TestPoint:TestPoint_THTPad_D1.0mm_Drill0.5mm, symbol bt_misc:TestPoint_THD
- D6001: footprint LED_SMD:LED_0201_0603Metric -> LED_SMD:LED_0603_1608Metric
Connections:
- net +3.3V: now also C6015.1
- net EECLK: now also TP6003.1
- net EECS: now also TP6001.1
- net EEDATA: now also TP6004.1
- net EEDATA_OUT: now also TP6002.1
- net GND: now also U6003.65 (EP), C6015.2
- net at R6005.1, U6003.14 (~{RESET}): now also TP6005.1
- net +1V8A renamed +1V8B
- net UART_B_1.RX renamed I2C_B_1.SDA
- removed net UART_B_1.TX: U6003.16 (ADBUS0), U6003.26 (BDBUS0), U6003.38 (CDBUS0)
- net UART_B_2.RX renamed I2C_B_2.SDA
- new net I2C_B_1.SCL: U6003.16 (ADBUS0)
- new net I2C_B_2.SCL: U6003.26 (BDBUS0)
- new net UART_B_3.TX: U6003.38 (CDBUS0)

Commit message: .
Parts:
- added TP6006, TP6007: TestPoint, TestPoint:TestPoint_THTPad_1.0x1.0mm_Drill0.5mm, symbol bt_misc:TestPoint_SQU
Connections:
- net GND: now also TP6006.1, TP6007.1
- no-connect marks 0 -> 24
