File: HW/CC_Debug/CC_Debug/usb2uart.kicad_sch (KiCad schematic)
At the start: 31 parts, among them U5001 12Mhz,50ppm, U5002 FT4232H_QFN, U5003 93AA46BT-I/OT

Commit message: .
Parts:
- added C5015: 100n 25V, Capacitor_SMD:C_0603_1608Metric, symbol bt_capacitor:C;M;100n;10p;25V;S;0603
Connections:
- net +3.3V: now also C5015.1
- net GND: now also U5002.65 (EP), C5015.2
- net UART_A_1.TX: no longer U5002.26 (BDBUS0), U5002.38 (CDBUS0)
- new net UART_A_2.TX: U5002.26 (BDBUS0)
- new net UART_A_3.TX: U5002.38 (CDBUS0)
Changed lines of the file:
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@@
 	)
 	(junction
+		(at 196.85 205.74)
+		(diameter 0)
+		(color 0 0 0 0)
+	)
+	(junction
 		(at 96.52 82.55)
 		(diameter 0)
@@
 	)
 	(junction
+		(at 269.24 45.72)
+		(diameter 0)
+		(color 0 0 0 0)
+	)
+	(junction
 		(at 92.71 237.49)
 		(diameter 0)
@@
 	)
 	(junction
+		(at 269.24 64.77)
+		(diameter 0)
+		(color 0 0 0 0)
+	)
+	(junction
 		(at 114.3 234.95)
 		(diameter 0)
@@
 	(wire
 		(pts
+			(xy 203.2 196.85) (xy 203.2 205.74)
+		)
+		(stroke
+			(width 0)
+			(type default)
+		)
+	)
+	(wire
+		(pts
 			(xy 303.53 45.72) (xy 320.04 45.72)
 		)
@@
 	(wire
 		(pts
+			(xy 255.27 59.69) (xy 255.27 64.77)
+		)
+		(stroke
+			(width 0)
+			(type default)
+		)
+	)
+	(wire
+		(pts
 			(xy 194.31 87.63) (xy 194.31 78.74)
 		)
@@
 		)
 	)
+	(wire
+		(pts
+			(xy 255.27 64.77) (xy 269.24 64.77)
+		)
+		(stroke
+			(width 0)
+			(type default)
+		)
+	)
 	(bus
 		(pts
@@
 	(wire
 		(pts
+			(xy 269.24 45.72) (xy 255.27 45.72)
+		)
+		(stroke
+			(width 0)
+			(type default)
+		)
+	)
+	(wire
+		(pts
+			(xy 196.85 205.74) (xy 203.2 205.74)
+		)
+		(stroke
+			(width 0)
+			(type default)
+		)
+	)
+	(wire
+		(pts
 			(xy 134.62 163.83) (xy 158.75 163.83)
 		)
@@
 	(wire
 		(pts
+			(xy 255.27 45.72) (xy 255.27 52.07)
+		)
+		(stroke
+			(width 0)
+			(type default)
+		)
+	)
+	(wire
+		(pts
 			(xy 181.61 205.74) (xy 184.15 205.74)
 		)
@@
 		)
 	)
-	(label "UART_A_1.TX"
+	(label "UART_A_3.TX"
 		(at 260.35 140.97 0)
 		(fields_autoplaced yes)
@@
 		)
 	)
-	(label "UART_A_1.TX"
+	(label "UART_A_2.TX"
 		(at 260.35 118.11 0)
 		(fields_autoplaced yes)
@@
 	)
 	(symbol
+		(lib_id "bt_capacitor:C;M;100n;10p;25V;S;0603")
+		(at 255.27 55.88 0)
+		(unit 1)
+		(exclude_from_sim no)
+		(in_bom yes)
+		(on_board yes)
+		(dnp no)
+		(fields_autoplaced yes)
+		(property "Reference" "C5015"
+			(at 259.08 54.6099 0)
+			(effects
+				(font
+					(size 1.27 1.27)
+				)
+				(justify left)
+			)
+		)
+		(property "Value" "100n 25V"
+			(at 259.08 57.1499 0)
+			(effects
+				(font
+					(size 1.27 1.27)
+				)
+				(justify left)
+			)
+		)
+		(property "Footprint" "Capacitor_SMD:C_0603_1608Metric"
+			(at 252.492 55.88 90)
+			(effects
+				(font
+					(size 1.27 1.27)
+				)
+				(hide yes)
+			)
+		)
+		(property "Datasheet" "~"
+			(at 255.27 55.88 0)
+			(effects
+				(font
+					(size 1.27 1.27)
+				)
+				(hide yes)
+			)
+		)
+		(property "Description" "Capacitor"
+			(at 255.27 55.88 0)
+			(effects
+				(font
+					(size 1.27 1.27)
+				)
+				(hide yes)
+			)
+		)
+		(property "MPN" "C;C;T1;S;P0603;NA"
+			(at 259.27 55.88 90)
+			(effects
+				(font
+					(size 1.27 1.27)
+				)
+				(hide yes)
+			)
+		)
+		(property "CPN" "BT00008-090680"
+			(at 259.27 55.88 90)
+			(effects
+				(font
+					(size 1.27 1.27)
+				)
+				(hide yes)
+			)
+		)
+		(pin "2"
+		)
+		(pin "1"
+		)
+		(instances
+			(project "CC_Debug"
+				(path "/333523da-fbe0-4b62-b707-15c1b23f3b41/94c11654-df98-40df-80fb-fde9e439ebc2"
+					(reference "C5015")
+					(unit 1)
+				)
+			)
+		)
+	)
+	(symbol
 		(lib_id "power:+3.3V")
 		(at 67.31 222.25 0)
@@
 		(pin "9"
 		)
+		(pin "65"
+		)
 		(instances

Commit message: .
Connections:
- no-connect marks 0 -> 26
Changed lines of the file:
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@@
 		(color 0 0 0 0)
+	)
+	(no_connect
+		(at 158.75 184.15)
+	)
+	(no_connect
+		(at 219.71 107.95)
+	)
+	(no_connect
+		(at 219.71 100.33)
+	)
+	(no_connect
+		(at 219.71 153.67)
+	)
+	(no_connect
+		(at 219.71 151.13)
+	)
+	(no_connect
+		(at 219.71 156.21)
+	)
+	(no_connect
+		(at 219.71 125.73)
+	)
+	(no_connect
+		(at 219.71 105.41)
+	)
+	(no_connect
+		(at 219.71 171.45)
+	)
+	(no_connect
+		(at 219.71 158.75)
+	)
+	(no_connect
+		(at 219.71 148.59)
+	)
+	(no_connect
+		(at 219.71 102.87)
+	)
+	(no_connect
+		(at 219.71 110.49)
+	)
+	(no_connect
+		(at 219.71 168.91)
+	)
+	(no_connect
+		(at 219.71 146.05)
+	)
+	(no_connect
+		(at 219.71 181.61)
+	)
+	(no_connect
+		(at 219.71 179.07)
+	)
+	(no_connect
+		(at 219.71 189.23)
+	)
+	(no_connect
+		(at 219.71 173.99)
+	)
+	(no_connect
+		(at 219.71 176.53)
+	)
+	(no_connect
+		(at 219.71 133.35)
+	)
+	(no_connect
+		(at 219.71 123.19)
+	)
+	(no_connect
+		(at 219.71 130.81)
+	)
+	(no_connect
+		(at 219.71 135.89)
+	)
+	(no_connect
+		(at 219.71 128.27)
+	)
+	(no_connect
+		(at 219.71 113.03)
 	)
 	(bus_entry
