File: HW/CC_Debug/CC_Debug/CC_Debug.kicad_pcb (KiCad board)
At the start: 2 copper layers, 46 parts, among them J3001 USB_B, U2001 USB2514B/M2, U2002 24Mhz,50ppm, U5001 12Mhz,50ppm, U5002 FT4232H_QFN

Commit message: .
Parts:
- added C5009: 100n 25V, Capacitor_SMD:C_0603_1608Metric, F.Cu at (148.7, 120.8)
- added C5010: 10u 10V, Capacitor_SMD:C_0603_1608Metric, F.Cu at (132.9, 114.6)
- added C5011: 100n 25V, Capacitor_SMD:C_0603_1608Metric, F.Cu at (130.7, 117.8)
- added C5012: 100n 25V, Capacitor_SMD:C_0603_1608Metric, F.Cu at (133.1, 117.7)
- added C5013: 10u 10V, Capacitor_SMD:C_0603_1608Metric, F.Cu at (131.4, 114.7)
- added C5014: 10u 10V, Capacitor_SMD:C_0603_1608Metric, F.Cu at (137.9, 129.4)
- added C6001: 100n 25V, Capacitor_SMD:C_0603_1608Metric, F.Cu at (134.9, 71.4)
- added C6002: 100n 25V, Capacitor_SMD:C_0603_1608Metric, F.Cu at (134.9, 73.9)
- added C6003: 100n 25V, Capacitor_SMD:C_0603_1608Metric, F.Cu at (134.9, 76.5)
- added C6004: 100n 25V, Capacitor_SMD:C_0603_1608Metric, F.Cu at (134.9, 79.0)
- added C6005: 100n 25V, Capacitor_SMD:C_0603_1608Metric, F.Cu at (134.9, 81.5)
- added C6006: 10u 10V, Capacitor_SMD:C_0603_1608Metric, F.Cu at (134.9, 84.0)
- added C6007: 100n 25V, Capacitor_SMD:C_0603_1608Metric, F.Cu at (134.9, 86.5)
- added C6008: 100n 25V, Capacitor_SMD:C_0603_1608Metric, F.Cu at (138.9, 71.4)
- added C6009: 10u 10V, Capacitor_SMD:C_0603_1608Metric, F.Cu at (138.9, 73.9)
- added C6010: 100n 25V, Capacitor_SMD:C_0603_1608Metric, F.Cu at (138.9, 76.5)
- added C6011: 100n 25V, Capacitor_SMD:C_0603_1608Metric, F.Cu at (138.9, 79.0)
- added C6012: 100n 25V, Capacitor_SMD:C_0603_1608Metric, F.Cu at (138.9, 81.5)
- added C6013: 100n 25V, Capacitor_SMD:C_0603_1608Metric, F.Cu at (138.9, 84.0)
- added C6014: 10u 10V, Capacitor_SMD:C_0603_1608Metric, F.Cu at (174.2, 69.3)
- added D5001: LED, LED_SMD:LED_0603_1608Metric, F.Cu at (144.6, 126.1)
- added D6001: LED, LED_SMD:LED_0201_0603Metric, F.Cu at (165.8, 95.5)
- added H4001: MountingHole, MountingHole:MountingHole_3.2mm_M3, F.Cu at (239.3, 69.8)
- added H4002: MountingHole, MountingHole:MountingHole_3.2mm_M3, F.Cu at (239.0, 135.1)
- added H4003: MountingHole, MountingHole:MountingHole_3.2mm_M3, F.Cu at (91.2, 67.6)
- added H4004: MountingHole, MountingHole:MountingHole_3.2mm_M3, F.Cu at (91.2, 137.2)
- added R5004: 10K, Resistor_SMD:R_0603_1608Metric, F.Cu at (144.7, 119.0)
- added R5005: 2K2, Resistor_SMD:R_0603_1608Metric, F.Cu at (141.9, 122.5)
- added R5006: 510R, Resistor_SMD:R_0603_1608Metric, F.Cu at (141.0, 126.1)
- added R6001: 10K, Resistor_SMD:R_0603_1608Metric, F.Cu at (138.9, 86.5)
- added R6002: 10K, Resistor_SMD:R_0603_1608Metric, F.Cu at (142.9, 71.4)
- added R6003: 2K2, Resistor_SMD:R_0603_1608Metric, F.Cu at (142.9, 73.9)
- added R6004: 12K, Resistor_SMD:R_0603_1608Metric, F.Cu at (142.9, 76.5)
- added R6005: 10K, Resistor_SMD:R_0603_1608Metric, F.Cu at (142.9, 79.0)
- added R6006: 510R, Resistor_SMD:R_0603_1608Metric, F.Cu at (142.9, 81.5)
- added TP5001: TestPoint, TestPoint:TestPoint_THTPad_D1.0mm_Drill0.5mm, F.Cu at (148.4, 122.8)
- added TP5002: TestPoint, TestPoint:TestPoint_THTPad_D1.0mm_Drill0.5mm, F.Cu at (141.8, 120.0)
- added TP5003: TestPoint, TestPoint:TestPoint_THTPad_1.0x1.0mm_Drill0.5mm, F.Cu at (149.6, 125.0)
- added TP5004: TestPoint, TestPoint:TestPoint_THTPad_D1.0mm_Drill0.5mm, F.Cu at (147.3, 124.8)
- added TP5005: TestPoint, TestPoint:TestPoint_THTPad_D1.0mm_Drill0.5mm, F.Cu at (138.7, 122.8)
- added TP5006: TestPoint, TestPoint:TestPoint_THTPad_1.0x1.0mm_Drill0.5mm, F.Cu at (122.7, 116.2)
- added TP5007: TestPoint, TestPoint:TestPoint_THTPad_D1.0mm_Drill0.5mm, F.Cu at (122.7, 118.4)
- added U5003: 93AA46BT-I/OT, Package_TO_SOT_SMD:SOT-23-6, F.Cu at (145.0, 121.9)
- added U6001: 93AA46BT-I/OT, Package_TO_SOT_SMD:SOT-23-6, F.Cu at (160.6, 88.0)
- added U6002: 12Mhz,50ppm, Oscillator:Oscillator_SMD_SeikoEpson_SG8002CE-4Pin_3.2x2.5mm, F.Cu at (155.3, 88.0)
- added U6003: FT4232H_QFN, Package_DFN_QFN:QFN-64-1EP_9x9mm_P0.5mm_EP4.35x4.35mm, F.Cu at (158.2, 80.0)
- C5001, C5002, C5003, C5004, C5005, C5006, C5007, C5008: footprint Capacitor_SMD:C_0805_2012Metric -> Capacitor_SMD:C_0603_1608Metric
- moved FID4002 76.2 mm to (222.5, 135.9)
- moved FID4003 69.4 mm to (227.3, 68.8)
- moved C5003 39.9 mm to (140.4, 118.0)
- moved C5007 38.7 mm to (137.7, 124.8)
- moved C5004 37.8 mm to (137.9, 120.0)
- moved C5006 37.4 mm to (137.9, 127.8)
- moved R5001 37.4 mm to (139.6, 115.4), turned to 90 degrees
- moved R5002 36.9 mm to (132.9, 111.6), turned to 90 degrees
- moved R5003 30.9 mm to (127.5, 117.7), turned to 90 degrees
- moved C5005 30.8 mm to (131.9, 131.4), turned to -90 degrees
- moved C5002 29.8 mm to (129.3, 131.4), turned to -90 degrees
- moved C5001 28.2 mm to (129.2, 117.8), turned to 90 degrees
- moved C5008 26.2 mm to (124.2, 127.8), turned to 180 degrees
- moved FID4004 21.2 mm to (115.1, 73.7)
- moved FID4001 19.3 mm to (96.8, 131.8)
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Connections:
- net Net-(U5001-OUT) renamed /USB2UART1/12Mhz
- net Net-(U5002-REF) renamed /USB2UART1/REF
- net Net-(U5002-~{RESET}) renamed /USB2UART1/RESET#
- U2001 pad 3: /USB hub/USB2.D- -> /USB2.D-
- U2001 pad 4: /USB hub/USB2.D+ -> /USB2.D+
- U5002 pad 16: unconnected-(U5002-ADBUS0-Pad16) -> /USB2UART1/UART_A_1.TX
- U5002 pad 17: unconnected-(U5002-ADBUS1-Pad17) -> /USB2UART1/UART_A_1.RX
- U5002 pad 26: unconnected-(U5002-BDBUS0-Pad26) -> /USB2UART1/UART_A_1.TX
- U5002 pad 27: unconnected-(U5002-BDBUS1-Pad27) -> /USB2UART1/UART_A_2.RX
- U5002 pad 38: unconnected-(U5002-CDBUS0-Pad38) -> /USB2UART1/UART_A_1.TX
- U5002 pad 39: unconnected-(U5002-CDBUS1-Pad39) -> /USB2UART1/UART_A_3.RX
- U5002 pad 48: unconnected-(U5002-DDBUS0-Pad48) -> /USB2UART1/UART_A_4.TX
- U5002 pad 52: unconnected-(U5002-DDBUS1-Pad52) -> /USB2UART1/UART_A_4.RX
- U5002 pad 60: unconnected-(U5002-~{PWREN}-Pad60) -> Net-(U5002-~{PWREN})
- U5002 pad 61: unconnected-(U5002-EEDATA-Pad61) -> /USB2UART1/EEDATA
- U5002 pad 62: unconnected-(U5002-EECLK-Pad62) -> /USB2UART1/EECLK
- U5002 pad 63: unconnected-(U5002-EECS-Pad63) -> /USB2UART1/EECS
Routing:
- net +1V8A: track 0.00 -> 11.1 mm
Other:
- board outline added: 160 x 80 mm
- copper layers 2 -> 4

Commit message: .
Parts:
- added C2011: 10u 10V, Capacitor_SMD:C_0603_1608Metric, F.Cu at (97.1, 85.5)
- added C2012: 10u 10V, Capacitor_SMD:C_0603_1608Metric, F.Cu at (99.4, 84.7)
- added C2013: 10u 10V, Capacitor_SMD:C_0603_1608Metric, F.Cu at (98.7, 82.3)
- added C2014: 10u 10V, Capacitor_SMD:C_0603_1608Metric, F.Cu at (98.7, 80.8)
- added C5015: 100n 25V, Capacitor_SMD:C_0603_1608Metric, F.Cu at (123.4, 125.6)
- added C6015: 100n 25V, Capacitor_SMD:C_0603_1608Metric, F.Cu at (121.0, 68.9)
- added C7001: 100n 25V, Capacitor_SMD:C_0603_1608Metric, F.Cu at (140.6, 133.7)
- added C7002: 100n 25V, Capacitor_SMD:C_0603_1608Metric, F.Cu at (140.6, 126.9)
- added C7003: 100n 25V, Capacitor_SMD:C_0603_1608Metric, F.Cu at (140.6, 120.0)
- added C7004: 100n 25V, Capacitor_SMD:C_0603_1608Metric, F.Cu at (140.6, 113.2)
- added C7005: 100n 25V, Capacitor_SMD:C_0603_1608Metric, F.Cu at (140.1, 89.0)
- added C7006: 100n 25V, Capacitor_SMD:C_0603_1608Metric, F.Cu at (140.3, 82.2)
- added C7007: 100n 25V, Capacitor_SMD:C_0603_1608Metric, F.Cu at (139.8, 75.1)
- added C7008: 100n 25V, Capacitor_SMD:C_0603_1608Metric, F.Cu at (140.3, 67.9)
- added J8001: 62684-401100ALF, bt_footprints:62684-401100ALF, F.Cu at (222.7, 103.7)
- added L2001: 1uH, Inductor_SMD:L_0805_2012Metric, F.Cu at (101.2, 85.3)
- added R2016: 22K, Resistor_SMD:R_0603_1608Metric, F.Cu at (94.1, 87.0)
- added R2017: 430K, Resistor_SMD:R_0603_1608Metric, F.Cu at (94.1, 88.5)
- added R2018: 100K, Resistor_SMD:R_0603_1608Metric, F.Cu at (94.1, 90.0)
- added TP6001: TestPoint, TestPoint:TestPoint_THTPad_D1.0mm_Drill0.5mm, F.Cu at (102.2, 76.6)
- added TP6002: TestPoint, TestPoint:TestPoint_THTPad_D1.0mm_Drill0.5mm, F.Cu at (108.6, 80.1)
- added TP6003: TestPoint, TestPoint:TestPoint_THTPad_D1.0mm_Drill0.5mm, F.Cu at (103.2, 74.6)
- added TP6004: TestPoint, TestPoint:TestPoint_THTPad_D1.0mm_Drill0.5mm, F.Cu at (112.7, 77.8)
- added TP6005: TestPoint, TestPoint:TestPoint_THTPad_D1.0mm_Drill0.5mm, F.Cu at (128.3, 82.2)
- added U2003: TPS62A01, Package_TO_SOT_SMD:SOT-23-6, F.Cu at (98.1, 88.0)
- added U7001: ADuM1201BR, Package_SO:SOIC-8_3.9x4.9mm_P1.27mm, F.Cu at (145.9, 128.9)
- added U7002: ADuM1201BR, Package_SO:SOIC-8_3.9x4.9mm_P1.27mm, F.Cu at (145.9, 122.0)
- added U7003: ADuM1201BR, Package_SO:SOIC-8_3.9x4.9mm_P1.27mm, F.Cu at (145.9, 115.1)
- added U7004: ADuM1201BR, Package_SO:SOIC-8_3.9x4.9mm_P1.27mm, F.Cu at (145.9, 135.8)
- added U7005: ADuM1254ASA+, Package_SO:SOIC-8_3.9x4.9mm_P1.27mm, F.Cu at (145.5, 90.9)
- added U7006: ADuM1254ASA+, Package_SO:SOIC-8_3.9x4.9mm_P1.27mm, F.Cu at (145.7, 84.1)
- added U7007: ADuM1201BR, Package_SO:SOIC-8_3.9x4.9mm_P1.27mm, F.Cu at (145.7, 77.0)
- added U7008: ADuM1201BR, Package_SO:SOIC-8_3.9x4.9mm_P1.27mm, F.Cu at (145.7, 70.0)
- D6001: footprint LED_SMD:LED_0201_0603Metric -> LED_SMD:LED_0603_1608Metric
- FID4001, FID4003: moved to B.Cu
- moved C6014 59.5 mm to (114.8, 71.2), turned to 180 degrees
- moved U6001 55.8 mm to (105.8, 77.5), turned to 180 degrees
- moved D6001 55.2 mm to (114.9, 74.2)
- moved TP5003 52.7 mm to (97.0, 122.8), turned to 180 degrees
- moved C5009 51.2 mm to (97.9, 127.0), turned to 180 degrees
- moved TP5001 50.2 mm to (98.2, 125.0), turned to 180 degrees
- moved TP5004 48.1 mm to (99.3, 123.0), turned to 180 degrees
- moved R5004 43.8 mm to (101.9, 128.8), turned to 180 degrees
- moved U5003 43.7 mm to (101.6, 125.9), turned to 180 degrees
- moved U6002 39.5 mm to (116.0, 83.3)
- moved TP5002 37.7 mm to (104.9, 127.8), turned to 180 degrees
- moved R5005 37.2 mm to (104.7, 125.3), turned to 90 degrees
- moved U6003 36.8 mm to (121.6, 75.8), turned to 90 degrees
- moved R5001 35.8 mm to (108.1, 132.4), turned to -90 degrees
- moved D5001 35.2 mm to (109.7, 121.5)
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Connections:
- net /USB Connector/USB_IN.D+ renamed /USB.D+
- net /USB Connector/USB_IN.D- renamed /USB.D-
- net /USB Connector/USB_IN.VBUS renamed /USB.VBUS
- net /USB2UART2/UART_B_1.RX renamed /Isolation_output/I2C_B_1.SDA
- net /USB2UART2/UART_B_2.RX renamed /Isolation_output/I2C_B_2.SDA
- C6002 pad 1: +1V8A -> +1V8B
- C6003 pad 1: +1V8A -> +1V8B
- C6005 pad 1: +1V8A -> +1V8B
- C6014 pad 1: +1V8A -> +1V8B
- U5002 pad 16: /USB2UART1/UART_A_1.TX -> /Isolation_output/UART_A_1.TX
- U5002 pad 17: /USB2UART1/UART_A_1.RX -> /Isolation_output/UART_A_1.RX
- U5002 pad 26: /USB2UART1/UART_A_1.TX -> /Isolation_output/UART_A_2.TX
- U5002 pad 27: /USB2UART1/UART_A_2.RX -> /Isolation_output/UART_A_2.RX
- U5002 pad 38: /USB2UART1/UART_A_1.TX -> /Isolation_output/UART_A_3.TX
- U5002 pad 39: /USB2UART1/UART_A_3.RX -> /Isolation_output/UART_A_3.RX
- U5002 pad 48: /USB2UART1/UART_A_4.TX -> /Isolation_output/UART_A_4.TX
- U5002 pad 52: /USB2UART1/UART_A_4.RX -> /Isolation_output/UART_A_4.RX
- U5002 pad 65: (no net) -> GND
- U6003 pad 12: +1V8A -> +1V8B
- U6003 pad 16: /USB2UART2/UART_B_1.TX -> /Isolation_output/I2C_B_1.SCL
- U6003 pad 26: /USB2UART2/UART_B_1.TX -> /Isolation_output/I2C_B_2.SCL
- U6003 pad 37: +1V8A -> +1V8B
- U6003 pad 38: /USB2UART2/UART_B_1.TX -> /Isolation_output/UART_B_3.TX
- U6003 pad 39: /USB2UART2/UART_B_3.RX -> /Isolation_output/UART_B_3.RX
- U6003 pad 48: /USB2UART2/UART_B_4.TX -> /Isolation_output/UART_B_4.TX
- U6003 pad 49: +1V8A -> +1V8B
- U6003 pad 52: /USB2UART2/UART_B_4.RX -> /Isolation_output/UART_B_4.RX
- U6003 pad 64: +1V8A -> +1V8B
- U6003 pad 65: (no net) -> GND
Routing:
- net +3.3V: track 0.00 -> 524.4 mm, vias 0 -> 34
- net GND: track 0.00 -> 198.5 mm, vias 0 -> 59
- net /USB2.D-: track 0.00 -> 56.0 mm, vias 0 -> 2
- net /USB2.D+: track 0.00 -> 52.1 mm, vias 0 -> 2
- net /Isolation_output/UART_A_4.TX: track 0.00 -> 49.6 mm, vias 0 -> 2
- net /USB.VBUS: track 0.00 -> 42.7 mm
- net /Isolation_output/UART_A_4.RX: track 0.00 -> 39.1 mm, vias 0 -> 2
- net /Isolation_output/UART_A_3.TX: track 0.00 -> 31.6 mm, vias 0 -> 2
- net /Isolation_output/UART_A_3.RX: track 0.00 -> 30.8 mm, vias 0 -> 2
- net /USB1.D+: track 0.00 -> 27.1 mm, vias 0 -> 2
- net /USB1.D-: track 0.00 -> 27.1 mm, vias 0 -> 2
- net /Isolation_output/UART_A_1.TX: track 0.00 -> 23.9 mm
- net /Isolation_output/UART_A_1.RX: track 0.00 -> 22.9 mm
- net /Isolation_output/UART_A_2.RX: track 0.00 -> 22.6 mm
- net /Isolation_output/UART_A_2.TX: track 0.00 -> 22.4 mm
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- added copper zone on In2.Cu, net +1V8A
- added copper zone on In2.Cu, net +1V8B
- added copper zone on B.Cu, net GND
- added copper zone on F.Cu, net GND
- added copper zone on In1.Cu, net GND
- added copper zone on In2.Cu, net GND

Commit message: .
Parts:
- added C7009: 100n 25V, Capacitor_SMD:C_0603_1608Metric, F.Cu at (151.4, 67.8)
- added C7010: 100n 25V, Capacitor_SMD:C_0603_1608Metric, F.Cu at (151.4, 74.9)
- added C7011: 100n 25V, Capacitor_SMD:C_0603_1608Metric, F.Cu at (151.4, 82.0)
- added C7012: 100n 25V, Capacitor_SMD:C_0603_1608Metric, F.Cu at (151.4, 88.9)
- added C7013: 100n 25V, Capacitor_SMD:C_0603_1608Metric, F.Cu at (151.4, 133.6)
- added C7014: 100n 25V, Capacitor_SMD:C_0603_1608Metric, F.Cu at (151.4, 113.3)
- added C7015: 100n 25V, Capacitor_SMD:C_0603_1608Metric, F.Cu at (151.4, 119.9)
- added C7016: 100n 25V, Capacitor_SMD:C_0603_1608Metric, F.Cu at (151.4, 126.7)
- added C7017: 100n 25V, Capacitor_SMD:C_0603_1608Metric, F.Cu at (138.2, 103.1)
- added C7018: 10u 10V, Capacitor_SMD:C_0603_1608Metric, F.Cu at (136.4, 103.1)
- added C7019: 100n 25V, Capacitor_SMD:C_0603_1608Metric, F.Cu at (154.7, 103.1)
- added C7020: 10u 10V, Capacitor_SMD:C_0603_1608Metric, F.Cu at (153.2, 103.1)
- added D8001: LED, LED_SMD:LED_0603_1608Metric, F.Cu at (193.3, 68.8)
- added D8002: LED, LED_SMD:LED_0603_1608Metric, F.Cu at (193.3, 96.7)
- added D8003: LED, LED_SMD:LED_0603_1608Metric, F.Cu at (193.3, 124.7)
- added D8004: LED, LED_SMD:LED_0603_1608Metric, F.Cu at (193.3, 83.1)
- added D8005: LED, LED_SMD:LED_0603_1608Metric, F.Cu at (193.5, 111.0)
- added J8002: Conn_02x10_Odd_Even, Connector_IDC:IDC-Header_2x10_P2.54mm_Vertical, F.Cu at (199.9, 73.4)
- added J8003: Conn_02x10_Odd_Even, Connector_IDC:IDC-Header_2x10_P2.54mm_Vertical, F.Cu at (199.9, 87.4)
- added J8004: Conn_02x10_Odd_Even, Connector_IDC:IDC-Header_2x10_P2.54mm_Vertical, F.Cu at (199.9, 101.4)
- added J8005: Conn_02x10_Odd_Even, Connector_IDC:IDC-Header_2x10_P2.54mm_Vertical, F.Cu at (199.9, 115.3)
- added J8006: Conn_02x10_Odd_Even, Connector_IDC:IDC-Header_2x10_P2.54mm_Vertical, F.Cu at (199.9, 129.3)
- added J8007: Conn_02x05_Odd_Even, Connector_IDC:IDC-Header_2x05_P2.54mm_Vertical, F.Cu at (185.9, 98.8)
- added J8008: Conn_02x05_Odd_Even, Connector_IDC:IDC-Header_2x05_P2.54mm_Vertical, F.Cu at (185.9, 74.9)
- added Q8001: BSS138, Package_TO_SOT_SMD:SOT-23, F.Cu at (190.3, 67.0)
- added Q8002: BSS138, Package_TO_SOT_SMD:SOT-23, F.Cu at (194.7, 93.3)
- added Q8003: BSS138, Package_TO_SOT_SMD:SOT-23, F.Cu at (194.3, 121.2)
- added Q8004: BSS138, Package_TO_SOT_SMD:SOT-23, F.Cu at (195.9, 79.0)
- added Q8005: BSS138, Package_TO_SOT_SMD:SOT-23, F.Cu at (194.6, 107.4)
- added R7001: 100R, Resistor_SMD:R_0603_1608Metric, F.Cu at (151.4, 128.3)
- added R7002: 100R, Resistor_SMD:R_0603_1608Metric, F.Cu at (151.4, 129.8)
- added R7003: 100R, Resistor_SMD:R_0603_1608Metric, F.Cu at (151.4, 114.8)
- added R7004: 100R, Resistor_SMD:R_0603_1608Metric, F.Cu at (151.4, 116.3)
- added R7005: 100R, Resistor_SMD:R_0603_1608Metric, F.Cu at (151.4, 135.4)
- added R7006: 100R, Resistor_SMD:R_0603_1608Metric, F.Cu at (151.4, 136.9)
- added R7007: 100R, Resistor_SMD:R_0603_1608Metric, F.Cu at (151.4, 90.4)
- added R7008: 100R, Resistor_SMD:R_0603_1608Metric, F.Cu at (151.4, 91.9)
- added R7009: 100R, Resistor_SMD:R_0603_1608Metric, F.Cu at (151.4, 76.5)
- added R7010: 100R, Resistor_SMD:R_0603_1608Metric, F.Cu at (151.4, 78.0)
- added R7011: 100R, Resistor_SMD:R_0603_1608Metric, F.Cu at (151.4, 69.3)
- added R7012: 100R, Resistor_SMD:R_0603_1608Metric, F.Cu at (151.4, 70.9)
- added R7013: 100R, Resistor_SMD:R_0603_1608Metric, F.Cu at (151.4, 83.6)
- added R7014: 100R, Resistor_SMD:R_0603_1608Metric, F.Cu at (151.4, 85.1)
- added R7015: 100R, Resistor_SMD:R_0603_1608Metric, F.Cu at (151.4, 121.4)
- added R7016: 100R, Resistor_SMD:R_0603_1608Metric, F.Cu at (151.4, 122.9)
- added R8001: 10K, Resistor_SMD:R_0603_1608Metric, F.Cu at (205.0, 78.7)
- added R8002: 10K, Resistor_SMD:R_0603_1608Metric, F.Cu at (215.1, 78.7)
- added R8003: 10K, Resistor_SMD:R_0603_1608Metric, F.Cu at (222.8, 78.7)
- added R8004: 10K, Resistor_SMD:R_0603_1608Metric, F.Cu at (205.0, 92.7)
- added R8005: 10K, Resistor_SMD:R_0603_1608Metric, F.Cu at (215.1, 92.7)
- added R8006: 10K, Resistor_SMD:R_0603_1608Metric, F.Cu at (222.8, 92.7)
- added R8007: 10K, Resistor_SMD:R_0603_1608Metric, F.Cu at (205.0, 106.7)
- added R8008: 10K, Resistor_SMD:R_0603_1608Metric, F.Cu at (215.2, 106.7)
- added R8009: 10K, Resistor_SMD:R_0603_1608Metric, F.Cu at (222.8, 106.7)
- added R8010: 10K, Resistor_SMD:R_0603_1608Metric, F.Cu at (205.0, 120.7)
- added R8011: 10K, Resistor_SMD:R_0603_1608Metric, F.Cu at (215.1, 120.7)
- added R8012: 10K, Resistor_SMD:R_0603_1608Metric, F.Cu at (222.8, 120.7)
- added R8013: 10K, Resistor_SMD:R_0603_1608Metric, F.Cu at (212.6, 134.6)
- added R8014: 10K, Resistor_SMD:R_0603_1608Metric, F.Cu at (222.8, 134.6)
- added R8015: 10K, Resistor_SMD:R_0603_1608Metric, F.Cu at (202.4, 78.7)
- added R8016: 10K, Resistor_SMD:R_0603_1608Metric, F.Cu at (212.6, 78.7)
- added R8017: 10K, Resistor_SMD:R_0603_1608Metric, F.Cu at (220.2, 78.7)
- added R8018: 10K, Resistor_SMD:R_0603_1608Metric, F.Cu at (202.4, 92.7)
- added R8019: 10K, Resistor_SMD:R_0603_1608Metric, F.Cu at (212.6, 92.7)
- added R8020: 10K, Resistor_SMD:R_0603_1608Metric, F.Cu at (220.2, 92.7)
- added R8021: 10K, Resistor_SMD:R_0603_1608Metric, F.Cu at (202.4, 106.7)
- added R8022: 10K, Resistor_SMD:R_0603_1608Metric, F.Cu at (212.6, 106.7)
- added R8023: 10K, Resistor_SMD:R_0603_1608Metric, F.Cu at (220.2, 106.7)
- added R8024: 10K, Resistor_SMD:R_0603_1608Metric, F.Cu at (202.4, 120.7)
- added R8025: 10K, Resistor_SMD:R_0603_1608Metric, F.Cu at (212.6, 120.7)
- added R8026: 10K, Resistor_SMD:R_0603_1608Metric, F.Cu at (220.2, 120.7)
- added R8027: 10K, Resistor_SMD:R_0603_1608Metric, F.Cu at (220.2, 134.6)
- added R8028: 10K, Resistor_SMD:R_0603_1608Metric, F.Cu at (195.9, 66.0)
- added R8029: 10K, Resistor_SMD:R_0603_1608Metric, F.Cu at (198.4, 94.2)
- added R8030: 10K, Resistor_SMD:R_0603_1608Metric, F.Cu at (197.1, 121.0)
- added R8031: 510R, Resistor_SMD:R_0603_1608Metric, F.Cu at (193.3, 71.8)
- added R8032: 510R, Resistor_SMD:R_0603_1608Metric, F.Cu at (193.3, 99.9)
- added R8033: 510R, Resistor_SMD:R_0603_1608Metric, F.Cu at (193.3, 128.0)
- added R8034: 10K, Resistor_SMD:R_0603_1608Metric, F.Cu at (198.6, 78.8)
- added R8035: 10K, Resistor_SMD:R_0603_1608Metric, F.Cu at (171.7, 132.1)
- added R8036: 510R, Resistor_SMD:R_0603_1608Metric, F.Cu at (193.3, 86.2)
- added R8037: 510R, Resistor_SMD:R_0603_1608Metric, F.Cu at (193.5, 114.1)
- added SW8001: M;SW;3;SPST, bt_footprints:SW_DS04-254-2-03BK-SMT, F.Cu at (165.1, 69.1)
- added SW8002: M;SW;3;SPST, bt_footprints:SW_DS04-254-2-03BK-SMT, F.Cu at (238.3, 124.2)
- added SW8003: M;SW;3;SPST, bt_footprints:SW_DS04-254-2-03BK-SMT, F.Cu at (165.1, 79.9)
- added SW8004: M;SW;3;SPST, bt_footprints:SW_DS04-254-2-03BK-SMT, F.Cu at (165.1, 133.9)
- added SW8005: M;SW;3;SPST, bt_footprints:SW_DS04-254-2-03BK-SMT, F.Cu at (165.1, 101.5)
- added SW8006: M;SW;3;SPST, bt_footprints:SW_DS04-254-2-03BK-SMT, F.Cu at (165.1, 112.3)
- added SW8007: M;SW;3;SPST, bt_footprints:SW_DS04-254-2-03BK-SMT, F.Cu at (165.1, 123.1)
- added SW8008: M;SW;3;SPST, bt_footprints:SW_DS04-254-2-03BK-SMT, F.Cu at (165.1, 90.7)
- added SW8009: M;SW;3;SPST, bt_footprints:SW_DS04-254-2-03BK-SMT, F.Cu at (176.5, 81.3)
- added TP2001: TestPoint, TestPoint:TestPoint_THTPad_D1.0mm_Drill0.5mm, F.Cu at (97.8, 78.2)
- added TP2002: TestPoint, TestPoint:TestPoint_THTPad_1.0x1.0mm_Drill0.5mm, F.Cu at (109.2, 73.7)
- added TP6006: TestPoint, TestPoint:TestPoint_THTPad_1.0x1.0mm_Drill0.5mm, F.Cu at (95.5, 78.2)
- added TP6007: TestPoint, TestPoint:TestPoint_THTPad_1.0x1.0mm_Drill0.5mm, F.Cu at (130.0, 84.1)
- added U7009: ADuM6028-3, Package_SO:SOIC-8_7.5x5.85mm_P1.27mm, F.Cu at (145.8, 101.5)
- FID4001, FID4003: moved to F.Cu
- moved J8001 18.5 mm to (241.0, 101.3)
- moved FID4003 14.9 mm to (237.7, 79.5), turned to 0 degrees
- moved FID4004 5.83 mm to (98.8, 65.8)
- moved FID4002 5.35 mm to (232.4, 137.4)
- moved H4001 2.30 mm to (239.0, 67.6)
- moved H4004 1.49 mm to (92.2, 135.1)
- moved H4003 1.34 mm to (92.2, 67.6)
- moved U7005 0.44 mm to (145.9, 90.9)
- moved U7006 0.19 mm to (145.9, 84.1)
- moved U7007 0.19 mm to (145.9, 77.0)
- moved U7008 0.19 mm to (145.9, 70.0)
- turned FID4001 to 0 degrees
Connections:
- J8001 pad 01: unconnected-(J8001-Pad01) -> /Isolation_output/Debug_connector/FORCE#
- J8001 pad 02: unconnected-(J8001-Pad02) -> /Isolation_output/Debug_connector/E_RESET#
- J8001 pad 03: unconnected-(J8001-Pad03) -> /Isolation_output/Debug_connector/E_TRST#
- J8001 pad 04: unconnected-(J8001-Pad04) -> /Isolation_output/Debug_connector/E_TCK
- J8001 pad 05: unconnected-(J8001-Pad05) -> /Isolation_output/Debug_connector/E_TMS
- J8001 pad 06: unconnected-(J8001-Pad06) -> /Isolation_output/Debug_connector/E_TDO
- J8001 pad 07: unconnected-(J8001-Pad07) -> /Isolation_output/Debug_connector/E_TDI
- J8001 pad 08: unconnected-(J8001-Pad08) -> GND2
- J8001 pad 09: unconnected-(J8001-Pad09) -> E_VCC
- J8001 pad 10: unconnected-(J8001-Pad10) -> /Isolation_output/Debug_connector/E_RX
- J8001 pad 11: unconnected-(J8001-Pad11) -> /Isolation_output/Debug_connector/E_TX
- J8001 pad 12: unconnected-(J8001-Pad12) -> /Isolation_output/Debug_connector/D_IO/F_VCC
- J8001 pad 13: unconnected-(J8001-Pad13) -> /Isolation_output/Debug_connector/D_RESET#
- J8001 pad 14: unconnected-(J8001-Pad14) -> /Isolation_output/Debug_connector/D_SWCLK
- J8001 pad 15: unconnected-(J8001-Pad15) -> /Isolation_output/Debug_connector/D_SWDIO
- J8001 pad 16: unconnected-(J8001-Pad16) -> GND2
- J8001 pad 17: unconnected-(J8001-Pad17) -> D_VCC
- J8001 pad 18: unconnected-(J8001-Pad18) -> /Isolation_output/Debug_connector/D_RX
- J8001 pad 19: unconnected-(J8001-Pad19) -> /Isolation_output/Debug_connector/D_TX
- J8001 pad 20: unconnected-(J8001-Pad20) -> /Isolation_output/Debug_connector/C_RESET#
- J8001 pad 21: unconnected-(J8001-Pad21) -> /Isolation_output/Debug_connector/C_SWCLK
- J8001 pad 22: unconnected-(J8001-Pad22) -> /Isolation_output/Debug_connector/C_SWDIO
- J8001 pad 23: unconnected-(J8001-Pad23) -> GND2
- J8001 pad 24: unconnected-(J8001-Pad24) -> C_VCC
- J8001 pad 25: unconnected-(J8001-Pad25) -> /Isolation_output/Debug_connector/C_RX
- J8001 pad 26: unconnected-(J8001-Pad26) -> /Isolation_output/Debug_connector/C_TX
- J8001 pad 27: unconnected-(J8001-Pad27) -> /Isolation_output/Debug_connector/B_RESET#
- J8001 pad 28: unconnected-(J8001-Pad28) -> /Isolation_output/Debug_connector/B_SWCLK
- J8001 pad 29: unconnected-(J8001-Pad29) -> /Isolation_output/Debug_connector/B_SWDIO
- J8001 pad 30: unconnected-(J8001-Pad30) -> GND2
- J8001 pad 31: unconnected-(J8001-Pad31) -> B_VCC
- J8001 pad 32: unconnected-(J8001-Pad32) -> /Isolation_output/Debug_connector/B_RX
- J8001 pad 33: unconnected-(J8001-Pad33) -> /Isolation_output/Debug_connector/B_TX
- J8001 pad 34: unconnected-(J8001-Pad34) -> /Isolation_output/Debug_connector/A_RESET#
- J8001 pad 35: unconnected-(J8001-Pad35) -> /Isolation_output/Debug_connector/A_SWCLK
- J8001 pad 36: unconnected-(J8001-Pad36) -> /Isolation_output/Debug_connector/A_SWDIO
- J8001 pad 37: unconnected-(J8001-Pad37) -> GND2
- J8001 pad 38: unconnected-(J8001-Pad38) -> A_VCC
- J8001 pad 39: unconnected-(J8001-Pad39) -> /Isolation_output/Debug_connector/A_RX
- J8001 pad 40: unconnected-(J8001-Pad40) -> /Isolation_output/Debug_connector/A_TX
- J8001 pad S1: unconnected-(J8001-PadS1) -> GND2
- J8001 pad S2: unconnected-(J8001-PadS2) -> GND2
- U7001 pad 5: unconnected-(U7001-GND2-Pad5) -> GND2
- U7001 pad 6: unconnected-(U7001-VOB-Pad6) -> Net-(U7001-VOB)
- U7001 pad 7: unconnected-(U7001-VIA-Pad7) -> Net-(U7001-VIA)
- U7001 pad 8: unconnected-(U7001-VDD2-Pad8) -> SW_A_VCC
- U7002 pad 5: unconnected-(U7002-GND2-Pad5) -> GND2
- U7002 pad 6: unconnected-(U7002-VOB-Pad6) -> Net-(U7002-VOB)
- U7002 pad 7: unconnected-(U7002-VIA-Pad7) -> Net-(U7002-VIA)
- U7002 pad 8: unconnected-(U7002-VDD2-Pad8) -> SW_B_VCC
- U7003 pad 5: unconnected-(U7003-GND2-Pad5) -> GND2
- U7003 pad 6: unconnected-(U7003-VOB-Pad6) -> Net-(U7003-VOB)
- U7003 pad 7: unconnected-(U7003-VIA-Pad7) -> Net-(U7003-VIA)
- U7003 pad 8: unconnected-(U7003-VDD2-Pad8) -> SW_C_VCC
- U7004 pad 5: unconnected-(U7004-GND2-Pad5) -> GND2
- U7004 pad 6: unconnected-(U7004-VOB-Pad6) -> Net-(U7004-VOB)
- U7004 pad 7: unconnected-(U7004-VIA-Pad7) -> Net-(U7004-VIA)
- U7004 pad 8: unconnected-(U7004-VDD2-Pad8) -> SW_D_VCC
- U7005 pad 5: unconnected-(U7005-GND2-Pad5) -> GND2
- U7005 pad 6: unconnected-(U7005-SCL2-Pad6) -> Net-(U7005-SCL2)
- U7005 pad 7: unconnected-(U7005-SDA2-Pad7) -> Net-(U7005-SDA2)
- U7005 pad 8: unconnected-(U7005-VDD2-Pad8) -> SW_D_I2C2_VCC
- U7006 pad 5: unconnected-(U7006-GND2-Pad5) -> GND2
- U7006 pad 6: unconnected-(U7006-SCL2-Pad6) -> Net-(U7006-SCL2)
- U7006 pad 7: unconnected-(U7006-SDA2-Pad7) -> Net-(U7006-SDA2)
- U7006 pad 8: unconnected-(U7006-VDD2-Pad8) -> SW_D_I2C1_VCC
- U7007 pad 5: unconnected-(U7007-GND2-Pad5) -> GND2
- U7007 pad 6: unconnected-(U7007-VOB-Pad6) -> Net-(U7007-VOB)
- U7007 pad 7: unconnected-(U7007-VIA-Pad7) -> Net-(U7007-VIA)
- U7007 pad 8: unconnected-(U7007-VDD2-Pad8) -> SW_E_VCC
- U7008 pad 5: unconnected-(U7008-GND2-Pad5) -> GND2
- U7008 pad 6: unconnected-(U7008-VOB-Pad6) -> Net-(U7008-VOB)
- U7008 pad 7: unconnected-(U7008-VIA-Pad7) -> Net-(U7008-VIA)
- U7008 pad 8: unconnected-(U7008-VDD2-Pad8) -> SW_F_VCC
Routing:
- net GND2: track 0.00 -> 228.5 mm, vias 0 -> 115
- net D_VCC: track 0.00 -> 160.9 mm, vias 0 -> 3
- net E_VCC: track 0.00 -> 155.0 mm, vias 0 -> 2
- net A_VCC: track 0.00 -> 139.4 mm, vias 0 -> 1
- net /Isolation_output/Debug_connector/D_IO/F_VCC: track 0.00 -> 125.1 mm, vias 0 -> 4
- net /Isolation_output/Debug_connector/E_RX: track 0.00 -> 119.4 mm, vias 0 -> 2
- net /Isolation_output/Debug_connector/E_TX: track 0.00 -> 119.0 mm, vias 0 -> 2
- net /Isolation_output/Debug_connector/D_SWCLK: track 0.00 -> 114.2 mm, vias 0 -> 6
- net /Isolation_output/Debug_connector/D_SWDIO: track 0.00 -> 108.6 mm
- net VCC_LED: track 0.00 -> 108.5 mm, vias 0 -> 4
- net /Isolation_output/Debug_connector/D_TX: track 0.00 -> 106.9 mm
- net B_VCC: track 0.00 -> 106.8 mm, vias 0 -> 2
- net /Isolation_output/Debug_connector/D_RX: track 0.00 -> 105.2 mm
- net /Isolation_output/Debug_connector/D_RESET#: track 0.00 -> 97.4 mm, vias 0 -> 1
- net /Isolation_output/Debug_connector/A_TX: track 0.00 -> 89.2 mm, vias 0 -> 2
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- added copper zone on B.Cu, net GND2
- added copper zone on F.Cu, net GND2
- added copper zone on In1.Cu, net GND2
- added copper zone on In2.Cu, net GND2
Other:
- board text added: "1"
- board text added: "2"
- board text added: "3"
- board text added: "4"
- board text added: "DEBUG board for CC"
- board text added: "FORCE"
- board text added: "I2C"
- board text added: "MCU A SWD: SS"
- board text added: "MCU B SWD: DMCU"
- board text added: "MCU C SWD: IO-MCU"
- board text added: "MCU D SWD: SS"
- board text added: "MCU E SWD/ JTAG"
- board text added: "SW1 UART F"
- board text added: "SW2 UART E"
- board text added: "SW3 I2C"
- board text added: "SW4 I2C"
- board text added: "SW5 UART C"
- board text added: "SW6 UART B"
- board text added: "SW6 UART D"
- board text added: "SW7 UART B"
- board text added: "USB A CH A:UART D CH B:UART C CH C:UART B CH D:UART A"
- board text added: "USB B CH A:I2C CH B:I2C CH C:UART F CH D:UART E"

Commit message: .
Parts:
- added C7021: 1n, Capacitor_SMD:C_1812_4532Metric, F.Cu at (145.8, 108.5)
- added R7017: 1M, Resistor_SMD:R_1210_3225Metric, F.Cu at (145.8, 96.0)
Routing:
- net GND: track 206.5 -> 209.9 mm
Other:
- board text added: "Version 0.1"
