File: HW/CC_Debug/CC_Debug/Isolation_output.kicad_sch (KiCad schematic)
At the start: 16 parts, among them U7001 ADuM1201BR, U7002 ADuM1201BR, U7003 ADuM1201BR, U7004 ADuM1201BR, U7005 ADuM1254ASA+, U7006 ADuM1254ASA+, U7007 ADuM1201BR, U7008 ADuM1201BR

Commit message: .
Parts:
- added C7009, C7010, C7011, C7012, C7013, C7014, C7015, C7016, C7017, C7019: 100n 25V, Capacitor_SMD:C_0603_1608Metric, symbol bt_capacitor:C;M;100n;10p;25V;S;0603
- added C7018, C7020: 10u 10V, Capacitor_SMD:C_0603_1608Metric, symbol bt_capacitor:C;M;10u;10p;10V;S;0603
- added R7001, R7002, R7003, R7004, R7005, R7006, R7007, R7008, R7009, R7010, R7011, R7012, R7013, R7014, R7015, R7016: 100R, Resistor_SMD:R_0603_1608Metric, symbol bt_resistors:R;G;100R;10P0;S;0603
- added U7009: ADuM6028-3, Package_SO:SOIC-8_7.5x5.85mm_P1.27mm, symbol bt_power:ADuM6028-3
Connections:
- net +3.3V: now also C7017.1, C7018.1, U7009.1 (PDIS), U7009.3 (VDDp)
- net GND: now also C7017.2, C7018.2, U7009.2 (GND), U7009.4 (GND)
- net GND2: now reaches U7007.5 (GND2)
- net GND2: now also U7001.5 (GND2), U7002.5 (GND2), U7003.5 (GND2), U7004.5 (GND2), U7005.5 (GND2), U7006.5 (GND2), U7008.5 (GND2), C7009.2, C7010.2, C7011.2, C7012.2, C7013.2, C7014.2, C7015.2, C7016.2, C7019.2, C7020.2, U7009.5 (GND_ISO), U7009.7 (GND_ISO), U7009.8 (V_SEL)
- net at U7007.6 (VOB): now also R7010.1
- net at U7007.7 (VIA): now also R7009.1
- net SW_E_VCC: now reaches U7007.8 (VDD2)
- net SW_E_VCC: now also C7010.1
- net at U7006.6 (SCL2): now also R7014.1
- net at U7006.7 (SDA2): now also R7013.1
- net SW_D_I2C1_VCC: now reaches U7006.8 (VDD2)
- net SW_D_I2C1_VCC: now also C7011.1
- net at U7004.6 (VOB): now also R7006.1
- net at U7004.7 (VIA): now also R7005.1
- net SW_D_VCC: now reaches U7004.8 (VDD2)
- net SW_D_VCC: now also C7013.1
- net at U7001.6 (VOB): now also R7002.1
- net at U7001.7 (VIA): now also R7001.1
- net SW_A_VCC: now reaches U7001.8 (VDD2)
- net SW_A_VCC: now also C7016.1
- net at U7008.6 (VOB): now also R7012.1
- net at U7008.7 (VIA): now also R7011.1
- net SW_F_VCC: now reaches U7008.8 (VDD2)
- net SW_F_VCC: now also C7009.1
- net at U7005.6 (SCL2): now also R7008.1
- net at U7005.7 (SDA2): now also R7007.1
- net SW_D_I2C2_VCC: now reaches U7005.8 (VDD2)
- net SW_D_I2C2_VCC: now also C7012.1
- net at U7002.6 (VOB): now also R7016.1
- net at U7002.7 (VIA): now also R7015.1
- net SW_B_VCC: now reaches U7002.8 (VDD2)
- net SW_B_VCC: now also C7015.1
- net at U7003.6 (VOB): now also R7004.1
- net at U7003.7 (VIA): now also R7003.1
- net SW_C_VCC: now reaches U7003.8 (VDD2)
- net SW_C_VCC: now also C7014.1
- new net I2C1.SCL: R7014.2
- new net I2C1.SDA: R7013.2
- new net I2C2.SCL: R7008.2
- new net I2C2.SDA: R7007.2
- new net SW_A.RX: R7001.2
- new net SW_A.TX: R7002.2
- new net SW_B.RX: R7015.2
- new net SW_B.TX: R7016.2
- new net SW_C.RX: R7003.2
- new net SW_C.TX: R7004.2
- new net SW_D.RX: R7005.2
- new net SW_D.TX: R7006.2
- new net SW_E.RX: R7009.2
- new net SW_E.TX: R7010.2
- new net SW_F.RX: R7011.2
- new net SW_F.TX: R7012.2
- new net VCC_LED: C7019.1, C7020.1, U7009.6 (V_ISO)
Other:
- sheet Debug_connector ports: added I2C1{I2C}, I2C2{I2C}, SW_A{UART}, SW_B{UART}, SW_C{UART}, SW_D{UART}, SW_E{UART}, SW_F{UART}; removed none

Commit message: .
Parts:
- added C7021: 1n, Capacitor_SMD:C_1812_4532Metric, symbol Device:C
- added R7017: 1M, Resistor_SMD:R_1210_3225Metric, symbol Device:R
Connections:
- net GND: now also C7021.1, R7017.1
- net GND2: now also C7021.2, R7017.2
Other:
- moved on the sheet: U7009
