File: HW/PIC18F_ETH/PIC18F_ETH/MCU_core.kicad_sch (KiCad schematic)
At the start: 3 parts

Commit message: .
Parts:
- added C? (x9): 100n 25V, Capacitor_SMD:C_0603_1608Metric, symbol bt_capacitor:C;M;100n;10p;25V;S;0603
- added C?: 10u 10V, Capacitor_SMD:C_0603_1608Metric, symbol bt_capacitor:C;M;10u;10p;10V;S;0603
- added J?: Conn_01x06, symbol Connector_Generic:Conn_01x06
- added R2001, R?: 10K, Resistor_SMD:R_0603_1608Metric, symbol bt_resistors:R;G;10K;10P0;S;0603
- added U?: 93AA46BT-I/OT, Package_TO_SOT_SMD:SOT-23-6, symbol bt_memory:93AA46BT-I/OT
- gave numbers to parts that had none: 2
Connections:
- net at U2002.1 (ST#): now also R2001.2
- net GND: now reaches U2002.2 (GND)
- net GND: now also U2001.20 (AVSS), U2001.25 (VSS), U2001.41 (VSS), U2001.45 (VSSRX), U2001.52 (VSSTX), U2001.55 (VSSPLL), U2001.56 (VSS), U2001.9 (VSS), C?.2, C?.2, C?.2, J?.3 (Pin_3), R?.2, U?.2 (GND)
- net at U2002.3 (OUT): now also U2001.39 (OSC1/CLKI)
- net +3.3V: now reaches U2002.4 (Vcc)
- net +3.3V: now also U2001.18 (ENVREG), U2001.19 (AVDD), U2001.26 (VDD), U2001.38 (VDD), U2001.48 (VDDRX), U2001.49 (VDDTX), U2001.54 (VDDPLL), U2001.57 (VDD), C?.1, C?.1, C?.1, C?.1, C?.1, C?.1, C?.1, C?.1, C?.1, C?.2, C?.2, C?.2, C?.2, C?.2, C?.2, C?.2, J?.2 (Pin_2), R2001.1, U?.6 (VCC)
- net at U2001.10 (VDDCORE/VCAP): now also C?.1
- net SPI_SS1: now reaches U2001.11 (RF7/*SS1)
- net SPI_SS1: now also R?.1, U?.5 (CS)
- net LED_B: now reaches U2001.23 (RA1/LEDB/AN1)
- net LED_A: now reaches U2001.24 (RA0/LEDA/AN0)
- net SPI_SS3: now reaches U2001.29 (RC1/T1OSI/ECCP2/P2A)
- net SPI_SS4: now reaches U2001.30 (RC0/T1OSO/T13CKI)
- net UART_TX: now reaches U2001.31 (RC6/TX1/CK1)
- net UART_RX: now reaches U2001.32 (RC7/RX1/DT1)
- net SPI_SS2: now reaches U2001.33 (RC2/ECCP1/P1A)
- net SPI_SCK: now reaches U2001.34 (RC3/SCK1/SCL1)
- net SPI_SCK: now also U?.4 (CLK)
- net SPI_MISO: now reaches U2001.35 (RC4/SDI1/SDA1)
- net SPI_MISO: now also U?.1 (DO), U?.3 (DI)
- net SPI_MOSI: now reaches U2001.36 (RC5/SDO1)
- net PGD: now reaches U2001.37 (RB7/KBI3/PGD)
- net PGD: now also J?.4 (Pin_4)
- net PGC: now reaches U2001.42 (RB6/KBI2/PGC)
- net PGC: now also J?.5 (Pin_5)
- net ETH.RX+: now reaches U2001.46 (TPIN-)
- net ETH.RX+: now also U2001.47 (TPIN+)
- net ETH.TX-: now reaches U2001.50 (TPOUT-)
- net ETH.TX+: now reaches U2001.51 (TPOUT+)
- net RST#: now reaches U2001.7 (*MCLR)
Other:
- moved on the sheet: U2002

Commit message: .
Parts:
- added R2003: 10K, Resistor_SMD:R_0603_1608Metric, symbol bt_resistors:R;G;10K;10P0;S;0603
- added R2004: 2K2, Resistor_SMD:R_0603_1608Metric, symbol bt_resistors:R;G;2K2;10P0;S;0603
- added R2005: 620R, Resistor_SMD:R_0603_1608Metric, symbol bt_resistors:R;G;620R;10P0;S;0603
- gave numbers to parts that had none: 13
Connections:
- net +3.3V: now also R2003.1
- net GND: now also R2005.2
- net RST#: now also J2001.1 (Pin_1), R2003.2
- net at U2001.53 (RBIAS): now also R2004.1
- new net: R2004.2, R2005.1

Commit message: .
Parts:
- added C2011: 100n 25V, Capacitor_SMD:C_0603_1608Metric, symbol bt_capacitor:C;M;100n;10p;25V;S;0603
- J2001: footprint (none) -> Connector_PinHeader_2.54mm:PinHeader_1x06_P2.54mm_Vertical
Connections:
- net SPI_SS4 is gone; now on net SPI_SS3: U2001.30 (RC0/T1OSO/T13CKI)
- net +3.3V: now also C2011.1
- net GND: now also C2011.2
- net SPI_SS1: now also U2001.33 (RC2/ECCP1/P1A); no longer U2001.11 (RF7/*SS1)
- net SPI_SS2: now also U2001.29 (RC1/T1OSI/ECCP2/P2A); no longer U2001.33 (RC2/ECCP1/P1A)
- net SPI_SS3: no longer U2001.29 (RC1/T1OSI/ECCP2/P2A)
- net MCU_25Mhz: now reaches U2001.39 (OSC1/CLKI), U2002.3 (OUT)
- net AD5: now reaches U2001.16 (RF2/AN7/C1OUT)
- net AD4: now reaches U2001.17 (RF1/AN6/C2OUT)
- net AD1: now reaches U2001.21 (RA3/AN3/VREF+)
- net AD0: now reaches U2001.22 (RA2/AN2/VREF-)
- net AD3: now reaches U2001.27 (RA5/AN4)
- net AD2: now reaches U2001.28 (RA4/T0CKI)
- net DI0: now reaches U2001.3 (RB0/INT0/FLT0)
- net DI1: now reaches U2001.4 (RB1/INT1)
- net DI6: now reaches U2001.43 (RB5/KBI1)
- net DI5: now reaches U2001.44 (RB4/KBI0)
- net DI3: now reaches U2001.5 (RB2/INT2)
- net DI4: now reaches U2001.6 (RB3/INT3)
- net PGC renamed DI7
- net PGD renamed DI8
- no-connect marks 0 -> 1

Commit message: .
Connections:
- net DI0: now also U2001.15 (RF3/AN8); no longer U2001.3 (RB0/INT0/FLT0)
- net DO1: now reaches U2001.1 (RE1/P2C)
- net DI11: now reaches U2001.12 (RF6/AN11)
- net DI10: now reaches U2001.13 (RF5/AN10/CVREF)
- net DI9: now reaches U2001.14 (RF4/AN9)
- net DO0: now reaches U2001.2 (RE0/P2D)
- net DO8: now reaches U2001.58 (RD2/CCP4/P3D)
- net DO7: now reaches U2001.59 (RD1/ECCP3/P3A)
- net DO6: now reaches U2001.60 (RD0/P1B)
- net DO5: now reaches U2001.61 (RE5/P1C)
- net DO4: now reaches U2001.62 (RE4/P3B)
- net DO3: now reaches U2001.63 (RE3/P3C)
- net DO2: now reaches U2001.64 (RE2/P2B)
- net SPI_MISO renamed CAN_CTRL.MISO
- net CAN_CTRL.MISO: no longer U2003.3 (DI)
- net SPI_MOSI renamed CAN_CTRL.MOSI
- net CAN_CTRL.MOSI: now also U2003.3 (DI)
- net SPI_SCK renamed CAN_CTRL.SCK
- net SPI_SS2 renamed CAN_CTRL.CS#
- new net CAN_CTRL.INT#: U2001.3 (RB0/INT0/FLT0)
Other:
- moved on the sheet: C2002

Commit message: .
Connections:
- net +3.3V: no longer C2003.2, C2004.2, C2005.2, C2006.2, C2007.2, C2008.2, C2009.2
- net GND: now also C2003.2, C2004.2, C2005.2, C2006.2, C2007.2, C2008.2, C2009.2
- net RBIAS: now reaches R2004.1, U2001.53 (RBIAS)
- net RB_Split: now reaches R2004.2, R2005.1
Other:
- moved on the sheet: R2005
Changed lines of the file:
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@@
 	)
 	(junction
-		(at 351.79 46.99)
-		(diameter 0)
-		(color 0 0 0 0)
-	)
-	(junction
 		(at 121.92 257.81)
 		(diameter 0)
@@
 	)
 	(junction
-		(at 365.76 46.99)
-		(diameter 0)
-		(color 0 0 0 0)
-	)
-	(junction
 		(at 370.84 57.15)
 		(diameter 0)
@@
 	)
 	(junction
+		(at 323.85 46.99)
+		(diameter 0)
+		(color 0 0 0 0)
+	)
+	(junction
 		(at 228.6 82.55)
 		(diameter 0)
@@
 	(wire
 		(pts
-			(xy 328.93 46.99) (xy 318.77 46.99)
+			(xy 328.93 46.99) (xy 323.85 46.99)
 		)
 		(stroke
@@
 	(wire
 		(pts
+			(xy 236.22 177.8) (xy 248.92 177.8)
+		)
+		(stroke
+			(width 0)
+			(type default)
+		)
+	)
+	(wire
+		(pts
 			(xy 76.2 151.13) (xy 110.49 151.13)
 		)
@@
 	(wire
 		(pts
+			(xy 323.85 46.99) (xy 318.77 46.99)
+		)
+		(stroke
+			(width 0)
+			(type default)
+		)
+	)
+	(wire
+		(pts
 			(xy 365.76 26.67) (xy 365.76 29.21)
 		)
@@
 	(wire
 		(pts
+			(xy 323.85 46.99) (xy 323.85 52.07)
+		)
+		(stroke
+			(width 0)
+			(type default)
+		)
+	)
+	(wire
+		(pts
 			(xy 76.2 156.21) (xy 110.49 156.21)
 		)
@@
 	(wire
 		(pts
-			(xy 365.76 46.99) (xy 351.79 46.99)
-		)
-		(stroke
-			(width 0)
-			(type default)
-		)
-	)
-	(wire
-		(pts
 			(xy 260.35 96.52) (xy 260.35 99.06)
 		)
@@
 	(wire
 		(pts
-			(xy 255.27 177.8) (xy 255.27 181.61)
+			(xy 261.62 177.8) (xy 261.62 181.61)
 		)
 		(stroke
@@
 		)
 	)
-	(wire
-		(pts
-			(xy 236.22 177.8) (xy 242.57 177.8)
-		)
-		(stroke
-			(width 0)
-			(type default)
-		)
-	)
 	(bus
 		(pts
@@
 	(wire
 		(pts
-			(xy 250.19 177.8) (xy 255.27 177.8)
+			(xy 256.54 177.8) (xy 261.62 177.8)
 		)
 		(stroke
@@
 	(label "CAN_CTRL.SCK"
 		(at 210.82 229.87 180)
+		(fields_autoplaced yes)
 		(effects
 			(font
@@
 	(label "DO1"
 		(at 201.93 163.83 0)
+		(fields_autoplaced yes)
 		(effects
 			(font
@@
 	(label "DO3"
 		(at 201.93 168.91 0)
+		(fields_autoplaced yes)
 		(effects
 			(font
@@
 	(label "DO5"
 		(at 201.93 173.99 0)
+		(fields_autoplaced yes)
 		(effects
 			(font
@@
 	(label "CAN_CTRL.CS#"
 		(at 210.82 237.49 180)
+		(fields_autoplaced yes)
 		(effects
 			(font
@@
 	(label "CAN_CTRL.MOSI"
 		(at 210.82 234.95 180)
+		(fields_autoplaced yes)
 		(effects
 			(font
@@
 	(label "DI10"
 		(at 240.03 130.81 0)
+		(fields_autoplaced yes)
 		(effects
 			(font
@@
 		)
 	)
+	(label "RBIAS"
+		(at 205.74 177.8 0)
+		(fields_autoplaced yes)
+		(effects
+			(font
+				(size 1.27 1.27)
+			)
+			(justify left bottom)
+		)
+	)
 	(label "SPI_SCK"
 		(at 86.36 156.21 0)
@@
 	(label "CAN_CTRL.INT#"
 		(at 209.55 227.33 180)
+		(fields_autoplaced yes)
 		(effects
 			(font
@@
 		)
 	)
+	(label "RB_Split"
+		(at 238.76 177.8 0)
+		(fields_autoplaced yes)
+		(effects
+			(font
+				(size 1.27 1.27)
+			)
+			(justify left bottom)
+		)
+	)
 	(label "DI11"
 		(at 96.52 184.15 0)
@@
 	(label "DI9"
 		(at 240.03 128.27 0)
+		(fields_autoplaced yes)
 		(effects
 			(font
@@
 	(label "DO6"
 		(at 201.93 151.13 0)
+		(fields_autoplaced yes)
 		(effects
 			(font
@@
 	(label "DI11"
 		(at 240.03 133.35 0)
+		(fields_autoplaced yes)
 		(effects
 			(font
@@
 	(label "CAN_CTRL.MISO"
 		(at 210.82 232.41 180)
+		(fields_autoplaced yes)
 		(effects
 			(font
@@
 	(label "DO2"
 		(at 201.93 166.37 0)
+		(fields_autoplaced yes)
 		(effects
 			(font
@@
 	(label "DO4"
 		(at 201.93 171.45 0)
+		(fields_autoplaced yes)
 		(effects
 			(font
@@
 	(label "DO0"
 		(at 201.93 161.29 0)
+		(fields_autoplaced yes)
 		(effects
 			(font
@@
 	(label "DO7"
 		(at 201.93 153.67 0)
+		(fields_autoplaced yes)
 		(effects
 			(font
@@
 	(label "DO8"
 		(at 201.93 156.21 0)
+		(fields_autoplaced yes)
 		(effects
 			(font
@@
 	(symbol
 		(lib_id "power:GND")
+		(at 323.85 52.07 0)
+		(unit 1)
+		(exclude_from_sim no)
+		(in_bom yes)
+		(on_board yes)
+		(dnp no)
+		(fields_autoplaced yes)
+		(property "Reference" "#PWR02016"
+			(at 323.85 58.42 0)
+			(effects
+				(font
+					(size 1.27 1.27)
+				)
+				(hide yes)
+			)
+		)
+		(property "Value" "GND"
+			(at 323.85 57.15 0)
+			(effects
+				(font
+					(size 1.27 1.27)
+				)
+			)
+		)
+		(property "Footprint" ""
+			(at 323.85 52.07 0)
+			(effects
+				(font
+					(size 1.27 1.27)
+				)
+				(hide yes)
+			)
+		)
+		(property "Datasheet" ""
+			(at 323.85 52.07 0)
+			(effects
+				(font
+					(size 1.27 1.27)
+				)
+				(hide yes)
+			)
+		)
+		(property "Description" "Power symbol creates a global label with name \"GND\" , ground"
+			(at 323.85 52.07 0)
+			(effects
+				(font
+					(size 1.27 1.27)
+				)
+				(hide yes)
+			)
+		)
+		(pin "1"
+		)
+		(instances
+			(project "PIC18F_ETH"
+				(path "/26a36835-4e01-4565-9612-f38560505464/ad2b3e7b-516f-4805-aaab-2158978e44df"
+					(reference "#PWR02016")
+					(unit 1)
+				)
+			)
+		)
+	)
+	(symbol
+		(lib_id "power:GND")
 		(at 370.84 69.85 0)
 		(unit 1)
@@
 	(symbol
 		(lib_id "power:GND")
-		(at 255.27 181.61 0)
+		(at 261.62 181.61 0)
 		(unit 1)
 		(exclude_from_sim no)
@@
 		(fields_autoplaced yes)
 		(property "Reference" "#PWR02013"
-			(at 255.27 187.96 0)
+			(at 261.62 187.96 0)
 			(effects
 				(font
@@
 		)
 		(property "Value" "GND"
-			(at 255.27 186.69 0)
+			(at 261.62 186.69 0)
 			(effects
 				(font
@@
 		)
 		(property "Footprint" ""
-			(at 255.27 181.61 0)
+			(at 261.62 181.61 0)
 			(effects
 				(font
@@
 		)
 		(property "Datasheet" ""
-			(at 255.27 181.61 0)
+			(at 261.62 181.61 0)
 			(effects
 				(font
@@
 		)
 		(property "Description" "Power symbol creates a global label with name \"GND\" , ground"
-			(at 255.27 181.61 0)
+			(at 261.62 181.61 0)
 			(effects
 				(font
@@
 	(symbol
 		(lib_id "bt_resistors:R;G;620R;10P0;S;0603")
-		(at 246.38 177.8 90)
+		(at 252.73 177.8 90)
 		(unit 1)
 		(exclude_from_sim no)
@@
 		(fields_autoplaced yes)
 		(property "Reference" "R2005"
-			(at 246.38 171.45 90)
+			(at 252.73 171.45 90)
 			(effects
 				(font
@@
 		)
 		(property "Value" "620R"
-			(at 246.38 173.99 90)
+			(at 252.73 173.99 90)
 			(effects
 				(font
@@
 		)
 		(property "Footprint" "Resistor_SMD:R_0603_1608Metric"
-			(at 246.38 179.578 90)
+			(at 252.73 179.578 90)
 			(effects
 				(font
@@
 		)
 		(property "Datasheet" "~"
-			(at 246.38 177.8 0)
+			(at 252.73 177.8 0)
 			(effects
 				(font
@@
 		)
 		(property "Description" "Resistor"
-			(at 246.38 177.8 0)
+			(at 252.73 177.8 0)
 			(effects
 				(font
@@
 		)
 		(property "MPN" "R;G;T1;S;P0603;NA"
-			(at 246.38 177.8 90)
+			(at 252.73 177.8 90)
 			(effects
 				(font
@@
 		)
 		(property "CPN" "BT00002-06200"
-			(at 246.38 177.8 90)
+			(at 252.73 177.8 90)
 			(effects
 				(font

Commit message: .
Connections:
- net ETH.RX+: no longer U2001.46 (TPIN-)
- new net ETH.RX-: U2001.46 (TPIN-)
Changed lines of the file:
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@@
 		)
 	)
-	(label "ETH.RX+"
+	(label "ETH.RX-"
 		(at 214.63 189.23 0)
 		(fields_autoplaced yes)

Commit message: .
Parts:
- renumbered C2011 to C2003, C2003 to C2004, C2004 to C2005, C2005 to C2006, C2006 to C2007, C2007 to C2008, C2008 to C2009, C2009 to C2010, C2010 to C2011, R2002 to R2001, R2003 to R2002, R2004 to R2003, R2001 to R2004, U2003 to U2001, U2001 to U2002, U2002 to U2003

Commit message: .
Connections:
- net DI0: no longer names the net of U2002.15 (RF3/AN8)
- net DI1 renamed SPI_DI.INT#
- net DI10: no longer names the net of U2002.13 (RF5/AN10/CVREF)
- net DI11: no longer names the net of U2002.12 (RF6/AN11)
- net DI3 renamed SPI_INT2#
- net DI4: no longer names the net of U2002.6 (RB3/INT3)
- net DI5: no longer names the net of U2002.44 (RB4/KBI0)
- net DI6: no longer names the net of U2002.43 (RB5/KBI1)
- net DI7 renamed PGC
- net DI8 renamed PGD
- net DI9: no longer names the net of U2002.14 (RF4/AN9)
- no-connect marks 1 -> 2
