File: HW/PIC18F_ETH/PIC18F_ETH/MCU_core.kicad_sch (KiCad schematic)
At the start: 20 parts, among them J2001 Conn_01x06, U2001 93AA46BT-I/OT, U2002 PIC18F67J60T-I, U2003 25Mhz,50ppm

Commit message: .
Connections:
- net SPI_INT2# renamed SPI_DI.INT1#

Commit message: .
Connections:
- net CAN_CTRL.CS#: now also U2002.33 (RC2/ECCP1/P1A); no longer U2002.29 (RC1/T1OSI/ECCP2/P2A)
- net SPI_SS0: now reaches U2002.11 (RF7/*SS1)
- net SPI_SS0: now also R2001.1, U2001.5 (CS)
- removed net SPI_SS1: R2001.1, U2001.5 (CS), U2002.33 (RC2/ECCP1/P1A)
- new net SPI_DI.CS#: U2002.29 (RC1/T1OSI/ECCP2/P2A)
Changed lines of the file:
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@@
+		)
+	)
+	(label "SPI_SS0"
+		(at 86.36 186.69 0)
+		(fields_autoplaced yes)
+		(effects
+			(font
+				(size 1.27 1.27)
+			)
+			(justify left bottom)
 		)
 	)
@@
 		)
 	)
-	(label "SPI_SS1"
+	(label "SPI_SS0"
 		(at 41.91 257.81 0)
 		(fields_autoplaced yes)
@@
 		)
 	)
-	(label "SPI_SS2"
+	(label "SPI_SS1"
 		(at 163.83 237.49 0)
 		(fields_autoplaced yes)
@@
 	(label "SPI_DI.INT1#"
 		(at 314.96 125.73 0)
-		(effects
-			(font
+		(fields_autoplaced yes)
+		(effects
+			(font

Commit message: .
Parts:
- added TP2001, TP2002, TP2003, TP2004, TP2006, TP2007, TP2008, TP2009, TP2010, TP2011, TP2012: TestPoint, TestPoint:TestPoint_THTPad_D1.0mm_Drill0.5mm, symbol bt_misc:TestPoint_THD
- added TP2005, TP2015, TP2016: TestPoint, TestPoint:TestPoint_THTPad_1.0x1.0mm_Drill0.5mm, symbol bt_misc:TestPoint_SQU
Connections:
- net CAN_CTRL.CS#: now also TP2007.1
- net CAN_CTRL.MISO: now also TP2009.1
- net CAN_CTRL.MOSI: now also TP2010.1
- net CAN_CTRL.SCK: now also TP2008.1
- net GND: now also TP2005.1, TP2015.1, TP2016.1
- net LED_A: now also TP2001.1
- net LED_B: now also TP2002.1
- net RST#: now also TP2012.1
- net SPI_DI.CS#: now also TP2006.1
- net SPI_SS0: now also TP2011.1
- net UART_RX: now also TP2003.1
- net UART_TX: now also TP2004.1

Commit message: .
Parts:
- added C2012: 100n 25V, Capacitor_SMD:C_0603_1608Metric, symbol bt_capacitor:C;M;100n;10p;25V;S;0603
Connections:
- net GND: now also C2012.2
- net RST#: now also C2012.1
Changed lines of the file:
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@@
 	)
 	(junction
+		(at 107.95 123.19)
+		(diameter 0)
+		(color 0 0 0 0)
+	)
+	(junction
 		(at 228.6 82.55)
 		(diameter 0)
@@
 		)
 	)
+	(wire
+		(pts
+			(xy 107.95 123.19) (xy 110.49 123.19)
+		)
+		(stroke
+			(width 0)
+			(type default)
+		)
+	)
 	(bus
 		(pts
@@
 	(wire
 		(pts
+			(xy 73.66 125.73) (xy 107.95 125.73)
+		)
+		(stroke
+			(width 0)
+			(type default)
+		)
+	)
+	(wire
+		(pts
 			(xy 323.85 46.99) (xy 323.85 52.07)
 		)
@@
 	(wire
 		(pts
+			(xy 107.95 125.73) (xy 107.95 123.19)
+		)
+		(stroke
+			(width 0)
+			(type default)
+		)
+	)
+	(wire
+		(pts
 			(xy 242.57 85.09) (xy 242.57 82.55)
 		)
@@
 	(wire
 		(pts
-			(xy 92.71 123.19) (xy 110.49 123.19)
+			(xy 92.71 123.19) (xy 107.95 123.19)
 		)
 		(stroke
@@
 	)
 	(symbol
+		(lib_id "bt_capacitor:C;M;100n;10p;25V;S;0603")
+		(at 69.85 125.73 270)
+		(unit 1)
+		(exclude_from_sim no)
+		(in_bom yes)
+		(on_board yes)
+		(dnp no)
+		(property "Reference" "C2012"
+			(at 72.136 127.254 90)
+			(effects
+				(font
+					(size 1.27 1.27)
+				)
+				(justify left)
+			)
+		)
+		(property "Value" "100n 25V"
+			(at 65.024 121.92 90)
+			(effects
+				(font
+					(size 1.27 1.27)
+				)
+				(justify left)
+			)
+		)
+		(property "Footprint" "Capacitor_SMD:C_0603_1608Metric"
+			(at 69.85 122.952 90)
+			(effects
+				(font
+					(size 1.27 1.27)
+				)
+				(hide yes)
+			)
+		)
+		(property "Datasheet" "~"
+			(at 69.85 125.73 0)
+			(effects
+				(font
+					(size 1.27 1.27)
+				)
+				(hide yes)
+			)
+		)
+		(property "Description" "Capacitor"
+			(at 69.85 125.73 0)
+			(effects
+				(font
+					(size 1.27 1.27)
+				)
+				(hide yes)
+			)
+		)
+		(property "MPN" "C;C;T1;S;P0603;NA"
+			(at 69.85 129.73 90)
+			(effects
+				(font
+					(size 1.27 1.27)
+				)
+				(hide yes)
+			)
+		)
+		(property "CPN" "BT00008-090680"
+			(at 69.85 129.73 90)
+			(effects
+				(font
+					(size 1.27 1.27)
+				)
+				(hide yes)
+			)
+		)
+		(pin "1"
+		)
+		(pin "2"
+		)
+		(instances
+			(project "PIC18F_ETH"
+				(path "/26a36835-4e01-4565-9612-f38560505464/ad2b3e7b-516f-4805-aaab-2158978e44df"
+					(reference "C2012")
+					(unit 1)
+				)
+			)
+		)
+	)
+	(symbol
 		(lib_id "bt_misc:TestPoint_SQU")
 		(at 67.31 162.56 0)
@@
 					(unit 1)
 				)
+			)
+		)
+	)
+	(symbol
+		(lib_id "power:GND")
+		(at 66.04 125.73 270)
+		(unit 1)
+		(exclude_from_sim no)
+		(in_bom yes)
+		(on_board yes)
+		(dnp no)
+		(fields_autoplaced yes)
+		(property "Reference" "#PWR02020"
+			(at 59.69 125.73 0)
+			(effects
+				(font
+					(size 1.27 1.27)
+				)
+				(hide yes)
+			)
+		)
+		(property "Value" "GND"
+			(at 60.96 125.73 0)
+			(effects
+				(font
+					(size 1.27 1.27)
+				)
+			)
+		)
+		(property "Footprint" ""
+			(at 66.04 125.73 0)
+			(effects
+				(font
+					(size 1.27 1.27)
+				)
+				(hide yes)
+			)
+		)
+		(property "Datasheet" ""
+			(at 66.04 125.73 0)
+			(effects
+				(font
+					(size 1.27 1.27)
+				)
+				(hide yes)
+			)
+		)
+		(property "Description" "Power symbol creates a global label with name \"GND\" , ground"
+			(at 66.04 125.73 0)
+			(effects
+				(font
+					(size 1.27 1.27)
+				)
+				(hide yes)
+			)
+		)
+		(pin "1"
+		)
+		(instances
+			(project "PIC18F_ETH"
+				(path "/26a36835-4e01-4565-9612-f38560505464/ad2b3e7b-516f-4805-aaab-2158978e44df"
+					(reference "#PWR02020")
+					(unit 1)
+				)

Commit message: .
Connections:
- no-connect marks 2 -> 22

Commit message: .
Connections:
- net DO0: no longer names the net of U2002.2 (RE0/P2D)
- net DO1: no longer names the net of U2002.1 (RE1/P2C)
- net DO2: no longer names the net of U2002.64 (RE2/P2B)
- net DO3: no longer names the net of U2002.63 (RE3/P3C)
- net DO4: no longer names the net of U2002.62 (RE4/P3B)
- net DO5: no longer names the net of U2002.61 (RE5/P1C)
- net DO6: no longer names the net of U2002.60 (RD0/P1B)
- net DO7: no longer names the net of U2002.59 (RD1/ECCP3/P3A)
- net DO8: no longer names the net of U2002.58 (RD2/CCP4/P3D)
Other:
- title: (none) -> BT_ADDX
- moved on the sheet: C2001, C2002, J2001, R2001, TP2005, TP2015, U2001

Commit message: .
Parts:
- removed TP2003, TP2004: TestPoint, TestPoint:TestPoint_THTPad_D1.0mm_Drill0.5mm, symbol bt_misc:TestPoint_THD
- removed TP2015: TestPoint, TestPoint:TestPoint_THTPad_1.0x1.0mm_Drill0.5mm, symbol bt_misc:TestPoint_SQU
- added J2002: JST,2.54, Connector_JST:JST_EH_B3B-EH-A_1x03_P2.50mm_Vertical, symbol bt_connector:M;JST;01x03;2.54
Connections:
- net GND: now also J2002.1 (Pin_1)
- net UART_RX: now also J2002.2 (Pin_2)
- net UART_TX: now also J2002.3 (Pin_3)
Other:
- title: BT_ADDX -> BT_AD/DX

Commit message: .
Parts:
- added R2006, R2007, R2008, R2009, R2010: 10K, Resistor_SMD:R_0603_1608Metric, symbol bt_resistors:R;G;10K;10P0;S;0603
Connections:
- net +3.3V: now also R2006.1, R2007.1, R2008.1, R2009.1, R2010.1
- net CAN_CTRL.CS#: now also R2007.2
- net CAN_CTRL.INT#: now also R2009.2
- net SPI_DI.CS#: now also R2006.2
- net SPI_DI.INT#: now also R2008.2
- net SPI_DI.INT1#: now also R2010.2
- net SPI_SS3: no longer names the net of U2002.30 (RC0/T1OSO/T13CKI)
- no-connect marks 22 -> 20
