File: HW/PIC18F_ETH/PIC18F_ETH/MCU_core.kicad_sch (KiCad schematic)
At the start: 38 parts, among them J2001 Conn_01x06, J2002 JST,2.54, U2001 93AA46BT-I/OT, U2002 PIC18F67J60T-I, U2003 25Mhz,50ppm

Commit message: .
Parts:
- C2001, C2002, C2003, C2004, C2005, C2006, C2007, C2008, C2009, C2010, C2012: MPN C;C;T1;S;P0603;NA -> C;M;100n;10p;25V;S;0603
- C2011: MPN C;C;T1;S;P0603;NA -> C;M;10u;10p;10V;S;0603
- R2001, R2002, R2004, R2006, R2007, R2008, R2009, R2010: MPN R;G;T1;S;P0603;NA -> R;G;10K;10P0;S;0603
- R2003: MPN R;G;T1;S;P0603;NA -> R;G;2K2;10P0;S;0603
- R2005: MPN R;G;T1;S;P0603;NA -> R;G;620R;10P0;S;0603
- U2002: CPN BT01004-00001 -> BT01005-00001
Connections:
- net +3.3V: no longer U2002.18 (ENVREG), U2002.38 (VDD), U2002.48 (VDDRX), U2002.49 (VDDTX), U2002.54 (VDDPLL), U2002.57 (VDD)
- net GND: no longer U2002.20 (AVSS), U2002.25 (VSS), U2002.41 (VSS), U2002.45 (VSSRX), U2002.52 (VSSTX), U2002.55 (VSSPLL), U2002.56 (VSS), U2002.9 (VSS)
- net at U2002.10 (VDDCORE/VCAP): no longer C2011.1
Changed lines of the file:
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@@
 			)
 		)
-		(property "MPN" "C;C;T1;S;P0603;NA"
+		(property "MPN" "C;M;100n;10p;25V;S;0603"
 			(at 69.85 129.73 90)
 			(effects
@@
 			)
 		)
-		(property "MPN" "R;G;T1;S;P0603;NA"
+		(property "MPN" "R;G;10K;10P0;S;0603"
 			(at 276.86 166.37 90)
 			(effects
@@
 			)
 		)
-		(property "MPN" "R;G;T1;S;P0603;NA"
+		(property "MPN" "R;G;10K;10P0;S;0603"
 			(at 242.57 88.9 90)
 			(effects
@@
 			)
 		)
-		(property "MPN" "R;G;T1;S;P0603;NA"
+		(property "MPN" "R;G;10K;10P0;S;0603"
 			(at 92.71 113.03 90)
 			(effects
@@
 			)
 		)
-		(property "MPN" "C;C;T1;S;P0603;NA"
+		(property "MPN" "C;M;100n;10p;25V;S;0603"
 			(at 311.34 38.1 90)
 			(effects
@@
 			)
 		)
-		(property "MPN" "R;G;T1;S;P0603;NA"
+		(property "MPN" "R;G;10K;10P0;S;0603"
 			(at 274.32 116.84 90)
 			(effects
@@
 			)
 		)
-		(property "CPN" "BT01004-00001"
+		(property "CPN" "BT01005-00001"
 			(at 374.65 33.02 0)
 			(effects
@@
 			)
 		)
-		(property "MPN" "R;G;T1;S;P0603;NA"
+		(property "MPN" "R;G;10K;10P0;S;0603"
 			(at 62.23 237.49 90)
 			(effects
@@
 			)
 		)
-		(property "CPN" "BT01004-00001"
+		(property "CPN" "BT01005-00001"
 			(at 110.49 123.19 0)
 			(effects
@@
 			)
 		)
-		(property "MPN" "C;C;T1;S;P0603;NA"
+		(property "MPN" "C;M;100n;10p;25V;S;0603"
 			(at 170.37 243.84 90)
 			(effects
@@
 			)
 		)
-		(property "MPN" "R;G;T1;S;P0603;NA"
+		(property "MPN" "R;G;10K;10P0;S;0603"
 			(at 290.83 167.64 90)
 			(effects
@@
 			)
 		)
-		(property "MPN" "C;C;T1;S;P0603;NA"
+		(property "MPN" "C;M;100n;10p;25V;S;0603"
 			(at 344.36 38.1 90)
 			(effects
@@
 			)
 		)
-		(property "MPN" "R;G;T1;S;P0603;NA"
+		(property "MPN" "R;G;10K;10P0;S;0603"
 			(at 281.94 116.84 90)
 			(effects
@@
 			)
 		)
-		(property "MPN" "C;C;T1;S;P0603;NA"
+		(property "MPN" "C;M;100n;10p;25V;S;0603"
 			(at 322.77 38.1 90)
 			(effects
@@
 			)
 		)
-		(property "MPN" "C;C;T1;S;P0603;NA"
+		(property "MPN" "C;M;100n;10p;25V;S;0603"
 			(at 288.48 38.1 90)
 			(effects
@@
 			)
 		)
-		(property "MPN" "C;C;T1;S;P0603;NA"
+		(property "MPN" "C;M;100n;10p;25V;S;0603"
 			(at 264.35 92.71 90)
 			(effects
@@
 			)
 		)
-		(property "MPN" "R;G;T1;S;P0603;NA"
+		(property "MPN" "R;G;2K2;10P0;S;0603"
 			(at 232.41 177.8 90)
 			(effects
@@
 			)
 		)
-		(property "MPN" "C;C;T1;S;P0603;NA"
+		(property "MPN" "C;M;100n;10p;25V;S;0603"
 			(at 101.79 247.65 90)
 			(effects
@@
 			)
 		)
-		(property "MPN" "C;C;T1;S;P0603;NA"
+		(property "MPN" "C;M;100n;10p;25V;S;0603"
 			(at 332.93 38.1 90)
 			(effects
@@
 			)
 		)
-		(property "MPN" "C;C;T1;S;P0603;NA"
+		(property "MPN" "C;M;100n;10p;25V;S;0603"
 			(at 355.79 38.1 90)
 			(effects
@@
 			)
 		)
-		(property "MPN" "C;C;T1;S;P0603;NA"
+		(property "MPN" "C;M;100n;10p;25V;S;0603"
 			(at 299.91 38.1 90)
 			(effects
@@
 			)
 		)
-		(property "MPN" "C;C;T1;S;P0603;NA"
+		(property "MPN" "C;M;10u;10p;10V;S;0603"
 			(at 355.79 53.34 90)
 			(effects
@@
 			)
 		)
-		(property "MPN" "R;G;T1;S;P0603;NA"
+		(property "MPN" "R;G;620R;10P0;S;0603"
 			(at 252.73 177.8 90)
 			(effects
@@
 			)
 		)
-		(property "MPN" "R;G;T1;S;P0603;NA"
+		(property "MPN" "R;G;10K;10P0;S;0603"
 			(at 292.1 116.84 90)
 			(effects

Commit message: .
Connections:
- net +3.3V: now also U2002.38 (VDD), U2002.48 (VDDRX), U2002.49 (VDDTX), U2002.54 (VDDPLL), U2002.57 (VDD)
- net GND: now also U2002.20 (AVSS), U2002.25 (VSS), U2002.41 (VSS), U2002.45 (VSSRX), U2002.52 (VSSTX), U2002.55 (VSSPLL), U2002.56 (VSS), U2002.9 (VSS)
- net at U2002.10 (VDDCORE/VCAP): now also C2011.1
Other:
- moved on the sheet: C2004, C2005, C2006, C2007, C2008, C2009, C2010, C2011, C2012, R2002, TP2012, TP2016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
