File: HW/PIC18F_ETH/PIC18F_ETH/Power.kicad_sch (KiCad schematic)
At the start: 18 parts, among them J3001 Jack-DC, U3001 LMR51610-Q1, U3002 TPS62A01

Commit message: .
Parts:
- removed J3001: Jack-DC, Connector_BarrelJack:BarrelJack_Horizontal, symbol Connector:Jack-DC
- added D3001: D, Diode_SMD:D_0805_2012Metric, symbol Device:D
- added J3001: Screw_Terminal_01x02, Connector_Samtec_HPM_THT:Samtec_HPM-02-01-x-S_Straight_1x02_Pitch5.08mm, symbol Connector:Screw_Terminal_01x02
- renumbered C3006 to C3002, C3002 to C3003, C3003 to C3004, C3007 to C3005, C3004 to C3006, C3008 to C3007, C3005 to C3008, R3006 to R3003, R3007 to R3004, R3008 to R3005
Connections:
- net GND: now also J3001.1 (Pin_1)
- net at C3001.1, U3001.4 (EN), U3001.5 (V_{IN}): now also D3001.1 (K)
- new net: D3001.2 (A), J3001.2 (Pin_2)
