File: HW/PIC18F_ETH/PIC18F_ETH/Power.kicad_sch (KiCad schematic)
At the start: 19 parts, among them J3001 Screw_Terminal_01x02, U3001 LMR51610-Q1, U3002 TPS62A01

Commit message: .
Parts:
- added D3002: LED G, LED_SMD:LED_0603_1608Metric, symbol bt_opto:D;LED;G;2V;25mA
- added R3006: 200R, Resistor_SMD:R_0603_1608Metric, symbol bt_resistors:R;G;200R;10P0;S;0603
Connections:
- net +3.3V: now also R3006.2
- net GND: now also D3002.1 (K)
- new net: D3002.2 (A), R3006.1

Commit message: .
Parts:
- added C3009: 3n3 50V, Capacitor_SMD:C_0603_1608Metric, symbol bt_capacitor:C;M;3n3;10p;50V;S;0603
- added TP3001, TP3003, TP3005: TestPoint, TestPoint:TestPoint_THTPad_D1.0mm_Drill0.5mm, symbol bt_misc:TestPoint_THD
- added TP3002, TP3004: TestPoint, TestPoint:TestPoint_THTPad_1.0x1.0mm_Drill0.5mm, symbol bt_misc:TestPoint_SQU
Connections:
- net +3.3V: now also TP3005.1
- net +5V: now also TP3003.1
- net GND: now also C3009.2, TP3002.1, TP3004.1
- net at C3001.1, D3001.1 (K), U3001.4 (EN)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: now also C3009.1
- net at D3001.2 (A), J3001.2 (Pin_2): now also TP3001.1

Commit message: .
Parts:
- added J3002: JST,2.54, Connector_JST:JST_EH_B2B-EH-A_1x02_P2.50mm_Vertical, symbol bt_connector:M;JST;01x02;2.54
- added TP3006: TestPoint, TestPoint:TestPoint_THTPad_1.0x1.0mm_Drill0.5mm, symbol bt_misc:TestPoint_SQU
Connections:
- net +3.3V: now also J3002.1 (Pin_1)
- net GND: now also J3002.2 (Pin_2), TP3006.1
