File: HW/PIC18F_ETH/PIC18F_ETH/Power.kicad_sch (KiCad schematic)
At the start: 29 parts, among them J3001 Screw_Terminal_01x02, J3002 JST,2.54, U3001 LMR51610-Q1, U3002 TPS62A01

Commit message: .
Other:
- moved on the sheet: TP3005
Changed lines of the file:
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@@
 	)
 	(junction
-		(at 270.51 196.85)
+		(at 265.43 195.58)
 		(diameter 0)
 		(color 0 0 0 0)
@@
 	)
 	(junction
+		(at 265.43 201.93)
+		(diameter 0)
+		(color 0 0 0 0)
+	)
+	(junction
 		(at 173.99 121.92)
 		(diameter 0)
@@
 	(wire
 		(pts
+			(xy 265.43 201.93) (xy 270.51 201.93)
+		)
+		(stroke
+			(width 0)
+			(type default)
+		)
+	)
+	(wire
+		(pts
 			(xy 115.57 213.36) (xy 115.57 222.25)
 		)
@@
 	(wire
 		(pts
-			(xy 270.51 193.04) (xy 270.51 196.85)
+			(xy 265.43 191.77) (xy 265.43 195.58)
 		)
 		(stroke
@@
 	(wire
 		(pts
-			(xy 270.51 196.85) (xy 270.51 201.93)
+			(xy 265.43 195.58) (xy 265.43 201.93)
 		)
 		(stroke
@@
 	(wire
 		(pts
-			(xy 242.57 201.93) (xy 270.51 201.93)
+			(xy 242.57 201.93) (xy 265.43 201.93)
 		)
 		(stroke
@@
 	(symbol
 		(lib_id "bt_misc:TestPoint_THD")
-		(at 270.51 196.85 0)
+		(at 265.43 195.58 0)
 		(unit 1)
 		(exclude_from_sim no)
@@
 		(fields_autoplaced yes)
 		(property "Reference" "TP3005"
-			(at 273.05 196.8499 0)
+			(at 267.97 195.5799 0)
 			(effects
 				(font
@@
 		)
 		(property "Value" "TestPoint"
-			(at 270.51 194.818 0)
+			(at 265.43 193.548 0)
 			(effects
 				(font
@@
 		)
 		(property "Footprint" "TestPoint:TestPoint_THTPad_D1.0mm_Drill0.5mm"
-			(at 275.844 200.914 0)
+			(at 270.764 199.644 0)
 			(effects
 				(font
@@
 		)
 		(property "Datasheet" "~"
-			(at 275.59 196.85 0)
+			(at 270.51 195.58 0)
 			(effects
 				(font
@@
 		)
 		(property "Description" "test point"
-			(at 263.906 198.374 0)
+			(at 258.826 197.104 0)
 			(effects
 				(font
@@
 	(symbol
 		(lib_id "power:+3.3V")
-		(at 270.51 193.04 0)
+		(at 265.43 191.77 0)
 		(unit 1)
 		(exclude_from_sim no)
@@
 		(fields_autoplaced yes)
 		(property "Reference" "#PWR03010"
-			(at 270.51 196.85 0)
+			(at 265.43 195.58 0)
 			(effects
 				(font
@@
 		)
 		(property "Value" "+3.3V"
-			(at 270.51 187.96 0)
+			(at 265.43 186.69 0)
 			(effects
 				(font
@@
 		)
 		(property "Footprint" ""
-			(at 270.51 193.04 0)
+			(at 265.43 191.77 0)
 			(effects
 				(font
@@
 		)
 		(property "Datasheet" ""
-			(at 270.51 193.04 0)
+			(at 265.43 191.77 0)
 			(effects
 				(font
@@
 		)
 		(property "Description" "Power symbol creates a global label with name \"+3.3V\""
-			(at 270.51 193.04 0)
+			(at 265.43 191.77 0)
 			(effects
 				(font

Commit message: .
Parts:
- C3001: value C_Polarized -> 4,7uF 100V
- C3002, C3004, C3006, C3008: value 10u 10V -> 10u 50V; symbol bt_capacitor:C;M;10u;10p;10V;S;0603 -> bt_capacitor:C;M;10u;10p;50V;S;0603; CPN BT00010-060100 -> BT00007-060100
- C3009: value 3n3 50V -> 100n 100V; symbol bt_capacitor:C;M;3n3;10p;50V;S;0603 -> bt_capacitor:C;M;100n;10p;100V;S;0603; CPN BT00007-090033 -> BT00013-090680; MPN C;C;T1;S;P0603;NA -> C;M;100n;10p;100V;S;0603
- J3001: value Screw_Terminal_01x02 -> 6-40V
- R3001: value 160K -> 16K; symbol bt_resistors:R;G;160K;10P0;S;0603 -> bt_resistors:R;G;16K;10P0;S;0603; CPN BT00002-31600 -> BT00002-30160
- R3002: value 30K -> 3K; symbol bt_resistors:R;G;30K;10P0;S;0603 -> bt_resistors:R;G;3K;10P0;S;0603; CPN BT00002-30300 -> BT00002-30030
Other:
- title: (none) -> BT_ADDX
Changed lines of the file:
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@@
 	(generator_version "8.0")
 	(paper "A3")
+	(title_block
+		(title "BT_ADDX")
+		(rev "Rev:P1")
+	)
 	(junction
 		(at 90.17 119.38)
@@
 	)
 	(symbol
-		(lib_id "bt_resistors:R;G;30K;10P0;S;0603")
+		(lib_id "bt_resistors:R;G;3K;10P0;S;0603")
 		(at 204.47 138.43 0)
 		(unit 1)
@@
 			)
 		)
-		(property "Value" "30K"
+		(property "Value" "3K"
 			(at 207.01 139.6999 0)
 			(effects
@@
 			)
 		)
-		(property "CPN" "BT00002-30300"
+		(property "CPN" "BT00002-30030"
 			(at 204.47 138.43 90)
 			(effects
@@
 	)
 	(symbol
-		(lib_id "bt_capacitor:C;M;10u;10p;10V;S;0603")
+		(lib_id "bt_capacitor:C;M;10u;10p;50V;S;0603")
 		(at 219.71 133.35 0)
 		(unit 1)
@@
 			)
 		)
-		(property "Value" "10u 10V"
+		(property "Value" "10u 50V"
 			(at 223.52 134.6199 0)
 			(effects
@@
 			)
 		)
-		(property "CPN" "BT00010-060100"
+		(property "CPN" "BT00007-060100"
 			(at 223.71 133.35 90)
 			(effects
@@
 			)
 		)
-		(property "Value" "C_Polarized"
+		(property "Value" "4,7uF 100V"
 			(at 110.49 129.9209 0)
 			(effects
@@
 	)
 	(symbol
-		(lib_id "bt_capacitor:C;M;10u;10p;10V;S;0603")
+		(lib_id "bt_capacitor:C;M;10u;10p;50V;S;0603")
 		(at 236.22 133.35 0)
 		(unit 1)
@@
 			)
 		)
-		(property "Value" "10u 10V"
+		(property "Value" "10u 50V"
 			(at 240.03 134.6199 0)
 			(effects
@@
 			)
 		)
-		(property "CPN" "BT00010-060100"
+		(property "CPN" "BT00007-060100"
 			(at 240.22 133.35 90)
 			(effects
@@
 	)
 	(symbol
-		(lib_id "bt_resistors:R;G;160K;10P0;S;0603")
+		(lib_id "bt_resistors:R;G;16K;10P0;S;0603")
 		(at 204.47 128.27 0)
 		(unit 1)
@@
 			)
 		)
-		(property "Value" "160K"
+		(property "Value" "16K"
 			(at 207.01 129.5399 0)
 			(effects
@@
 			)
 		)
-		(property "CPN" "BT00002-31600"
+		(property "CPN" "BT00002-30160"
 			(at 204.47 128.27 90)
 			(effects
@@
 	)
 	(symbol
-		(lib_id "bt_capacitor:C;M;3n3;10p;50V;S;0603")
+		(lib_id "bt_capacitor:C;M;100n;10p;100V;S;0603")
 		(at 124.46 129.54 0)
 		(unit 1)
@@
 			)
 		)
-		(property "Value" "3n3 50V"
+		(property "Value" "100n 100V"
 			(at 128.27 130.8099 0)
 			(effects
@@
 			)
 		)
-		(property "MPN" "C;C;T1;S;P0603;NA"
+		(property "MPN" "C;M;100n;10p;100V;S;0603"
 			(at 128.46 129.54 90)
 			(effects
@@
 			)
 		)
-		(property "CPN" "BT00007-090033"
+		(property "CPN" "BT00013-090680"
 			(at 128.46 129.54 90)
 			(effects
@@
 	)
 	(symbol
-		(lib_id "bt_capacitor:C;M;10u;10p;10V;S;0603")
+		(lib_id "bt_capacitor:C;M;10u;10p;50V;S;0603")
 		(at 115.57 209.55 0)
 		(unit 1)
@@
 			)
 		)
-		(property "Value" "10u 10V"
+		(property "Value" "10u 50V"
 			(at 119.38 210.8199 0)
 			(effects
@@
 			)
 		)
-		(property "CPN" "BT00010-060100"
+		(property "CPN" "BT00007-060100"
 			(at 119.57 209.55 90)
 			(effects
@@
 		(on_board yes)
 		(dnp no)
-		(fields_autoplaced yes)
 		(property "Reference" "J3001"
-			(at 82.55 113.03 0)
-			(effects
-				(font
-					(size 1.27 1.27)
-				)
-			)
-		)
-		(property "Value" "Screw_Terminal_01x02"
-			(at 82.55 115.57 0)
+			(at 80.264 116.586 0)
+			(effects
+				(font
+					(size 1.27 1.27)
+				)
+			)
+		)
+		(property "Value" "6-40V"
+			(at 77.47 120.396 0)
 			(effects
 				(font
@@
 		(on_board yes)
 		(dnp no)
-		(fields_autoplaced yes)
 		(property "Reference" "TP3001"
-			(at 92.71 119.3799 0)
+			(at 87.63 117.094 0)
 			(effects
 				(font
@@
 	)
 	(symbol
-		(lib_id "bt_capacitor:C;M;10u;10p;10V;S;0603")
+		(lib_id "bt_capacitor:C;M;10u;10p;50V;S;0603")
 		(at 251.46 133.35 0)
 		(unit 1)
@@
 			)
 		)
-		(property "Value" "10u 10V"
+		(property "Value" "10u 50V"
 			(at 255.27 134.6199 0)
 			(effects
@@
 			)
 		)
-		(property "CPN" "BT00010-060100"
+		(property "CPN" "BT00007-060100"
 			(at 255.46 133.35 90)
 			(effects

Commit message: .
Other:
- title: BT_ADDX -> BT_AD/DX
Changed lines of the file:
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@@
 	(paper "A3")
 	(title_block
-		(title "BT_ADDX")
+		(title "BT_AD/DX")
 		(rev "Rev:P1")
+		(comment 1 "BT_0001-1")
 	)
 	(junction

Commit message: .
Parts:
- C3002, C3004, C3006, C3008: MPN C;C;T1;S;P0603;NA -> C;M;10u;10p;50V;S;0603
- C3003: MPN C;C;T1;S;P0603;NA -> C;M;100n;10p;25V;S;0603
- C3005, C3007: MPN C;C;T1;S;P0603;NA -> C;M;10u;10p;10V;S;0603
- R3001: MPN R;G;T1;S;P0603;NA -> R;G;16K;10P0;S;0603
- R3002: MPN R;G;T1;S;P0603;NA -> R;G;3K;10P0;S;0603
- R3003: MPN R;G;T1;S;P0603;NA -> R;G;2K2;10P0;S;0603
- R3004: MPN R;G;T1;S;P0603;NA -> R;G;43K;10P0;S;0603
- R3005: MPN R;G;T1;S;P0603;NA -> R;G;10K;10P0;S;0603
- R3006: MPN R;G;T1;S;P0603;NA -> R;G;200R;10P0;S;0603
Changed lines of the file:
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@@
 			)
 		)
-		(property "MPN" "R;G;T1;S;P0603;NA"
+		(property "MPN" "R;G;3K;10P0;S;0603"
 			(at 204.47 138.43 90)
 			(effects
@@
 			)
 		)
-		(property "MPN" "C;C;T1;S;P0603;NA"
+		(property "MPN" "C;M;10u;10p;50V;S;0603"
 			(at 223.71 133.35 90)
 			(effects
@@
 			)
 		)
-		(property "MPN" "R;G;T1;S;P0603;NA"
+		(property "MPN" "R;G;10K;10P0;S;0603"
 			(at 209.55 228.6 90)
 			(effects
@@
 			)
 		)
-		(property "MPN" "R;G;T1;S;P0603;NA"
+		(property "MPN" "R;G;2K2;10P0;S;0603"
 			(at 209.55 209.55 90)
 			(effects
@@
 			)
 		)
-		(property "MPN" "R;G;T1;S;P0603;NA"
+		(property "MPN" "R;G;200R;10P0;S;0603"
 			(at 270.51 210.82 90)
 			(effects
@@
 			)
 		)
-		(property "MPN" "C;C;T1;S;P0603;NA"
+		(property "MPN" "C;M;10u;10p;50V;S;0603"
 			(at 240.22 133.35 90)
 			(effects
@@
 			)
 		)
-		(property "MPN" "R;G;T1;S;P0603;NA"
+		(property "MPN" "R;G;16K;10P0;S;0603"
 			(at 204.47 128.27 90)
 			(effects
@@
 			)
 		)
-		(property "MPN" "C;C;T1;S;P0603;NA"
+		(property "MPN" "C;M;10u;10p;50V;S;0603"
 			(at 119.57 209.55 90)
 			(effects
@@
 			)
 		)
-		(property "MPN" "C;C;T1;S;P0603;NA"
+		(property "MPN" "C;M;10u;10p;10V;S;0603"
 			(at 246.57 210.82 90)
 			(effects
@@
 			)
 		)
-		(property "MPN" "C;C;T1;S;P0603;NA"
+		(property "MPN" "C;M;100n;10p;25V;S;0603"
 			(at 166.37 107.76 90)
 			(effects
@@
 			)
 		)
-		(property "MPN" "C;C;T1;S;P0603;NA"
+		(property "MPN" "C;M;10u;10p;50V;S;0603"
 			(at 255.46 133.35 90)
 			(effects
@@
 			)
 		)
-		(property "MPN" "C;C;T1;S;P0603;NA"
+		(property "MPN" "C;M;10u;10p;10V;S;0603"
 			(at 228.79 210.82 90)
 			(effects
@@
 			)
 		)
-		(property "MPN" "R;G;T1;S;P0603;NA"
+		(property "MPN" "R;G;43K;10P0;S;0603"
 			(at 209.55 218.44 90)
 			(effects
