File: HW/PIC18F_ETH/PIC18F_ETH/PIC18F_ETH.kicad_pcb (KiCad board)
At the start: 2 copper layers, 114 parts, among them J2001 Conn_01x06, J4001 Conn_01x03, J4002 Conn_01x03, J4003 Conn_01x03, J4004 Conn_01x03, J4005 Conn_01x03, J4006 Conn_01x03, J4007 Conn_01x08, J4008 Conn_01x08, J4009 Conn_01x08, J4010 Conn_01x08, J4011 Conn_01x08, J5001 RJ45_LED_ETH_Shielded, U2001 PIC18F67J60T-I, U2002 25Mhz,50ppm, U2003 93AA46BT-I/OT, U4001 TLP241B, U4002 TLP241B, U4003 TLP241B, U4004 TLP241B, U4005 TLP241B, U4006 TLP241B, U4007 TLP241B, U4008 TLP241B, U6001 MCP2515T-E/ML

Commit message: .
Parts:
- added R6001: 10K, Resistor_SMD:R_0603_1608Metric, F.Cu at (65.7, 181.1)
- added R6002: 10K, Resistor_SMD:R_0603_1608Metric, F.Cu at (65.7, 183.6)
- added R6003: 0R, Resistor_SMD:R_0603_1608Metric, F.Cu at (85.2, 176.1)
- added R6004: 0R, Resistor_SMD:R_0603_1608Metric, F.Cu at (85.2, 178.6)
- added R6005: 10K, Resistor_SMD:R_0603_1608Metric, F.Cu at (85.2, 181.1)
- added U6002: 25Mhz,50ppm, Oscillator:Oscillator_SMD_SeikoEpson_SG8002CE-4Pin_3.2x2.5mm, F.Cu at (61.0, 182.2)
- added U6003: ATA6561-GAQW, bt_footprints:SOIC8_4P9X3P9MC_MCH, F.Cu at (62.5, 176.6)
- J4001, J4002, J4003, J4004, J4005, J4006: value Conn_01x03 -> JST,2.54; footprint Connector_Samtec_HPM_THT:Samtec_HPM-03-01-x-S_Straight_1x03_Pitch5.08mm -> Connector_JST:JST_EH_B3B-EH-A_1x03_P2.50mm_Vertical
- moved R5006 94.5 mm to (52.6, 151.1), turned to 180 degrees
- moved R5005 80.7 mm to (52.3, 129.5), turned to 180 degrees
- moved J4006 69.9 mm to (159.5, 105.9), turned to 90 degrees
- moved D4001 67.8 mm to (157.5, 111.1)
- moved R4005 67.8 mm to (155.0, 110.5)
- moved R4006 67.8 mm to (160.0, 110.5)
- moved J4005 66.4 mm to (154.7, 105.9), turned to 90 degrees
- moved J4004 62.8 mm to (149.9, 105.9), turned to 90 degrees
- moved D4002 60.0 mm to (147.9, 111.1)
- moved R4003 60.0 mm to (145.4, 110.5)
- moved R4004 60.0 mm to (150.4, 110.5)
- moved J4003 59.3 mm to (145.0, 105.9), turned to 90 degrees
- moved J4002 55.9 mm to (140.0, 105.9), turned to 90 degrees
- moved R4029 55.1 mm to (224.0, 183.9), turned to -90 degrees
- moved D4003 53.5 mm to (137.8, 111.0)
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Connections:
- U2001 pad 1: unconnected-(U2001A-RE1/P2C-Pad1) -> /DO1
- U2001 pad 12: unconnected-(U2001A-RF6/AN11-Pad12) -> /DI11
- U2001 pad 13: unconnected-(U2001A-RF5/AN10/CVREF-Pad13) -> /DI10
- U2001 pad 14: unconnected-(U2001A-RF4/AN9-Pad14) -> /DI9
- U2001 pad 15: unconnected-(U2001A-RF3/AN8-Pad15) -> /DI0
- U2001 pad 2: unconnected-(U2001A-RE0/P2D-Pad2) -> /DO0
- U2001 pad 29: /MCU_core/SPI_SS2 -> /CAN_CTRL.CS#
- U2001 pad 3: /DI0 -> /CAN_CTRL.INT#
- U2001 pad 34: /MCU_core/SPI_SCK -> /CAN_CTRL.SCK
- U2001 pad 35: /MCU_core/SPI_MISO -> /CAN_CTRL.MISO
- U2001 pad 36: /MCU_core/SPI_MOSI -> /CAN_CTRL.MOSI
- U2001 pad 58: unconnected-(U2001A-RD2/CCP4/P3D-Pad58) -> /MCU_core/DO8
- U2001 pad 59: unconnected-(U2001A-RD1/ECCP3/P3A-Pad59) -> /DO7
- U2001 pad 60: unconnected-(U2001A-RD0/P1B-Pad60) -> /DO6
- U2001 pad 61: unconnected-(U2001A-RE5/P1C-Pad61) -> /DO5
- U2001 pad 62: unconnected-(U2001A-RE4/P3B-Pad62) -> /DO4
- U2001 pad 63: unconnected-(U2001A-RE3/P3C-Pad63) -> /DO3
- U2001 pad 64: unconnected-(U2001A-RE2/P2B-Pad64) -> /DO2
- U2003 pad 1: /MCU_core/SPI_MISO -> /CAN_CTRL.MISO
- U2003 pad 3: /MCU_core/SPI_MISO -> /CAN_CTRL.MOSI
- U2003 pad 4: /MCU_core/SPI_SCK -> /CAN_CTRL.SCK
- U6001 pad 10: unconnected-(U6001-*RX0BF-Pad10) -> Net-(U6001-*RX0BF)
- U6001 pad 11: unconnected-(U6001-*INT-Pad11) -> /CAN_CTRL.INT#
- U6001 pad 12: unconnected-(U6001-SCK-Pad12) -> /CAN_CTRL.SCK
- U6001 pad 14: unconnected-(U6001-SI-Pad14) -> /CAN_CTRL.MOSI
- U6001 pad 15: unconnected-(U6001-SO-Pad15) -> /CAN_CTRL.MISO
- U6001 pad 16: unconnected-(U6001-*CS-Pad16) -> /CAN_CTRL.CS#
- U6001 pad 17: unconnected-(U6001-*RESET-Pad17) -> Net-(U6001-*RESET)
- U6001 pad 18: unconnected-(U6001-VDD-Pad18) -> +3.3V
- U6001 pad 19: unconnected-(U6001-TXCAN-Pad19) -> /CAN/CAN_TX
- U6001 pad 20: unconnected-(U6001-RXCAN-Pad20) -> /CAN/CAN_RX
- U6001 pad 21: unconnected-(U6001-EPAD-Pad21) -> GND
- U6001 pad 7: unconnected-(U6001-OSC1-Pad7) -> /CAN/25Mhz_CAN
- U6001 pad 8: unconnected-(U6001-GND-Pad8) -> GND

Commit message: .
Parts:
- added J4012: JST,2.54, Connector_JST:JST_EH_B2B-EH-A_1x02_P2.50mm_Vertical, F.Cu at (108.8, 169.4)
- added J4013: JST,2.54, Connector_JST:JST_EH_B2B-EH-A_1x02_P2.50mm_Vertical, F.Cu at (113.8, 169.4)
- added J4014: JST,2.54, Connector_JST:JST_EH_B2B-EH-A_1x02_P2.50mm_Vertical, F.Cu at (118.6, 169.4)
- added J4015: JST,2.54, Connector_JST:JST_EH_B2B-EH-A_1x02_P2.50mm_Vertical, F.Cu at (144.1, 169.4)
- added J4016: JST,2.54, Connector_JST:JST_EH_B2B-EH-A_1x02_P2.50mm_Vertical, F.Cu at (149.0, 169.4)
- added J4017: JST,2.54, Connector_JST:JST_EH_B2B-EH-A_1x02_P2.50mm_Vertical, F.Cu at (154.2, 169.5)
- added J4018: JST,2.54, Connector_JST:JST_EH_B2B-EH-A_1x02_P2.50mm_Vertical, F.Cu at (159.0, 169.5)
- added J4019: JST,2.54, Connector_JST:JST_EH_B2B-EH-A_1x02_P2.50mm_Vertical, F.Cu at (200.6, 106.7)
- added J4020: JST,2.54, Connector_JST:JST_EH_B2B-EH-A_1x02_P2.50mm_Vertical, F.Cu at (176.5, 113.3)
- added J4021: JST,2.54, Connector_JST:JST_EH_B2B-EH-A_1x02_P2.50mm_Vertical, F.Cu at (187.9, 125.8)
- added J4022: JST,2.54, Connector_JST:JST_EH_B2B-EH-A_1x02_P2.50mm_Vertical, F.Cu at (178.3, 132.9)
- added J4023: JST,2.54, Connector_JST:JST_EH_B2B-EH-A_1x02_P2.50mm_Vertical, F.Cu at (177.5, 153.5)
- added J4024: JST,2.54, Connector_JST:JST_EH_B2B-EH-A_1x02_P2.50mm_Vertical, F.Cu at (177.5, 134.4)
- added J4025: JST,2.54, Connector_JST:JST_EH_B2B-EH-A_1x02_P2.50mm_Vertical, F.Cu at (177.5, 140.3)
- added J4026: JST,2.54, Connector_JST:JST_EH_B2B-EH-A_1x02_P2.50mm_Vertical, F.Cu at (177.5, 146.1)
- J4007, J4008, J4009, J4010, J4011: value Conn_01x08 -> JST,2.54; footprint Connector_Samtec_HPM_THT:Samtec_HPM-08-01-x-S_Straight_1x08_Pitch5.08mm -> Connector_JST:JST_EH_B2B-EH-A_1x02_P2.50mm_Vertical
- moved J4011 182.8 mm to (103.9, 169.4), turned to 90 degrees
- moved J4010 166.9 mm to (138.9, 169.4), turned to 90 degrees
- moved C4010 139.8 mm to (124.7, 158.9)
- moved C4007 113.1 mm to (104.4, 158.8)
- moved R4019 110.6 mm to (154.2, 107.0)
- moved U4001 110.6 mm to (162.0, 108.5)
- moved R4020 109.6 mm to (154.1, 112.5)
- moved U4002 109.6 mm to (161.9, 114.0)
- moved R4013 109.4 mm to (120.7, 161.2), turned to -90 degrees
- moved R4021 108.8 mm to (154.2, 118.0)
- moved U4003 108.8 mm to (162.0, 119.5)
- moved C4008 108.8 mm to (108.2, 158.8), turned to 180 degrees
- moved R4023 108.1 mm to (154.1, 128.9)
- moved U4005 108.1 mm to (161.9, 130.4)
- moved R4022 108.0 mm to (154.4, 123.4)
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Connections:
- net Net-(R2004-Pad2) renamed /MCU_core/RB_Split
- net Net-(U2001A-RBIAS) renamed /MCU_core/RBIAS
- C2003 pad 2: +3.3V -> GND
- C2004 pad 2: +3.3V -> GND
- C2005 pad 2: +3.3V -> GND
- C2006 pad 2: +3.3V -> GND
- C2007 pad 2: +3.3V -> GND
- C2008 pad 2: +3.3V -> GND
- C2009 pad 2: +3.3V -> GND
- C4007 pad 1: /IO_core/DI4x -> /DI4
- C4008 pad 1: /IO_core/DI5x -> /DI5
- C4009 pad 1: /IO_core/DI8x -> /DI8
- C4010 pad 1: /IO_core/DI0x -> /DI0
- C4011 pad 1: /IO_core/DI6x -> /DI6
- C4012 pad 1: /IO_core/DI9x -> /DI9
- C4013 pad 1: /IO_core/DI1x -> /DI1
- C4014 pad 1: /IO_core/DI7x -> /DI7
- C4015 pad 1: /IO_core/DI10x -> /DI10
- C4016 pad 1: /IO_core/DI2x -> /DI2
- C4017 pad 1: /IO_core/DI11x -> /DI11
- C4018 pad 1: /IO_core/DI3x -> /DI3
- J4007 pad 2: /IO_core/DI4x -> /IO_core/DI0x
- J4008 pad 2: /IO_core/DI0x -> /IO_core/DI1x
- J4009 pad 2: /IO_core/DI8x -> /IO_core/DI2x
- J4010 pad 1: Net-(J4010-Pin_1) -> GND
- J4010 pad 2: Net-(J4010-Pin_2) -> /IO_core/DI3x
- J4011 pad 1: Net-(J4011-Pin_1) -> GND
- J4011 pad 2: Net-(J4011-Pin_2) -> /IO_core/DI4x
- U4001 pad 3: Net-(J4010-Pin_2) -> Net-(J4019-Pin_2)
- U4001 pad 4: Net-(J4010-Pin_1) -> Net-(J4019-Pin_1)
- U4002 pad 3: Net-(J4010-Pin_4) -> Net-(J4020-Pin_2)
- U4002 pad 4: Net-(J4010-Pin_3) -> Net-(J4020-Pin_1)
- U4003 pad 3: Net-(J4010-Pin_6) -> Net-(J4021-Pin_2)
- U4003 pad 4: Net-(J4010-Pin_5) -> Net-(J4021-Pin_1)
- U4004 pad 3: Net-(J4010-Pin_8) -> Net-(J4022-Pin_2)
- U4004 pad 4: Net-(J4010-Pin_7) -> Net-(J4022-Pin_1)
- U4005 pad 3: Net-(J4011-Pin_2) -> Net-(J4023-Pin_2)
- U4005 pad 4: Net-(J4011-Pin_1) -> Net-(J4023-Pin_1)
- U4006 pad 3: Net-(J4011-Pin_4) -> Net-(J4024-Pin_2)
- U4006 pad 4: Net-(J4011-Pin_3) -> Net-(J4024-Pin_1)
- U4007 pad 3: Net-(J4011-Pin_6) -> Net-(J4025-Pin_2)
- U4007 pad 4: Net-(J4011-Pin_5) -> Net-(J4025-Pin_1)
- U4008 pad 3: Net-(J4011-Pin_8) -> Net-(J4026-Pin_2)
- U4008 pad 4: Net-(J4011-Pin_7) -> Net-(J4026-Pin_1)
Other:
- board outline added: 160 x 80 mm

Commit message: .
Parts:
- added C6001: 100n 25V, Capacitor_SMD:C_0603_1608Metric, F.Cu at (116.1, 124.7)
- added C6002: 100n 25V, Capacitor_SMD:C_0603_1608Metric, F.Cu at (122.2, 115.9)
- added C6003: 100n 25V, Capacitor_SMD:C_0603_1608Metric, F.Cu at (138.2, 119.9)
- added C6004: 100n 25V, Capacitor_SMD:C_0603_1608Metric, F.Cu at (134.6, 126.2)
- added FID7001: Fiducial_05_1, Fiducial:Fiducial_0.5mm_Mask1mm, F.Cu at (119.2, 142.8)
- added FID7002: Fiducial_05_1, Fiducial:Fiducial_0.5mm_Mask1mm, F.Cu at (119.2, 145.3)
- added FID7003: Fiducial_05_1, Fiducial:Fiducial_0.5mm_Mask1mm, F.Cu at (119.2, 147.9)
- added FID7004: Fiducial_05_1, Fiducial:Fiducial_0.5mm_Mask1mm, F.Cu at (119.2, 150.4)
- added H7001: MountingHole_Pad, MountingHole:MountingHole_3.2mm_M3_ISO7380_Pad, F.Cu at (52.3, 105.9)
- added H7002: MountingHole_Pad, MountingHole:MountingHole_3.2mm_M3_ISO7380_Pad, F.Cu at (196.6, 105.9)
- added H7003: MountingHole_Pad, MountingHole:MountingHole_3.2mm_M3_ISO7380_Pad, F.Cu at (197.1, 173.2)
- added H7004: MountingHole_Pad, MountingHole:MountingHole_3.2mm_M3_ISO7380_Pad, F.Cu at (51.1, 174.0)
- added J6001: JST,2.54, Connector_JST:JST_EH_B3B-EH-A_1x03_P2.50mm_Vertical, F.Cu at (133.1, 109.5)
- added J6002: JST,2.54, Connector_JST:JST_EH_B3B-EH-A_1x03_P2.50mm_Vertical, F.Cu at (133.1, 114.5)
- added R6006: 120R, Resistor_SMD:R_0603_1608Metric, F.Cu at (134.4, 105.9)
- moved U6003 90.7 mm to (134.6, 121.5), turned to 90 degrees
- moved R6002 89.1 mm to (123.7, 115.9), turned to -90 degrees
- moved U6002 81.8 mm to (120.1, 125.6)
- moved R6005 75.8 mm to (128.5, 118.9)
- moved R6004 74.5 mm to (130.8, 119.7), turned to 90 degrees
- moved R6001 74.1 mm to (116.1, 126.7)
- moved U6001 73.3 mm to (121.9, 120.1)
- moved R6003 70.4 mm to (129.3, 121.2), turned to -90 degrees
- moved J4011 60.4 mm to (164.2, 172.0), turned to 180 degrees
- moved J4006 57.6 mm to (142.5, 172.0), turned to 0 degrees
- moved J4012 55.5 mm to (164.2, 167.1), turned to 180 degrees
- moved R4007 55.3 mm to (156.1, 173.7), turned to 0 degrees
- moved R4034 53.5 mm to (156.1, 172.2), turned to 0 degrees
- moved J4005 53.3 mm to (142.5, 167.2), turned to 0 degrees
- moved J4018 52.9 mm to (164.3, 116.8), turned to 180 degrees
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Connections:
- net Net-(U6001-*RESET) renamed /CAN/CAN_CTRL_RST#
- U2001 pad 46: /ETH_Connector/ETH.RX+ -> /ETH_Connector/ETH.RX-
Other:
- copper layers 2 -> 4

Commit message: .
Parts:
- added C3001: C_Polarized, Capacitor_SMD:CP_Elec_4x3, F.Cu at (65.2, 111.8)
- added C3002: 100n 25V, Capacitor_SMD:C_0603_1608Metric, F.Cu at (72.0, 110.7)
- added C3003: 10u 10V, Capacitor_SMD:C_0603_1608Metric, F.Cu at (91.0, 115.7)
- added C3004: 10u 10V, Capacitor_SMD:C_0603_1608Metric, F.Cu at (93.0, 115.7)
- added C3005: 10u 10V, Capacitor_SMD:C_0603_1608Metric, F.Cu at (89.0, 115.7)
- added C3006: 10u 10V, Capacitor_SMD:C_0603_1608Metric, F.Cu at (94.5, 118.5)
- added C3007: 10u 10V, Capacitor_SMD:C_0603_1608Metric, F.Cu at (101.8, 121.3)
- added C3008: 10u 10V, Capacitor_SMD:C_0603_1608Metric, F.Cu at (100.2, 121.3)
- added J3001: Jack-DC, Connector_BarrelJack:BarrelJack_Horizontal, F.Cu at (58.5, 117.5)
- added L3001: 33uH, Inductor_SMD:L_Bourns_SRR1208_12.7x12.7mm, F.Cu at (80.0, 115.0)
- added L3002: 1uH, Inductor_SMD:L_0805_2012Metric, F.Cu at (97.8, 120.5)
- added R3001: 160K, Resistor_SMD:R_0603_1608Metric, F.Cu at (68.8, 106.0)
- added R3002: 30K, Resistor_SMD:R_0603_1608Metric, F.Cu at (68.8, 107.5)
- added R3006: 2K2, Resistor_SMD:R_0603_1608Metric, F.Cu at (95.8, 122.5)
- added R3007: 43K, Resistor_SMD:R_0603_1608Metric, F.Cu at (92.8, 122.5)
- added R3008: 10K, Resistor_SMD:R_0603_1608Metric, F.Cu at (92.2, 120.2)
- added U3001: LMR51610-Q1, Package_TO_SOT_SMD:SOT-23-6, F.Cu at (69.5, 111.0)
- added U3002: TPS62A01, Package_TO_SOT_SMD:SOT-563, F.Cu at (94.5, 120.5)
- C2010: value 10u 10V -> 100n 25V
- C2011: value 100n 25V -> 10u 10V
- R2003: value 10K -> 2K2
- R2004: value 2K2 -> 10K
- R4007, R4008, R4009, R4010, R4011, R4012, R4013, R4014, R4015, R4016, R4017, R4018: value 10K -> 200R
- R4019, R4020, R4021, R4022, R4023, R4024, R4025, R4026, R4027, R4028, R4029, R4030: value 200R -> 10K
- R5001, R5002: value 49R9 -> 510K
- R5005, R5006: value 510K -> 49R9
- U2001: value PIC18F67J60T-I -> 93AA46BT-I/OT; footprint bt_footprints:TQFP64_10x10MC_MCH -> Package_TO_SOT_SMD:SOT-23-6
- U2002: value 25Mhz,50ppm -> PIC18F67J60T-I; footprint Oscillator:Oscillator_SMD_SeikoEpson_SG8002CE-4Pin_3.2x2.5mm -> bt_footprints:TQFP64_10x10MC_MCH
- U2003: value 93AA46BT-I/OT -> 25Mhz,50ppm; footprint Package_TO_SOT_SMD:SOT-23-6 -> Oscillator:Oscillator_SMD_SeikoEpson_SG8002CE-4Pin_3.2x2.5mm
- U6001: value MCP2515T-E/ML -> 25Mhz,50ppm; footprint bt_footprints:QFN20_4x4MC_MCH -> Oscillator:Oscillator_SMD_SeikoEpson_SG8002CE-4Pin_3.2x2.5mm
- U6002: value 25Mhz,50ppm -> MCP2515T-E/ML; footprint Oscillator:Oscillator_SMD_SeikoEpson_SG8002CE-4Pin_3.2x2.5mm -> bt_footprints:QFN20_4x4MC_MCH
- moved R6006 90.2 mm to (78.3, 176.6), turned to 180 degrees
- moved FID7002 85.0 mm to (197.0, 111.0)
- moved J6001 83.1 mm to (79.5, 173.0), turned to 180 degrees
- moved FID7003 79.9 mm to (197.0, 166.0)
- moved C6003 76.7 mm to (74.5, 162.6), turned to 90 degrees
- moved J6002 75.8 mm to (79.5, 168.0), turned to 180 degrees
- moved FID7001 71.8 mm to (57.5, 106.0)
- moved U6003 68.9 mm to (78.0, 161.0), turned to -90 degrees
- moved FID7004 67.2 mm to (56.5, 174.5)
- moved R6004 65.3 mm to (81.8, 162.9), turned to -90 degrees
- moved C6004 64.1 mm to (78.0, 156.3), turned to 0 degrees
- moved R6005 63.1 mm to (84.1, 163.6), turned to 180 degrees
- moved R6002 61.4 mm to (88.9, 166.6), turned to 90 degrees
- moved R6003 61.0 mm to (83.3, 161.3), turned to 90 degrees
- moved C6002 59.8 mm to (90.5, 166.6), turned to -90 degrees
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Connections:
- C2010 pad 1: Net-(U2001B-VDDCORE/VCAP) -> +3.3V
- C2011 pad 1: +3.3V -> Net-(U2002B-VDDCORE/VCAP)
- C4007 pad 1: /DI4 -> /DI0
- C4008 pad 1: /DI5 -> /DI4
- C4010 pad 1: /DI0 -> /DI9
- C4011 pad 1: /DI6 -> /DI1
- C4012 pad 1: /DI9 -> /DI5
- C4013 pad 1: /DI1 -> /DI2
- C4014 pad 1: /DI7 -> /DI6
- C4016 pad 1: /DI2 -> /DI3
- C4017 pad 1: /DI11 -> /DI7
- C4018 pad 1: /DI3 -> /DI11
- D4001 pad 1: /IO_core/AD5x -> /IO_core/AD3x
- D4001 pad 2: /IO_core/AD4x -> /IO_core/AD0x
- D4003 pad 1: /IO_core/AD3x -> /IO_core/AD5x
- D4003 pad 2: /IO_core/AD0x -> /IO_core/AD4x
- D4004 pad 1: /IO_core/DI10x -> /IO_core/DI6x
- D4004 pad 2: /IO_core/DI11x -> /IO_core/DI7x
- D4005 pad 1: /IO_core/DI8x -> /IO_core/DI10x
- D4005 pad 2: /IO_core/DI9x -> /IO_core/DI11x
- D4006 pad 1: /IO_core/DI6x -> /IO_core/DI4x
- D4006 pad 2: /IO_core/DI7x -> /IO_core/DI5x
- D4007 pad 1: /IO_core/DI4x -> /IO_core/DI8x
- D4007 pad 2: /IO_core/DI5x -> /IO_core/DI9x
- R2001 pad 1: +3.3V -> /MCU_core/SPI_SS1
- R2001 pad 2: Net-(U2002-ST#) -> GND
- R2002 pad 1: /MCU_core/SPI_SS1 -> +3.3V
- R2002 pad 2: GND -> /MCU_core/RST#
- R2003 pad 1: +3.3V -> /MCU_core/RBIAS
- R2003 pad 2: /MCU_core/RST# -> /MCU_core/RB_Split
- R2004 pad 1: /MCU_core/RBIAS -> +3.3V
- R2004 pad 2: /MCU_core/RB_Split -> Net-(U2003-ST#)
- R4007 pad 1: +3.3V -> /DI4
- R4008 pad 1: +3.3V -> /DI5
- R4009 pad 1: +3.3V -> /DI6
- R4009 pad 2: /IO_core/DI8x -> /IO_core/DI6x
- R4010 pad 1: +3.3V -> /DI7
- R4010 pad 2: /IO_core/DI6x -> /IO_core/DI7x
- R4011 pad 1: +3.3V -> /DI8
- R4011 pad 2: /IO_core/DI0x -> /IO_core/DI8x
- R4012 pad 1: +3.3V -> /DI9
- R4013 pad 1: +3.3V -> /DI10
- R4013 pad 2: /IO_core/DI7x -> /IO_core/DI10x
- R4014 pad 1: +3.3V -> /DI11
- R4014 pad 2: /IO_core/DI1x -> /IO_core/DI11x
- R4015 pad 1: +3.3V -> /DI0
- R4015 pad 2: /IO_core/DI10x -> /IO_core/DI0x
- R4016 pad 1: +3.3V -> /DI1
- R4016 pad 2: /IO_core/DI2x -> /IO_core/DI1x
- R4017 pad 1: +3.3V -> /DI2
- R4017 pad 2: /IO_core/DI11x -> /IO_core/DI2x
- R4018 pad 1: +3.3V -> /DI3
- R4019 pad 1: /DO0 -> +3.3V
- R4019 pad 2: /IO_core/DO0x -> /IO_core/DI4x
- R4020 pad 1: /DO1 -> +3.3V
- R4020 pad 2: /IO_core/DO1x -> /IO_core/DI8x
- R4021 pad 1: /DO2 -> +3.3V
- R4021 pad 2: /IO_core/DO2x -> /IO_core/DI0x
- R4022 pad 1: /DO3 -> +3.3V
- R4022 pad 2: /IO_core/DO3x -> /IO_core/DI5x
- R4023 pad 1: /DO4 -> +3.3V
- R4023 pad 2: /IO_core/DO4x -> /IO_core/DI9x
- R4024 pad 1: /DO5 -> +3.3V
- R4024 pad 2: /IO_core/DO5x -> /IO_core/DI1x
- R4025 pad 1: /DO6 -> +3.3V
- R4025 pad 2: /IO_core/DO6x -> /IO_core/DI6x
- R4026 pad 1: /DO7 -> +3.3V
- R4026 pad 2: /IO_core/DO7x -> /IO_core/DI10x
- R4027 pad 1: /DI11 -> +3.3V
- R4027 pad 2: /IO_core/DI11x -> /IO_core/DI2x
- R4028 pad 1: /DI10 -> +3.3V
- R4028 pad 2: /IO_core/DI10x -> /IO_core/DI7x
- R4029 pad 1: /DI9 -> +3.3V
- R4029 pad 2: /IO_core/DI9x -> /IO_core/DI11x
- R4030 pad 1: /DI8 -> +3.3V
- R4030 pad 2: /IO_core/DI8x -> /IO_core/DI3x
- R4031 pad 1: /DI7 -> /DO0
- R4031 pad 2: /IO_core/DI7x -> /IO_core/DO0x
- R4032 pad 1: /DI6 -> /DO1
- R4032 pad 2: /IO_core/DI6x -> /IO_core/DO1x
- R4033 pad 1: /DI5 -> /DO2
- R4033 pad 2: /IO_core/DI5x -> /IO_core/DO2x
- R4034 pad 1: /DI4 -> /DO3
- R4034 pad 2: /IO_core/DI4x -> /IO_core/DO3x
- R4035 pad 1: /DI3 -> /DO4
- R4035 pad 2: /IO_core/DI3x -> /IO_core/DO4x
- R4036 pad 1: /DI2 -> /DO5
- R4036 pad 2: /IO_core/DI2x -> /IO_core/DO5x
- R4037 pad 1: /DI1 -> /DO6
- R4037 pad 2: /IO_core/DI1x -> /IO_core/DO6x
- R4038 pad 1: /DI0 -> /DO7
- R4038 pad 2: /IO_core/DI0x -> /IO_core/DO7x
- R5001 pad 1: /ETH_Connector/ETH.RX- -> /ETH_Connector/LED_Y
- R5001 pad 2: /ETH_Connector/RX_C -> Net-(J5001-Pad9)
- R5002 pad 1: /ETH_Connector/RX_C -> /ETH_Connector/LED_G
- R5002 pad 2: /ETH_Connector/ETH.RX+ -> Net-(J5001-Pad11)
- R5003 pad 1: /ETH_Connector/ETH.TX- -> /ETH_Connector/ETH.RX-
- R5003 pad 2: /ETH_Connector/TX_C -> /ETH_Connector/RX_C
- R5004 pad 1: /ETH_Connector/TX_C -> /ETH_Connector/RX_C
- R5004 pad 2: /ETH_Connector/ETH.TX+ -> /ETH_Connector/ETH.RX+
- R5005 pad 1: /ETH_Connector/LED_Y -> /ETH_Connector/ETH.TX-
- R5005 pad 2: Net-(J5001-Pad9) -> /ETH_Connector/TX_C
- R5006 pad 1: /ETH_Connector/LED_G -> /ETH_Connector/TX_C
- R5006 pad 2: Net-(J5001-Pad11) -> /ETH_Connector/ETH.TX+
- R6001 pad 2: Net-(U6002-ST#) -> Net-(U6001-ST#)
- R6003 pad 2: Net-(U6001-*RX0BF) -> Net-(U6002-*RX0BF)
- U2001 pad 1: /DO1 -> /CAN_CTRL.MISO
- U2001 pad 2: /DO0 -> GND
- U2001 pad 3: /CAN_CTRL.INT# -> /CAN_CTRL.MOSI
- U2001 pad 4: /DI1 -> /CAN_CTRL.SCK
- U2001 pad 5: /DI3 -> /MCU_core/SPI_SS1
- U2001 pad 6: /DI4 -> +3.3V
- U2002 pad 1: Net-(U2002-ST#) -> /DO1
- U2002 pad 2: GND -> /DO0
- U2002 pad 3: /MCU_core/MCU_25Mhz -> /CAN_CTRL.INT#
- U2002 pad 4: +3.3V -> /DI1
- U2003 pad 1: /CAN_CTRL.MISO -> Net-(U2003-ST#)
- U2003 pad 3: /CAN_CTRL.MOSI -> /MCU_core/MCU_25Mhz
- U2003 pad 4: /CAN_CTRL.SCK -> +3.3V
- U6001 pad 1: unconnected-(U6001-CLKOUT-Pad1) -> Net-(U6001-ST#)
- U6001 pad 2: unconnected-(U6001-*TX0RTS-Pad2) -> GND
- U6001 pad 3: unconnected-(U6001-*TX1RTS-Pad3) -> /CAN/25Mhz_CAN
- U6001 pad 4: unconnected-(U6001-NC-Pad4) -> +3.3V
- U6002 pad 1: Net-(U6002-ST#) -> unconnected-(U6002-CLKOUT-Pad1)
- U6002 pad 2: GND -> unconnected-(U6002-*TX0RTS-Pad2)
- U6002 pad 3: /CAN/25Mhz_CAN -> unconnected-(U6002-*TX1RTS-Pad3)
- U6002 pad 4: +3.3V -> unconnected-(U6002-NC-Pad4)
Routing:
- net +5V: track 0.00 -> 33.8 mm

Commit message: .
Parts:
- removed C4009, C4010, C4011, C4012, C4013, C4014, C4015, C4016, C4017, C4018: 100n 25V, Capacitor_SMD:C_0603_1608Metric
- removed D4004, D4005, D4006, D4007, D4008, D4009: PESD2USB3UXT-Q, Package_TO_SOT_SMD:SOT-23-3
- removed J4007, J4008, J4009, J4010, J4011, J4012, J4013, J4014, J4015, J4016, J4017, J4018, J4019, J4020, J4021, J4022, J4023, J4024, J4025, J4026: JST,2.54, Connector_JST:JST_EH_B2B-EH-A_1x02_P2.50mm_Vertical
- removed R4009, R4010, R4011, R4012, R4013, R4014, R4015, R4016, R4017, R4018, R4031, R4032, R4033, R4034, R4035, R4036, R4037, R4038: 200R, Resistor_SMD:R_0603_1608Metric
- removed R4019, R4020, R4021, R4022, R4023, R4024, R4025, R4026, R4027, R4028, R4029, R4030: 10K, Resistor_SMD:R_0603_1608Metric
- removed U4003, U4004, U4005, U4006, U4007, U4008: TLP241B, Package_SO:SO-4_7.6x3.6mm_P2.54mm
- added C8001: 100n 25V, Capacitor_SMD:C_0603_1608Metric, F.Cu at (121.2, 162.8)
- added C8002: 100n 25V, Capacitor_SMD:C_0603_1608Metric, F.Cu at (141.2, 162.8)
- added C8003: 100n 25V, Capacitor_SMD:C_0603_1608Metric, F.Cu at (125.0, 162.8)
- added C8004: 100n 25V, Capacitor_SMD:C_0603_1608Metric, F.Cu at (145.0, 162.8)
- added C8005: 100n 25V, Capacitor_SMD:C_0603_1608Metric, F.Cu at (131.3, 162.8)
- added C8006: 100n 25V, Capacitor_SMD:C_0603_1608Metric, F.Cu at (151.6, 162.8)
- added C8007: 100n 25V, Capacitor_SMD:C_0603_1608Metric, F.Cu at (135.1, 162.8)
- added C8008: 100n 25V, Capacitor_SMD:C_0603_1608Metric, F.Cu at (155.4, 162.8)
- added C8009: 100n 25V, Capacitor_SMD:C_0603_1608Metric, F.Cu at (155.2, 116.9)
- added C8010: 100n 25V, Capacitor_SMD:C_0603_1608Metric, F.Cu at (134.9, 116.9)
- added C8011: 100n 25V, Capacitor_SMD:C_0603_1608Metric, F.Cu at (151.7, 116.9)
- added C8012: 100n 25V, Capacitor_SMD:C_0603_1608Metric, F.Cu at (131.4, 116.9)
- added C8013: 100n 25V, Capacitor_SMD:C_0603_1608Metric, F.Cu at (145.1, 116.9)
- added C8014: 100n 25V, Capacitor_SMD:C_0603_1608Metric, F.Cu at (124.8, 116.9)
- added C8015: 100n 25V, Capacitor_SMD:C_0603_1608Metric, F.Cu at (141.5, 116.9)
- added C8016: 100n 25V, Capacitor_SMD:C_0603_1608Metric, F.Cu at (121.0, 116.9)
- added D8001: PESD2USB3UXT-Q, Package_TO_SOT_SMD:SOT-23-3, F.Cu at (153.5, 166.0)
- added D8002: PESD2USB3UXT-Q, Package_TO_SOT_SMD:SOT-23-3, F.Cu at (143.2, 166.0)
- added D8003: PESD2USB3UXT-Q, Package_TO_SOT_SMD:SOT-23-3, F.Cu at (123.0, 166.0)
- added D8004: PESD2USB3UXT-Q, Package_TO_SOT_SMD:SOT-23-3, F.Cu at (133.2, 166.0)
- added D8005: PESD2USB3UXT-Q, Package_TO_SOT_SMD:SOT-23-3, F.Cu at (143.3, 113.7)
- added D8006: PESD2USB3UXT-Q, Package_TO_SOT_SMD:SOT-23-3, F.Cu at (153.5, 113.7)
- added D8007: PESD2USB3UXT-Q, Package_TO_SOT_SMD:SOT-23-3, F.Cu at (122.9, 113.7)
- added D8008: PESD2USB3UXT-Q, Package_TO_SOT_SMD:SOT-23-3, F.Cu at (133.1, 113.7)
- added J8001: JST,2.54, Connector_JST:JST_EH_B2B-EH-A_1x02_P2.50mm_Vertical, F.Cu at (120.1, 173.7)
- added J8002: JST,2.54, Connector_JST:JST_EH_B2B-EH-A_1x02_P2.50mm_Vertical, F.Cu at (125.2, 173.8)
- added J8003: JST,2.54, Connector_JST:JST_EH_B2B-EH-A_1x02_P2.50mm_Vertical, F.Cu at (130.3, 173.8)
- added J8004: JST,2.54, Connector_JST:JST_EH_B2B-EH-A_1x02_P2.50mm_Vertical, F.Cu at (135.4, 173.8)
- added J8005: JST,2.54, Connector_JST:JST_EH_B2B-EH-A_1x02_P2.50mm_Vertical, F.Cu at (140.5, 173.8)
- added J8006: JST,2.54, Connector_JST:JST_EH_B2B-EH-A_1x02_P2.50mm_Vertical, F.Cu at (145.5, 173.8)
- added J8007: JST,2.54, Connector_JST:JST_EH_B2B-EH-A_1x02_P2.50mm_Vertical, F.Cu at (150.6, 173.8)
- added J8008: JST,2.54, Connector_JST:JST_EH_B2B-EH-A_1x02_P2.50mm_Vertical, F.Cu at (155.7, 173.7)
- added J8009: JST,2.54, Connector_JST:JST_EH_B2B-EH-A_1x02_P2.50mm_Vertical, F.Cu at (156.3, 106.0)
- added J8010: JST,2.54, Connector_JST:JST_EH_B2B-EH-A_1x02_P2.50mm_Vertical, F.Cu at (151.2, 106.0)
- added J8011: JST,2.54, Connector_JST:JST_EH_B2B-EH-A_1x02_P2.50mm_Vertical, F.Cu at (146.1, 106.0)
- added J8012: JST,2.54, Connector_JST:JST_EH_B2B-EH-A_1x02_P2.50mm_Vertical, F.Cu at (141.0, 106.0)
- added J8013: JST,2.54, Connector_JST:JST_EH_B2B-EH-A_1x02_P2.50mm_Vertical, F.Cu at (136.0, 106.0)
- added J8014: JST,2.54, Connector_JST:JST_EH_B2B-EH-A_1x02_P2.50mm_Vertical, F.Cu at (130.9, 106.0)
- added J8015: JST,2.54, Connector_JST:JST_EH_B2B-EH-A_1x02_P2.50mm_Vertical, F.Cu at (125.8, 106.0)
- added J8016: JST,2.54, Connector_JST:JST_EH_B2B-EH-A_1x02_P2.50mm_Vertical, F.Cu at (120.7, 106.0)
- added J9001: JST,2.54, Connector_JST:JST_EH_B2B-EH-A_1x02_P2.50mm_Vertical, F.Cu at (163.6, 171.3)
- added J9002: JST,2.54, Connector_JST:JST_EH_B2B-EH-A_1x02_P2.50mm_Vertical, F.Cu at (168.7, 171.2)
- added J9003: JST,2.54, Connector_JST:JST_EH_B2B-EH-A_1x02_P2.50mm_Vertical, F.Cu at (173.7, 171.2)
- added J9004: JST,2.54, Connector_JST:JST_EH_B2B-EH-A_1x02_P2.50mm_Vertical, F.Cu at (178.8, 171.2)
- added J9005: JST,2.54, Connector_JST:JST_EH_B2B-EH-A_1x02_P2.50mm_Vertical, F.Cu at (183.9, 171.2)
- added J9006: JST,2.54, Connector_JST:JST_EH_B2B-EH-A_1x02_P2.50mm_Vertical, F.Cu at (189.0, 171.2)
- added J9007: JST,2.54, Connector_JST:JST_EH_B2B-EH-A_1x02_P2.50mm_Vertical, F.Cu at (194.1, 162.4)
- added J9008: JST,2.54, Connector_JST:JST_EH_B2B-EH-A_1x02_P2.50mm_Vertical, F.Cu at (199.1, 162.4)
- added J9009: JST,2.54, Connector_JST:JST_EH_B2B-EH-A_1x02_P2.50mm_Vertical, F.Cu at (198.5, 117.1)
- added J9010: JST,2.54, Connector_JST:JST_EH_B2B-EH-A_1x02_P2.50mm_Vertical, F.Cu at (193.5, 117.1)
- added J9011: JST,2.54, Connector_JST:JST_EH_B2B-EH-A_1x02_P2.50mm_Vertical, F.Cu at (188.4, 108.5)
- added J9012: JST,2.54, Connector_JST:JST_EH_B2B-EH-A_1x02_P2.50mm_Vertical, F.Cu at (183.3, 108.5)
- added J9013: JST,2.54, Connector_JST:JST_EH_B2B-EH-A_1x02_P2.50mm_Vertical, F.Cu at (178.5, 108.5)
- added J9014: JST,2.54, Connector_JST:JST_EH_B2B-EH-A_1x02_P2.50mm_Vertical, F.Cu at (173.4, 108.5)
- added J9015: JST,2.54, Connector_JST:JST_EH_B2B-EH-A_1x02_P2.50mm_Vertical, F.Cu at (168.3, 108.5)
- added J9016: JST,2.54, Connector_JST:JST_EH_B2B-EH-A_1x02_P2.50mm_Vertical, F.Cu at (163.3, 108.5)
- added R8001: 200R, Resistor_SMD:R_0603_1608Metric, F.Cu at (140.5, 165.1)
- added R8002: 200R, Resistor_SMD:R_0603_1608Metric, F.Cu at (145.8, 165.1)
- added R8003: 200R, Resistor_SMD:R_0603_1608Metric, F.Cu at (150.9, 165.1)
- added R8004: 200R, Resistor_SMD:R_0603_1608Metric, F.Cu at (156.2, 165.1)
- added R8005: 200R, Resistor_SMD:R_0603_1608Metric, F.Cu at (120.4, 165.1)
- added R8006: 200R, Resistor_SMD:R_0603_1608Metric, F.Cu at (125.7, 165.1)
- added R8007: 200R, Resistor_SMD:R_0603_1608Metric, F.Cu at (130.6, 165.1)
- added R8008: 200R, Resistor_SMD:R_0603_1608Metric, F.Cu at (135.9, 165.1)
- added R8009: 10K, Resistor_SMD:R_0603_1608Metric, F.Cu at (139.8, 167.4)
- added R8010: 10K, Resistor_SMD:R_0603_1608Metric, F.Cu at (119.7, 167.4)
- added R8011: 10K, Resistor_SMD:R_0603_1608Metric, F.Cu at (146.6, 167.4)
- added R8012: 10K, Resistor_SMD:R_0603_1608Metric, F.Cu at (126.2, 167.4)
- added R8013: 10K, Resistor_SMD:R_0603_1608Metric, F.Cu at (150.1, 167.4)
- added R8014: 10K, Resistor_SMD:R_0603_1608Metric, F.Cu at (129.9, 167.4)
- added R8015: 10K, Resistor_SMD:R_0603_1608Metric, F.Cu at (156.8, 167.4)
- added R8016: 10K, Resistor_SMD:R_0603_1608Metric, F.Cu at (136.4, 167.4)
- added R8017: 200R, Resistor_SMD:R_0603_1608Metric, F.Cu at (156.0, 114.6)
- added R8018: 200R, Resistor_SMD:R_0603_1608Metric, F.Cu at (150.9, 114.6)
- added R8019: 200R, Resistor_SMD:R_0603_1608Metric, F.Cu at (145.8, 114.6)
- added R8020: 200R, Resistor_SMD:R_0603_1608Metric, F.Cu at (140.8, 114.7)
- added R8021: 200R, Resistor_SMD:R_0603_1608Metric, F.Cu at (135.7, 114.6)
- added R8022: 200R, Resistor_SMD:R_0603_1608Metric, F.Cu at (130.6, 114.6)
- added R8023: 200R, Resistor_SMD:R_0603_1608Metric, F.Cu at (125.5, 114.6)
- added R8024: 200R, Resistor_SMD:R_0603_1608Metric, F.Cu at (120.2, 114.6)
- added R8025: 10K, Resistor_SMD:R_0603_1608Metric, F.Cu at (156.8, 112.3)
- added R8026: 10K, Resistor_SMD:R_0603_1608Metric, F.Cu at (136.4, 112.3)
- added R8027: 10K, Resistor_SMD:R_0603_1608Metric, F.Cu at (150.2, 112.3)
- added R8028: 10K, Resistor_SMD:R_0603_1608Metric, F.Cu at (129.9, 112.3)
- added R8029: 10K, Resistor_SMD:R_0603_1608Metric, F.Cu at (146.6, 112.3)
- added R8030: 10K, Resistor_SMD:R_0603_1608Metric, F.Cu at (126.3, 112.3)
- added R8031: 10K, Resistor_SMD:R_0603_1608Metric, F.Cu at (140.0, 112.3)
- added R8032: 10K, Resistor_SMD:R_0603_1608Metric, F.Cu at (119.4, 112.3)
- added R9001: 200R, Resistor_SMD:R_0603_1608Metric, F.Cu at (164.6, 154.5)
- added R9002: 200R, Resistor_SMD:R_0603_1608Metric, F.Cu at (169.7, 154.4)
- added R9003: 200R, Resistor_SMD:R_0603_1608Metric, F.Cu at (174.8, 154.4)
- added R9004: 200R, Resistor_SMD:R_0603_1608Metric, F.Cu at (179.8, 154.4)
- added R9005: 200R, Resistor_SMD:R_0603_1608Metric, F.Cu at (184.9, 154.4)
- added R9006: 200R, Resistor_SMD:R_0603_1608Metric, F.Cu at (190.0, 154.4)
- added R9007: 200R, Resistor_SMD:R_0603_1608Metric, F.Cu at (195.1, 145.6)
- added R9008: 200R, Resistor_SMD:R_0603_1608Metric, F.Cu at (200.2, 145.6)
- added R9009: 200R, Resistor_SMD:R_0603_1608Metric, F.Cu at (197.6, 133.9)
- added R9010: 200R, Resistor_SMD:R_0603_1608Metric, F.Cu at (192.5, 133.9)
- added R9011: 200R, Resistor_SMD:R_0603_1608Metric, F.Cu at (187.4, 125.2)
- added R9012: 200R, Resistor_SMD:R_0603_1608Metric, F.Cu at (182.3, 125.2)
- added R9013: 200R, Resistor_SMD:R_0603_1608Metric, F.Cu at (177.5, 125.2)
- added R9014: 200R, Resistor_SMD:R_0603_1608Metric, F.Cu at (172.4, 125.2)
- added R9015: 200R, Resistor_SMD:R_0603_1608Metric, F.Cu at (167.3, 125.2)
- added R9016: 200R, Resistor_SMD:R_0603_1608Metric, F.Cu at (162.3, 125.2)
- added U9001: TLP241B, Package_SO:SO-4_7.6x3.6mm_P2.54mm, F.Cu at (163.3, 162.2)
- added U9002: TLP241B, Package_SO:SO-4_7.6x3.6mm_P2.54mm, F.Cu at (168.4, 162.1)
- added U9003: TLP241B, Package_SO:SO-4_7.6x3.6mm_P2.54mm, F.Cu at (173.5, 162.1)
- added U9004: TLP241B, Package_SO:SO-4_7.6x3.6mm_P2.54mm, F.Cu at (178.6, 162.1)
- added U9005: TLP241B, Package_SO:SO-4_7.6x3.6mm_P2.54mm, F.Cu at (183.6, 162.1)
- added U9006: TLP241B, Package_SO:SO-4_7.6x3.6mm_P2.54mm, F.Cu at (188.7, 162.1)
- added U9007: TLP241B, Package_SO:SO-4_7.6x3.6mm_P2.54mm, F.Cu at (193.8, 153.3)
- added U9008: TLP241B, Package_SO:SO-4_7.6x3.6mm_P2.54mm, F.Cu at (198.9, 153.3)
- added U9009: TLP241B, Package_SO:SO-4_7.6x3.6mm_P2.54mm, F.Cu at (198.8, 126.2)
- added U9010: TLP241B, Package_SO:SO-4_7.6x3.6mm_P2.54mm, F.Cu at (193.8, 126.2)
- added U9011: TLP241B, Package_SO:SO-4_7.6x3.6mm_P2.54mm, F.Cu at (188.7, 117.5)
- added U9012: TLP241B, Package_SO:SO-4_7.6x3.6mm_P2.54mm, F.Cu at (183.6, 117.5)
- added U9013: TLP241B, Package_SO:SO-4_7.6x3.6mm_P2.54mm, F.Cu at (178.8, 117.5)
- added U9014: TLP241B, Package_SO:SO-4_7.6x3.6mm_P2.54mm, F.Cu at (173.7, 117.5)
- added U9015: TLP241B, Package_SO:SO-4_7.6x3.6mm_P2.54mm, F.Cu at (168.6, 117.5)
- added U9016: TLP241B, Package_SO:SO-4_7.6x3.6mm_P2.54mm, F.Cu at (163.5, 117.5)
- R4007, R4008: value 200R -> 10K
- U4001, U4002: value TLP241B -> MCP23S17-E/ML; footprint Package_SO:SO-4_7.6x3.6mm_P2.54mm -> bt_footprints:QFN28_6x6MC_MCH
- moved R6006 68.3 mm to (95.5, 110.5), turned to 90 degrees
- moved C6003 66.0 mm to (109.4, 106.6), turned to 0 degrees
- moved J6001 64.3 mm to (99.0, 111.7), turned to 90 degrees
- moved J6002 61.4 mm to (104.0, 111.7), turned to 90 degrees
- moved U6003 60.5 mm to (111.1, 110.2), turned to 180 degrees
- moved C6004 59.6 mm to (115.8, 110.2), turned to -90 degrees
- moved R6004 56.0 mm to (109.2, 114.0), turned to 180 degrees
- moved R6003 53.3 mm to (110.8, 115.5), turned to 0 degrees
- moved R6005 53.2 mm to (108.4, 116.3), turned to 90 degrees
- moved J4006 51.4 mm to (91.3, 168.7), turned to -90 degrees
- moved U4001 48.6 mm to (142.0, 140.2), turned to -90 degrees
- moved R6002 48.4 mm to (105.5, 121.1), turned to 0 degrees
- moved J2001 47.8 mm to (67.8, 125.0)
- moved R4006 47.0 mm to (90.8, 163.0), turned to -90 degrees
- moved J4005 46.5 mm to (96.1, 168.7), turned to -90 degrees
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Connections:
- net /DI7 renamed /MCU_core/PGC
- net /DI8 renamed /MCU_core/PGD
- C4007 pad 1: /DI0 -> +3.3V
- C4008 pad 1: /DI4 -> +3.3V
- R4007 pad 1: /DI4 -> +3.3V
- R4007 pad 2: /IO_core/DI4x -> Net-(U4001-*RESET)
- R4008 pad 1: /DI5 -> +3.3V
- R4008 pad 2: /IO_core/DI5x -> Net-(U4002-*RESET)
- U2002 pad 1: /DO1 -> /MCU_core/DO1
- U2002 pad 12: /DI11 -> unconnected-(U2002A-RF6/AN11-Pad12)
- U2002 pad 13: /DI10 -> unconnected-(U2002A-RF5/AN10/CVREF-Pad13)
- U2002 pad 14: /DI9 -> unconnected-(U2002A-RF4/AN9-Pad14)
- U2002 pad 15: /DI0 -> unconnected-(U2002A-RF3/AN8-Pad15)
- U2002 pad 2: /DO0 -> /MCU_core/DO0
- U2002 pad 4: /DI1 -> /MCU_core/SPI_DI.INT#
- U2002 pad 43: /DI6 -> unconnected-(U2002A-RB5/KBI1-Pad43)
- U2002 pad 44: /DI5 -> unconnected-(U2002A-RB4/KBI0-Pad44)
- U2002 pad 5: /DI3 -> /MCU_core/SPI_INT2#
- U2002 pad 59: /DO7 -> /MCU_core/DO7
- U2002 pad 6: /DI4 -> unconnected-(U2002A-RB3/INT3-Pad6)
- U2002 pad 60: /DO6 -> /MCU_core/DO6
- U2002 pad 61: /DO5 -> /MCU_core/DO5
- U2002 pad 62: /DO4 -> /MCU_core/DO4
- U2002 pad 63: /DO3 -> /MCU_core/DO3
- U2002 pad 64: /DO2 -> /MCU_core/DO2
- U4001 pad 1: /IO_core/DO0x -> /IO_core/DI12
- U4001 pad 2: GND -> /IO_core/DI13
- U4001 pad 3: Net-(J4019-Pin_2) -> /IO_core/DI14
- U4001 pad 4: Net-(J4019-Pin_1) -> /IO_core/DI15
- U4002 pad 1: /IO_core/DO1x -> /IO_core/DO12
- U4002 pad 2: GND -> /IO_core/DO13
- U4002 pad 3: Net-(J4020-Pin_2) -> /IO_core/DO14
- U4002 pad 4: Net-(J4020-Pin_1) -> /IO_core/DO15
