File: HW/PIC18F_ETH/PIC18F_ETH/PIC18F_ETH.kicad_pcb (KiCad board)
At the start: 4 copper layers, 160 x 80 mm, 217 parts, among them J2001 Conn_01x06, J3001 Jack-DC, J4001 JST,2.54, J4002 JST,2.54, J4003 JST,2.54, J4004 JST,2.54, J4005 JST,2.54, J4006 JST,2.54, J5001 RJ45_LED_ETH_Shielded, J6001 JST,2.54, J6002 JST,2.54, J8001 JST,2.54, J8002 JST,2.54, J8003 JST,2.54, J8004 JST,2.54, J8005 JST,2.54, J8006 JST,2.54, J8007 JST,2.54, J8008 JST,2.54, J8009 JST,2.54, J8010 JST,2.54, J8011 JST,2.54, J8012 JST,2.54, J8013 JST,2.54, J8014 JST,2.54, J8015 JST,2.54, J8016 JST,2.54, J9001 JST,2.54, J9002 JST,2.54, J9003 JST,2.54, J9004 JST,2.54, J9005 JST,2.54, J9006 JST,2.54, J9007 JST,2.54, J9008 JST,2.54, J9009 JST,2.54, J9010 JST,2.54, J9011 JST,2.54, J9012 JST,2.54, J9013 JST,2.54, J9014 JST,2.54, J9015 JST,2.54, J9016 JST,2.54, U2001 93AA46BT-I/OT, U2002 PIC18F67J60T-I, U2003 25Mhz,50ppm, U3001 LMR51610-Q1, U3002 TPS62A01, U4001 MCP23S17-E/ML, U4002 MCP23S17-E/ML, U6001 25Mhz,50ppm, U6002 MCP2515T-E/ML, U6003 ATA6561-GAQW, U9001 TLP241B, U9002 TLP241B, U9003 TLP241B, U9004 TLP241B, U9005 TLP241B, U9006 TLP241B, U9007 TLP241B, U9008 TLP241B, U9009 TLP241B, U9010 TLP241B, U9011 TLP241B, U9012 TLP241B, U9013 TLP241B, U9014 TLP241B, U9015 TLP241B, U9016 TLP241B

Commit message: .
Parts:
- removed R3006: 2K2, Resistor_SMD:R_0603_1608Metric
- removed R3007: 43K, Resistor_SMD:R_0603_1608Metric
- removed R3008: 10K, Resistor_SMD:R_0603_1608Metric
- added D3001: D, Diode_SMD:D_0805_2012Metric, F.Cu at (59.4, 114.0)
- added R3003: 2K2, Resistor_SMD:R_0603_1608Metric, F.Cu at (94.0, 123.5)
- added R3004: 43K, Resistor_SMD:R_0603_1608Metric, F.Cu at (91.5, 122.5)
- added R3005: 10K, Resistor_SMD:R_0603_1608Metric, F.Cu at (90.0, 122.5)
- C3002: value 100n 25V -> 10u 10V
- C3003: value 10u 10V -> 100n 25V
- J3001: value Jack-DC -> Screw_Terminal_01x02; footprint Connector_BarrelJack:BarrelJack_Horizontal -> Connector_Samtec_HPM_THT:Samtec_HPM-02-01-x-S_Straight_1x02_Pitch5.08mm
- moved J2001 35.2 mm to (63.9, 160.0)
- moved R5001 22.7 mm to (53.0, 129.2), turned to 180 degrees
- moved R5006 22.2 mm to (70.0, 137.2), turned to 90 degrees
- moved C3003 19.6 mm to (72.0, 110.7)
- moved C3002 18.7 mm to (90.0, 115.7)
- moved R5002 18.3 mm to (52.8, 151.2)
- moved R5005 18.3 mm to (68.5, 138.0), turned to -90 degrees
- moved C3005 12.3 mm to (99.5, 122.2)
- moved R6001 11.3 mm to (105.2, 126.5), turned to 0 degrees
- moved C2002 10.8 mm to (96.2, 139.2)
- moved C3008 10.3 mm to (91.5, 115.7)
- moved C6001 9.75 mm to (105.2, 125.0), turned to 180 degrees
- moved C2010 8.30 mm to (96.2, 144.2), turned to 0 degrees
- moved R5004 8.20 mm to (68.5, 143.2), turned to -90 degrees
- moved J3001 7.89 mm to (51.0, 120.0), turned to 180 degrees
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Connections:
- net /IO_core/Digital Input/D12x renamed /IO_core/Digital Input/DI12x
- net /IO_core/SPI_DO.INT# renamed /SPI_DO.INT#
- net /IO_core/SPI_DO.INT1# renamed /SPI_DO.INT1#
- C3001 pad 1: Net-(U3001-EN) -> Net-(D3001-K)
- C3002 pad 1: Net-(U3001-BOOST) -> +5V
- C3002 pad 2: Net-(U3001-SW) -> GND
- C3003 pad 1: +5V -> Net-(U3001-BOOST)
- C3003 pad 2: GND -> Net-(U3001-SW)
- C3005 pad 1: +5V -> +3.3V
- C3008 pad 1: +3.3V -> +5V
- D8006 pad 1: /IO_core/Digital Input/DI8x -> /IO_core/Digital Input/DI14x
- D8006 pad 2: /IO_core/Digital Input/DI9x -> /IO_core/Digital Input/DI15x
- D8007 pad 1: /IO_core/Digital Input/DI14x -> /IO_core/Digital Input/DI8x
- D8007 pad 2: /IO_core/Digital Input/DI15x -> /IO_core/Digital Input/DI9x
- J3001 pad 1: Net-(U3001-EN) -> GND
- J3001 pad 2: GND -> Net-(D3001-A)
- U2002 pad 4: /MCU_core/SPI_DI.INT# -> /SPI_DI.INT#
- U2002 pad 5: /MCU_core/SPI_INT2# -> /SPI_DI.INT1#
- U3001 pad 4: Net-(U3001-EN) -> Net-(D3001-K)
- U3001 pad 5: Net-(U3001-EN) -> Net-(D3001-K)
- U4001 pad 10: /IO_core/SPI_DI.MISO -> /CAN_CTRL.MISO
- U4001 pad 15: /IO_core/SPI_DI.INT1# -> /SPI_DI.INT1#
- U4001 pad 16: /IO_core/SPI_DI.INT# -> /SPI_DI.INT#
- U4001 pad 7: /IO_core/SPI_DI.CS# -> /CAN_CTRL.CS#
- U4001 pad 8: /IO_core/SPI_DI.SCK -> /CAN_CTRL.SCK
- U4001 pad 9: /IO_core/SPI_DI.MOSI -> /CAN_CTRL.MOSI
- U4002 pad 10: /IO_core/SPI_DO.MISO -> /CAN_CTRL.MISO
- U4002 pad 7: /IO_core/SPI_DO.CS# -> /CAN_CTRL.CS#
- U4002 pad 8: /IO_core/SPI_DO.SCK -> /CAN_CTRL.SCK
- U4002 pad 9: /IO_core/SPI_DO.MOSI -> /CAN_CTRL.MOSI

Commit message: .
Parts:
- added D3002: LED G, LED_SMD:LED_0603_1608Metric, F.Cu at (59.2, 120.7)
- added D9001: LED G, LED_SMD:LED_0603_1608Metric, F.Cu at (198.6, 145.5)
- added D9002: LED G, LED_SMD:LED_0603_1608Metric, F.Cu at (188.5, 154.4)
- added D9003: LED G, LED_SMD:LED_0603_1608Metric, F.Cu at (163.1, 154.4)
- added D9004: LED G, LED_SMD:LED_0603_1608Metric, F.Cu at (168.1, 154.4)
- added D9005: LED G, LED_SMD:LED_0603_1608Metric, F.Cu at (173.2, 154.4)
- added D9006: LED G, LED_SMD:LED_0603_1608Metric, F.Cu at (178.3, 154.4)
- added D9007: LED G, LED_SMD:LED_0603_1608Metric, F.Cu at (183.4, 154.4)
- added D9008: LED G, LED_SMD:LED_0603_1608Metric, F.Cu at (193.5, 145.5)
- added D9009: LED G, LED_SMD:LED_0603_1608Metric, F.Cu at (199.1, 133.9)
- added D9010: LED G, LED_SMD:LED_0603_1608Metric, F.Cu at (194.1, 133.9)
- added D9011: LED G, LED_SMD:LED_0603_1608Metric, F.Cu at (189.0, 125.2)
- added D9012: LED G, LED_SMD:LED_0603_1608Metric, F.Cu at (183.9, 125.2)
- added D9013: LED G, LED_SMD:LED_0603_1608Metric, F.Cu at (179.1, 125.2)
- added D9014: LED G, LED_SMD:LED_0603_1608Metric, F.Cu at (174.0, 125.2)
- added D9015: LED G, LED_SMD:LED_0603_1608Metric, F.Cu at (168.9, 125.2)
- added D9016: LED G, LED_SMD:LED_0603_1608Metric, F.Cu at (163.8, 125.2)
- added R3006: 200R, Resistor_SMD:R_0603_1608Metric, F.Cu at (59.2, 122.4)
- added R9017: 200R, Resistor_SMD:R_0603_1608Metric, F.Cu at (199.3, 143.3)
- added R9018: 200R, Resistor_SMD:R_0603_1608Metric, F.Cu at (189.4, 152.1)
- added R9019: 200R, Resistor_SMD:R_0603_1608Metric, F.Cu at (163.8, 152.1)
- added R9020: 200R, Resistor_SMD:R_0603_1608Metric, F.Cu at (168.9, 152.1)
- added R9021: 200R, Resistor_SMD:R_0603_1608Metric, F.Cu at (174.0, 152.1)
- added R9022: 200R, Resistor_SMD:R_0603_1608Metric, F.Cu at (179.0, 152.1)
- added R9023: 200R, Resistor_SMD:R_0603_1608Metric, F.Cu at (184.1, 152.1)
- added R9024: 200R, Resistor_SMD:R_0603_1608Metric, F.Cu at (194.3, 143.3)
- added R9025: 200R, Resistor_SMD:R_0603_1608Metric, F.Cu at (198.4, 136.1)
- added R9026: 200R, Resistor_SMD:R_0603_1608Metric, F.Cu at (193.3, 136.1)
- added R9027: 200R, Resistor_SMD:R_0603_1608Metric, F.Cu at (188.2, 127.5)
- added R9028: 200R, Resistor_SMD:R_0603_1608Metric, F.Cu at (183.1, 127.5)
- added R9029: 200R, Resistor_SMD:R_0603_1608Metric, F.Cu at (178.2, 127.5)
- added R9030: 200R, Resistor_SMD:R_0603_1608Metric, F.Cu at (173.2, 127.5)
- added R9031: 200R, Resistor_SMD:R_0603_1608Metric, F.Cu at (168.1, 127.5)
- added R9032: 200R, Resistor_SMD:R_0603_1608Metric, F.Cu at (163.1, 127.5)
- moved D8006 30.5 mm to (122.9, 113.7)
- moved D8007 30.5 mm to (153.4, 113.7)
- moved R2001 4.59 mm to (105.1, 134.5), turned to 0 degrees
- moved J4002 4.45 mm to (106.3, 168.7)
- moved J4006 4.45 mm to (86.8, 168.7)
- moved C4001 4.45 mm to (110.3, 160.5)
- moved C4002 4.45 mm to (106.8, 160.5)
- moved C4003 4.45 mm to (100.3, 160.5)
- moved C4004 4.45 mm to (96.8, 160.5)
- moved C4005 4.45 mm to (90.6, 160.5)
- moved C4006 4.45 mm to (87.1, 160.5)
- moved D4001 4.45 mm to (88.9, 163.5)
- moved D4002 4.45 mm to (98.5, 163.5)
- moved D4003 4.45 mm to (108.6, 163.5)
- moved J4001 4.45 mm to (111.2, 168.7)
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Connections:
- net /CAN_CTRL.MISO renamed /SPI_DO.MISO
- net /CAN_CTRL.MOSI renamed /SPI_DO.MOSI
- net /CAN_CTRL.SCK renamed /SPI_DO.SCK
- R2001 pad 1: /MCU_core/SPI_SS1 -> /MCU_core/SPI_SS0
- U2001 pad 5: /MCU_core/SPI_SS1 -> /MCU_core/SPI_SS0
- U2002 pad 11: unconnected-(U2002A-RF7/*SS1-Pad11) -> /MCU_core/SPI_SS0
- U2002 pad 29: /CAN_CTRL.CS# -> /SPI_DO.CS#
- U2002 pad 33: /MCU_core/SPI_SS1 -> /CAN_CTRL.CS#
- U4001 pad 7: /CAN_CTRL.CS# -> /SPI_DO.CS#
- U4002 pad 7: /CAN_CTRL.CS# -> /SPI_DO.CS#
Routing:
- net /SPI_DO.MOSI: track 0.00 -> 92.1 mm, vias 0 -> 4
- net /SPI_DO.MISO: track 0.00 -> 88.3 mm, vias 0 -> 4
- net /SPI_DO.SCK: track 0.00 -> 88.2 mm, vias 0 -> 6
- net /IO_core/DI0: track 0.00 -> 45.0 mm
- net /IO_core/DI15: track 0.00 -> 40.8 mm
- net /IO_core/DI1: track 0.00 -> 39.8 mm
- net /IO_core/DO7: track 0.00 -> 35.7 mm
- net /IO_core/DI14: track 0.00 -> 35.6 mm
- net /IO_core/DI2: track 0.00 -> 35.1 mm
- net /IO_core/DI8: track 0.00 -> 35.1 mm
- net /IO_core/DO8: track 0.00 -> 33.4 mm
- net /IO_core/DO10: track 0.00 -> 32.1 mm
- net /IO_core/DO5: track 0.00 -> 32.0 mm
- net /IO_core/DI7: track 0.00 -> 31.6 mm
- net /IO_core/DO6: track 0.00 -> 30.8 mm
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
Commit message: .
Parts:
- added C3009: 3n3 50V, Capacitor_SMD:C_0603_1608Metric, F.Cu at (67.1, 111.5)
- added TP2001: TestPoint, TestPoint:TestPoint_THTPad_D1.0mm_Drill0.5mm, F.Cu at (67.3, 150.1)
- added TP2002: TestPoint, TestPoint:TestPoint_THTPad_D1.0mm_Drill0.5mm, F.Cu at (67.3, 152.4)
- added TP2003: TestPoint, TestPoint:TestPoint_THTPad_D1.0mm_Drill0.5mm, F.Cu at (98.6, 136.7)
- added TP2004: TestPoint, TestPoint:TestPoint_THTPad_D1.0mm_Drill0.5mm, F.Cu at (96.5, 136.7)
- added TP2005: TestPoint, TestPoint:TestPoint_THTPad_1.0x1.0mm_Drill0.5mm, F.Cu at (132.6, 142.5)
- added TP2006: TestPoint, TestPoint:TestPoint_THTPad_D1.0mm_Drill0.5mm, F.Cu at (108.0, 137.9)
- added TP2007: TestPoint, TestPoint:TestPoint_THTPad_D1.0mm_Drill0.5mm, F.Cu at (114.0, 118.1)
- added TP2008: TestPoint, TestPoint:TestPoint_THTPad_D1.0mm_Drill0.5mm, F.Cu at (131.6, 139.7)
- added TP2009: TestPoint, TestPoint:TestPoint_THTPad_D1.0mm_Drill0.5mm, F.Cu at (136.1, 140.7)
- added TP2010: TestPoint, TestPoint:TestPoint_THTPad_D1.0mm_Drill0.5mm, F.Cu at (134.1, 140.0)
- added TP2011: TestPoint, TestPoint:TestPoint_THTPad_D1.0mm_Drill0.5mm, F.Cu at (108.2, 135.6)
- added TP2012: TestPoint, TestPoint:TestPoint_THTPad_D1.0mm_Drill0.5mm, F.Cu at (84.8, 147.8)
- added TP2015: TestPoint, TestPoint:TestPoint_THTPad_1.0x1.0mm_Drill0.5mm, F.Cu at (100.6, 136.7)
- added TP2016: TestPoint, TestPoint:TestPoint_THTPad_1.0x1.0mm_Drill0.5mm, F.Cu at (82.0, 150.1)
- added TP3001: TestPoint, TestPoint:TestPoint_THTPad_D1.0mm_Drill0.5mm, F.Cu at (55.9, 115.1)
- added TP3002: TestPoint, TestPoint:TestPoint_THTPad_1.0x1.0mm_Drill0.5mm, F.Cu at (55.9, 118.4)
- added TP3003: TestPoint, TestPoint:TestPoint_THTPad_D1.0mm_Drill0.5mm, F.Cu at (94.7, 115.1)
- added TP3004: TestPoint, TestPoint:TestPoint_THTPad_1.0x1.0mm_Drill0.5mm, F.Cu at (98.6, 126.7)
- added TP3005: TestPoint, TestPoint:TestPoint_THTPad_D1.0mm_Drill0.5mm, F.Cu at (101.1, 126.7)
- moved J2001 24.2 mm to (87.1, 153.2)
- moved R5001 23.7 mm to (52.6, 152.9)
- moved D4001 19.8 mm to (108.6, 163.5)
- moved D4003 19.8 mm to (88.8, 163.5)
- moved FID7002 9.93 mm to (193.0, 110.0)
- moved FID7003 7.55 mm to (192.8, 170.2)
- moved R6003 1.73 mm to (109.2, 112.8), turned to -90 degrees
- moved R6004 1.72 mm to (110.7, 112.8), turned to 90 degrees
- moved R6005 1.70 mm to (107.7, 112.8)
- moved C3001 1.40 mm to (63.8, 111.8)
- moved D3001 0.85 mm to (59.2, 114.8), turned to 180 degrees
- moved R2002 0.60 mm to (87.0, 148.4)
- moved R5002 0.11 mm to (52.6, 151.2)
Routing:
- net GND: track 0.00 -> 223.0 mm, vias 0 -> 133
- net +3.3V: track 10.3 -> 80.2 mm, vias 0 -> 57
- net /SPI_DI.INT#: track 0.00 -> 57.6 mm, vias 0 -> 2
- net /SPI_DI.INT1#: track 0.00 -> 56.1 mm, vias 0 -> 2
- net +5V: track 33.8 -> 83.5 mm
- net /SPI_DO.CS#: track 24.5 -> 70.7 mm
- net /ETH_Connector/LED_Y: track 0.00 -> 46.0 mm
- net /ETH_Connector/LED_G: track 0.00 -> 45.5 mm
- net /CAN_CTRL.INT#: track 0.00 -> 40.1 mm, vias 0 -> 2
- net /AD5: track 0.00 -> 38.7 mm
- net /AD0: track 0.00 -> 35.5 mm, vias 0 -> 2
- net /AD4: track 0.00 -> 35.0 mm
- net /AD3: track 0.00 -> 35.0 mm
- net /MCU_core/PGC: track 0.00 -> 33.4 mm, vias 0 -> 1
- net /MCU_core/PGD: track 0.00 -> 32.3 mm, vias 0 -> 1
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- added copper zone on B.Cu, net +3.3V
- added copper zone on F.Cu, net +3.3V
- added copper zone on F.Cu, net GND
- added copper zone on In1.Cu, net GND
- added copper zone on In2.Cu, net GND
Other:
- board text added: "10k"
- board text added: "200"
- board text added: "3V3"
- board text added: "3V3 ADC, Digital I/O"
- board text added: "3V3 I/O"
- board text added: "AC/DC 80V 1.5A"
- board text added: "AD1"
- board text added: "AD2"
- board text added: "AD3"
- board text added: "AD4"
- board text added: "AD5"
- board text added: "AD6/ DX"
- board text added: "CAN"
- board text added: "CAN H"
- board text added: "CAN L"
- board text added: "DO1"
- board text added: "DX1"
- board text added: "GND"
- board text added: "Power Led"
- board text added: "Vin DC 6-50V"
- board text added: "opto Relay"
