File: HW/PIC18F_ETH/PIC18F_ETH/PIC18F_ETH.kicad_pcb (KiCad board)
At the start: 4 copper layers, 160 x 80 mm, 272 parts, among them J2001 Conn_01x06, J3001 Screw_Terminal_01x02, J4001 JST,2.54, J4002 JST,2.54, J4003 JST,2.54, J4004 JST,2.54, J4005 JST,2.54, J4006 JST,2.54, J5001 RJ45_LED_ETH_Shielded, J6001 JST,2.54, J6002 JST,2.54, J8001 JST,2.54, J8002 JST,2.54, J8003 JST,2.54, J8004 JST,2.54, J8005 JST,2.54, J8006 JST,2.54, J8007 JST,2.54, J8008 JST,2.54, J8009 JST,2.54, J8010 JST,2.54, J8011 JST,2.54, J8012 JST,2.54, J8013 JST,2.54, J8014 JST,2.54, J8015 JST,2.54, J8016 JST,2.54, J9001 JST,2.54, J9002 JST,2.54, J9003 JST,2.54, J9004 JST,2.54, J9005 JST,2.54, J9006 JST,2.54, J9007 JST,2.54, J9008 JST,2.54, J9009 JST,2.54, J9010 JST,2.54, J9011 JST,2.54, J9012 JST,2.54, J9013 JST,2.54, J9014 JST,2.54, J9015 JST,2.54, J9016 JST,2.54, U2001 93AA46BT-I/OT, U2002 PIC18F67J60T-I, U2003 25Mhz,50ppm, U3001 LMR51610-Q1, U3002 TPS62A01, U4001 MCP23S17-E/ML, U4002 MCP23S17-E/ML, U6001 25Mhz,50ppm, U6002 MCP2515T-E/ML, U6003 ATA6561-GAQW, U9001 TLP241B, U9002 TLP241B, U9003 TLP241B, U9004 TLP241B, U9005 TLP241B, U9006 TLP241B, U9007 TLP241B, U9008 TLP241B, U9009 TLP241B, U9010 TLP241B, U9011 TLP241B, U9012 TLP241B, U9013 TLP241B, U9014 TLP241B, U9015 TLP241B, U9016 TLP241B

Commit message: .
Parts:
- added J3002: JST,2.54, Connector_JST:JST_EH_B2B-EH-A_1x02_P2.50mm_Vertical, F.Cu at (52.2, 163.0)
- added TP3006: TestPoint, TestPoint:TestPoint_THTPad_1.0x1.0mm_Drill0.5mm, F.Cu at (90.2, 114.8)
- moved C3004 11.8 mm to (84.5, 107.5), turned to 180 degrees
- moved D3002 10.4 mm to (50.8, 126.8)
- moved R3006 10.4 mm to (50.7, 128.5)
- moved C3008 10.1 mm to (86.8, 106.8), turned to 90 degrees
- moved C3002 9.13 mm to (88.2, 106.8), turned to 90 degrees
- moved TP3003 2.02 mm to (92.8, 114.8)
Routing:
- net +5V: track 83.5 -> 95.8 mm, vias 0 -> 2
- net GND: track 223.0 -> 229.1 mm, vias 133 -> 140
- net /MCU_core/RST#: track 9.91 -> 10.5 mm
- net +3.3V: vias 57 -> 58
Other:
- board text added: "1"
- board text added: "2"
- board text added: "3"
- board text added: "3,3V"
- board text added: "4"
- board text added: "AD/DX board Version:1.0.0 (c) Björn Thor 2024"
- board text added: "AD1/ DX1"
- board text added: "AD2/ DX2"
- board text added: "AD3/ DX3"
- board text added: "AD4/ DX4"
- board text added: "AD5/ DX5"
- board text added: "AD6/ DX6"
- board text added: "DO10"
- board text added: "DO11"
- board text added: "DO12"
- board text added: "DO13"
- board text added: "DO14"
- board text added: "DO15"
- board text added: "DO16"
- board text added: "DO2"
- board text added: "DO3"
- board text added: "DO4"
- board text added: "DO5"
- board text added: "DO6"
- board text added: "DO7"
- board text added: "DO8"
- board text added: "DO9"
- board text added: "DX10"
- board text added: "DX11"
- board text added: "DX12"
- board text added: "DX13"
- board text added: "DX14"
- board text added: "DX7"
- board text added: "DX8"
- board text added: "DX9"
- board text added: "RX"
- board text added: "TX"
- board text added: "Vin DC 6-40V"
- board text removed: "AD1"
- board text removed: "AD2"
- board text removed: "AD3"
- board text removed: "AD4"
- board text removed: "AD5"
- board text removed: "AD6/ DX"
- board text removed: "Vin DC 6-50V"

Commit message: .
Parts:
- added C2012: 100n 25V, Capacitor_SMD:C_0603_1608Metric, F.Cu at (83.6, 153.2)
- added C4009: 100n 25V, Capacitor_SMD:C_0603_1608Metric, F.Cu at (137.9, 145.8)
- added C4010: 100n 25V, Capacitor_SMD:C_0603_1608Metric, F.Cu at (160.5, 146.1)
- added C6005: 100n 25V, Capacitor_SMD:C_0603_1608Metric, F.Cu at (114.5, 116.1)
Routing:
- net GND: track 229.1 -> 234.9 mm, vias 140 -> 143
- net /MCU_core/RST#: track 10.5 -> 13.3 mm
- net /CAN/CAN_CTRL_RST#: track 2.37 -> 5.00 mm
- net Net-(U4002-*RESET): track 1.71 -> 3.35 mm
- net Net-(U4001-*RESET): track 1.85 -> 3.39 mm
Other:
- board text added: "DX15"
- board text added: "DX16"
- board text added: "DX17"
- board text added: "DX18"
- board text added: "DX19"
- board text added: "DX20"
- board text added: "DX21"
- board text added: "DX22"
- board text removed: "DX1"

Commit message: .
Connections:
- D4001 pad 1: /IO_core/AD3x -> /IO_core/AD1x
- D4002 pad 1: /IO_core/AD2x -> /IO_core/AD3x
- D4002 pad 2: /IO_core/AD1x -> /IO_core/AD2x
- J4002 pad 2: /IO_core/AD3x -> /IO_core/AD1x
- J4003 pad 2: /IO_core/AD1x -> /IO_core/AD2x
- J4004 pad 2: /IO_core/AD2x -> /IO_core/AD3x
- R4002 pad 2: /IO_core/AD3x -> /IO_core/AD1x
- R4003 pad 2: /IO_core/AD1x -> /IO_core/AD2x
- R4004 pad 2: /IO_core/AD2x -> /IO_core/AD3x
Changed lines of the file:
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@@
 			(layers "F.Cu" "F.Paste" "F.Mask")
 			(roundrect_rratio 0.25)
-			(net 73 "/IO_core/AD2x")
+			(net 74 "/IO_core/AD3x")
 			(pintype "passive")
 		)
@@
 			(layers "F.Cu" "F.Paste" "F.Mask")
 			(roundrect_rratio 0.25)
-			(net 74 "/IO_core/AD3x")
+			(net 72 "/IO_core/AD1x")
 			(pintype "passive")
 		)
@@
 			(layers "F.Cu" "F.Paste" "F.Mask")
 			(roundrect_rratio 0.25)
-			(net 72 "/IO_core/AD1x")
+			(net 73 "/IO_core/AD2x")
 			(pintype "passive")
 		)
@@
 			(layers "F.Cu" "F.Paste" "F.Mask")
 			(roundrect_rratio 0.25)
-			(net 73 "/IO_core/AD2x")
+			(net 74 "/IO_core/AD3x")
 			(pinfunction "K1")
 			(pintype "passive")
@@
 			(layers "F.Cu" "F.Paste" "F.Mask")
 			(roundrect_rratio 0.25)
-			(net 72 "/IO_core/AD1x")
+			(net 73 "/IO_core/AD2x")
 			(pinfunction "K2")
 			(pintype "passive")
@@
 			(layers "*.Cu" "*.Mask")
 			(remove_unused_layers no)
-			(net 72 "/IO_core/AD1x")
+			(net 73 "/IO_core/AD2x")
 			(pinfunction "Pin_2")
 			(pintype "passive")
@@
 			(net 190 "/SPI_DO.INT1#")
 			(pinfunction "INTB")
-			(pintype "open_collector")
+			(pintype "open_collector+no_connect")
 		)
 		(pad "16" smd rect
@@
 			(net 189 "/SPI_DO.INT#")
 			(pinfunction "INTA")
-			(pintype "open_collector")
+			(pintype "open_collector+no_connect")
 		)
 		(pad "17" smd rect
@@
 			(layers "F.Cu" "F.Paste" "F.Mask")
 			(roundrect_rratio 0.25)
-			(net 74 "/IO_core/AD3x")
+			(net 72 "/IO_core/AD1x")
 			(pinfunction "K1")
 			(pintype "passive")
@@
 			(net 166 "/MCU_core/DO1")
 			(pinfunction "RE1/P2C")
-			(pintype "unspecified")
+			(pintype "unspecified+no_connect")
 		)
 		(pad "2" smd rect
@@
 			(net 164 "/MCU_core/DO0")
 			(pinfunction "RE0/P2D")
-			(pintype "unspecified")
+			(pintype "unspecified+no_connect")
 		)
 		(pad "3" smd rect
@@
 			(net 163 "unconnected-(U2002A-RB3{slash}INT3-Pad6)")
 			(pinfunction "RB3/INT3")
-			(pintype "unspecified")
+			(pintype "unspecified+no_connect")
 		)
 		(pad "7" smd rect
@@
 			(net 107 "unconnected-(U2002A-RG4{slash}CCP5{slash}P1D-Pad8)")
 			(pinfunction "RG4/CCP5/P1D")
-			(pintype "unspecified")
+			(pintype "unspecified+no_connect")
 		)
 		(pad "9" smd rect
@@
 			(net 158 "unconnected-(U2002A-RF6{slash}AN11-Pad12)")
 			(pinfunction "RF6/AN11")
-			(pintype "unspecified")
+			(pintype "unspecified+no_connect")
 		)
 		(pad "13" smd rect
@@
 			(net 157 "unconnected-(U2002A-RF5{slash}AN10{slash}CVREF-Pad13)")
 			(pinfunction "RF5/AN10/CVREF")
-			(pintype "unspecified")
+			(pintype "unspecified+no_connect")
 		)
 		(pad "14" smd rect
@@
 			(net 161 "unconnected-(U2002A-RF4{slash}AN9-Pad14)")
 			(pinfunction "RF4/AN9")
-			(pintype "unspecified")
+			(pintype "unspecified+no_connect")
 		)
 		(pad "15" smd rect
@@
 			(net 167 "unconnected-(U2002A-RF3{slash}AN8-Pad15)")
 			(pinfunction "RF3/AN8")
-			(pintype "unspecified")
+			(pintype "unspecified+no_connect")
 		)
 		(pad "16" smd rect
@@
 			(net 50 "/MCU_core/SPI_SS3")
 			(pinfunction "RC0/T1OSO/T13CKI")
-			(pintype "unspecified")
+			(pintype "unspecified+no_connect")
 		)
 		(pad "31" smd rect
@@
 			(net 156 "unconnected-(U2002A-RB5{slash}KBI1-Pad43)")
 			(pinfunction "RB5/KBI1")
-			(pintype "unspecified")
+			(pintype "unspecified+no_connect")
 		)
 		(pad "44" smd rect
@@
 			(net 162 "unconnected-(U2002A-RB4{slash}KBI0-Pad44)")
 			(pinfunction "RB4/KBI0")
-			(pintype "unspecified")
+			(pintype "unspecified+no_connect")
 		)
 		(pad "45" smd rect
@@
 			(net 46 "/MCU_core/DO8")
 			(pinfunction "RD2/CCP4/P3D")
-			(pintype "unspecified")
+			(pintype "unspecified+no_connect")
 		)
 		(pad "59" smd rect
@@
 			(net 168 "/MCU_core/DO7")
 			(pinfunction "RD1/ECCP3/P3A")
-			(pintype "unspecified")
+			(pintype "unspecified+no_connect")
 		)
 		(pad "60" smd rect
@@
 			(net 155 "/MCU_core/DO6")
 			(pinfunction "RD0/P1B")
-			(pintype "unspecified")
+			(pintype "unspecified+no_connect")
 		)
 		(pad "61" smd rect
@@
 			(net 165 "/MCU_core/DO5")
 			(pinfunction "RE5/P1C")
-			(pintype "unspecified")
+			(pintype "unspecified+no_connect")
 		)
 		(pad "62" smd rect
@@
 			(net 154 "/MCU_core/DO4")
 			(pinfunction "RE4/P3B")
-			(pintype "unspecified")
+			(pintype "unspecified+no_connect")
 		)
 		(pad "63" smd rect
@@
 			(net 160 "/MCU_core/DO3")
 			(pinfunction "RE3/P3C")
-			(pintype "unspecified")
+			(pintype "unspecified+no_connect")
 		)
 		(pad "64" smd rect
@@
 			(net 159 "/MCU_core/DO2")
 			(pinfunction "RE2/P2B")
-			(pintype "unspecified")
+			(pintype "unspecified+no_connect")
 		)
 	)
@@
 			(layers "*.Cu" "*.Mask")
 			(remove_unused_layers no)
-			(net 74 "/IO_core/AD3x")
+			(net 72 "/IO_core/AD1x")
 			(pinfunction "Pin_2")
 			(pintype "passive")
@@
 			(layers "*.Cu" "*.Mask")
 			(remove_unused_layers no)
-			(net 73 "/IO_core/AD2x")
+			(net 74 "/IO_core/AD3x")
 			(pinfunction "Pin_2")
 			(pintype "passive")
@@
 		(tags "capacitor")
 		(property "Reference" "C2012"
-			(at 0 -1.43 360)
+			(at 0 -1.43 0)
 			(layer "F.SilkS")
 			(hide yes)
@@
 		)
 		(property "Value" "100n 25V"
-			(at 0 1.43 360)
+			(at 0 1.43 0)
 			(layer "F.Fab")
 			(hide yes)
@@
 		)
 		(fp_text user "${REFERENCE}"
-			(at 0 0 360)
+			(at 0 0 0)
 			(layer "F.Fab")
 			(effects
@@
 	)
 	(segment
-		(start 99.472 164.6585)
-		(end 100.3545 163.776)
+		(start 106.8135 163.776)
+		(end 106.09 163.776)
 		(width 0.15)
 		(layer "F.Cu")
@@
 	)
 	(segment
-		(start 101.346 171.156)
-		(end 99.472 169.282)
+		(start 107.696 169.804)
+		(end 107.696 164.6585)
 		(width 0.15)
 		(layer "F.Cu")
@@
 	)
 	(segment
-		(start 100.3545 163.776)
-		(end 101.022 163.776)
+		(start 106.344 171.156)
+		(end 107.696 169.804)
 		(width 0.15)
 		(layer "F.Cu")
@@
 	)
 	(segment
-		(start 99.472 169.282)
-		(end 99.472 164.6585)
+		(start 107.696 164.6585)
+		(end 106.8135 163.776)
 		(width 0.15)
 		(layer "F.Cu")
@@
 	)
 	(segment
-		(start 96.52 171.156)
-		(end 96.52 170.588968)
+		(start 99.472 164.6585)
+		(end 100.3545 163.776)
 		(width 0.15)
 		(layer "F.Cu")
@@
 	)
 	(segment
-		(start 97.67 169.438968)
-		(end 97.67 164.7565)
+		(start 101.346 171.156)
+		(end 99.472 169.282)
 		(width 0.15)
 		(layer "F.Cu")
@@
 	)
 	(segment
-		(start 96.6895 163.776)
-		(end 96.022 163.776)
+		(start 100.3545 163.776)
+		(end 101.022 163.776)
 		(width 0.15)
 		(layer "F.Cu")
@@
 	)
 	(segment
-		(start 97.572 164.6585)
-		(end 96.6895 163.776)
+		(start 99.472 169.282)
+		(end 99.472 164.6585)
 		(width 0.15)
 		(layer "F.Cu")
@@
 	)
 	(segment
-		(start 97.67 164.7565)
-		(end 97.572 164.6585)
+		(start 96.52 171.156)
+		(end 96.52 170.588968)
 		(width 0.15)
 		(layer "F.Cu")
-		(net 73)
+		(net 74)
 	)
 	(segment
-		(start 96.52 170.588968)
-		(end 97.67 169.438968)
+		(start 97.67 169.438968)
+		(end 97.67 164.7565)
 		(width 0.15)
 		(layer "F.Cu")
-		(net 73)
+		(net 74)
 	)
 	(segment
-		(start 106.8135 163.776)
-		(end 106.09 163.776)
+		(start 96.6895 163.776)
+		(end 96.022 163.776)
 		(width 0.15)
 		(layer "F.Cu")
@@
 	)
 	(segment
-		(start 107.696 169.804)
-		(end 107.696 164.6585)
+		(start 97.572 164.6585)
+		(end 96.6895 163.776)
 		(width 0.15)
 		(layer "F.Cu")
@@
 	)
 	(segment
-		(start 106.344 171.156)
-		(end 107.696 169.804)
+		(start 97.67 164.7565)
+		(end 97.572 164.6585)
 		(width 0.15)
 		(layer "F.Cu")
@@
 	)
 	(segment
-		(start 107.696 164.6585)
-		(end 106.8135 163.776)
+		(start 96.52 170.588968)
+		(end 97.67 169.438968)
 		(width 0.15)
 		(layer "F.Cu")
