File: HW/PIC18F_ETH/PIC18F_ETH/PIC18F_ETH.kicad_pcb (KiCad board)
At the start: 4 copper layers, 160 x 80 mm, 278 parts, among them J2001 Conn_01x06, J3001 Screw_Terminal_01x02, J3002 JST,2.54, J4001 JST,2.54, J4002 JST,2.54, J4003 JST,2.54, J4004 JST,2.54, J4005 JST,2.54, J4006 JST,2.54, J5001 RJ45_LED_ETH_Shielded, J6001 JST,2.54, J6002 JST,2.54, J8001 JST,2.54, J8002 JST,2.54, J8003 JST,2.54, J8004 JST,2.54, J8005 JST,2.54, J8006 JST,2.54, J8007 JST,2.54, J8008 JST,2.54, J8009 JST,2.54, J8010 JST,2.54, J8011 JST,2.54, J8012 JST,2.54, J8013 JST,2.54, J8014 JST,2.54, J8015 JST,2.54, J8016 JST,2.54, J9001 JST,2.54, J9002 JST,2.54, J9003 JST,2.54, J9004 JST,2.54, J9005 JST,2.54, J9006 JST,2.54, J9007 JST,2.54, J9008 JST,2.54, J9009 JST,2.54, J9010 JST,2.54, J9011 JST,2.54, J9012 JST,2.54, J9013 JST,2.54, J9014 JST,2.54, J9015 JST,2.54, J9016 JST,2.54, U2001 93AA46BT-I/OT, U2002 PIC18F67J60T-I, U2003 25Mhz,50ppm, U3001 LMR51610-Q1, U3002 TPS62A01, U4001 MCP23S17-E/ML, U4002 MCP23S17-E/ML, U6001 25Mhz,50ppm, U6002 MCP2515T-E/ML, U6003 ATA6561-GAQW, U9001 TLP241B, U9002 TLP241B, U9003 TLP241B, U9004 TLP241B, U9005 TLP241B, U9006 TLP241B, U9007 TLP241B, U9008 TLP241B, U9009 TLP241B, U9010 TLP241B, U9011 TLP241B, U9012 TLP241B, U9013 TLP241B, U9014 TLP241B, U9015 TLP241B, U9016 TLP241B

Commit message: .
Parts:
- C3001: value C_Polarized -> 4,7uF 100V
- C3002, C3004, C3006, C3008: value 10u 10V -> 10u 50V
- C3009: value 3n3 50V -> 100n 100V
Changed lines of the file:
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@@
 			)
 		)
-		(property "Value" "10u 10V"
+		(property "Value" "10u 50V"
 			(at 0 1.43 90)
 			(layer "F.Fab")
@@
 			)
 		)
-		(property "CPN" "BT00010-060100"
+		(property "CPN" "BT00007-060100"
 			(at 0 0 90)
 			(unlocked yes)
@@
 			)
 		)
-		(property "Value" "3n3 50V"
+		(property "Value" "100n 100V"
 			(at 0 1.43 90)
 			(layer "F.Fab")
@@
 			)
 		)
-		(property "MPN" "C;C;T1;S;P0603;NA"
+		(property "MPN" "C;M;100n;10p;100V;S;0603"
 			(at 0 0 90)
 			(unlocked yes)
@@
 			)
 		)
-		(property "CPN" "BT00007-090033"
+		(property "CPN" "BT00013-090680"
 			(at 0 0 90)
 			(unlocked yes)
@@
 			)
 		)
-		(property "Value" "10u 10V"
+		(property "Value" "10u 50V"
 			(at 0 1.43 90)
 			(layer "F.Fab")
@@
 			)
 		)
-		(property "CPN" "BT00010-060100"
+		(property "CPN" "BT00007-060100"
 			(at 0 0 90)
 			(unlocked yes)
@@
 			)
 		)
-		(property "Value" "10u 10V"
+		(property "Value" "10u 50V"
 			(at 0 1.43 180)
 			(layer "F.Fab")
@@
 			)
 		)
-		(property "CPN" "BT00010-060100"
+		(property "CPN" "BT00007-060100"
 			(at 0 0 180)
 			(unlocked yes)
@@
 			)
 		)
-		(property "Value" "10u 10V"
+		(property "Value" "10u 50V"
 			(at 0 1.43 0)
 			(layer "F.Fab")
@@
 			)
 		)
-		(property "CPN" "BT00010-060100"
+		(property "CPN" "BT00007-060100"
 			(at 0 0 180)
 			(unlocked yes)
@@
 			)
 		)
-		(property "Value" "C_Polarized"
+		(property "Value" "4,7uF 100V"
 			(at 0 3.2 -90)
 			(layer "F.Fab")
@@
 	)
 	(segment
-		(start 93.688999 138.18)
-		(end 94.996 138.18)
-		(width 0.1)
+		(start 94.742 138.176)
+		(end 94.667999 138.250001)
+		(width 0.15)
 		(layer "F.Cu")
 		(net 5)
 	)
 	(segment
-		(start 97.385554 138.18)
-		(end 94.996 138.18)
+		(start 94.667999 138.250001)
+		(end 93.618998 138.250001)
 		(width 0.15)
 		(layer "F.Cu")
@@
 	)
 	(segment
-		(start 103.116 143.910446)
-		(end 97.385554 138.18)
+		(start 94.746 138.18)
+		(end 94.742 138.176)
 		(width 0.15)
 		(layer "F.Cu")
@@
 	)
 	(segment
-		(start 101.047 159.811)
-		(end 103.116 157.742)
+		(start 101.047 160.528)
+		(end 101.047 159.811)
 		(width 0.15)
 		(layer "F.Cu")
@@
 	)
 	(segment
-		(start 93.618998 138.250001)
-		(end 93.688999 138.18)
-		(width 0.1)
+		(start 97.385554 138.18)
+		(end 94.746 138.18)
+		(width 0.15)
 		(layer "F.Cu")
 		(net 5)
@@
 	)
 	(segment
-		(start 101.047 160.528)
-		(end 101.047 159.811)
+		(start 103.116 143.910446)
+		(end 97.385554 138.18)
+		(width 0.15)
+		(layer "F.Cu")
+		(net 5)
+	)
+	(segment
+		(start 93.618998 138.250001)
+		(end 93.688999 138.18)
+		(width 0.1)
+		(layer "F.Cu")
+		(net 5)
+	)
+	(segment
+		(start 101.047 159.811)
+		(end 103.116 157.742)
 		(width 0.15)
 		(layer "F.Cu")

Commit message: .
Parts:
- removed TP2003, TP2004: TestPoint, TestPoint:TestPoint_THTPad_D1.0mm_Drill0.5mm
- removed TP2015: TestPoint, TestPoint:TestPoint_THTPad_1.0x1.0mm_Drill0.5mm
- added J2002: JST,2.54, Connector_JST:JST_EH_B3B-EH-A_1x03_P2.50mm_Vertical, F.Cu at (115.6, 129.3)
- J3001: value Screw_Terminal_01x02 -> 6-40V
- R3001: value 160K -> 16K
- R3002: value 30K -> 3K
- moved TP2006 29.0 mm to (136.9, 136.4)
- moved TP2011 2.05 mm to (108.0, 133.6)
- moved TP2007 1.30 mm to (114.3, 119.4)
Connections:
- net /ETH_Connector/LED_G renamed /LED_G
- net /ETH_Connector/LED_Y renamed /LED_Y
- U2002 pad 1: /MCU_core/DO1 -> unconnected-(U2002A-RE1/P2C-Pad1)
- U2002 pad 2: /MCU_core/DO0 -> unconnected-(U2002A-RE0/P2D-Pad2)
- U2002 pad 58: /MCU_core/DO8 -> unconnected-(U2002A-RD2/CCP4/P3D-Pad58)
- U2002 pad 59: /MCU_core/DO7 -> unconnected-(U2002A-RD1/ECCP3/P3A-Pad59)
- U2002 pad 60: /MCU_core/DO6 -> unconnected-(U2002A-RD0/P1B-Pad60)
- U2002 pad 61: /MCU_core/DO5 -> unconnected-(U2002A-RE5/P1C-Pad61)
- U2002 pad 62: /MCU_core/DO4 -> unconnected-(U2002A-RE4/P3B-Pad62)
- U2002 pad 63: /MCU_core/DO3 -> unconnected-(U2002A-RE3/P3C-Pad63)
- U2002 pad 64: /MCU_core/DO2 -> unconnected-(U2002A-RE2/P2B-Pad64)
Routing:
- net /MCU_core/UART_TX: track 2.94 -> 23.0 mm
- net /MCU_core/UART_RX: track 5.33 -> 23.9 mm
- net /SPI_DO.CS#: track 70.7 -> 73.5 mm
- net GND: track 234.9 -> 235.3 mm, vias 143 -> 144

Commit message: .
Parts:
- added R2006: 10K, Resistor_SMD:R_0603_1608Metric, F.Cu at (222.3, 131.0)
- added R2007: 10K, Resistor_SMD:R_0603_1608Metric, F.Cu at (199.5, 114.0)
- added R2008: 10K, Resistor_SMD:R_0603_1608Metric, F.Cu at (225.9, 143.2)
- added R2009: 10K, Resistor_SMD:R_0603_1608Metric, F.Cu at (169.5, 144.8)
- added R2010: 10K, Resistor_SMD:R_0603_1608Metric, F.Cu at (224.1, 143.2)
- moved H7002 85.0 mm to (281.5, 103.6)
- moved C2004 84.9 mm to (175.1, 128.9)
- moved H7004 84.6 mm to (135.5, 169.6)
- moved H7003 84.5 mm to (281.5, 169.6)
- moved D9001 84.5 mm to (283.0, 141.9)
- moved R9008 84.5 mm to (284.6, 142.0)
- moved R9014 84.5 mm to (256.8, 121.7)
- moved R9023 84.5 mm to (268.5, 148.6)
- moved U9011 84.5 mm to (273.1, 114.0)
- moved C2001 84.5 mm to (188.8, 128.5)
- moved C2002 84.5 mm to (180.7, 135.7)
- moved C2005 84.5 mm to (163.4, 137.1)
- moved C2006 84.5 mm to (163.4, 135.6)
- moved C2007 84.5 mm to (180.7, 139.2)
- moved C2010 84.5 mm to (180.6, 140.7)
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Connections:
- C5001 pad 1: /ETH_Connector/RX_C -> Net-(C5001-Pad1)
- C5002 pad 1: /ETH_Connector/TX_C -> +3.3V
- C5002 pad 2: +3.3V -> GND
- J5001 pad 3: /ETH_Connector/TX_C -> +3.3V
- R5003 pad 2: /ETH_Connector/RX_C -> Net-(C5001-Pad1)
- R5004 pad 1: /ETH_Connector/RX_C -> Net-(C5001-Pad1)
- R5005 pad 2: /ETH_Connector/TX_C -> +3.3V
- R5006 pad 1: /ETH_Connector/TX_C -> +3.3V
- U2002 pad 30: /MCU_core/SPI_SS3 -> unconnected-(U2002A-RC0/T1OSO/T13CKI-Pad30)
- U4002 pad 15: /SPI_DO.INT1# -> unconnected-(U4002-INTB-Pad15)
- U4002 pad 16: /SPI_DO.INT# -> unconnected-(U4002-INTA-Pad16)
Routing:
- net +3.3V: track 80.2 -> 94.3 mm
- net /ETH_Connector/TX_C: track 14.0 -> 0.00 mm
- net /ETH_Connector/RX_C: track 10.4 -> 0.00 mm
- net Net-(C5001-Pad1): track 0.00 -> 3.00 mm
- net /SPI_DI.INT#: track 57.6 -> 59.6 mm
- net /CAN_CTRL.INT#: track 40.1 -> 42.1 mm
- net /SPI_DO.CS#: track 73.5 -> 75.3 mm
- net Net-(J5001-Pad11): track 7.40 -> 9.22 mm
- net /CAN_CTRL.CS#: track 30.7 -> 32.5 mm
- net /SPI_DI.INT1#: track 56.1 -> 57.5 mm
- net GND: track 235.3 -> 235.2 mm, vias 144 -> 176
Other:
- board text added: "7mA max"
