File: HW/PIC18F_ETH/PIC18F_ETH/CAN.kicad_sch (KiCad schematic)
At the start: 1 part

Commit message: .
Parts:
- gave numbers to parts that had none: 1
Changed lines of the file:
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@@
 		(dnp no)
 		(fields_autoplaced yes)
-		(property "Reference" "U?"
+		(property "Reference" "U6001"
 			(at 208.28 100.33 0)
 			(effects
@@
 			(project "PIC18F_ETH"
 				(path "/26a36835-4e01-4565-9612-f38560505464/ab2c46cb-188d-485d-996b-6193419384b9"
-					(reference "U?")
+					(reference "U6001")
 					(unit 1)
 				)

Commit message: .
Parts:
- U6001: footprint QFN20_4x4MC_MCH -> bt_footprints:QFN20_4x4MC_MCH
Changed lines of the file:
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@@
 			)
 		)
-		(property "Footprint" "QFN20_4x4MC_MCH"
+		(property "Footprint" "bt_footprints:QFN20_4x4MC_MCH"
 			(at 182.88 110.49 0)
 			(effects

Commit message: .
Parts:
- added R6001, R6002, R6005: 10K, Resistor_SMD:R_0603_1608Metric, symbol bt_resistors:R;G;10K;10P0;S;0603
- added R6003, R6004: 0R, Resistor_SMD:R_0603_1608Metric, symbol bt_resistors:R;G;0R;10P0;S;0603
- added U6002: 25Mhz,50ppm, Oscillator:Oscillator_SMD_SeikoEpson_SG8002CE-4Pin_3.2x2.5mm, symbol bt_oscillator:OSC;25Mhz;50ppm;3v3;SG3225CAN
- added U6003: ATA6561-GAQW, bt_footprints:SOIC8_4P9X3P9MC_MCH, symbol bt_communication:ATA6561-GAQW
- U6001: footprint bt_footprints:QFN20_4x4MC_MCH -> QFN20_4x4MC_MCH; CPN (none) -> BT02006-00001 MCP2515; MPN (none) -> MCP2515T-E/ML; SMT (none) -> y
Connections:
- net at U6001.10 (*RX0BF): now also R6003.2
- net CAN_CTRL.INT#: now reaches U6001.11 (*INT)
- net CAN_CTRL.SCK: now reaches U6001.12 (SCK)
- net CAN_CTRL.MOSI: now reaches U6001.14 (SI)
- net CAN_CTRL.MISO: now reaches U6001.15 (SO)
- net CAN_CTRL.CS#: now reaches U6001.16 (*CS)
- net at U6001.17 (*RESET): now also R6002.2
- net +3.3V: now reaches U6001.18 (VDD)
- net +3.3V: now also R6001.1, R6002.1, R6005.1, U6002.4 (Vcc), U6003.5 (VIO)
- net CAN_TX: now reaches U6001.19 (TXCAN)
- net CAN_TX: now also U6003.1 (TXD)
- net CAN_RX: now reaches U6001.20 (RXCAN)
- net CAN_RX: now also U6003.4 (RXD)
- net GND: now reaches U6001.21 (EPAD)
- net GND: now also U6001.8 (GND), R6004.1, U6002.2 (GND), U6003.2 (GND)
- net 25Mhz_CAN: now reaches U6001.7 (OSC1)
- net 25Mhz_CAN: now also U6002.3 (OUT)
- new net: R6001.2, U6002.1 (ST#)
- new net +5V: U6003.3 (VCC)
- new net CAN_H: U6003.7 (CANH)
- new net CAN_L: U6003.6 (CANL)
- new net CAN_STBY: R6003.1, R6004.2, R6005.2, U6003.8 (STBY)

Commit message: .
Parts:
- added C6001, C6002, C6003, C6004: 100n 25V, Capacitor_SMD:C_0603_1608Metric, symbol bt_capacitor:C;M;100n;10p;25V;S;0603
- added J6001, J6002: JST,2.54, Connector_JST:JST_EH_B3B-EH-A_1x03_P2.50mm_Vertical, symbol bt_connector:M;JST;01x03;2.54
- added R6006: 120R, Resistor_SMD:R_0603_1608Metric, symbol bt_resistors:R;G;120R;10P0;S;0603
Connections:
- net +3.3V: now also C6001.1, C6002.1, C6003.1
- net +5V: now also C6004.1
- net CAN_H: now also J6001.1 (Pin_1), J6002.1 (Pin_1), R6006.1
- net CAN_L: now also J6001.2 (Pin_2), J6002.2 (Pin_2), R6006.2
- net GND: now also C6001.2, C6002.2, C6003.2, C6004.2, J6001.3 (Pin_3), J6002.3 (Pin_3)
- net CAN_CTRL_RST#: now reaches R6002.2, U6001.17 (*RESET)
- no-connect marks 0 -> 6

Commit message: .
Parts:
- U6002: renamed from U6001; footprint QFN20_4x4MC_MCH -> bt_footprints:QFN20_4x4MC_MCH
- renumbered U6002 to U6001
Changed lines of the file:
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@@
 		(dnp no)
 		(fields_autoplaced yes)
-		(property "Reference" "#PWR06001"
+		(property "Reference" "#PWR06009"
 			(at 233.68 100.33 0)
 			(effects
@@
 			(project "PIC18F_ETH"
 				(path "/26a36835-4e01-4565-9612-f38560505464/ab2c46cb-188d-485d-996b-6193419384b9"
-					(reference "#PWR06001")
+					(reference "#PWR06009")
 					(unit 1)
 				)
@@
 		(dnp no)
 		(fields_autoplaced yes)
-		(property "Reference" "#PWR06002"
+		(property "Reference" "#PWR06011"
 			(at 259.08 93.98 0)
 			(effects
@@
 			(project "PIC18F_ETH"
 				(path "/26a36835-4e01-4565-9612-f38560505464/ab2c46cb-188d-485d-996b-6193419384b9"
-					(reference "#PWR06002")
+					(reference "#PWR06011")
 					(unit 1)
 				)
@@
 		(dnp no)
 		(fields_autoplaced yes)
-		(property "Reference" "#PWR06016"
+		(property "Reference" "#PWR06013"
 			(at 269.24 97.79 0)
 			(effects
@@
 			(project "PIC18F_ETH"
 				(path "/26a36835-4e01-4565-9612-f38560505464/ab2c46cb-188d-485d-996b-6193419384b9"
-					(reference "#PWR06016")
+					(reference "#PWR06013")
 					(unit 1)
 				)
@@
 		(dnp no)
 		(fields_autoplaced yes)
-		(property "Reference" "#PWR06018"
+		(property "Reference" "#PWR06017"
 			(at 316.23 97.79 0)
 			(effects
@@
 			(project "PIC18F_ETH"
 				(path "/26a36835-4e01-4565-9612-f38560505464/ab2c46cb-188d-485d-996b-6193419384b9"
-					(reference "#PWR06018")
+					(reference "#PWR06017")
 					(unit 1)
 				)
@@
 		(dnp no)
 		(fields_autoplaced yes)
-		(property "Reference" "#PWR06017"
+		(property "Reference" "#PWR06016"
 			(at 316.23 87.63 0)
 			(effects
@@
 			(project "PIC18F_ETH"
 				(path "/26a36835-4e01-4565-9612-f38560505464/ab2c46cb-188d-485d-996b-6193419384b9"
-					(reference "#PWR06017")
+					(reference "#PWR06016")
 					(unit 1)
 				)
@@
 		(dnp no)
 		(fields_autoplaced yes)
-		(property "Reference" "#PWR06012"
+		(property "Reference" "#PWR06004"
 			(at 149.86 171.45 0)
 			(effects
@@
 			(project "PIC18F_ETH"
 				(path "/26a36835-4e01-4565-9612-f38560505464/ab2c46cb-188d-485d-996b-6193419384b9"
-					(reference "#PWR06012")
+					(reference "#PWR06004")
 					(unit 1)
 				)
@@
 		(dnp no)
 		(fields_autoplaced yes)
-		(property "Reference" "#PWR06006"
+		(property "Reference" "#PWR06001"
 			(at 133.35 134.62 0)
 			(effects
@@
 			(project "PIC18F_ETH"
 				(path "/26a36835-4e01-4565-9612-f38560505464/ab2c46cb-188d-485d-996b-6193419384b9"
-					(reference "#PWR06006")
+					(reference "#PWR06001")
 					(unit 1)
 				)
@@
 		(dnp no)
 		(fields_autoplaced yes)
-		(property "Reference" "#PWR06013"
+		(property "Reference" "#PWR06007"
 			(at 223.52 83.82 0)
 			(effects
@@
 			(project "PIC18F_ETH"
 				(path "/26a36835-4e01-4565-9612-f38560505464/ab2c46cb-188d-485d-996b-6193419384b9"
-					(reference "#PWR06013")
+					(reference "#PWR06007")
 					(unit 1)
 				)
@@
 		(dnp no)
 		(fields_autoplaced yes)
-		(property "Reference" "#PWR06014"
+		(property "Reference" "#PWR06008"
 			(at 223.52 93.98 0)
 			(effects
@@
 			(project "PIC18F_ETH"
 				(path "/26a36835-4e01-4565-9612-f38560505464/ab2c46cb-188d-485d-996b-6193419384b9"
-					(reference "#PWR06014")
+					(reference "#PWR06008")
 					(unit 1)
 				)
@@
 		(dnp no)
 		(fields_autoplaced yes)
-		(property "Reference" "#PWR06015"
+		(property "Reference" "#PWR06012"
 			(at 269.24 87.63 0)
 			(effects
@@
 			(project "PIC18F_ETH"
 				(path "/26a36835-4e01-4565-9612-f38560505464/ab2c46cb-188d-485d-996b-6193419384b9"
-					(reference "#PWR06015")
+					(reference "#PWR06012")
 					(unit 1)
 				)
@@
 		(dnp no)
 		(fields_autoplaced yes)
-		(property "Reference" "#PWR06003"
+		(property "Reference" "#PWR06006"
 			(at 210.82 152.4 0)
 			(effects
@@
 			(project "PIC18F_ETH"
 				(path "/26a36835-4e01-4565-9612-f38560505464/ab2c46cb-188d-485d-996b-6193419384b9"
-					(reference "#PWR06003")
+					(reference "#PWR06006")
 					(unit 1)
 				)
@@
 		(on_board yes)
 		(dnp no)
-		(property "Reference" "U6002"
+		(property "Reference" "U6001"
 			(at 126.492 136.652 0)
 			(effects
@@
 			(project "PIC18F_ETH"
 				(path "/26a36835-4e01-4565-9612-f38560505464/ab2c46cb-188d-485d-996b-6193419384b9"
-					(reference "U6002")
+					(reference "U6001")
 					(unit 1)
 				)
@@
 		(dnp no)
 		(fields_autoplaced yes)
-		(property "Reference" "#PWR06004"
+		(property "Reference" "#PWR06014"
 			(at 279.4 134.62 0)
 			(effects
@@
 			(project "PIC18F_ETH"
 				(path "/26a36835-4e01-4565-9612-f38560505464/ab2c46cb-188d-485d-996b-6193419384b9"
-					(reference "#PWR06004")
+					(reference "#PWR06014")
 					(unit 1)
 				)
@@
 		(dnp no)
 		(fields_autoplaced yes)
-		(property "Reference" "#PWR06007"
+		(property "Reference" "#PWR06002"
 			(at 133.35 166.37 0)
 			(effects
@@
 			(project "PIC18F_ETH"
 				(path "/26a36835-4e01-4565-9612-f38560505464/ab2c46cb-188d-485d-996b-6193419384b9"
-					(reference "#PWR06007")
+					(reference "#PWR06002")
 					(unit 1)
 				)
@@
 		(dnp no)
 		(fields_autoplaced yes)
-		(property "Reference" "#PWR06009"
+		(property "Reference" "#PWR06010"
 			(at 254 134.62 0)
 			(effects
@@
 			(project "PIC18F_ETH"
 				(path "/26a36835-4e01-4565-9612-f38560505464/ab2c46cb-188d-485d-996b-6193419384b9"
-					(reference "#PWR06009")
+					(reference "#PWR06010")
 					(unit 1)
 				)
@@
 		(dnp no)
 		(fields_autoplaced yes)
-		(property "Reference" "#PWR06008"
+		(property "Reference" "#PWR06015"
 			(at 303.53 99.06 0)
 			(effects
@@
 			(project "PIC18F_ETH"
 				(path "/26a36835-4e01-4565-9612-f38560505464/ab2c46cb-188d-485d-996b-6193419384b9"
-					(reference "#PWR06008")
+					(reference "#PWR06015")
 					(unit 1)
 				)
@@
 		(dnp no)
 		(fields_autoplaced yes)
-		(property "Reference" "#PWR06010"
+		(property "Reference" "#PWR06018"
 			(at 328.93 134.62 0)
 			(effects
@@
 			(project "PIC18F_ETH"
 				(path "/26a36835-4e01-4565-9612-f38560505464/ab2c46cb-188d-485d-996b-6193419384b9"
-					(reference "#PWR06010")
+					(reference "#PWR06018")
 					(unit 1)
 				)
@@
 		(on_board yes)
 		(dnp no)
-		(property "Reference" "U6001"
+		(property "Reference" "U6002"
 			(at 209.55 96.012 0)
 			(effects
@@
 			)
 		)
-		(property "Footprint" "QFN20_4x4MC_MCH"
+		(property "Footprint" "bt_footprints:QFN20_4x4MC_MCH"
 			(at 195.58 106.68 0)
 			(effects
@@
 			(project "PIC18F_ETH"
 				(path "/26a36835-4e01-4565-9612-f38560505464/ab2c46cb-188d-485d-996b-6193419384b9"
-					(reference "U6001")
+					(reference "U6002")
 					(unit 1)
 				)
@@
 		(dnp no)
 		(fields_autoplaced yes)
-		(property "Reference" "#PWR06011"
+		(property "Reference" "#PWR06003"
 			(at 149.86 161.29 0)
 			(effects
@@
 			(project "PIC18F_ETH"
 				(path "/26a36835-4e01-4565-9612-f38560505464/ab2c46cb-188d-485d-996b-6193419384b9"
-					(reference "#PWR06011")
-					(unit 1)
-				)
+					(reference "#PWR06003")
+					(unit 1)
+				)

Commit message: .
Parts:
- added C6005: 100n 25V, Capacitor_SMD:C_0603_1608Metric, symbol bt_capacitor:C;M;100n;10p;25V;S;0603
Connections:
- net CAN_CTRL_RST#: now also C6005.1
- net GND: now also C6005.2
Changed lines of the file:
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@@
 		(color 0 0 0 0)
 	)
+	(junction
+		(at 175.26 107.95)
+		(diameter 0)
+		(color 0 0 0 0)
+	)
 	(no_connect
 		(at 195.58 125.73)
@@
 	(wire
 		(pts
+			(xy 167.64 107.95) (xy 175.26 107.95)
+		)
+		(stroke
+			(width 0)
+			(type default)
+		)
+	)
+	(wire
+		(pts
 			(xy 332.74 118.11) (xy 328.93 118.11)
 		)
@@
 	)
 	(symbol
+		(lib_id "power:GND")
+		(at 160.02 107.95 270)
+		(unit 1)
+		(exclude_from_sim no)
+		(in_bom yes)
+		(on_board yes)
+		(dnp no)
+		(fields_autoplaced yes)
+		(property "Reference" "#PWR06019"
+			(at 153.67 107.95 0)
+			(effects
+				(font
+					(size 1.27 1.27)
+				)
+				(hide yes)
+			)
+		)
+		(property "Value" "GND"
+			(at 154.94 107.95 0)
+			(effects
+				(font
+					(size 1.27 1.27)
+				)
+			)
+		)
+		(property "Footprint" ""
+			(at 160.02 107.95 0)
+			(effects
+				(font
+					(size 1.27 1.27)
+				)
+				(hide yes)
+			)
+		)
+		(property "Datasheet" ""
+			(at 160.02 107.95 0)
+			(effects
+				(font
+					(size 1.27 1.27)
+				)
+				(hide yes)
+			)
+		)
+		(property "Description" "Power symbol creates a global label with name \"GND\" , ground"
+			(at 160.02 107.95 0)
+			(effects
+				(font
+					(size 1.27 1.27)
+				)
+				(hide yes)
+			)
+		)
+		(pin "1"
+		)
+		(instances
+			(project "PIC18F_ETH"
+				(path "/26a36835-4e01-4565-9612-f38560505464/ab2c46cb-188d-485d-996b-6193419384b9"
+					(reference "#PWR06019")
+					(unit 1)
+				)
+			)
+		)
+	)
+	(symbol
 		(lib_id "bt_connector:M;JST;01x03;2.54")
 		(at 350.52 115.57 0)
@@
 					(unit 1)
 				)
+			)
+		)
+	)
+	(symbol
+		(lib_id "bt_capacitor:C;M;100n;10p;25V;S;0603")
+		(at 163.83 107.95 270)
+		(unit 1)
+		(exclude_from_sim no)
+		(in_bom yes)
+		(on_board yes)
+		(dnp no)
+		(property "Reference" "C6005"
+			(at 165.1001 111.76 0)
+			(effects
+				(font
+					(size 1.27 1.27)
+				)
+				(justify left)
+			)
+		)
+		(property "Value" "100n 25V"
+			(at 159.004 104.14 90)
+			(effects
+				(font
+					(size 1.27 1.27)
+				)
+				(justify left)
+			)
+		)
+		(property "Footprint" "Capacitor_SMD:C_0603_1608Metric"
+			(at 163.83 105.172 90)
+			(effects
+				(font
+					(size 1.27 1.27)
+				)
+				(hide yes)
+			)
+		)
+		(property "Datasheet" "~"
+			(at 163.83 107.95 0)
+			(effects
+				(font
+					(size 1.27 1.27)
+				)
+				(hide yes)
+			)
+		)
+		(property "Description" "Capacitor"
+			(at 163.83 107.95 0)
+			(effects
+				(font
+					(size 1.27 1.27)
+				)
+				(hide yes)
+			)
+		)
+		(property "MPN" "C;C;T1;S;P0603;NA"
+			(at 163.83 111.95 90)
+			(effects
+				(font
+					(size 1.27 1.27)
+				)
+				(hide yes)
+			)
+		)
+		(property "CPN" "BT00008-090680"
+			(at 163.83 111.95 90)
+			(effects
+				(font
+					(size 1.27 1.27)
+				)
+				(hide yes)
+			)
+		)
+		(pin "1"
+		)
+		(pin "2"
+		)
+		(instances
+			(project "PIC18F_ETH"
+				(path "/26a36835-4e01-4565-9612-f38560505464/ab2c46cb-188d-485d-996b-6193419384b9"
+					(reference "C6005")
+					(unit 1)
+				)
