File: HW/PIC18F_ETH/PIC18F_ETH/CAN.kicad_sch (KiCad schematic)
At the start: 16 parts, among them J6001 JST,2.54, J6002 JST,2.54, U6001 25Mhz,50ppm, U6002 MCP2515T-E/ML, U6003 ATA6561-GAQW

Commit message: .
Other:
- title: (none) -> BT_ADDX
Changed lines of the file:
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@@
 	(generator_version "8.0")
 	(paper "A3")
+	(title_block
+		(title "BT_ADDX")
+		(rev "Rev:P1")
+	)
 	(bus_alias "SPI"
 		(members "CS#" "MOSI" "MISO" "SCK" "INT#" "INT1#")

Commit message: .
Other:
- title: BT_ADDX -> BT_AD/DX
Changed lines of the file:
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@@
 	(paper "A3")
 	(title_block
-		(title "BT_ADDX")
+		(title "BT_AD/DX")
 		(rev "Rev:P1")
+		(comment 1 "BT_0001-1")
 	)
 	(bus_alias "SPI"

Commit message: .
Parts:
- C6001, C6002, C6003, C6004, C6005: MPN C;C;T1;S;P0603;NA -> C;M;100n;10p;25V;S;0603
- R6001, R6002, R6005: MPN R;G;T1;S;P0603;NA -> R;G;10K;10P0;S;0603
- R6003, R6004: MPN R;G;T1;S;P0603;NA -> R;G;0R;10P0;S;0603
- R6006: MPN R;G;T1;S;P0603;NA -> R;G;120R;10P0;S;0603
- U6002: CPN BT02006-00001 MCP2515 -> BT02006-00001
Changed lines of the file:
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@@
 			)
 		)
-		(property "MPN" "R;G;T1;S;P0603;NA"
+		(property "MPN" "R;G;120R;10P0;S;0603"
 			(at 360.68 113.03 90)
 			(effects
@@
 			)
 		)
-		(property "MPN" "R;G;T1;S;P0603;NA"
+		(property "MPN" "R;G;10K;10P0;S;0603"
 			(at 119.38 139.7 90)
 			(effects
@@
 			)
 		)
-		(property "MPN" "C;C;T1;S;P0603;NA"
+		(property "MPN" "C;M;100n;10p;25V;S;0603"
 			(at 320.23 87.63 90)
 			(effects
@@
 			)
 		)
-		(property "MPN" "R;G;T1;S;P0603;NA"
+		(property "MPN" "R;G;10K;10P0;S;0603"
 			(at 175.26 100.33 90)
 			(effects
@@
 			)
 		)
-		(property "MPN" "R;G;T1;S;P0603;NA"
+		(property "MPN" "R;G;0R;10P0;S;0603"
 			(at 250.952 130.048 90)
 			(effects
@@
 			)
 		)
-		(property "MPN" "R;G;T1;S;P0603;NA"
+		(property "MPN" "R;G;10K;10P0;S;0603"
 			(at 255.27 101.6 90)
 			(effects
@@
 			)
 		)
-		(property "MPN" "R;G;T1;S;P0603;NA"
+		(property "MPN" "R;G;0R;10P0;S;0603"
 			(at 169.672 118.872 90)
 			(effects
@@
 			)
 		)
-		(property "MPN" "C;C;T1;S;P0603;NA"
+		(property "MPN" "C;M;100n;10p;25V;S;0603"
 			(at 273.24 87.63 90)
 			(effects
@@
 			)
 		)
-		(property "MPN" "C;C;T1;S;P0603;NA"
+		(property "MPN" "C;M;100n;10p;25V;S;0603"
 			(at 153.86 161.29 90)
 			(effects
@@
 			)
 		)
-		(property "CPN" "BT02006-00001 MCP2515"
+		(property "CPN" "BT02006-00001"
 			(at 195.58 106.68 0)
 			(effects
@@
 			)
 		)
-		(property "MPN" "C;C;T1;S;P0603;NA"
+		(property "MPN" "C;M;100n;10p;25V;S;0603"
 			(at 227.52 83.82 90)
 			(effects
@@
 			)
 		)
-		(property "MPN" "C;C;T1;S;P0603;NA"
+		(property "MPN" "C;M;100n;10p;25V;S;0603"
 			(at 163.83 111.95 90)
 			(effects

Commit message: .
Parts:
- U6002: footprint bt_footprints:QFN20_4x4MC_MCH -> QFN20_4x4MC_MCH
Changed lines of the file:
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@@
 			)
 		)
-		(property "Footprint" "bt_footprints:QFN20_4x4MC_MCH"
+		(property "Footprint" "QFN20_4x4MC_MCH"
 			(at 195.58 106.68 0)
 			(effects
