File: HW/PIC18F_ETH/PIC18F_ETH/IO-core.kicad_sch (KiCad schematic)
At the start: 0 parts

Commit message: .
Parts:
- added C4001, C4002, C4003, C4004, C4005, C4006, C4007, C4008, C4009, C4010, C4011, C4012, C4013, C4014, C4015, C4016, C4017, C4018: 100n 25V, Capacitor_SMD:C_0603_1608Metric, symbol bt_capacitor:C;M;100n;10p;25V;S;0603
- added J4001, J4002, J4003, J4004, J4005, J4006: Conn_01x03, symbol Connector_Generic:Conn_01x03
- added J4007, J4008, J4009, J4010, J4011: Conn_01x08, symbol Connector_Generic:Conn_01x08
- added R4001, R4002, R4003, R4004, R4005, R4006, R4019, R4020, R4021, R4022, R4023, R4024, R4025, R4026: 200R, Resistor_SMD:R_0603_1608Metric, symbol bt_resistors:R;G;200R;10P0;S;0603
- added R4007, R4008, R4009, R4010, R4011, R4012, R4013, R4014, R4015, R4016, R4017, R4018: 10K, Resistor_SMD:R_0603_1608Metric, symbol bt_resistors:R;G;10K;10P0;S;0603
- added U4001, U4002, U4003, U4004, U4005, U4006, U4007, U4008: TLP241B, Package_SO:SO-4_7.6x3.6mm_P2.54mm, symbol bt_relay:TLP241B-D4-LF1
Connections:
- new net: C4015.1, J4009.6 (Pin_6), R4015.2
- new net: C4005.1, R4005.1
- new net: J4005.2 (Pin_2), R4005.2
- new net: C4003.1, R4003.1
- new net: J4003.2 (Pin_2), R4003.2
- new net: R4026.2, U4008.1
- new net: J4002.2 (Pin_2), R4002.2
- new net: J4006.2 (Pin_2), R4006.2
- new net: R4022.2, U4004.1
- new net: J4010.8 (Pin_8), U4004.3
- new net: J4010.7 (Pin_7), U4004.4
- new net: C4004.1, R4004.1
- new net: R4020.2, U4002.1
- new net: C4012.1, J4009.4 (Pin_4), R4012.2
- new net: R4019.2, U4001.1
- new net: C4009.1, J4009.2 (Pin_2), R4009.2
- new net: C4017.1, J4009.8 (Pin_8), R4017.2
- new net: C4016.1, J4008.6 (Pin_6), R4016.2
- new net: C4007.1, J4007.2 (Pin_2), R4007.2
- new net: R4023.2, U4005.1
- new net: J4011.2 (Pin_2), U4005.3
- new net: J4011.1 (Pin_1), U4005.4
- new net: C4006.1, R4006.1
- new net: R4025.2, U4007.1
- new net: J4011.6 (Pin_6), U4007.3
- new net: J4011.5 (Pin_5), U4007.4
- new net: R4021.2, U4003.1
- new net: C4010.1, J4008.2 (Pin_2), R4011.2
- new net: C4008.1, J4007.4 (Pin_4), R4008.2
- new net: J4010.6 (Pin_6), U4003.3
- new net: C4002.1, R4002.1
- new net: J4010.2 (Pin_2), U4001.3
- new net: J4010.1 (Pin_1), U4001.4
- new net: C4018.1, J4008.8 (Pin_8), R4018.2
- new net: C4011.1, J4007.6 (Pin_6), R4010.2
- new net: C4014.1, J4007.8 (Pin_8), R4013.2
- new net: J4010.3 (Pin_3), U4002.4
- new net: J4010.4 (Pin_4), U4002.3
- new net: C4013.1, J4008.4 (Pin_4), R4014.2
- new net: C4001.1, R4001.1
- new net: R4024.2, U4006.1
- new net: J4011.4 (Pin_4), U4006.3
- new net: J4011.3 (Pin_3), U4006.4
- new net: J4001.2 (Pin_2), R4001.2
- new net: J4004.2 (Pin_2), R4004.2
- new net: J4011.7 (Pin_7), U4008.4
- new net: J4011.8 (Pin_8), U4008.3
- new net +3.3V: J4001.1 (Pin_1), J4002.1 (Pin_1), J4003.1 (Pin_1), J4004.1 (Pin_1), J4005.1 (Pin_1), J4006.1 (Pin_1), R4007.1, R4008.1, R4009.1, R4010.1, R4011.1, R4012.1, R4013.1, R4014.1, R4015.1, R4016.1, R4017.1, R4018.1
- new net GND: C4001.2, C4002.2, C4003.2, C4004.2, C4005.2, C4006.2, C4007.2, C4008.2, C4009.2, C4010.2, C4011.2, C4012.2, C4013.2, C4014.2, C4015.2, C4016.2, C4017.2, C4018.2, J4001.3 (Pin_3), J4002.3 (Pin_3), J4003.3 (Pin_3), J4004.3 (Pin_3), J4005.3 (Pin_3), J4006.3 (Pin_3), J4007.1 (Pin_1), J4007.3 (Pin_3), J4007.5 (Pin_5), J4007.7 (Pin_7), J4008.1 (Pin_1), J4008.3 (Pin_3), J4008.5 (Pin_5), J4008.7 (Pin_7), J4009.1 (Pin_1), J4009.3 (Pin_3), J4009.5 (Pin_5), J4009.7 (Pin_7), U4001.2, U4002.2, U4003.2, U4004.2, U4005.2, U4006.2, U4007.2, U4008.2

Commit message: .
Parts:
- added D4001, D4002, D4003, D4004, D4005, D4006, D4007, D4008, D4009: PESD2USB3UXT-Q, Package_TO_SOT_SMD:SOT-23-3, symbol bt_ESD_protection:PESD2USB3UXT-Q
- added R4027, R4028, R4029, R4030, R4031, R4032, R4033, R4034, R4035, R4036, R4037, R4038: 200R, Resistor_SMD:R_0603_1608Metric, symbol bt_resistors:R;G;200R;10P0;S;0603
- J4001, J4002, J4003, J4004, J4005, J4006: footprint (none) -> Connector_Samtec_HPM_THT:Samtec_HPM-03-01-x-S_Straight_1x03_Pitch5.08mm
- J4007, J4008, J4009, J4010, J4011: footprint (none) -> Connector_Samtec_HPM_THT:Samtec_HPM-08-01-x-S_Straight_1x08_Pitch5.08mm
Connections:
- net GND: now also D4001.3 (CA), D4002.3 (CA), D4003.3 (CA), D4004.3 (CA), D4005.3 (CA), D4006.3 (CA), D4007.3 (CA), D4008.3 (CA), D4009.3 (CA)
- net DI10x: now reaches C4015.1, J4009.6 (Pin_6), R4015.2
- net DI10x: now also D4004.1 (K1), R4028.2
- net AD4: now reaches C4005.1, R4005.1
- net AD4x: now reaches J4005.2 (Pin_2), R4005.2
- net AD4x: now also D4001.2 (K2)
- net AD2: now reaches C4003.1, R4003.1
- net AD1x: now reaches J4003.2 (Pin_2), R4003.2
- net AD1x: now also D4002.2 (K2)
- net DO7: now reaches R4026.1
- net DO7x: now reaches R4026.2, U4008.1
- net AD3x: now reaches J4002.2 (Pin_2), R4002.2
- net AD3x: now also D4003.1 (K1)
- net AD5x: now reaches J4006.2 (Pin_2), R4006.2
- net AD5x: now also D4001.1 (K1)
- net DO3x: now reaches R4022.2, U4004.1
- net AD3: now reaches C4004.1, R4004.1
- net DO1: now reaches R4020.1
- net DO1x: now reaches R4020.2, U4002.1
- net DI9x: now reaches C4012.1, J4009.4 (Pin_4), R4012.2
- net DI9x: now also D4005.2 (K2), R4029.2
- net DO0: now reaches R4019.1
- net DO0x: now reaches R4019.2, U4001.1
- net DI8x: now reaches C4009.1, J4009.2 (Pin_2), R4009.2
- net DI8x: now also D4005.1 (K1), R4030.2
- net DI11x: now reaches C4017.1, J4009.8 (Pin_8), R4017.2
- net DI11x: now also D4004.2 (K2), R4027.2
- net DI2x: now reaches C4016.1, J4008.6 (Pin_6), R4016.2
- net DI2x: now also D4009.1 (K1), R4036.2
- net DI4x: now reaches C4007.1, J4007.2 (Pin_2), R4007.2
- net DI4x: now also D4007.1 (K1), R4034.2
- net DO4x: now reaches R4023.2, U4005.1
- net AD5: now reaches C4006.1, R4006.1
- net DO6x: now reaches R4025.2, U4007.1
- net DO2: now reaches R4021.1
- net DO2x: now reaches R4021.2, U4003.1
- net DI0x: now reaches C4010.1, J4008.2 (Pin_2), R4011.2
- net DI0x: now also D4008.1 (K1), R4038.2
- net DI5x: now reaches C4008.1, J4007.4 (Pin_4), R4008.2
- net DI5x: now also D4007.2 (K2), R4033.2
- net at U4003.4: now also J4010.5 (Pin_5)
- net AD1: now reaches C4002.1, R4002.1
- net DI3x: now reaches C4018.1, J4008.8 (Pin_8), R4018.2
- net DI3x: now also D4009.2 (K2), R4035.2
- net DI6x: now reaches C4011.1, J4007.6 (Pin_6), R4010.2
- net DI6x: now also D4006.1 (K1), R4032.2
- net DI7x: now reaches C4014.1, J4007.8 (Pin_8), R4013.2
- net DI7x: now also D4006.2 (K2), R4031.2
- net DI1x: now reaches C4013.1, J4008.4 (Pin_4), R4014.2
- net DI1x: now also D4008.2 (K2), R4037.2
- net DO4: now reaches R4023.1
- net AD0: now reaches C4001.1, R4001.1
- net DO5x: now reaches R4024.2, U4006.1
- net AD0x: now reaches J4001.2 (Pin_2), R4001.2
- net AD0x: now also D4003.2 (K2)
- net DO5: now reaches R4024.1
- net AD2x: now reaches J4004.2 (Pin_2), R4004.2
- net AD2x: now also D4002.1 (K1)
- net DO6: now reaches R4025.1
- net DO3: now reaches R4022.1
- new net DI0: R4038.1
- new net DI1: R4037.1
- new net DI10: R4028.1
- new net DI11: R4027.1
- new net DI2: R4036.1
- new net DI3: R4035.1
- new net DI4: R4034.1
- new net DI5: R4033.1
- new net DI6: R4032.1
- new net DI7: R4031.1
- new net DI8: R4030.1
- new net DI9: R4029.1
Other:
- moved on the sheet: C4001, C4002, C4003, C4004, C4005, C4006, C4007, C4008, C4009, C4010, C4011, C4012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

Commit message: .
Parts:
- J4001, J4002, J4003, J4004, J4005, J4006: value Conn_01x03 -> JST,2.54; footprint Connector_Samtec_HPM_THT:Samtec_HPM-03-01-x-S_Straight_1x03_Pitch5.08mm -> Connector_JST:JST_EH_B3B-EH-A_1x03_P2.50mm_Vertical; symbol Connector_Generic:Conn_01x03 -> bt_connector:M;JST;01x03;2.54; CPN (none) -> BT10003-00003; MPN (none) -> JST 3 pin; SMT (none) -> n
Changed lines of the file:
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@@
 	(label "DI7"
 		(at 137.16 153.67 0)
+		(fields_autoplaced yes)
 		(effects
 			(font
@@
 	(label "DO3"
 		(at 306.07 113.03 0)
+		(fields_autoplaced yes)
 		(effects
 			(font
@@
 	(label "DI10"
 		(at 137.16 227.33 0)
+		(fields_autoplaced yes)
 		(effects
 			(font
@@
 	(label "DO4"
 		(at 306.07 143.51 0)
+		(fields_autoplaced yes)
 		(effects
 			(font
@@
 	(label "DI4"
 		(at 137.16 138.43 0)
+		(fields_autoplaced yes)
 		(effects
 			(font
@@
 	(label "AD5"
 		(at 41.91 247.65 0)
+		(fields_autoplaced yes)
 		(effects
 			(font
@@
 	(label "DO1"
 		(at 306.07 59.69 0)
+		(fields_autoplaced yes)
 		(effects
 			(font
@@
 	(label "DI8"
 		(at 137.16 217.17 0)
+		(fields_autoplaced yes)
 		(effects
 			(font
@@
 	(label "DO7"
 		(at 306.07 229.87 0)
+		(fields_autoplaced yes)
 		(effects
 			(font
@@
 	(label "AD1"
 		(at 41.91 77.47 0)
+		(fields_autoplaced yes)
 		(effects
 			(font
@@
 	(label "DI0"
 		(at 137.16 58.42 0)
+		(fields_autoplaced yes)
 		(effects
 			(font
@@
 	(label "AD4"
 		(at 41.91 204.47 0)
+		(fields_autoplaced yes)
 		(effects
 			(font
@@
 	(label "AD3"
 		(at 41.91 162.56 0)
+		(fields_autoplaced yes)
 		(effects
 			(font
@@
 	(label "DI11"
 		(at 137.16 231.14 0)
+		(fields_autoplaced yes)
 		(effects
 			(font
@@
 	(label "DI1"
 		(at 137.16 63.5 0)
+		(fields_autoplaced yes)
 		(effects
 			(font
@@
 	(label "AD0"
 		(at 41.91 36.83 0)
+		(fields_autoplaced yes)
 		(effects
 			(font
@@
 	(label "DI9"
 		(at 137.16 222.25 0)
+		(fields_autoplaced yes)
 		(effects
 			(font
@@
 	(label "DO5"
 		(at 306.07 171.45 0)
+		(fields_autoplaced yes)
 		(effects
 			(font
@@
 	(label "DO2"
 		(at 306.07 87.63 0)
+		(fields_autoplaced yes)
 		(effects
 			(font
@@
 	(label "DO6"
 		(at 306.07 201.93 0)
+		(fields_autoplaced yes)
 		(effects
 			(font
@@
 	(label "DI3"
 		(at 137.16 73.66 0)
+		(fields_autoplaced yes)
 		(effects
 			(font
@@
 	(label "AD2"
 		(at 41.91 118.11 0)
+		(fields_autoplaced yes)
 		(effects
 			(font
@@
 	(label "DI5"
 		(at 137.16 143.51 0)
+		(fields_autoplaced yes)
 		(effects
 			(font
@@
 	(label "DI2"
 		(at 137.16 68.58 0)
+		(fields_autoplaced yes)
 		(effects
 			(font
@@
 	(label "DO0"
 		(at 306.07 36.83 0)
+		(fields_autoplaced yes)
 		(effects
 			(font
@@
 	(label "DI6"
 		(at 137.16 148.59 0)
+		(fields_autoplaced yes)
 		(effects
 			(font
@@
 	)
 	(symbol
-		(lib_id "Connector_Generic:Conn_01x03")
+		(lib_id "bt_connector:M;JST;01x03;2.54")
 		(at 88.9 77.47 0)
 		(unit 1)
@@
 			)
 		)
-		(property "Value" "Conn_01x03"
+		(property "Value" "JST,2.54"
 			(at 91.44 78.7399 0)
 			(effects
@@
 			)
 		)
-		(property "Footprint" "Connector_Samtec_HPM_THT:Samtec_HPM-03-01-x-S_Straight_1x03_Pitch5.08mm"
+		(property "Footprint" "Connector_JST:JST_EH_B3B-EH-A_1x03_P2.50mm_Vertical"
 			(at 88.9 77.47 0)
 			(effects
@@
 			)
 		)
+		(property "CPN" "BT10003-00003"
+			(at 88.9 77.47 0)
+			(effects
+				(font
+					(size 1.27 1.27)
+				)
+				(hide yes)
+			)
+		)
+		(property "MPN" "JST 3 pin"
+			(at 88.9 77.47 0)
+			(effects
+				(font
+					(size 1.27 1.27)
+				)
+				(hide yes)
+			)
+		)
+		(property "SMT" "n"
+			(at 88.9 77.47 0)
+			(effects
+				(font
+					(size 1.27 1.27)
+				)
+				(hide yes)
+			)
+		)
 		(pin "3"
 		)
@@
 	)
 	(symbol
-		(lib_id "Connector_Generic:Conn_01x03")
+		(lib_id "bt_connector:M;JST;01x03;2.54")
 		(at 88.9 247.65 0)
 		(unit 1)
@@
 			)
 		)
-		(property "Value" "Conn_01x03"
+		(property "Value" "JST,2.54"
 			(at 91.44 248.9199 0)
 			(effects
@@
 			)
 		)
-		(property "Footprint" "Connector_Samtec_HPM_THT:Samtec_HPM-03-01-x-S_Straight_1x03_Pitch5.08mm"
+		(property "Footprint" "Connector_JST:JST_EH_B3B-EH-A_1x03_P2.50mm_Vertical"
 			(at 88.9 247.65 0)
 			(effects
@@
 			)
 		)
+		(property "CPN" "BT10003-00003"
+			(at 88.9 247.65 0)
+			(effects
+				(font
+					(size 1.27 1.27)
+				)
+				(hide yes)
+			)
+		)
+		(property "MPN" "JST 3 pin"
+			(at 88.9 247.65 0)
+			(effects
+				(font
+					(size 1.27 1.27)
+				)
+				(hide yes)
+			)
+		)
+		(property "SMT" "n"
+			(at 88.9 247.65 0)
+			(effects
+				(font
+					(size 1.27 1.27)
+				)
+				(hide yes)
+			)
+		)
 		(pin "3"
 		)
@@
 	)
 	(symbol
-		(lib_id "Connector_Generic:Conn_01x03")
+		(lib_id "bt_connector:M;JST;01x03;2.54")
 		(at 88.9 204.47 0)
 		(unit 1)
@@
 			)
 		)
-		(property "Value" "Conn_01x03"
+		(property "Value" "JST,2.54"
 			(at 91.44 205.7399 0)
 			(effects
@@
 			)
 		)
-		(property "Footprint" "Connector_Samtec_HPM_THT:Samtec_HPM-03-01-x-S_Straight_1x03_Pitch5.08mm"
+		(property "Footprint" "Connector_JST:JST_EH_B3B-EH-A_1x03_P2.50mm_Vertical"
 			(at 88.9 204.47 0)
 			(effects
@@
 			)
 		)
+		(property "CPN" "BT10003-00003"
+			(at 88.9 204.47 0)
+			(effects
+				(font
+					(size 1.27 1.27)
+				)
+				(hide yes)
+			)
+		)
+		(property "MPN" "JST 3 pin"
+			(at 88.9 204.47 0)
+			(effects
+				(font
+					(size 1.27 1.27)
+				)
+				(hide yes)
+			)
+		)
+		(property "SMT" "n"
+			(at 88.9 204.47 0)
+			(effects
+				(font
+					(size 1.27 1.27)
+				)
+				(hide yes)
+			)
+		)
 		(pin "3"
 		)
@@
 	)
 	(symbol
-		(lib_id "Connector_Generic:Conn_01x03")
+		(lib_id "bt_connector:M;JST;01x03;2.54")
 		(at 88.9 118.11 0)
 		(unit 1)
@@
 			)
 		)
-		(property "Value" "Conn_01x03"
+		(property "Value" "JST,2.54"
 			(at 91.44 119.3799 0)
 			(effects
@@
 			)
 		)
-		(property "Footprint" "Connector_Samtec_HPM_THT:Samtec_HPM-03-01-x-S_Straight_1x03_Pitch5.08mm"
+		(property "Footprint" "Connector_JST:JST_EH_B3B-EH-A_1x03_P2.50mm_Vertical"
 			(at 88.9 118.11 0)
 			(effects
@@
 			)
 		)
+		(property "CPN" "BT10003-00003"
+			(at 88.9 118.11 0)
+			(effects
+				(font
+					(size 1.27 1.27)
+				)
+				(hide yes)
+			)
+		)
+		(property "MPN" "JST 3 pin"
+			(at 88.9 118.11 0)
+			(effects
+				(font
+					(size 1.27 1.27)
+				)
+				(hide yes)
+			)
+		)
+		(property "SMT" "n"
+			(at 88.9 118.11 0)
+			(effects
+				(font
+					(size 1.27 1.27)
+				)
+				(hide yes)
+			)
+		)
 		(pin "3"
 		)
@@
 	)
 	(symbol
-		(lib_id "Connector_Generic:Conn_01x03")
+		(lib_id "bt_connector:M;JST;01x03;2.54")
 		(at 88.9 36.83 0)
 		(unit 1)
@@
 			)
 		)
-		(property "Value" "Conn_01x03"
+		(property "Value" "JST,2.54"
 			(at 91.44 38.0999 0)
 			(effects
@@
 			)
 		)
-		(property "Footprint" "Connector_Samtec_HPM_THT:Samtec_HPM-03-01-x-S_Straight_1x03_Pitch5.08mm"
+		(property "Footprint" "Connector_JST:JST_EH_B3B-EH-A_1x03_P2.50mm_Vertical"
 			(at 88.9 36.83 0)
 			(effects
@@
 			)
 		)
+		(property "CPN" "BT10003-00003"
+			(at 88.9 36.83 0)
+			(effects
+				(font
+					(size 1.27 1.27)
+				)
+				(hide yes)
+			)
+		)
+		(property "MPN" "JST 3 pin"
+			(at 88.9 36.83 0)
+			(effects
+				(font
+					(size 1.27 1.27)
+				)
+				(hide yes)
+			)
+		)
+		(property "SMT" "n"
+			(at 88.9 36.83 0)
+			(effects
+				(font
+					(size 1.27 1.27)
+				)
+				(hide yes)
+			)
+		)
 		(pin "3"
 		)
@@
 	)
 	(symbol
-		(lib_id "Connector_Generic:Conn_01x03")
+		(lib_id "bt_connector:M;JST;01x03;2.54")
 		(at 88.9 162.56 0)
 		(unit 1)
@@
 			)
 		)
-		(property "Value" "Conn_01x03"
+		(property "Value" "JST,2.54"
 			(at 91.44 163.8299 0)
 			(effects
@@
 			)
 		)
-		(property "Footprint" "Connector_Samtec_HPM_THT:Samtec_HPM-03-01-x-S_Straight_1x03_Pitch5.08mm"
+		(property "Footprint" "Connector_JST:JST_EH_B3B-EH-A_1x03_P2.50mm_Vertical"
 			(at 88.9 162.56 0)
 			(effects
@@
 			(at 88.9 162.56 0)
 			(effects
+				(font
+					(size 1.27 1.27)
+				)
+				(hide yes)
+			)
+		)
+		(property "CPN" "BT10003-00003"
+			(at 88.9 162.56 0)
+			(effects
+				(font
+					(size 1.27 1.27)
+				)
+				(hide yes)
+			)
+		)
+		(property "MPN" "JST 3 pin"
+			(at 88.9 162.56 0)
+			(effects
+				(font
+					(size 1.27 1.27)
+				)
+				(hide yes)
+			)
+		)
+		(property "SMT" "n"
+			(at 88.9 162.56 0)
+			(effects

Commit message: .
Parts:
- removed J4007, J4008, J4009, J4010, J4011: Conn_01x08, Connector_Samtec_HPM_THT:Samtec_HPM-08-01-x-S_Straight_1x08_Pitch5.08mm, symbol Connector_Generic:Conn_01x08
- added J4007, J4008, J4009, J4010, J4011, J4012, J4013, J4014, J4015, J4016, J4017, J4018, J4019, J4020, J4021, J4022, J4023, J4024, J4025, J4026: JST,2.54, Connector_JST:JST_EH_B2B-EH-A_1x02_P2.50mm_Vertical, symbol bt_connector:M;JST;01x02;2.54
Connections:
- net DI0: now also C4010.1
- net DI0x: now also J4007.2 (Pin_2); no longer C4010.1
- net DI1: now also C4013.1
- net DI10: now also C4015.1
- net DI10x: now also J4017.2 (Pin_2); no longer C4015.1
- net DI11: now also C4017.1
- net DI11x: now also J4018.2 (Pin_2); no longer C4017.1
- net DI1x: now also J4008.2 (Pin_2); no longer C4013.1
- net DI2: now also C4016.1
- net DI2x: now also J4009.2 (Pin_2); no longer C4016.1
- net DI3: now also C4018.1
- net DI3x: now also J4010.2 (Pin_2); no longer C4018.1
- net DI4: now also C4007.1
- net DI4x: now also J4011.2 (Pin_2); no longer C4007.1
- net DI5: now also C4008.1
- net DI5x: now also J4012.2 (Pin_2); no longer C4008.1
- net DI6: now also C4011.1
- net DI6x: now also J4013.2 (Pin_2); no longer C4011.1
- net DI7: now also C4014.1
- net DI7x: now also J4014.2 (Pin_2); no longer C4014.1
- net DI8: now also C4009.1
- net DI8x: now also J4015.2 (Pin_2); no longer C4009.1
- net DI9: now also C4012.1
- net DI9x: now also J4016.2 (Pin_2); no longer C4012.1
- net GND: now also J4007.1 (Pin_1), J4008.1 (Pin_1), J4009.1 (Pin_1), J4010.1 (Pin_1), J4011.1 (Pin_1), J4012.1 (Pin_1), J4013.1 (Pin_1), J4014.1 (Pin_1), J4015.1 (Pin_1), J4016.1 (Pin_1), J4017.1 (Pin_1), J4018.1 (Pin_1)
- net at U4004.3: now also J4022.2 (Pin_2)
- net at U4004.4: now also J4022.1 (Pin_1)
- net at U4005.3: now also J4023.2 (Pin_2)
- net at U4005.4: now also J4023.1 (Pin_1)
- net at U4007.3: now also J4025.2 (Pin_2)
- net at U4007.4: now also J4025.1 (Pin_1)
- net at U4003.3: now also J4021.2 (Pin_2)
- net at U4003.4: now also J4021.1 (Pin_1)
- net at U4001.3: now also J4019.2 (Pin_2)
- net at U4001.4: now also J4019.1 (Pin_1)
- net at U4002.4: now also J4020.1 (Pin_1)
- net at U4002.3: now also J4020.2 (Pin_2)
- net at U4006.3: now also J4024.2 (Pin_2)
- net at U4006.4: now also J4024.1 (Pin_1)
- net at U4008.4: now also J4026.1 (Pin_1)
- net at U4008.3: now also J4026.2 (Pin_2)
Other:
- moved on the sheet: C4007, C4008, C4009, C4010, C4011, C4012, C4013, C4014, C4015, C4016, C4017, C4018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

Commit message: .
Parts:
- renumbered C4010 to C4007, C4007 to C4008, C4012 to C4010, C4013 to C4011, C4008 to C4012, C4016 to C4013, C4011 to C4014, C4018 to C4016, C4014 to C4017, C4017 to C4018, D4003 to D4001, D4001 to D4003, D4006 to D4004, D4004 to D4005, D4007 to D4006, D4005 to D4007, R4034 to R4007, R4033 to R4008, R4032 to R4009, R4031 to R4010, R4030 to R4011, R4029 to R4012, R4028 to R4013, R4027 to R4014, R4038 to R4015, R4037 to R4016, R4036 to R4017, R4035 to R4018, R4007 to R4019, R4009 to R4020, R4011 to R4021, R4008 to R4022, R4012 to R4023, R4014 to R4024, R4010 to R4025, R4015 to R4026, R4016 to R4027, R4013 to R4028, R4017 to R4029, R4018 to R4030, R4019 to R4031, R4020 to R4032, R4021 to R4033, R4022 to R4034, R4023 to R4035, R4024 to R4036, R4025 to R4037, R4026 to R4038

Commit message: .
Parts:
- removed C4009, C4010, C4011, C4012, C4013, C4014, C4015, C4016, C4017, C4018: 100n 25V, Capacitor_SMD:C_0603_1608Metric, symbol bt_capacitor:C;M;100n;10p;25V;S;0603
- removed D4004, D4005, D4006, D4007, D4008, D4009: PESD2USB3UXT-Q, Package_TO_SOT_SMD:SOT-23-3, symbol bt_ESD_protection:PESD2USB3UXT-Q
- removed J4007, J4008, J4009, J4010, J4011, J4012, J4013, J4014, J4015, J4016, J4017, J4018, J4019, J4020, J4021, J4022, J4023, J4024, J4025, J4026: JST,2.54, Connector_JST:JST_EH_B2B-EH-A_1x02_P2.50mm_Vertical, symbol bt_connector:M;JST;01x02;2.54
- removed R4007, R4008, R4009, R4010, R4011, R4012, R4013, R4014, R4015, R4016, R4017, R4018, R4031, R4032, R4033, R4034, R4035, R4036, R4037, R4038: 200R, Resistor_SMD:R_0603_1608Metric, symbol bt_resistors:R;G;200R;10P0;S;0603
- removed R4019, R4020, R4021, R4022, R4023, R4024, R4025, R4026, R4027, R4028, R4029, R4030: 10K, Resistor_SMD:R_0603_1608Metric, symbol bt_resistors:R;G;10K;10P0;S;0603
- removed U4001, U4002, U4003, U4004, U4005, U4006, U4007, U4008: TLP241B, Package_SO:SO-4_7.6x3.6mm_P2.54mm, symbol bt_relay:TLP241B-D4-LF1
- added R4007, R4008: 10K, Resistor_SMD:R_0603_1608Metric, symbol bt_resistors:R;G;10K;10P0;S;0603
- added U4001, U4002: MCP23S17-E/ML, bt_footprints:QFN28_6x6MC_MCH, symbol bt_interface:MCP23S17-E_ML
Connections:
- net +3.3V: now also C4007.1, C4008.1, R4007.1, R4008.1, U4001.5 (VDD), U4002.11 (A0), U4002.5 (VDD)
- net DI0: now also U4001.17 (GPA0); no longer C4007.1
- net DI1: now also U4001.18 (GPA1)
- net DI10: now also U4001.27 (GPB2)
- net DI11: now also U4001.28 (GPB3)
- net DI2: now also U4001.19 (GPA2)
- net DI3: now also U4001.20 (GPA3)
- net DI4: now also U4001.21 (GPA4); no longer C4008.1
- net DI5: now also U4001.22 (GPA5)
- net DI6: now also U4001.23 (GPA6)
- net DI7: now also U4001.24 (GPA7)
- net DI8: now also U4001.25 (GPB0)
- net DI9: now also U4001.26 (GPB1)
- net DO0: now also U4002.17 (GPA0)
- net DO1: now also U4002.18 (GPA1)
- net DO2: now also U4002.19 (GPA2)
- net DO3: now also U4002.20 (GPA3)
- net DO4: now also U4002.21 (GPA4)
- net DO5: now also U4002.22 (GPA5)
- net DO6: now also U4002.23 (GPA6)
- net DO7: now also U4002.24 (GPA7)
- net GND: now also U4001.11 (A0), U4001.12 (A1), U4001.13 (A2), U4001.29 (HTAB), U4001.6 (VSS), U4002.12 (A1), U4002.13 (A2), U4002.29 (HTAB), U4002.6 (VSS)
- new net: R4007.2, U4001.14 (*RESET)
- new net: R4008.2, U4002.14 (*RESET)
- new net DI12: U4001.1 (GPB4)
- new net DI13: U4001.2 (GPB5)
- new net DI14: U4001.3 (GPB6)
- new net DI15: U4001.4 (GPB7)
- new net DO10: U4002.27 (GPB2)
- new net DO11: U4002.28 (GPB3)
- new net DO12: U4002.1 (GPB4)
- new net DO13: U4002.2 (GPB5)
- new net DO14: U4002.3 (GPB6)
- new net DO15: U4002.4 (GPB7)
- new net DO8: U4002.25 (GPB0)
- new net DO9: U4002.26 (GPB1)
- new net SPI_DI.CS#: U4001.7 (*CS)
- new net SPI_DI.INT#: U4001.16 (INTA)
- new net SPI_DI.INT1#: U4001.15 (INTB)
- new net SPI_DI.MISO: U4001.10 (SO)
- new net SPI_DI.MOSI: U4001.9 (SI)
- new net SPI_DI.SCK: U4001.8 (SCK)
- new net SPI_DO.CS#: U4002.7 (*CS)
- new net SPI_DO.INT#: U4002.16 (INTA)
- new net SPI_DO.INT1#: U4002.15 (INTB)
- new net SPI_DO.MISO: U4002.10 (SO)
- new net SPI_DO.MOSI: U4002.9 (SI)
- new net SPI_DO.SCK: U4002.8 (SCK)
Other:
- added sheet Digital Input (Digital_Input.kicad_sch)
- added sheet Digital Output (Digital_Output.kicad_sch)

Commit message: .
Parts:
- added C4009, C4010: 100n 25V, Capacitor_SMD:C_0603_1608Metric, symbol bt_capacitor:C;M;100n;10p;25V;S;0603
Connections:
- net GND: now also C4009.2, C4010.1
- net at R4007.2, U4001.14 (*RESET): now also C4009.1
- net at R4008.2, U4002.14 (*RESET): now also C4010.2
