File: HW/PIC18F_ETH/PIC18F_ETH/IO-core.kicad_sch (KiCad schematic)
At the start: 29 parts, among them J4001 JST,2.54, J4002 JST,2.54, J4003 JST,2.54, J4004 JST,2.54, J4005 JST,2.54, J4006 JST,2.54, U4001 MCP23S17-E/ML, U4002 MCP23S17-E/ML

Commit message: .
Connections:
- net AD1x: now also D4001.1 (K1), J4002.2 (Pin_2), R4002.2; no longer D4002.2 (K2), J4003.2 (Pin_2), R4003.2
- net AD2x: now also D4002.2 (K2), J4003.2 (Pin_2), R4003.2; no longer D4002.1 (K1), J4004.2 (Pin_2), R4004.2
- net AD3x: now also D4002.1 (K1), J4004.2 (Pin_2), R4004.2; no longer D4001.1 (K1), J4002.2 (Pin_2), R4002.2
Changed lines of the file:
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@@
 		)
 	)
-	(label "AD2x"
+	(label "AD3x"
 		(at 78.74 162.56 180)
 		(fields_autoplaced yes)
@@
 		)
 	)
-	(label "AD3x"
+	(label "AD1x"
 		(at 78.74 77.47 180)
 		(fields_autoplaced yes)
@@
 		)
 	)
-	(label "AD1x"
+	(label "AD2x"
 		(at 78.74 118.11 180)
 		(fields_autoplaced yes)

Commit message: .
Other:
- title: (none) -> BT_ADDX
Changed lines of the file:
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@@
 	(generator_version "8.0")
 	(paper "A3")
+	(title_block
+		(title "BT_ADDX")
+		(rev "Rev:P1")
+	)
 	(junction
 		(at 162.56 76.2)

Commit message: .
Other:
- title: BT_ADDX -> BT_AD/DX
Changed lines of the file:
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@@
 	(paper "A3")
 	(title_block
-		(title "BT_ADDX")
+		(title "BT_AD/DX")
 		(rev "Rev:P1")
+		(comment 1 "BT_0001-1")
 	)
 	(junction

Commit message: .
Connections:
- net SPI_DO.INT#: no longer names the net of U4002.16 (INTA)
- net SPI_DO.INT1#: no longer names the net of U4002.15 (INTB)
- no-connect marks 0 -> 2
Changed lines of the file:
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@@
 		(color 0 0 0 0)
+	)
+	(no_connect
+		(at 181.61 195.58)
+	)
+	(no_connect
+		(at 181.61 198.12)
 	)
 	(bus_entry
@@
 	)
 	(bus_entry
-		(at 140.97 195.58)
-		(size 2.54 2.54)
-		(stroke
-			(width 0)
-			(type default)
-		)
-	)
-	(bus_entry
 		(at 233.68 184.15)
 		(size -2.54 2.54)
@@
 	)
 	(bus_entry
-		(at 140.97 193.04)
-		(size 2.54 2.54)
-		(stroke
-			(width 0)
-			(type default)
-		)
-	)
-	(bus_entry
 		(at 31.75 115.57)
 		(size 2.54 2.54)
@@
 	(bus
 		(pts
-			(xy 140.97 195.58) (xy 140.97 193.04)
-		)
-		(stroke
-			(width 0)
-			(type default)
-		)
-	)
-	(bus
-		(pts
 			(xy 31.75 115.57) (xy 31.75 74.93)
 		)
@@
 		)
 	)
-	(wire
-		(pts
-			(xy 143.51 195.58) (xy 181.61 195.58)
-		)
-		(stroke
-			(width 0)
-			(type default)
-		)
-	)
 	(bus
 		(pts
@@
 		)
 	)
-	(bus
-		(pts
-			(xy 140.97 201.93) (xy 140.97 195.58)
-		)
-		(stroke
-			(width 0)
-			(type default)
-		)
-	)
 	(wire
 		(pts
@@
 	(bus
 		(pts
-			(xy 140.97 193.04) (xy 140.97 173.99)
+			(xy 140.97 173.99) (xy 140.97 201.93)
 		)
 		(stroke
@@
 		(pts
 			(xy 233.68 186.69) (xy 233.68 189.23)
-		)
-		(stroke
-			(width 0)
-			(type default)
-		)
-	)
-	(wire
-		(pts
-			(xy 143.51 198.12) (xy 181.61 198.12)
 		)
 		(stroke
@@
 		)
 	)
-	(label "SPI_DO.INT1#"
-		(at 165.1 198.12 0)
-		(fields_autoplaced yes)
-		(effects
-			(font
-				(size 1.27 1.27)
-			)
-			(justify left bottom)
-		)
-	)
 	(label "SPI_DO.MOSI"
 		(at 165.1 207.01 0)
@@
 		(fields_autoplaced yes)
 		(effects
-			(font
-				(size 1.27 1.27)
-			)
-			(justify left bottom)
-		)
-	)
-	(label "SPI_DO.INT#"
-		(at 165.1 195.58 0)
-		(fields_autoplaced yes)
-		(effects

Commit message: .
Parts:
- C4001, C4002, C4003, C4004, C4005, C4006, C4007, C4008, C4009, C4010: MPN C;C;T1;S;P0603;NA -> C;M;100n;10p;25V;S;0603
- R4001, R4002, R4003, R4004, R4005, R4006: MPN R;G;T1;S;P0603;NA -> R;G;200R;10P0;S;0603
- R4007, R4008: MPN R;G;T1;S;P0603;NA -> R;G;10K;10P0;S;0603
Changed lines of the file:
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@@
 			)
 		)
-		(property "MPN" "R;G;T1;S;P0603;NA"
+		(property "MPN" "R;G;200R;10P0;S;0603"
 			(at 60.96 204.47 90)
 			(effects
@@
 	)
 	(symbol
-		(lib_name "PESD2USB3UXT-Q_7")
 		(lib_id "bt_ESD_protection:PESD2USB3UXT-Q")
 		(at 59.69 63.5 180)
@@
 			)
 		)
-		(property "MPN" "R;G;T1;S;P0603;NA"
+		(property "MPN" "R;G;200R;10P0;S;0603"
 			(at 60.96 118.11 90)
 			(effects
@@
 			)
 		)
-		(property "MPN" "C;C;T1;S;P0603;NA"
+		(property "MPN" "C;M;100n;10p;25V;S;0603"
 			(at 56.07 167.64 90)
 			(effects
@@
 			)
 		)
-		(property "MPN" "C;C;T1;S;P0603;NA"
+		(property "MPN" "C;M;100n;10p;25V;S;0603"
 			(at 56.07 209.55 90)
 			(effects
@@
 			)
 		)
-		(property "MPN" "C;C;T1;S;P0603;NA"
+		(property "MPN" "C;M;100n;10p;25V;S;0603"
 			(at 191.96 162.56 90)
 			(effects
@@
 			)
 		)
-		(property "MPN" "C;C;T1;S;P0603;NA"
+		(property "MPN" "C;M;100n;10p;25V;S;0603"
 			(at 185.61 50.8 90)
 			(effects
@@
 			)
 		)
-		(property "MPN" "R;G;T1;S;P0603;NA"
+		(property "MPN" "R;G;200R;10P0;S;0603"
 			(at 60.96 247.65 90)
 			(effects
@@
 			)
 		)
-		(property "MPN" "C;C;T1;S;P0603;NA"
+		(property "MPN" "C;M;100n;10p;25V;S;0603"
 			(at 56.07 82.55 90)
 			(effects
@@
 			)
 		)
-		(property "MPN" "C;C;T1;S;P0603;NA"
+		(property "MPN" "C;M;100n;10p;25V;S;0603"
 			(at 155.13 66.04 90)
 			(effects
@@
 	)
 	(symbol
-		(lib_name "PESD2USB3UXT-Q_8")
 		(lib_id "bt_ESD_protection:PESD2USB3UXT-Q")
 		(at 59.69 143.51 180)
@@
 			)
 		)
-		(property "MPN" "C;C;T1;S;P0603;NA"
+		(property "MPN" "C;M;100n;10p;25V;S;0603"
 			(at 56.07 252.73 90)
 			(effects
@@
 			)
 		)
-		(property "MPN" "C;C;T1;S;P0603;NA"
+		(property "MPN" "C;M;100n;10p;25V;S;0603"
 			(at 162.75 184.15 90)
 			(effects
@@
 			)
 		)
-		(property "MPN" "R;G;T1;S;P0603;NA"
+		(property "MPN" "R;G;10K;10P0;S;0603"
 			(at 162.56 71.12 90)
 			(effects
@@
 			)
 		)
-		(property "MPN" "R;G;T1;S;P0603;NA"
+		(property "MPN" "R;G;200R;10P0;S;0603"
 			(at 60.96 77.47 90)
 			(effects
@@
 			)
 		)
-		(property "MPN" "R;G;T1;S;P0603;NA"
+		(property "MPN" "R;G;10K;10P0;S;0603"
 			(at 168.91 184.15 90)
 			(effects
@@
 	)
 	(symbol
-		(lib_name "PESD2USB3UXT-Q_6")
 		(lib_id "bt_ESD_protection:PESD2USB3UXT-Q")
 		(at 59.69 232.41 180)
@@
 			)
 		)
-		(property "MPN" "C;C;T1;S;P0603;NA"
+		(property "MPN" "C;M;100n;10p;25V;S;0603"
 			(at 56.07 41.91 90)
 			(effects
@@
 			)
 		)
-		(property "MPN" "R;G;T1;S;P0603;NA"
+		(property "MPN" "R;G;200R;10P0;S;0603"
 			(at 60.96 36.83 90)
 			(effects
@@
 			)
 		)
-		(property "MPN" "R;G;T1;S;P0603;NA"
+		(property "MPN" "R;G;200R;10P0;S;0603"
 			(at 60.96 162.56 90)
 			(effects
@@
 			)
 		)
-		(property "MPN" "C;C;T1;S;P0603;NA"
+		(property "MPN" "C;M;100n;10p;25V;S;0603"
 			(at 56.07 123.19 90)
 			(effects
