File: HW/PIC18F_ETH/PIC18F_ETH/PIC18F_ETH.kicad_sch (KiCad schematic)
At the start: 0 parts

Commit message: .
Other:
- title: BT_ADDX -> BT_AD/DX
Changed lines of the file:
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@@
 	(paper "A3")
 	(title_block
-		(title "BT_ADDX")
+		(title "BT_AD/DX")
 		(rev "Rev:P1")
+		(comment 1 "BT_0001-1")
 	)
 	(bus
