File: HW/PIC18F_ETH/PIC18F_ETH/Digital_Input.kicad_sch (KiCad schematic)
At the start: 72 parts, among them J8001 JST,2.54, J8002 JST,2.54, J8003 JST,2.54, J8004 JST,2.54, J8005 JST,2.54, J8006 JST,2.54, J8007 JST,2.54, J8008 JST,2.54, J8009 JST,2.54, J8010 JST,2.54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

Commit message: .
Parts:
- renumbered D8007 to D8006, D8006 to D8007
Changed lines of the file:
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@@
 		(on_board yes)
 		(dnp no)
-		(property "Reference" "D8006"
+		(property "Reference" "D8007"
 			(at 303.784 52.832 0)
 			(effects
@@
 			(project "PIC18F_ETH"
 				(path "/26a36835-4e01-4565-9612-f38560505464/1753a15f-d572-4c39-8cc7-77188589f279/1458a913-4d81-4cff-86ce-674c73f5e529"
-					(reference "D8006")
+					(reference "D8007")
 					(unit 1)
 				)
@@
 		(dnp no)
 		(fields_autoplaced yes)
-		(property "Reference" "#PWR08005"
+		(property "Reference" "#PWR08013"
 			(at 294.64 101.6 0)
 			(effects
@@
 			(project "PIC18F_ETH"
 				(path "/26a36835-4e01-4565-9612-f38560505464/1753a15f-d572-4c39-8cc7-77188589f279/1458a913-4d81-4cff-86ce-674c73f5e529"
-					(reference "#PWR08005")
+					(reference "#PWR08013")
 					(unit 1)
 				)
@@
 		(dnp no)
 		(fields_autoplaced yes)
-		(property "Reference" "#PWR08007"
+		(property "Reference" "#PWR08015"
 			(at 298.45 40.64 0)
 			(effects
@@
 			(project "PIC18F_ETH"
 				(path "/26a36835-4e01-4565-9612-f38560505464/1753a15f-d572-4c39-8cc7-77188589f279/1458a913-4d81-4cff-86ce-674c73f5e529"
-					(reference "#PWR08007")
+					(reference "#PWR08015")
 					(unit 1)
 				)
@@
 		(dnp no)
 		(fields_autoplaced yes)
-		(property "Reference" "#PWR08002"
+		(property "Reference" "#PWR08011"
 			(at 242.57 113.03 0)
 			(effects
@@
 			(project "PIC18F_ETH"
 				(path "/26a36835-4e01-4565-9612-f38560505464/1753a15f-d572-4c39-8cc7-77188589f279/1458a913-4d81-4cff-86ce-674c73f5e529"
-					(reference "#PWR08002")
+					(reference "#PWR08011")
 					(unit 1)
 				)
@@
 		(dnp no)
 		(fields_autoplaced yes)
-		(property "Reference" "#PWR08008"
+		(property "Reference" "#PWR08005"
 			(at 134.62 30.48 0)
 			(effects
@@
 			(project "PIC18F_ETH"
 				(path "/26a36835-4e01-4565-9612-f38560505464/1753a15f-d572-4c39-8cc7-77188589f279/1458a913-4d81-4cff-86ce-674c73f5e529"
-					(reference "#PWR08008")
+					(reference "#PWR08005")
 					(unit 1)
 				)
@@
 		(on_board yes)
 		(dnp no)
-		(property "Reference" "#PWR08011"
+		(property "Reference" "#PWR08017"
 			(at 322.58 40.64 0)
 			(effects
@@
 			(project "PIC18F_ETH"
 				(path "/26a36835-4e01-4565-9612-f38560505464/1753a15f-d572-4c39-8cc7-77188589f279/1458a913-4d81-4cff-86ce-674c73f5e529"
-					(reference "#PWR08011")
+					(reference "#PWR08017")
 					(unit 1)
 				)
@@
 		(dnp no)
 		(fields_autoplaced yes)
-		(property "Reference" "#PWR08006"
+		(property "Reference" "#PWR08004"
 			(at 129.54 111.76 0)
 			(effects
@@
 			(project "PIC18F_ETH"
 				(path "/26a36835-4e01-4565-9612-f38560505464/1753a15f-d572-4c39-8cc7-77188589f279/1458a913-4d81-4cff-86ce-674c73f5e529"
-					(reference "#PWR08006")
+					(reference "#PWR08004")
 					(unit 1)
 				)
@@
 		(dnp no)
 		(fields_autoplaced yes)
-		(property "Reference" "#PWR08012"
+		(property "Reference" "#PWR08008"
 			(at 157.48 34.29 0)
 			(effects
@@
 			(project "PIC18F_ETH"
 				(path "/26a36835-4e01-4565-9612-f38560505464/1753a15f-d572-4c39-8cc7-77188589f279/1458a913-4d81-4cff-86ce-674c73f5e529"
-					(reference "#PWR08012")
+					(reference "#PWR08008")
 					(unit 1)
 				)
@@
 		(dnp no)
 		(fields_autoplaced yes)
-		(property "Reference" "#PWR08018"
+		(property "Reference" "#PWR08016"
 			(at 298.45 111.76 0)
 			(effects
@@
 			(project "PIC18F_ETH"
 				(path "/26a36835-4e01-4565-9612-f38560505464/1753a15f-d572-4c39-8cc7-77188589f279/1458a913-4d81-4cff-86ce-674c73f5e529"
-					(reference "#PWR08018")
+					(reference "#PWR08016")
 					(unit 1)
 				)
@@
 		(dnp no)
 		(fields_autoplaced yes)
-		(property "Reference" "#PWR08016"
+		(property "Reference" "#PWR08012"
 			(at 247.65 180.34 0)
 			(effects
@@
 			(project "PIC18F_ETH"
 				(path "/26a36835-4e01-4565-9612-f38560505464/1753a15f-d572-4c39-8cc7-77188589f279/1458a913-4d81-4cff-86ce-674c73f5e529"
-					(reference "#PWR08016")
+					(reference "#PWR08012")
 					(unit 1)
 				)
@@
 		(dnp no)
 		(fields_autoplaced yes)
-		(property "Reference" "#PWR08009"
+		(property "Reference" "#PWR08006"
 			(at 134.62 92.71 0)
 			(effects
@@
 			(project "PIC18F_ETH"
 				(path "/26a36835-4e01-4565-9612-f38560505464/1753a15f-d572-4c39-8cc7-77188589f279/1458a913-4d81-4cff-86ce-674c73f5e529"
-					(reference "#PWR08009")
+					(reference "#PWR08006")
 					(unit 1)
 				)
@@
 		(dnp no)
 		(fields_autoplaced yes)
-		(property "Reference" "#PWR08017"
+		(property "Reference" "#PWR08014"
 			(at 294.64 172.72 0)
 			(effects
@@
 			(project "PIC18F_ETH"
 				(path "/26a36835-4e01-4565-9612-f38560505464/1753a15f-d572-4c39-8cc7-77188589f279/1458a913-4d81-4cff-86ce-674c73f5e529"
-					(reference "#PWR08017")
+					(reference "#PWR08014")
 					(unit 1)
 				)
@@
 		(on_board yes)
 		(dnp no)
-		(property "Reference" "#PWR08003"
+		(property "Reference" "#PWR08002"
 			(at 90.17 101.6 0)
 			(effects
@@
 			(project "PIC18F_ETH"
 				(path "/26a36835-4e01-4565-9612-f38560505464/1753a15f-d572-4c39-8cc7-77188589f279/1458a913-4d81-4cff-86ce-674c73f5e529"
-					(reference "#PWR08003")
+					(reference "#PWR08002")
 					(unit 1)
 				)
@@
 		(on_board yes)
 		(dnp no)
-		(property "Reference" "#PWR08019"
+		(property "Reference" "#PWR08018"
 			(at 328.93 107.95 0)
 			(effects
@@
 			(project "PIC18F_ETH"
 				(path "/26a36835-4e01-4565-9612-f38560505464/1753a15f-d572-4c39-8cc7-77188589f279/1458a913-4d81-4cff-86ce-674c73f5e529"
-					(reference "#PWR08019")
+					(reference "#PWR08018")
 					(unit 1)
 				)
@@
 		(dnp no)
 		(fields_autoplaced yes)
-		(property "Reference" "#PWR08013"
+		(property "Reference" "#PWR08009"
 			(at 176.53 165.1 0)
 			(effects
@@
 			(project "PIC18F_ETH"
 				(path "/26a36835-4e01-4565-9612-f38560505464/1753a15f-d572-4c39-8cc7-77188589f279/1458a913-4d81-4cff-86ce-674c73f5e529"
-					(reference "#PWR08013")
+					(reference "#PWR08009")
 					(unit 1)
 				)
@@
 		(dnp no)
 		(fields_autoplaced yes)
-		(property "Reference" "#PWR08014"
+		(property "Reference" "#PWR08019"
 			(at 344.17 88.9 0)
 			(effects
@@
 			(project "PIC18F_ETH"
 				(path "/26a36835-4e01-4565-9612-f38560505464/1753a15f-d572-4c39-8cc7-77188589f279/1458a913-4d81-4cff-86ce-674c73f5e529"
-					(reference "#PWR08014")
+					(reference "#PWR08019")
 					(unit 1)
 				)
@@
 		(dnp no)
 		(fields_autoplaced yes)
-		(property "Reference" "#PWR08004"
+		(property "Reference" "#PWR08003"
 			(at 125.73 175.26 0)
 			(effects
@@
 			(project "PIC18F_ETH"
 				(path "/26a36835-4e01-4565-9612-f38560505464/1753a15f-d572-4c39-8cc7-77188589f279/1458a913-4d81-4cff-86ce-674c73f5e529"
-					(reference "#PWR08004")
+					(reference "#PWR08003")
 					(unit 1)
 				)
@@
 		(dnp no)
 		(fields_autoplaced yes)
-		(property "Reference" "#PWR08015"
+		(property "Reference" "#PWR08010"
 			(at 179.07 85.09 0)
 			(effects
@@
 			(project "PIC18F_ETH"
 				(path "/26a36835-4e01-4565-9612-f38560505464/1753a15f-d572-4c39-8cc7-77188589f279/1458a913-4d81-4cff-86ce-674c73f5e529"
-					(reference "#PWR08015")
+					(reference "#PWR08010")
 					(unit 1)
 				)
@@
 		(on_board yes)
 		(dnp no)
-		(property "Reference" "D8007"
+		(property "Reference" "D8006"
 			(at 290.068 161.544 0)
 			(effects
@@
 			(project "PIC18F_ETH"
 				(path "/26a36835-4e01-4565-9612-f38560505464/1753a15f-d572-4c39-8cc7-77188589f279/1458a913-4d81-4cff-86ce-674c73f5e529"
-					(reference "D8007")
+					(reference "D8006")
 					(unit 1)
 				)
@@
 		(on_board yes)
 		(dnp no)
-		(property "Reference" "#PWR08010"
+		(property "Reference" "#PWR08007"
 			(at 154.94 114.3 0)
 			(effects
@@
 			(project "PIC18F_ETH"
 				(path "/26a36835-4e01-4565-9612-f38560505464/1753a15f-d572-4c39-8cc7-77188589f279/1458a913-4d81-4cff-86ce-674c73f5e529"
-					(reference "#PWR08010")
+					(reference "#PWR08007")
 					(unit 1)
 				)

Commit message: .
Other:
- title: (none) -> BT_ADDX
Changed lines of the file:
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@@
 	(generator_version "8.0")
 	(paper "A3")
+	(title_block
+		(title "BT_ADDX")
+		(rev "Rev:P1")
+	)
 	(junction
 		(at 326.39 72.39)

Commit message: .
Other:
- title: BT_ADDX -> BT_AD/DX
Changed lines of the file:
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@@
 	(paper "A3")
 	(title_block
-		(title "BT_ADDX")
+		(title "BT_AD/DX")
 		(rev "Rev:P1")
+		(comment 1 "BT_0001-1")
 	)
 	(junction

Commit message: .
Parts:
- C8001, C8002, C8003, C8004, C8005, C8006, C8007, C8008, C8009, C8010, C8011, C8012, C8013, C8014, C8015, C8016: MPN C;C;T1;S;P0603;NA -> C;M;100n;10p;25V;S;0603
- R8001, R8002, R8003, R8004, R8005, R8006, R8007, R8008, R8017, R8018, R8019, R8020, R8021, R8022, R8023, R8024: MPN R;G;T1;S;P0603;NA -> R;G;200R;10P0;S;0603
- R8009, R8010, R8011, R8012, R8013, R8014, R8015, R8016, R8025, R8026, R8027, R8028, R8029, R8030, R8031, R8032: MPN R;G;T1;S;P0603;NA -> R;G;10K;10P0;S;0603
Changed lines of the file:
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@@
 			)
 		)
-		(property "MPN" "C;C;T1;S;P0603;NA"
+		(property "MPN" "C;M;100n;10p;25V;S;0603"
 			(at 256.73 158.75 90)
 			(effects
@@
 			)
 		)
-		(property "MPN" "R;G;T1;S;P0603;NA"
+		(property "MPN" "R;G;200R;10P0;S;0603"
 			(at 276.86 72.39 90)
 			(effects
@@
 			)
 		)
-		(property "MPN" "R;G;T1;S;P0603;NA"
+		(property "MPN" "R;G;200R;10P0;S;0603"
 			(at 115.57 60.96 90)
 			(effects
@@
 			)
 		)
-		(property "MPN" "R;G;T1;S;P0603;NA"
+		(property "MPN" "R;G;200R;10P0;S;0603"
 			(at 115.57 66.04 90)
 			(effects
@@
 			)
 		)
-		(property "MPN" "R;G;T1;S;P0603;NA"
+		(property "MPN" "R;G;200R;10P0;S;0603"
 			(at 107.95 140.97 90)
 			(effects
@@
 			)
 		)
-		(property "MPN" "C;C;T1;S;P0603;NA"
+		(property "MPN" "C;M;100n;10p;25V;S;0603"
 			(at 246.57 158.75 90)
 			(effects
@@
 	)
 	(symbol
-		(lib_name "PESD2USB3UXT-Q_1")
 		(lib_id "bt_ESD_protection:PESD2USB3UXT-Q")
 		(at 298.45 55.88 90)
@@
 			)
 		)
-		(property "MPN" "R;G;T1;S;P0603;NA"
+		(property "MPN" "R;G;10K;10P0;S;0603"
 			(at 335.28 125.73 90)
 			(effects
@@
 			)
 		)
-		(property "MPN" "R;G;T1;S;P0603;NA"
+		(property "MPN" "R;G;200R;10P0;S;0603"
 			(at 115.57 55.88 90)
 			(effects
@@
 			)
 		)
-		(property "MPN" "R;G;T1;S;P0603;NA"
+		(property "MPN" "R;G;10K;10P0;S;0603"
 			(at 170.18 48.26 90)
 			(effects
@@
 			)
 		)
-		(property "MPN" "C;C;T1;S;P0603;NA"
+		(property "MPN" "C;M;100n;10p;25V;S;0603"
 			(at 99.25 80.01 90)
 			(effects
@@
 			)
 		)
-		(property "MPN" "R;G;T1;S;P0603;NA"
+		(property "MPN" "R;G;200R;10P0;S;0603"
 			(at 276.86 143.51 90)
 			(effects
@@
 			)
 		)
-		(property "MPN" "R;G;T1;S;P0603;NA"
+		(property "MPN" "R;G;10K;10P0;S;0603"
 			(at 167.64 128.27 90)
 			(effects
@@
 			)
 		)
-		(property "MPN" "C;C;T1;S;P0603;NA"
+		(property "MPN" "C;M;100n;10p;25V;S;0603"
 			(at 99.25 163.83 90)
 			(effects
@@
 			)
 		)
-		(property "MPN" "C;C;T1;S;P0603;NA"
+		(property "MPN" "C;M;100n;10p;25V;S;0603"
 			(at 70.04 163.83 90)
 			(effects
@@
 			)
 		)
-		(property "MPN" "C;C;T1;S;P0603;NA"
+		(property "MPN" "C;M;100n;10p;25V;S;0603"
 			(at 237.68 87.63 90)
 			(effects
@@
 			)
 		)
-		(property "MPN" "R;G;T1;S;P0603;NA"
+		(property "MPN" "R;G;200R;10P0;S;0603"
 			(at 276.86 138.43 90)
 			(effects
@@
 			)
 		)
-		(property "MPN" "R;G;T1;S;P0603;NA"
+		(property "MPN" "R;G;10K;10P0;S;0603"
 			(at 140.97 128.27 90)
 			(effects
@@
 			)
 		)
-		(property "MPN" "R;G;T1;S;P0603;NA"
+		(property "MPN" "R;G;10K;10P0;S;0603"
 			(at 335.28 54.61 90)
 			(effects
@@
 			)
 		)
-		(property "MPN" "C;C;T1;S;P0603;NA"
+		(property "MPN" "C;M;100n;10p;25V;S;0603"
 			(at 266.89 87.63 90)
 			(effects
@@
 			)
 		)
-		(property "MPN" "R;G;T1;S;P0603;NA"
+		(property "MPN" "R;G;200R;10P0;S;0603"
 			(at 107.95 146.05 90)
 			(effects
@@
 			)
 		)
-		(property "MPN" "R;G;T1;S;P0603;NA"
+		(property "MPN" "R;G;10K;10P0;S;0603"
 			(at 152.4 48.26 90)
 			(effects
@@
 			)
 		)
-		(property "MPN" "R;G;T1;S;P0603;NA"
+		(property "MPN" "R;G;200R;10P0;S;0603"
 			(at 276.86 67.31 90)
 			(effects
@@
 			)
 		)
-		(property "MPN" "R;G;T1;S;P0603;NA"
+		(property "MPN" "R;G;10K;10P0;S;0603"
 			(at 149.86 128.27 90)
 			(effects
@@
 			)
 		)
-		(property "MPN" "R;G;T1;S;P0603;NA"
+		(property "MPN" "R;G;200R;10P0;S;0603"
 			(at 107.95 151.13 90)
 			(effects
@@
 			)
 		)
-		(property "MPN" "C;C;T1;S;P0603;NA"
+		(property "MPN" "C;M;100n;10p;25V;S;0603"
 			(at 89.09 80.01 90)
 			(effects
@@
 	)
 	(symbol
-		(lib_name "PESD2USB3UXT-Q_5")
 		(lib_id "bt_ESD_protection:PESD2USB3UXT-Q")
 		(at 134.62 80.01 270)
@@
 			)
 		)
-		(property "MPN" "R;G;T1;S;P0603;NA"
+		(property "MPN" "R;G;200R;10P0;S;0603"
 			(at 276.86 148.59 90)
 			(effects
@@
 	)
 	(symbol
-		(lib_name "PESD2USB3UXT-Q_4")
 		(lib_id "bt_ESD_protection:PESD2USB3UXT-Q")
 		(at 134.62 46.99 90)
@@
 			)
 		)
-		(property "MPN" "R;G;T1;S;P0603;NA"
+		(property "MPN" "R;G;10K;10P0;S;0603"
 			(at 143.51 48.26 90)
 			(effects
@@
 			)
 		)
-		(property "MPN" "C;C;T1;S;P0603;NA"
+		(property "MPN" "C;M;100n;10p;25V;S;0603"
 			(at 266.89 158.75 90)
 			(effects
@@
 			)
 		)
-		(property "MPN" "R;G;T1;S;P0603;NA"
+		(property "MPN" "R;G;10K;10P0;S;0603"
 			(at 326.39 54.61 90)
 			(effects
@@
 			)
 		)
-		(property "MPN" "C;C;T1;S;P0603;NA"
+		(property "MPN" "C;M;100n;10p;25V;S;0603"
 			(at 80.2 80.01 90)
 			(effects
@@
 			)
 		)
-		(property "MPN" "R;G;T1;S;P0603;NA"
+		(property "MPN" "R;G;10K;10P0;S;0603"
 			(at 326.39 125.73 90)
 			(effects
@@
 			)
 		)
-		(property "MPN" "C;C;T1;S;P0603;NA"
+		(property "MPN" "C;M;100n;10p;25V;S;0603"
 			(at 80.2 163.83 90)
 			(effects
@@
 			)
 		)
-		(property "MPN" "C;C;T1;S;P0603;NA"
+		(property "MPN" "C;M;100n;10p;25V;S;0603"
 			(at 70.04 80.01 90)
 			(effects
@@
 			)
 		)
-		(property "MPN" "C;C;T1;S;P0603;NA"
+		(property "MPN" "C;M;100n;10p;25V;S;0603"
 			(at 256.73 87.63 90)
 			(effects
@@
 			)
 		)
-		(property "MPN" "R;G;T1;S;P0603;NA"
+		(property "MPN" "R;G;200R;10P0;S;0603"
 			(at 276.86 133.35 90)
 			(effects
@@
 			)
 		)
-		(property "MPN" "R;G;T1;S;P0603;NA"
+		(property "MPN" "R;G;200R;10P0;S;0603"
 			(at 107.95 135.89 90)
 			(effects
@@
 			)
 		)
-		(property "MPN" "R;G;T1;S;P0603;NA"
+		(property "MPN" "R;G;10K;10P0;S;0603"
 			(at 161.29 48.26 90)
 			(effects
@@
 			)
 		)
-		(property "MPN" "R;G;T1;S;P0603;NA"
+		(property "MPN" "R;G;200R;10P0;S;0603"
 			(at 115.57 71.12 90)
 			(effects
@@
 			)
 		)
-		(property "MPN" "R;G;T1;S;P0603;NA"
+		(property "MPN" "R;G;10K;10P0;S;0603"
 			(at 317.5 54.61 90)
 			(effects
@@
 			)
 		)
-		(property "MPN" "R;G;T1;S;P0603;NA"
+		(property "MPN" "R;G;10K;10P0;S;0603"
 			(at 308.61 125.73 90)
 			(effects
@@
 			)
 		)
-		(property "MPN" "C;C;T1;S;P0603;NA"
+		(property "MPN" "C;M;100n;10p;25V;S;0603"
 			(at 89.09 163.83 90)
 			(effects
@@
 	)
 	(symbol
-		(lib_name "PESD2USB3UXT-Q_1")
 		(lib_id "bt_ESD_protection:PESD2USB3UXT-Q")
 		(at 298.45 127 90)
@@
 			)
 		)
-		(property "MPN" "R;G;T1;S;P0603;NA"
+		(property "MPN" "R;G;200R;10P0;S;0603"
 			(at 276.86 77.47 90)
 			(effects
@@
 			)
 		)
-		(property "MPN" "R;G;T1;S;P0603;NA"
+		(property "MPN" "R;G;10K;10P0;S;0603"
 			(at 317.5 125.73 90)
 			(effects
@@
 			)
 		)
-		(property "MPN" "C;C;T1;S;P0603;NA"
+		(property "MPN" "C;M;100n;10p;25V;S;0603"
 			(at 246.57 87.63 90)
 			(effects
@@
 	)
 	(symbol
-		(lib_name "PESD2USB3UXT-Q_2")
 		(lib_id "bt_ESD_protection:PESD2USB3UXT-Q")
 		(at 294.64 157.48 270)
@@
 			)
 		)
-		(property "MPN" "R;G;T1;S;P0603;NA"
+		(property "MPN" "R;G;10K;10P0;S;0603"
 			(at 308.61 54.61 90)
 			(effects
@@
 			)
 		)
-		(property "MPN" "C;C;T1;S;P0603;NA"
+		(property "MPN" "C;M;100n;10p;25V;S;0603"
 			(at 237.68 158.75 90)
 			(effects
@@
 			)
 		)
-		(property "MPN" "R;G;T1;S;P0603;NA"
+		(property "MPN" "R;G;10K;10P0;S;0603"
 			(at 158.75 128.27 90)
 			(effects
@@
 	)
 	(symbol
-		(lib_name "PESD2USB3UXT-Q_2")
 		(lib_id "bt_ESD_protection:PESD2USB3UXT-Q")
 		(at 294.64 86.36 270)
@@
 			)
 		)
-		(property "MPN" "R;G;T1;S;P0603;NA"
+		(property "MPN" "R;G;200R;10P0;S;0603"
 			(at 276.86 62.23 90)
 			(effects
@@
 	)
 	(symbol
-		(lib_name "PESD2USB3UXT-Q_3")
 		(lib_id "bt_ESD_protection:PESD2USB3UXT-Q")
 		(at 129.54 125.73 90)
