File: HW/PIC18F_ETH/PIC18F_ETH/Digital_Output.kicad_sch (KiCad schematic)
At the start: 48 parts, among them J9001 JST,2.54, J9002 JST,2.54, J9003 JST,2.54, J9004 JST,2.54, J9005 JST,2.54, J9006 JST,2.54, J9007 JST,2.54, J9008 JST,2.54, J9009 JST,2.54, J9010 JST,2.54, J9011 JST,2.54, J9012 JST,2.54, J9013 JST,2.54, J9014 JST,2.54, J9015 JST,2.54, J9016 JST,2.54, U9001 TLP241B, U9002 TLP241B, U9003 TLP241B, U9004 TLP241B, U9005 TLP241B, U9006 TLP241B, U9007 TLP241B, U9008 TLP241B, U9009 TLP241B, U9010 TLP241B, U9011 TLP241B, U9012 TLP241B, U9013 TLP241B, U9014 TLP241B, U9015 TLP241B, U9016 TLP241B

Commit message: .
Parts:
- added D9001, D9002, D9003, D9004, D9005, D9006, D9007, D9008, D9009, D9010, D9011, D9012, D9013, D9014, D9015, D9016: LED G, LED_SMD:LED_0603_1608Metric, symbol bt_opto:D;LED;G;2V;25mA
- added R9017, R9018, R9019, R9020, R9021, R9022, R9023, R9024, R9025, R9026, R9027, R9028, R9029, R9030, R9031, R9032: 200R, Resistor_SMD:R_0603_1608Metric, symbol bt_resistors:R;G;200R;10P0;S;0603
Connections:
- net DO0: now also R9019.2
- net DO1: now also R9020.2
- net DO10: now also R9027.2
- net DO11: now also R9028.2
- net DO12: now also R9029.2
- net DO13: now also R9030.2
- net DO14: now also R9031.2
- net DO15: now also R9032.2
- net DO2: now also R9021.2
- net DO3: now also R9022.2
- net DO4: now also R9023.2
- net DO5: now also R9018.2
- net DO6: now also R9024.2
- net DO7: now also R9017.2
- net DO8: now also R9025.2
- net DO9: now also R9026.2
- net GND: now also D9001.1 (K), D9002.1 (K), D9003.1 (K), D9004.1 (K), D9005.1 (K), D9006.1 (K), D9007.1 (K), D9008.1 (K), D9009.1 (K), D9010.1 (K), D9011.1 (K), D9012.1 (K), D9013.1 (K), D9014.1 (K), D9015.1 (K), D9016.1 (K)
- new net: D9007.2 (A), R9023.1
- new net: D9005.2 (A), R9021.1
- new net: D9008.2 (A), R9024.1
- new net: D9012.2 (A), R9028.1
- new net: D9015.2 (A), R9031.1
- new net: D9002.2 (A), R9018.1
- new net: D9013.2 (A), R9029.1
- new net: D9006.2 (A), R9022.1
- new net: D9014.2 (A), R9030.1
- new net: D9009.2 (A), R9025.1
- new net: D9003.2 (A), R9019.1
- new net: D9016.2 (A), R9032.1
- new net: D9004.2 (A), R9020.1
- new net: D9001.2 (A), R9017.1
- new net: D9010.2 (A), R9026.1
- new net: D9011.2 (A), R9027.1

Commit message: .
Other:
- title: (none) -> BT_ADDX
Changed lines of the file:
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@@
 	(generator_version "8.0")
 	(paper "A3")
+	(title_block
+		(title "BT_ADDX")
+		(rev "Rev:P1")
+	)
 	(junction
 		(at 252.73 66.04)

Commit message: .
Other:
- title: BT_ADDX -> BT_AD/DX
Changed lines of the file:
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@@
 	(paper "A3")
 	(title_block
-		(title "BT_ADDX")
+		(title "BT_AD/DX")
 		(rev "Rev:P1")
+		(comment 1 "BT_0001-1")
 	)
 	(junction

Commit message: .
Parts:
- R9001, R9002, R9003, R9004, R9005, R9006, R9007, R9008, R9009, R9010, R9011, R9012, R9013, R9014, R9015, R9016, R9017, R9018, R9019, R9020, R9021, R9022, R9023, R9024, R9025, R9026, R9027, R9028, R9029, R9030, R9031, R9032: MPN R;G;T1;S;P0603;NA -> R;G;200R;10P0;S;0603
Changed lines of the file:
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@@
 			)
 		)
-		(property "MPN" "R;G;T1;S;P0603;NA"
+		(property "MPN" "R;G;200R;10P0;S;0603"
 			(at 74.93 87.63 90)
 			(effects
@@
 			)
 		)
-		(property "MPN" "R;G;T1;S;P0603;NA"
+		(property "MPN" "R;G;200R;10P0;S;0603"
 			(at 67.31 147.32 90)
 			(effects
@@
 			)
 		)
-		(property "MPN" "R;G;T1;S;P0603;NA"
+		(property "MPN" "R;G;200R;10P0;S;0603"
 			(at 67.31 91.44 90)
 			(effects
@@
 			)
 		)
-		(property "MPN" "R;G;T1;S;P0603;NA"
+		(property "MPN" "R;G;200R;10P0;S;0603"
 			(at 261.62 208.28 90)
 			(effects
@@
 			)
 		)
-		(property "MPN" "R;G;T1;S;P0603;NA"
+		(property "MPN" "R;G;200R;10P0;S;0603"
 			(at 252.73 123.19 90)
 			(effects
@@
 			)
 		)
-		(property "MPN" "R;G;T1;S;P0603;NA"
+		(property "MPN" "R;G;200R;10P0;S;0603"
 			(at 252.73 212.09 90)
 			(effects
@@
 			)
 		)
-		(property "MPN" "R;G;T1;S;P0603;NA"
+		(property "MPN" "R;G;200R;10P0;S;0603"
 			(at 261.62 149.86 90)
 			(effects
@@
 			)
 		)
-		(property "MPN" "R;G;T1;S;P0603;NA"
+		(property "MPN" "R;G;200R;10P0;S;0603"
 			(at 74.93 171.45 90)
 			(effects
@@
 			)
 		)
-		(property "MPN" "R;G;T1;S;P0603;NA"
+		(property "MPN" "R;G;200R;10P0;S;0603"
 			(at 261.62 177.8 90)
 			(effects
@@
 			)
 		)
-		(property "MPN" "R;G;T1;S;P0603;NA"
+		(property "MPN" "R;G;200R;10P0;S;0603"
 			(at 261.62 236.22 90)
 			(effects
@@
 			)
 		)
-		(property "MPN" "R;G;T1;S;P0603;NA"
+		(property "MPN" "R;G;200R;10P0;S;0603"
 			(at 252.73 153.67 90)
 			(effects
@@
 			)
 		)
-		(property "MPN" "R;G;T1;S;P0603;NA"
+		(property "MPN" "R;G;200R;10P0;S;0603"
 			(at 67.31 116.84 90)
 			(effects
@@
 			)
 		)
-		(property "MPN" "R;G;T1;S;P0603;NA"
+		(property "MPN" "R;G;200R;10P0;S;0603"
 			(at 67.31 205.74 90)
 			(effects
@@
 			)
 		)
-		(property "MPN" "R;G;T1;S;P0603;NA"
+		(property "MPN" "R;G;200R;10P0;S;0603"
 			(at 252.73 181.61 90)
 			(effects
@@
 			)
 		)
-		(property "MPN" "R;G;T1;S;P0603;NA"
+		(property "MPN" "R;G;200R;10P0;S;0603"
 			(at 252.73 46.99 90)
 			(effects
@@
 			)
 		)
-		(property "MPN" "R;G;T1;S;P0603;NA"
+		(property "MPN" "R;G;200R;10P0;S;0603"
 			(at 67.31 40.64 90)
 			(effects
@@
 			)
 		)
-		(property "MPN" "R;G;T1;S;P0603;NA"
+		(property "MPN" "R;G;200R;10P0;S;0603"
 			(at 74.93 143.51 90)
 			(effects
@@
 			)
 		)
-		(property "MPN" "R;G;T1;S;P0603;NA"
+		(property "MPN" "R;G;200R;10P0;S;0603"
 			(at 74.93 36.83 90)
 			(effects
@@
 			)
 		)
-		(property "MPN" "R;G;T1;S;P0603;NA"
+		(property "MPN" "R;G;200R;10P0;S;0603"
 			(at 261.62 43.18 90)
 			(effects
@@
 			)
 		)
-		(property "MPN" "R;G;T1;S;P0603;NA"
+		(property "MPN" "R;G;200R;10P0;S;0603"
 			(at 67.31 63.5 90)
 			(effects
@@
 			)
 		)
-		(property "MPN" "R;G;T1;S;P0603;NA"
+		(property "MPN" "R;G;200R;10P0;S;0603"
 			(at 261.62 119.38 90)
 			(effects
@@
 			)
 		)
-		(property "MPN" "R;G;T1;S;P0603;NA"
+		(property "MPN" "R;G;200R;10P0;S;0603"
 			(at 261.62 93.98 90)
 			(effects
@@
 			)
 		)
-		(property "MPN" "R;G;T1;S;P0603;NA"
+		(property "MPN" "R;G;200R;10P0;S;0603"
 			(at 74.93 229.87 90)
 			(effects
@@
 			)
 		)
-		(property "MPN" "R;G;T1;S;P0603;NA"
+		(property "MPN" "R;G;200R;10P0;S;0603"
 			(at 252.73 69.85 90)
 			(effects
@@
 			)
 		)
-		(property "MPN" "R;G;T1;S;P0603;NA"
+		(property "MPN" "R;G;200R;10P0;S;0603"
 			(at 252.73 97.79 90)
 			(effects
@@
 			)
 		)
-		(property "MPN" "R;G;T1;S;P0603;NA"
+		(property "MPN" "R;G;200R;10P0;S;0603"
 			(at 74.93 113.03 90)
 			(effects
@@
 			)
 		)
-		(property "MPN" "R;G;T1;S;P0603;NA"
+		(property "MPN" "R;G;200R;10P0;S;0603"
 			(at 60.96 233.68 90)
 			(effects
@@
 			)
 		)
-		(property "MPN" "R;G;T1;S;P0603;NA"
+		(property "MPN" "R;G;200R;10P0;S;0603"
 			(at 252.73 240.03 90)
 			(effects
@@
 			)
 		)
-		(property "MPN" "R;G;T1;S;P0603;NA"
+		(property "MPN" "R;G;200R;10P0;S;0603"
 			(at 66.04 175.26 90)
 			(effects
@@
 			)
 		)
-		(property "MPN" "R;G;T1;S;P0603;NA"
+		(property "MPN" "R;G;200R;10P0;S;0603"
 			(at 74.93 59.69 90)
 			(effects
@@
 			)
 		)
-		(property "MPN" "R;G;T1;S;P0603;NA"
+		(property "MPN" "R;G;200R;10P0;S;0603"
 			(at 261.62 66.04 90)
 			(effects
@@
 			)
 		)
-		(property "MPN" "R;G;T1;S;P0603;NA"
+		(property "MPN" "R;G;200R;10P0;S;0603"
 			(at 74.93 201.93 90)
 			(effects
