File: HW/PIC18F_ETH/PIC18F_ETH/ETH_Connector.kicad_sch (KiCad schematic)
At the start: 9 parts, among them J5001 RJ45_LED_ETH_Shielded

Commit message: .
Parts:
- gave numbers to parts that had none: 4
Connections:
- net GND: now also J5001.SH
Changed lines of the file:
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@@
+	(wire
+		(pts
+			(xy 130.81 111.76) (xy 130.81 114.3)
+		)
+		(stroke
+			(width 0)
+			(type default)
+		)
+	)
 	(wire
 		(pts
@@
 	)
 	(symbol
+		(lib_id "power:GND")
+		(at 130.81 114.3 0)
+		(unit 1)
+		(exclude_from_sim no)
+		(in_bom yes)
+		(on_board yes)
+		(dnp no)
+		(fields_autoplaced yes)
+		(property "Reference" "#PWR05005"
+			(at 130.81 120.65 0)
+			(effects
+				(font
+					(size 1.27 1.27)
+				)
+				(hide yes)
+			)
+		)
+		(property "Value" "GND"
+			(at 130.81 119.38 0)
+			(effects
+				(font
+					(size 1.27 1.27)
+				)
+			)
+		)
+		(property "Footprint" ""
+			(at 130.81 114.3 0)
+			(effects
+				(font
+					(size 1.27 1.27)
+				)
+				(hide yes)
+			)
+		)
+		(property "Datasheet" ""
+			(at 130.81 114.3 0)
+			(effects
+				(font
+					(size 1.27 1.27)
+				)
+				(hide yes)
+			)
+		)
+		(property "Description" "Power symbol creates a global label with name \"GND\" , ground"
+			(at 130.81 114.3 0)
+			(effects
+				(font
+					(size 1.27 1.27)
+				)
+				(hide yes)
+			)
+		)
+		(pin "1"
+		)
+		(instances
+			(project "PIC18F_ETH"
+				(path "/26a36835-4e01-4565-9612-f38560505464/fe5ea34d-21cf-4dac-9ef2-b9905ff3ffd8"
+					(reference "#PWR05005")
+					(unit 1)
+				)
+			)
+		)
+	)
+	(symbol
 		(lib_id "Device:R")
 		(at 179.07 93.98 0)
@@
 		(dnp no)
 		(fields_autoplaced yes)
-		(property "Reference" "R?"
+		(property "Reference" "R5005"
 			(at 104.14 85.09 90)
 			(effects
@@
 			(project "PIC18F_ETH"
 				(path "/26a36835-4e01-4565-9612-f38560505464/fe5ea34d-21cf-4dac-9ef2-b9905ff3ffd8"
-					(reference "R?")
+					(reference "R5005")
 					(unit 1)
 				)
@@
 		(dnp no)
 		(fields_autoplaced yes)
-		(property "Reference" "C?"
+		(property "Reference" "C5002"
 			(at 200.66 104.14 90)
 			(effects
@@
 			(project "PIC18F_ETH"
 				(path "/26a36835-4e01-4565-9612-f38560505464/fe5ea34d-21cf-4dac-9ef2-b9905ff3ffd8"
-					(reference "C?")
+					(reference "C5002")
 					(unit 1)
 				)
@@
 		(dnp no)
 		(fields_autoplaced yes)
-		(property "Reference" "C?"
+		(property "Reference" "C5001"
 			(at 200.66 81.28 90)
 			(effects
@@
 			(project "PIC18F_ETH"
 				(path "/26a36835-4e01-4565-9612-f38560505464/fe5ea34d-21cf-4dac-9ef2-b9905ff3ffd8"
-					(reference "C?")
+					(reference "C5001")
 					(unit 1)
 				)
@@
 		(dnp no)
 		(fields_autoplaced yes)
-		(property "Reference" "R?"
+		(property "Reference" "R5006"
 			(at 104.14 100.33 90)
 			(effects
@@
 			(project "PIC18F_ETH"
 				(path "/26a36835-4e01-4565-9612-f38560505464/fe5ea34d-21cf-4dac-9ef2-b9905ff3ffd8"
-					(reference "R?")
-					(unit 1)
-				)
+					(reference "R5006")
+					(unit 1)
+				)

Commit message: .
Parts:
- renumbered R5005 to R5001, R5006 to R5002, R5001 to R5003, R5002 to R5004, R5003 to R5005, R5004 to R5006
Changed lines of the file:
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@@
 		(dnp no)
 		(fields_autoplaced yes)
-		(property "Reference" "#PWR05001"
+		(property "Reference" "#PWR05004"
 			(at 205.74 96.52 0)
 			(effects
@@
 			(project "PIC18F_ETH"
 				(path "/26a36835-4e01-4565-9612-f38560505464/fe5ea34d-21cf-4dac-9ef2-b9905ff3ffd8"
-					(reference "#PWR05001")
+					(reference "#PWR05004")
 					(unit 1)
 				)
@@
 		(dnp no)
 		(fields_autoplaced yes)
-		(property "Reference" "#PWR05004"
+		(property "Reference" "#PWR05001"
 			(at 111.76 88.9 0)
 			(effects
@@
 			(project "PIC18F_ETH"
 				(path "/26a36835-4e01-4565-9612-f38560505464/fe5ea34d-21cf-4dac-9ef2-b9905ff3ffd8"
-					(reference "#PWR05004")
+					(reference "#PWR05001")
 					(unit 1)
 				)
@@
 		(dnp no)
 		(fields_autoplaced yes)
-		(property "Reference" "#PWR05003"
+		(property "Reference" "#PWR05002"
 			(at 111.76 104.14 0)
 			(effects
@@
 			(project "PIC18F_ETH"
 				(path "/26a36835-4e01-4565-9612-f38560505464/fe5ea34d-21cf-4dac-9ef2-b9905ff3ffd8"
-					(reference "#PWR05003")
+					(reference "#PWR05002")
 					(unit 1)
 				)
@@
 		(dnp no)
 		(fields_autoplaced yes)
-		(property "Reference" "#PWR05005"
+		(property "Reference" "#PWR05003"
 			(at 130.81 120.65 0)
 			(effects
@@
 			(project "PIC18F_ETH"
 				(path "/26a36835-4e01-4565-9612-f38560505464/fe5ea34d-21cf-4dac-9ef2-b9905ff3ffd8"
-					(reference "#PWR05005")
+					(reference "#PWR05003")
 					(unit 1)
 				)
@@
 		(on_board yes)
 		(dnp no)
-		(property "Reference" "R5002"
+		(property "Reference" "R5004"
 			(at 181.864 92.964 0)
 			(effects
@@
 			(project "PIC18F_ETH"
 				(path "/26a36835-4e01-4565-9612-f38560505464/fe5ea34d-21cf-4dac-9ef2-b9905ff3ffd8"
-					(reference "R5002")
+					(reference "R5004")
 					(unit 1)
 				)
@@
 		(dnp no)
 		(fields_autoplaced yes)
-		(property "Reference" "R5005"
+		(property "Reference" "R5001"
 			(at 104.14 85.09 90)
 			(effects
@@
 			(project "PIC18F_ETH"
 				(path "/26a36835-4e01-4565-9612-f38560505464/fe5ea34d-21cf-4dac-9ef2-b9905ff3ffd8"
-					(reference "R5005")
+					(reference "R5001")
 					(unit 1)
 				)
@@
 		(dnp no)
 		(fields_autoplaced yes)
-		(property "Reference" "#PWR05002"
+		(property "Reference" "#PWR05005"
 			(at 210.82 113.03 0)
 			(effects
@@
 			(project "PIC18F_ETH"
 				(path "/26a36835-4e01-4565-9612-f38560505464/fe5ea34d-21cf-4dac-9ef2-b9905ff3ffd8"
-					(reference "#PWR05002")
+					(reference "#PWR05005")
 					(unit 1)
 				)
@@
 		(dnp no)
 		(fields_autoplaced yes)
-		(property "Reference" "R5003"
+		(property "Reference" "R5005"
 			(at 181.61 104.1399 0)
 			(effects
@@
 			(project "PIC18F_ETH"
 				(path "/26a36835-4e01-4565-9612-f38560505464/fe5ea34d-21cf-4dac-9ef2-b9905ff3ffd8"
-					(reference "R5003")
+					(reference "R5005")
 					(unit 1)
 				)
@@
 		(dnp no)
 		(fields_autoplaced yes)
-		(property "Reference" "R5001"
+		(property "Reference" "R5003"
 			(at 181.61 81.2799 0)
 			(effects
@@
 			(project "PIC18F_ETH"
 				(path "/26a36835-4e01-4565-9612-f38560505464/fe5ea34d-21cf-4dac-9ef2-b9905ff3ffd8"
-					(reference "R5001")
+					(reference "R5003")
 					(unit 1)
 				)
@@
 		(dnp no)
 		(fields_autoplaced yes)
-		(property "Reference" "R5004"
+		(property "Reference" "R5006"
 			(at 181.61 115.5699 0)
 			(effects
@@
 			(project "PIC18F_ETH"
 				(path "/26a36835-4e01-4565-9612-f38560505464/fe5ea34d-21cf-4dac-9ef2-b9905ff3ffd8"
-					(reference "R5004")
+					(reference "R5006")
 					(unit 1)
 				)
@@
 		(dnp no)
 		(fields_autoplaced yes)
-		(property "Reference" "R5006"
+		(property "Reference" "R5002"
 			(at 104.14 100.33 90)
 			(effects
@@
 			(project "PIC18F_ETH"
 				(path "/26a36835-4e01-4565-9612-f38560505464/fe5ea34d-21cf-4dac-9ef2-b9905ff3ffd8"
-					(reference "R5006")
-					(unit 1)
-				)
+					(reference "R5002")
+					(unit 1)
+				)

Commit message: .
Other:
- title: (none) -> BT_ADDX
Changed lines of the file:
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@@
 	(generator "eeschema")
 	(generator_version "8.0")
-	(paper "A4")
+	(paper "A3")
+	(title_block
+		(title "BT_ADDX")
+		(rev "Rev:P1")
+	)
 	(bus_alias "ETH"
 		(members "RX-" "RX+" "TX-" "TX+")

Commit message: .
Other:
- title: BT_ADDX -> BT_AD/DX
Changed lines of the file:
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@@
 	(paper "A3")
 	(title_block
-		(title "BT_ADDX")
+		(title "BT_AD/DX")
 		(rev "Rev:P1")
+		(comment 1 "BT_0001-1")
 	)
 	(bus_alias "ETH"

Commit message: .
Connections:
- net TX_C is gone; now on net +3.3V: C5002.1, J5001.3, R5005.2, R5006.1
- net +3.3V: no longer C5002.2
- net GND: now also C5002.2
- net RX_C: no longer C5001.1, R5003.2, R5004.1
- new net: C5001.1, R5003.2, R5004.1
Changed lines of the file:
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@@
+	)
+	(junction
+		(at 190.5 111.76)
+		(diameter 0)
+		(color 0 0 0 0)
 	)
 	(junction
@@
 	)
 	(junction
-		(at 179.07 87.63)
-		(diameter 0)
-		(color 0 0 0 0)
-	)
-	(junction
 		(at 179.07 88.9)
 		(diameter 0)
@@
 		)
 	)
-	(wire
-		(pts
-			(xy 170.18 87.63) (xy 179.07 87.63)
-		)
-		(stroke
-			(width 0)
-			(type default)
-		)
-	)
 	(bus
 		(pts
@@
 	(wire
 		(pts
-			(xy 179.07 111.76) (xy 196.85 111.76)
+			(xy 179.07 111.76) (xy 190.5 111.76)
 		)
 		(stroke
@@
 	(wire
 		(pts
-			(xy 179.07 87.63) (xy 179.07 88.9)
-		)
-		(stroke
-			(width 0)
-			(type default)
-		)
-	)
-	(wire
-		(pts
-			(xy 210.82 111.76) (xy 210.82 109.22)
+			(xy 179.07 86.36) (xy 179.07 88.9)
 		)
 		(stroke
@@
 	(wire
 		(pts
+			(xy 190.5 109.22) (xy 190.5 111.76)
+		)
+		(stroke
+			(width 0)
+			(type default)
+		)
+	)
+	(wire
+		(pts
 			(xy 95.25 91.44) (xy 100.33 91.44)
 		)
@@
 	(wire
 		(pts
+			(xy 190.5 111.76) (xy 196.85 111.76)
+		)
+		(stroke
+			(width 0)
+			(type default)
+		)
+	)
+	(wire
+		(pts
 			(xy 160.02 120.65) (xy 179.07 120.65)
 		)
@@
 	(wire
 		(pts
+			(xy 210.82 111.76) (xy 210.82 113.03)
+		)
+		(stroke
+			(width 0)
+			(type default)
+		)
+	)
+	(wire
+		(pts
 			(xy 160.02 106.68) (xy 160.02 120.65)
 		)
@@
 		(pts
 			(xy 179.07 88.9) (xy 179.07 90.17)
-		)
-		(stroke
-			(width 0)
-			(type default)
-		)
-	)
-	(wire
-		(pts
-			(xy 179.07 86.36) (xy 179.07 87.63)
 		)
 		(stroke
@@
 	(label "TX+"
 		(at 144.78 106.68 0)
-		(fields_autoplaced yes)
-		(effects
-			(font
-				(size 1.27 1.27)
-			)
-			(justify left bottom)
-		)
-	)
-	(label "RX_C"
-		(at 170.18 87.63 0)
 		(fields_autoplaced yes)
 		(effects
@@
 				(path "/26a36835-4e01-4565-9612-f38560505464/fe5ea34d-21cf-4dac-9ef2-b9905ff3ffd8"
 					(reference "#PWR05004")
+					(unit 1)
+				)
+			)
+		)
+	)
+	(symbol
+		(lib_id "power:GND")
+		(at 210.82 113.03 0)
+		(unit 1)
+		(exclude_from_sim no)
+		(in_bom yes)
+		(on_board yes)
+		(dnp no)
+		(fields_autoplaced yes)
+		(property "Reference" "#PWR05005"
+			(at 210.82 119.38 0)
+			(effects
+				(font
+					(size 1.27 1.27)
+				)
+				(hide yes)
+			)
+		)
+		(property "Value" "GND"
+			(at 210.82 118.11 0)
+			(effects
+				(font
+					(size 1.27 1.27)
+				)
+			)
+		)
+		(property "Footprint" ""
+			(at 210.82 113.03 0)
+			(effects
+				(font
+					(size 1.27 1.27)
+				)
+				(hide yes)
+			)
+		)
+		(property "Datasheet" ""
+			(at 210.82 113.03 0)
+			(effects
+				(font
+					(size 1.27 1.27)
+				)
+				(hide yes)
+			)
+		)
+		(property "Description" "Power symbol creates a global label with name \"GND\" , ground"
+			(at 210.82 113.03 0)
+			(effects
+				(font
+					(size 1.27 1.27)
+				)
+				(hide yes)
+			)
+		)
+		(pin "1"
+		)
+		(instances
+			(project "PIC18F_ETH"
+				(path "/26a36835-4e01-4565-9612-f38560505464/fe5ea34d-21cf-4dac-9ef2-b9905ff3ffd8"
+					(reference "#PWR05005")
+					(unit 1)
+				)
+			)
+		)
+	)
+	(symbol
+		(lib_id "power:+3.3V")
+		(at 190.5 109.22 0)
+		(unit 1)
+		(exclude_from_sim no)
+		(in_bom yes)
+		(on_board yes)
+		(dnp no)
+		(fields_autoplaced yes)
+		(property "Reference" "#PWR05006"
+			(at 190.5 113.03 0)
+			(effects
+				(font
+					(size 1.27 1.27)
+				)
+				(hide yes)
+			)
+		)
+		(property "Value" "+3.3V"
+			(at 190.5 104.14 0)
+			(effects
+				(font
+					(size 1.27 1.27)
+				)
+			)
+		)
+		(property "Footprint" ""
+			(at 190.5 109.22 0)
+			(effects
+				(font
+					(size 1.27 1.27)
+				)
+				(hide yes)
+			)
+		)
+		(property "Datasheet" ""
+			(at 190.5 109.22 0)
+			(effects
+				(font
+					(size 1.27 1.27)
+				)
+				(hide yes)
+			)
+		)
+		(property "Description" "Power symbol creates a global label with name \"+3.3V\""
+			(at 190.5 109.22 0)
+			(effects
+				(font
+					(size 1.27 1.27)
+				)
+				(hide yes)
+			)
+		)
+		(pin "1"
+		)
+		(instances
+			(project "PIC18F_ETH"
+				(path "/26a36835-4e01-4565-9612-f38560505464/fe5ea34d-21cf-4dac-9ef2-b9905ff3ffd8"
+					(reference "#PWR05006")
 					(unit 1)
 				)
@@
 					(unit 1)
 				)
-			)
-		)
-	)
-	(symbol
-		(lib_id "power:+3.3V")
-		(at 210.82 109.22 0)
-		(unit 1)
-		(exclude_from_sim no)
-		(in_bom yes)
-		(on_board yes)
-		(dnp no)
-		(fields_autoplaced yes)
-		(property "Reference" "#PWR05005"
-			(at 210.82 113.03 0)
-			(effects
-				(font
-					(size 1.27 1.27)
-				)
-				(hide yes)
-			)
-		)
-		(property "Value" "+3.3V"
-			(at 210.82 104.14 0)
-			(effects
-				(font
-					(size 1.27 1.27)
-				)
-			)
-		)
-		(property "Footprint" ""
-			(at 210.82 109.22 0)
-			(effects
-				(font
-					(size 1.27 1.27)
-				)
-				(hide yes)
-			)
-		)
-		(property "Datasheet" ""
-			(at 210.82 109.22 0)
-			(effects
-				(font
-					(size 1.27 1.27)
-				)
-				(hide yes)
-			)
-		)
-		(property "Description" "Power symbol creates a global label with name \"+3.3V\""
-			(at 210.82 109.22 0)
-			(effects
-				(font
-					(size 1.27 1.27)
-				)
-				(hide yes)
-			)
-		)
-		(pin "1"
-		)
-		(instances
-			(project "PIC18F_ETH"
-				(path "/26a36835-4e01-4565-9612-f38560505464/fe5ea34d-21cf-4dac-9ef2-b9905ff3ffd8"
-					(reference "#PWR05005")
-					(unit 1)
-				)

Commit message: .
Parts:
- C5001, C5002: MPN C;C;T1;S;P0603;NA -> C;M;100n;10p;25V;S;0603
- R5001, R5002: MPN R;G;T1;S;P0603;NA -> R;G;510K;10P0;S;0603
Changed lines of the file:
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@@
 			)
 		)
-		(property "MPN" "R;G;T1;S;P0603;NA"
+		(property "MPN" "R;G;510K;10P0;S;0603"
 			(at 104.14 91.44 90)
 			(effects
@@
 			)
 		)
-		(property "MPN" "C;C;T1;S;P0603;NA"
+		(property "MPN" "C;M;100n;10p;25V;S;0603"
 			(at 200.66 107.76 90)
 			(effects
@@
 			)
 		)
-		(property "MPN" "C;C;T1;S;P0603;NA"
+		(property "MPN" "C;M;100n;10p;25V;S;0603"
 			(at 200.66 84.9 90)
 			(effects
@@
 			)
 		)
-		(property "MPN" "R;G;T1;S;P0603;NA"
+		(property "MPN" "R;G;510K;10P0;S;0603"
 			(at 104.14 106.68 90)
 			(effects

Commit message: .
Parts:
- J5001: CPN BT10000-00001 -> BT10001-00001; SMT (none) -> n
Changed lines of the file:
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@@
 			)
 		)
-		(property "Datasheet" "https://www.electrokit.com/uploads/productfile/41010/MagJack.pdf"
+		(property "Datasheet" "https://www.electrokit.com/upload/product/41010/41010276/MagJack.pdf"
 			(at 130.81 80.01 0)
 			(effects
@@
 			)
 		)
-		(property "CPN" "BT10000-00001"
+		(property "CPN" "BT10001-00001"
 			(at 130.81 97.79 0)
 			(effects
@@
 			)
 		)
+		(property "SMT" "n"
+			(at 130.81 97.79 0)
+			(effects
+				(font
+					(size 1.27 1.27)
+				)
+			)
+		)
