File: HW/DTS_Board/400hz_input.kicad_sch (KiCad schematic)
At the start: 13 parts, among them U3001 LM324A

Commit message: .
Changed lines of the file:
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@@
 	(wire
 		(pts
-			(xy 231.14 80.01) (xy 247.65 80.01)
+			(xy 231.14 80.01) (xy 248.92 80.01)
 		)
 		(stroke
@@
 	(hierarchical_label "Ch400Hz"
 		(shape output)
-		(at 247.65 80.01 0)
-		(fields_autoplaced yes)
+		(at 248.92 80.01 0)
 		(effects
 			(font
@@
 			(justify left)
 		)
-	)
+		(property "Intersheetrefs" "${INTERSHEET_REFS}"
+			(at 252.476 83.058 0)
+			(show_name yes)
+			(effects
+				(font
+					(size 1.27 1.27)
+					(italic yes)
+				)
+			)
+		)
+	)
