File: HW/LISN/LISN_5u/LISN_5u.kicad_pcb (KiCad board)
At the start: 2 copper layers, 90 x 50 mm, 43 parts, among them X101 Conn_Coaxial_Small, X102 SLB4,RED, X103 SLB4,RED, X104 SLB4,BLACK, X105 SLB4,BLACK

Commit message: .
Parts:
- moved D105 3.81 mm to (97.3, 75.2), turned to -135 degrees
Routing:
- net Net-(X103-Pin_1): track 14.2 -> 17.7 mm
- net GND: track 1.82 -> 2.65 mm, vias 318 -> 332
