File: HW/ETH_mPCIe_t1_Switch/mPCIe_T1Switch/PCIe_connector.kicad_sch (KiCad schematic)
At the start: 1 part

Commit message: .
Parts:
- gave numbers to parts that had none: 1
Changed lines of the file:
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@@
 	)
 	(hierarchical_label "PCIE{PCIE}"
-		(shape input)
+		(shape bidirectional)
 		(at 100.33 116.84 180)
 		(fields_autoplaced yes)
@@
 		(on_board yes)
 		(dnp no)
-		(property "Reference" "X?"
+		(property "Reference" "X4001"
 			(at 218.186 87.63 0)
 			(effects
@@
 			(project ""
 				(path "/35c16f53-2908-4c19-8371-633bea9adc2a/5373f408-5f1e-469a-8abd-82497cfedf8b"
-					(reference "X?")
+					(reference "X4001")
 					(unit 1)
 				)

Commit message: .
Other:
- note added: "Check Pinning"
Changed lines of the file:
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@@
+		)
+	)
+	(text "Check Pinning"
+		(exclude_from_sim no)
+		(at 159.258 118.364 0)
+		(effects
+			(font
+				(size 1.27 1.27)
+			)
 		)
 	)
