File: HW/ETH_mPCIe_t1_Switch/mPCIe_T1Switch/mPCIe_T1Switch.kicad_sch (KiCad schematic)
At the start: 0 parts

Commit message: .
Other:
- sheet PCIe_connector ports: added PCIE{PCIE}; removed none
Changed lines of the file:
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@@
+		)
+	)
+	(bus
+		(pts
+			(xy 90.17 104.14) (xy 111.76 104.14)
+		)
+		(stroke
+			(width 0)
+			(type default)
+		)
+	)
+	(label "PCIE{PCIE}"
+		(at 95.25 104.14 0)
+		(fields_autoplaced yes)
+		(effects
+			(font
+				(size 1.27 1.27)
+			)
+			(justify left bottom)
 		)
 	)
@@
 			)
 		)
-		(pin "PCIE{PCIE}" input
+		(pin "PCIE{PCIE}" bidirectional
 			(at 111.76 104.14 180)
 			(effects
@@
 			)
 		)
+		(pin "PCIE{PCIE}" bidirectional
+			(at 90.17 104.14 0)
+			(effects
+				(font
+					(size 1.27 1.27)
+				)
+				(justify right)
+			)
+		)

Commit message: .
Other:
- sheet 4Port_T1_switch ports: added INH, MDC, MDIO, PHY_Int#, PHY_Reset#, SPI{SPI}, WAKE_OUT; removed none
- sheet PCI_ETH_Controller ports: added MDC, MDIO, PHY_Int#, PHY_Reset#; removed none
- note added: "MDIO"
Changed lines of the file:
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@@
 	(generator_version "8.0")
 	(paper "A3")
+	(wire
+		(pts
+			(xy 160.02 107.95) (xy 222.25 107.95)
+		)
+		(stroke
+			(width 0)
+			(type default)
+		)
+	)
+	(wire
+		(pts
+			(xy 160.02 115.57) (xy 222.25 115.57)
+		)
+		(stroke
+			(width 0)
+			(type default)
+		)
+	)
+	(wire
+		(pts
+			(xy 160.02 113.03) (xy 222.25 113.03)
+		)
+		(stroke
+			(width 0)
+			(type default)
+		)
+	)
 	(bus
 		(pts
@@
 			(width 0)
 			(type default)
+		)
+	)
+	(wire
+		(pts
+			(xy 160.02 110.49) (xy 222.25 110.49)
+		)
+		(stroke
+			(width 0)
+			(type default)
+		)
+	)
+	(text "MDIO"
+		(exclude_from_sim no)
+		(at 183.896 115.062 0)
+		(effects
+			(font
+				(size 1.27 1.27)
+			)
+		)
+	)
+	(label "MDC"
+		(at 181.61 113.03 0)
+		(fields_autoplaced yes)
+		(effects
+			(font
+				(size 1.27 1.27)
+			)
+			(justify left bottom)
+		)
+	)
+	(label "PHY_Reset#"
+		(at 181.61 110.49 0)
+		(fields_autoplaced yes)
+		(effects
+			(font
+				(size 1.27 1.27)
+			)
+			(justify left bottom)
+		)
+	)
+	(label "PHY_Int#"
+		(at 181.61 107.95 0)
+		(fields_autoplaced yes)
+		(effects
+			(font
+				(size 1.27 1.27)
+			)
+			(justify left bottom)
 		)
 	)
@@
 		(pin "RGMII{RGMII}" input
 			(at 160.02 105.41 0)
+			(effects
+				(font
+					(size 1.27 1.27)
+				)
+				(justify right)
+			)
+		)
+		(pin "PHY_Int#" bidirectional
+			(at 160.02 107.95 0)
+			(effects
+				(font
+					(size 1.27 1.27)
+				)
+				(justify right)
+			)
+		)
+		(pin "PHY_Reset#" bidirectional
+			(at 160.02 110.49 0)
+			(effects
+				(font
+					(size 1.27 1.27)
+				)
+				(justify right)
+			)
+		)
+		(pin "MDC" bidirectional
+			(at 160.02 113.03 0)
+			(effects
+				(font
+					(size 1.27 1.27)
+				)
+				(justify right)
+			)
+		)
+		(pin "MDIO" bidirectional
+			(at 160.02 115.57 0)
 			(effects
 				(font
@@
 			)
 		)
+		(pin "MDC" bidirectional
+			(at 222.25 113.03 180)
+			(effects
+				(font
+					(size 1.27 1.27)
+				)
+				(justify left)
+			)
+		)
+		(pin "PHY_Int#" bidirectional
+			(at 222.25 107.95 180)
+			(effects
+				(font
+					(size 1.27 1.27)
+				)
+				(justify left)
+			)
+		)
+		(pin "MDIO" bidirectional
+			(at 222.25 115.57 180)
+			(effects
+				(font
+					(size 1.27 1.27)
+				)
+				(justify left)
+			)
+		)
+		(pin "PHY_Reset#" bidirectional
+			(at 222.25 110.49 180)
+			(effects
+				(font
+					(size 1.27 1.27)
+				)
+				(justify left)
+			)
+		)
+		(pin "WAKE_OUT" bidirectional
+			(at 246.38 90.17 90)
+			(effects
+				(font
+					(size 1.27 1.27)
+				)
+				(justify right)
+			)
+		)
+		(pin "INH" bidirectional
+			(at 248.92 90.17 90)
+			(effects
+				(font
+					(size 1.27 1.27)
+				)
+				(justify right)
+			)
+		)
+		(pin "SPI{SPI}" bidirectional
+			(at 254 90.17 90)
+			(effects
+				(font
+					(size 1.27 1.27)
+				)
+				(justify right)
+			)
+		)
