File: HW/ETH_mPCIe_t1_Switch/mPCIe_T1Switch/4Port_T1_switch.kicad_sch (KiCad schematic)
At the start: 9 parts, among them U301 LAN9370-V/KCXVAO, U302 TPS62A01

Commit message: .
Parts:
- added C3001, C3002, C3003, C3004, C3005, C3006, C3007, C3008, C3009, C3010, C3011, C3012, C3013, C3014, C3015, C3016, C3017, C3018, C3019, C3020: 100n 25V, Capacitor_SMD:C_0603_1608Metric, symbol bt_capacitor:C;M;100n;10p;25V;S;0603
Connections:
- net +1V1: now also U301.11 (VDD11ATXRX), U301.15 (E_VDDA), U301.17 (VDDCORE), U301.34 (VDDCORE), U301.39 (VDDCORE), U301.4 (VDD11ATXRX), U301.5 (VDD11ACOM), U301.57 (VDD11ATXRX), U301.58 (VDDCORE), C3001.1, C3002.1, C3003.1, C3004.1, C3005.1, C3006.1, C3007.1, C3008.1, C3009.1
- net +3V3: now also U301.1 (VDDATXRX), U301.14 (VDDATXRX), U301.22 (VDDRGMII), U301.28 (VDDRGMII), U301.33 (VDDRGMII), U301.35 (VDDIO), U301.43 (VDDIO), U301.53 (VDDIO), U301.54 (VDDATXRX), U301.64 (VBAT), U301.7 (VDDACOM), U301.8 (VDDATXRX), C3010.1, C3011.1, C3012.1, C3013.1, C3014.1, C3015.1, C3016.1, C3017.1, C3018.1, C3019.1, C3020.1
- net GND: now also C3001.2, C3002.2, C3003.2, C3004.2, C3005.2, C3006.2, C3007.2, C3008.2, C3009.2, C3010.2, C3011.2, C3012.2, C3013.2, C3014.2, C3015.2, C3016.2, C3017.2, C3018.2, C3019.2, C3020.2

Commit message: .
Parts:
- added R303: 10K, Resistor_SMD:R_0603_1608Metric, symbol bt_resistors:R;G;10K;10P0;S;0603
Connections:
- net +3V3: now also R303.1
- net SPI.CS#: now reaches U301.38 (SCS_N)
- net SPI.MOSI: now reaches U301.40 (SDI)
- net SPI.MISO: now reaches U301.41 (SDO/SWITCH_EN)
- net SPI.CLK: now reaches U301.42 (SCL)
- net PHY_Int#: now reaches U301.44 (IRQ_N)
- net PHY_Reset#: now reaches U301.45 (RESET_N)
- net PHY_Reset#: now also R303.2
- net MDIO: now reaches U301.49 (LED_3/MDIO)
- net MDC: now reaches U301.50 (LED_4/MDC)
- net WAKE_OUT: now reaches U301.61 (WAKE_OUT)
- net INH: now reaches U301.63 (INH)
- net RGMII.RX_ER: no longer names the net of U301.25 (RX_ER)

Commit message: .
Parts:
- C3001, C3002, C3003, C3004, C3005, C3006, C3007, C3008, C3009, C3010, C3011, C3012, C3013, C3014, C3015, C3016, C3017, C3018, C3019, C3020: footprint Capacitor_SMD:C_0603_1608Metric -> Capacitor_SMD:C_0402_1005Metric; symbol bt_capacitor:C;M;100n;10p;25V;S;0603 -> bt_capacitor:C;M;100n;10p;16V;S;0402; CPN BT00008-091000 -> BT00024-091000; MPN C;M;100n;10p;25V;S;0603 -> C;M;100n;10p;16V;S;0402
