File: HW/ETH_mPCIe_t1_Switch/mPCIe_T1Switch/untitled.kicad_sch (KiCad schematic)
At the start: 4 parts, among them U201 LAN7431/YXX

Commit message: .
Parts:
- added C2001, C2002, C2021, C2022: 10u 10V, Capacitor_SMD:C_0603_1608Metric, symbol bt_capacitor:C;M;10u;10p;10V;S;0603
- added C2003, C2004, C2005, C2006, C2007, C2008, C2009, C2010, C2011, C2012, C2013, C2014, C2015, C2016, C2017, C2018, C2019, C2020: 100n 25V, Capacitor_SMD:C_0603_1608Metric, symbol bt_capacitor:C;M;100n;10p;25V;S;0603
Connections:
- net GND is gone; now on net +3V3: C201.2, U201.26 (VSS), U201.29 (VSS), U201.33 (VSS), U201.EP (VSS)
- net +1V2: now also C2002.1, C2003.1, C2006.1, C2009.1, C2010.1, C2012.1, C2014.1, C2017.1, C2020.1
- net +2V5: now also C2001.1, C2016.1, C2019.1
- net +3V3: now also C2001.2, C2002.2, C2003.2, C2004.1, C2004.2, C2005.1, C2005.2, C2006.2, C2007.1, C2007.2, C2008.1, C2008.2, C2009.2, C2010.2, C2011.1, C2011.2, C2012.2, C2013.1, C2013.2, C2014.2, C2015.1, C2015.2, C2016.2, C2017.2, C2018.1, C2018.2, C2019.2, C2020.2, C2021.1, C2021.2, C2022.1, C2022.2

Commit message: .
Connections:
- net PHY_Int#: now reaches U201.41 (PHY_INT_N)
- net PHY_Reset#: now reaches U201.42 (PHY_RESET_N)
- net MDIO: now reaches U201.63 (MDIO)
- net MDC: now reaches U201.64 (MDC)
- net RGMII.RX_ER: no longer names the net of U201.20 (CLK125/RX_ER)
- no-connect marks 0 -> 4
Other:
- note added: "JTAG"

Commit message: .
Parts:
- C2003, C2004, C2005, C2006, C2007, C2008, C2009, C2010, C2011, C2012, C2013, C2014, C2015, C2016, C2017, C2018, C2019, C2020: footprint Capacitor_SMD:C_0603_1608Metric -> Capacitor_SMD:C_0402_1005Metric; symbol bt_capacitor:C;M;100n;10p;25V;S;0603 -> bt_capacitor:C;M;100n;10p;16V;S;0402; CPN BT00008-091000 -> BT00024-091000; MPN C;M;100n;10p;25V;S;0603 -> C;M;100n;10p;16V;S;0402
