File: HW/ETH_mPCIe_t1_Switch/mPCIe_T1Switch/mPCIe_T1Switch.kicad_pcb (KiCad board)
At the start: 4 copper layers, 13 parts, among them U201 LAN7431/YXX, U301 LAN9370-V/KCXVAO, U302 TPS62A01

Commit message: .
Parts:
- added C2001: 10u 10V, Capacitor_SMD:C_0603_1608Metric, F.Cu at (158.6, 113.9)
- added C2002: 10u 10V, Capacitor_SMD:C_0603_1608Metric, F.Cu at (158.6, 116.5)
- added X4001: ~, bt_footprints:M.2_KEY_E, F.Cu at (141.8, 147.2)
- U201: moved to B.Cu
- moved U201 41.1 mm to (137.2, 136.5)
- moved U301 30.1 mm to (147.8, 123.0), turned to 0 degrees
Connections:
- U201 pad 27: /PCI_ETH_Controller/PCIE.RX_P -> /PCIE.RX_P
- U201 pad 28: /PCI_ETH_Controller/PCIE.RX_N -> /PCIE.RX_N
- U201 pad 30: /PCI_ETH_Controller/PCIE.TX_P -> /PCIE.TX_P
- U201 pad 32: /PCI_ETH_Controller/PCIE.TX_N -> /PCIE.TX_N
- U201 pad 36: /PCI_ETH_Controller/PCIE.CLK_P -> /PCIE.CLK_P
- U201 pad 37: /PCI_ETH_Controller/PCIE.CLK_N -> /PCIE.CLK_N
- U201 pad 66: /PCI_ETH_Controller/PCIE.CLKREQ# -> /PCIE.CLKREQ#
- U201 pad 67: /PCI_ETH_Controller/PCIE.WAKE# -> /PCIE.WAKE#
- U201 pad 68: /PCI_ETH_Controller/PCIE.PERST# -> /PCIE.PERST#
Other:
- board outline added: 22 x 4 mm

Commit message: .
Parts:
- added C2003: 100n 25V, Capacitor_SMD:C_0603_1608Metric, F.Cu at (107.8, 115.4)
- added C2004: 100n 25V, Capacitor_SMD:C_0603_1608Metric, F.Cu at (81.7, 118.9)
- added C2005: 100n 25V, Capacitor_SMD:C_0603_1608Metric, F.Cu at (80.8, 125.0)
- added C2006: 100n 25V, Capacitor_SMD:C_0603_1608Metric, F.Cu at (80.1, 131.8)
- added C2007: 100n 25V, Capacitor_SMD:C_0603_1608Metric, F.Cu at (100.5, 140.5)
- added C2008: 100n 25V, Capacitor_SMD:C_0603_1608Metric, F.Cu at (111.9, 115.4)
- added C2009: 100n 25V, Capacitor_SMD:C_0603_1608Metric, F.Cu at (85.7, 118.9)
- added C2010: 100n 25V, Capacitor_SMD:C_0603_1608Metric, F.Cu at (84.8, 125.0)
- added C2011: 100n 25V, Capacitor_SMD:C_0603_1608Metric, F.Cu at (84.1, 131.8)
- added C2012: 100n 25V, Capacitor_SMD:C_0603_1608Metric, F.Cu at (104.5, 140.5)
- added C2013: 100n 25V, Capacitor_SMD:C_0603_1608Metric, F.Cu at (115.9, 115.4)
- added C2014: 100n 25V, Capacitor_SMD:C_0603_1608Metric, F.Cu at (89.7, 118.9)
- added C2015: 100n 25V, Capacitor_SMD:C_0603_1608Metric, F.Cu at (88.9, 125.0)
- added C2016: 100n 25V, Capacitor_SMD:C_0603_1608Metric, F.Cu at (88.1, 131.8)
- added C2017: 100n 25V, Capacitor_SMD:C_0603_1608Metric, F.Cu at (108.5, 140.5)
- added C2018: 100n 25V, Capacitor_SMD:C_0603_1608Metric, F.Cu at (119.9, 115.4)
- added C2019: 100n 25V, Capacitor_SMD:C_0603_1608Metric, F.Cu at (93.7, 118.9)
- added C2020: 100n 25V, Capacitor_SMD:C_0603_1608Metric, F.Cu at (92.9, 125.0)
- added C2021: 10u 10V, Capacitor_SMD:C_0603_1608Metric, F.Cu at (92.1, 131.8)
- added C2022: 10u 10V, Capacitor_SMD:C_0603_1608Metric, F.Cu at (112.5, 140.5)
- added C3001: 100n 25V, Capacitor_SMD:C_0603_1608Metric, F.Cu at (163.4, 123.6)
- added C3002: 100n 25V, Capacitor_SMD:C_0603_1608Metric, F.Cu at (163.4, 126.1)
- added C3003: 100n 25V, Capacitor_SMD:C_0603_1608Metric, F.Cu at (163.4, 128.6)
- added C3004: 100n 25V, Capacitor_SMD:C_0603_1608Metric, F.Cu at (163.4, 131.2)
- added C3005: 100n 25V, Capacitor_SMD:C_0603_1608Metric, F.Cu at (163.4, 133.7)
- added C3006: 100n 25V, Capacitor_SMD:C_0603_1608Metric, F.Cu at (163.4, 136.2)
- added C3007: 100n 25V, Capacitor_SMD:C_0603_1608Metric, F.Cu at (163.4, 138.7)
- added C3008: 100n 25V, Capacitor_SMD:C_0603_1608Metric, F.Cu at (167.4, 123.6)
- added C3009: 100n 25V, Capacitor_SMD:C_0603_1608Metric, F.Cu at (167.4, 126.1)
- added C3010: 100n 25V, Capacitor_SMD:C_0603_1608Metric, F.Cu at (167.4, 128.6)
- added C3011: 100n 25V, Capacitor_SMD:C_0603_1608Metric, F.Cu at (167.4, 131.2)
- added C3012: 100n 25V, Capacitor_SMD:C_0603_1608Metric, F.Cu at (167.4, 133.7)
- added C3013: 100n 25V, Capacitor_SMD:C_0603_1608Metric, F.Cu at (167.4, 136.2)
- added C3014: 100n 25V, Capacitor_SMD:C_0603_1608Metric, F.Cu at (167.4, 138.7)
- added C3015: 100n 25V, Capacitor_SMD:C_0603_1608Metric, F.Cu at (171.4, 123.6)
- added C3016: 100n 25V, Capacitor_SMD:C_0603_1608Metric, F.Cu at (171.4, 126.1)
- added C3017: 100n 25V, Capacitor_SMD:C_0603_1608Metric, F.Cu at (171.4, 128.6)
- added C3018: 100n 25V, Capacitor_SMD:C_0603_1608Metric, F.Cu at (171.4, 131.2)
- added C3019: 100n 25V, Capacitor_SMD:C_0603_1608Metric, F.Cu at (171.4, 133.7)
- added C3020: 100n 25V, Capacitor_SMD:C_0603_1608Metric, F.Cu at (171.4, 136.2)
- added R303: 10K, Resistor_SMD:R_0603_1608Metric, F.Cu at (171.4, 138.7)
Connections:
- C2001 pad 2: GND -> +3V3
- C2002 pad 2: GND -> +3V3
- C201 pad 2: GND -> +3V3
- C301 pad 2: GND -> +3V3
- C302 pad 2: GND -> +3V3
- C303 pad 2: GND -> +3V3
- C304 pad 2: GND -> +3V3
- R302 pad 2: GND -> +3V3
- U201 pad 20: /4Port_T1_switch/RGMII.RX_ER -> unconnected-(U201A-CLK125/RX_ER-Pad20)
- U201 pad 26: GND -> +3V3
- U201 pad 29: GND -> +3V3
- U201 pad 33: GND -> +3V3
- U201 pad 41: unconnected-(U201A-PHY_INT_N-Pad41) -> /PHY_Int#
- U201 pad 42: unconnected-(U201A-PHY_RESET_N-Pad42) -> /PHY_Reset#
- U201 pad 63: unconnected-(U201A-MDIO-Pad63) -> /4Port_T1_switch/MDIO
- U201 pad 64: unconnected-(U201A-MDC-Pad64) -> /MDC
- U201 pad EP: GND -> +3V3
- U301 pad 1: Net-(U301B-VBAT) -> +3V3
- U301 pad 11: Net-(U301B-E_VDDA) -> +1V1
- U301 pad 14: Net-(U301B-VBAT) -> +3V3
- U301 pad 15: Net-(U301B-E_VDDA) -> +1V1
- U301 pad 17: Net-(U301B-E_VDDA) -> +1V1
- U301 pad 22: Net-(U301B-VBAT) -> +3V3
- U301 pad 25: /4Port_T1_switch/RGMII.RX_ER -> unconnected-(U301A-RX_ER-Pad25)
- U301 pad 28: Net-(U301B-VBAT) -> +3V3
- U301 pad 33: Net-(U301B-VBAT) -> +3V3
- U301 pad 34: Net-(U301B-E_VDDA) -> +1V1
- U301 pad 35: Net-(U301B-VBAT) -> +3V3
- U301 pad 38: unconnected-(U301A-SCS_N-Pad38) -> /4Port_T1_switch/SPI.CS#
- U301 pad 39: Net-(U301B-E_VDDA) -> +1V1
- U301 pad 4: Net-(U301B-E_VDDA) -> +1V1
- U301 pad 40: unconnected-(U301A-SDI-Pad40) -> /4Port_T1_switch/SPI.MOSI
- U301 pad 41: unconnected-(U301A-SDO/SWITCH_EN-Pad41) -> /4Port_T1_switch/SPI.MISO
- U301 pad 42: unconnected-(U301A-SCL-Pad42) -> /4Port_T1_switch/SPI.CLK
- U301 pad 43: Net-(U301B-VBAT) -> +3V3
- U301 pad 44: unconnected-(U301A-IRQ_N-Pad44) -> /PHY_Int#
- U301 pad 45: unconnected-(U301A-RESET_N-Pad45) -> /PHY_Reset#
- U301 pad 46: GND -> +3V3
- U301 pad 49: unconnected-(U301A-LED_3/MDIO-Pad49) -> /4Port_T1_switch/MDIO
- U301 pad 5: Net-(U301B-E_VDDA) -> +1V1
- U301 pad 50: unconnected-(U301A-LED_4/MDC-Pad50) -> /MDC
- U301 pad 53: Net-(U301B-VBAT) -> +3V3
- U301 pad 54: Net-(U301B-VBAT) -> +3V3
- U301 pad 57: Net-(U301B-E_VDDA) -> +1V1
- U301 pad 58: Net-(U301B-E_VDDA) -> +1V1
- U301 pad 61: unconnected-(U301A-WAKE_OUT-Pad61) -> /4Port_T1_switch/WAKE_OUT
- U301 pad 63: unconnected-(U301A-INH-Pad63) -> /4Port_T1_switch/INH
- U301 pad 64: Net-(U301B-VBAT) -> +3V3
- U301 pad 7: Net-(U301B-VBAT) -> +3V3
- U301 pad 8: Net-(U301B-VBAT) -> +3V3
- U301 pad EP: GND -> +3V3
- U302 pad 2: GND -> +3V3
- X4001 pad 1: GND -> +3V3
- X4001 pad 18: GND -> +3V3
- X4001 pad 33: GND -> +3V3
- X4001 pad 39: GND -> +3V3
- X4001 pad 45: GND -> +3V3
- X4001 pad 51: GND -> +3V3
- X4001 pad 57: GND -> +3V3
- X4001 pad 63: GND -> +3V3
- X4001 pad 69: GND -> +3V3
- X4001 pad 7: GND -> +3V3
- X4001 pad 75: GND -> +3V3

Commit message: .
Parts:
- C2003, C2004, C2005, C2006, C2007, C2008, C2009, C2010, C2011, C2012, C2013, C2014, C2015, C2016, C2017, C2018, C2019, C2020, C3001, C3002, C3003, C3004, C3005, C3006, C3007, C3008, C3009, C3010, C3011, C3012, C3013, C3014, C3015, C3016, C3017, C3018, C3019, C3020: footprint Capacitor_SMD:C_0603_1608Metric -> Capacitor_SMD:C_0402_1005Metric
- U201: moved to F.Cu
- moved C301 53.0 mm to (161.0, 137.8), turned to 0 degrees
- moved L301 52.0 mm to (158.4, 132.5), turned to 90 degrees
- moved U302 50.5 mm to (161.0, 134.9), turned to -90 degrees
- moved R302 49.7 mm to (163.5, 137.3), turned to -90 degrees
- moved C304 49.1 mm to (159.4, 129.9), turned to 0 degrees
- moved C303 48.2 mm to (159.4, 128.4), turned to 0 degrees
- moved C302 47.4 mm to (159.4, 126.9), turned to 0 degrees
- moved R301 47.2 mm to (163.5, 134.3), turned to -90 degrees
- moved C3014 37.5 mm to (192.7, 111.0)
- moved R303 37.5 mm to (196.7, 111.0)
- moved C3007 37.5 mm to (188.7, 111.0)
- moved C3020 31.3 mm to (197.2, 118.4)
- moved C3006 31.3 mm to (189.2, 118.4)
- moved C3013 31.3 mm to (193.2, 118.4)
- moved C3010 30.9 mm to (195.5, 141.5)
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
Commit message: .
Parts:
- moved U301 12.6 mm to (135.1, 123.7)
- moved U201 8.66 mm to (145.8, 135.1)
Routing:
- net /4Port_T1_switch/RGMII.RXD3: track 0.00 -> 13.6 mm
- net /4Port_T1_switch/RGMII.RX_CTL: track 0.00 -> 13.6 mm, vias 0 -> 2
- net /4Port_T1_switch/RGMII.TX_CTL: track 0.00 -> 13.0 mm, vias 0 -> 2
- net /4Port_T1_switch/RGMII.RXD2: track 0.00 -> 12.9 mm
- net /4Port_T1_switch/RGMII.TX_CLK: track 0.00 -> 12.6 mm, vias 0 -> 2
- net /4Port_T1_switch/RGMII.TXD0: track 0.00 -> 12.6 mm, vias 0 -> 2
- net /4Port_T1_switch/RGMII.TXD1: track 0.00 -> 12.3 mm, vias 0 -> 2
- net /4Port_T1_switch/RGMII.RXD1: track 0.00 -> 12.3 mm
- net /4Port_T1_switch/RGMII.RX_CLK: track 0.00 -> 12.2 mm, vias 0 -> 2
- net /4Port_T1_switch/RGMII.RXD0: track 0.00 -> 11.6 mm
