File: HW/LED_Dimmer/LedDimmer/LedDimmer.kicad_pcb (KiCad board)
At the start: 2 copper layers, 40 x 50 mm, 48 parts, among them J1 Screw_Terminal_01x03, J2 Screw_Terminal_01x02, J3 Screw_Terminal_01x03, J4 Screw_Terminal_01x03, J5 Screw_Terminal_01x03, J6 Screw_Terminal_01x02, Q1 SSM3J133TU, Q2 BSS138, Q3 BSS138, Q4 SSM3J133TU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

Commit message: .
Parts:
- added C14: 10u 50V, Capacitor_SMD:C_0805_2012Metric, F.Cu at (47.4, 70.0)
- C1: value 22u 100V -> 10u 50V; footprint Capacitor_SMD:CP_Elec_8x10.5 -> Capacitor_SMD:C_0805_2012Metric
- moved C2 6.92 mm to (51.2, 70.5), turned to 90 degrees
- moved C10 4.82 mm to (68.4, 91.0)
- moved H1 4.76 mm to (75.4, 62.0)
- moved H4 4.76 mm to (40.4, 62.0)
- moved C9 4.24 mm to (68.4, 81.7)
- moved L1 4.01 mm to (59.4, 71.0)
- moved R4 4.01 mm to (68.1, 64.1)
- moved C3 4.01 mm to (66.7, 71.9)
- moved C4 4.01 mm to (68.3, 71.9)
- moved C6 4.01 mm to (68.2, 68.9)
- moved C7 4.01 mm to (66.7, 68.9)
- moved R2 4.01 mm to (69.8, 68.9)
- moved R3 4.01 mm to (69.1, 66.5)
- moved C5 4.01 mm to (53.9, 64.9)
- moved U1 4.01 mm to (51.8, 67.1)
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Routing:
- net /FB: track 0.00 -> 23.6 mm, vias 0 -> 2
- net +3.3V: track 8.70 -> 32.1 mm
- net GND: track 0.44 -> 21.7 mm, vias 0 -> 87
- net /CH1: track 0.00 -> 14.3 mm
- net /VIN: track 0.00 -> 11.8 mm
- net /CH2: track 0.00 -> 11.3 mm
- net Net-(U1-SW): track 0.00 -> 10.1 mm
- net Net-(D2-K): track 0.00 -> 6.78 mm
- net Net-(D6-K): track 0.00 -> 6.55 mm
- net Net-(J6-Pin_2): track 0.00 -> 6.29 mm
- net Net-(D5-K): track 0.00 -> 5.62 mm
- net Net-(D3-K): track 0.00 -> 5.61 mm
- net Net-(J1-Pin_1): track 0.00 -> 5.22 mm
- net Net-(J3-Pin_1): track 0.00 -> 5.00 mm
- net /PWR: track 0.00 -> 3.84 mm
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- added copper zone on F.Cu, net +3.3V
- added copper zone on B.Cu, net GND
- added copper zone on F.Cu, net GND
Other:
- board size 40 x 50 mm -> 40 x 45 mm
- board text added: "+5-12V GND"
- board text added: "AI1 V S G"
- board text added: "AI2 V S G"
- board text added: "Ch1 V S G"
- board text added: "Ch2 V S G"
- board text added: "Dx S G"
- board text added: "PWM-board Björn Thor (c) 2025"

Commit message: .
Parts:
- added R18: 10K, Resistor_SMD:R_0603_1608Metric, F.Cu at (55.6, 89.3)
- added R19: 10K, Resistor_SMD:R_0603_1608Metric, F.Cu at (55.6, 86.3)
- added R20: 10K, Resistor_SMD:R_0603_1608Metric, F.Cu at (54.1, 93.0)
- added R21: 10K, Resistor_SMD:R_0603_1608Metric, F.Cu at (55.7, 93.0)
- moved C10 5.19 mm to (71.7, 87.0), turned to 180 degrees
- moved C9 3.84 mm to (72.1, 80.6), turned to 180 degrees
Connections:
- net Net-(U2-RA3) renamed /RST#
Routing:
- net +3.3V: track 32.1 -> 42.8 mm
- net GND: track 21.7 -> 28.3 mm
- net /CH1: track 14.3 -> 15.1 mm
- net /AN0: track 15.3 -> 15.8 mm, vias 0 -> 2
- net /AN1: track 10.6 -> 10.9 mm, vias 0 -> 2
- net Net-(J6-Pin_2): vias 0 -> 1

Commit message: .
Parts:
- added Q5: BSS138, Package_TO_SOT_SMD:SOT-23, F.Cu at (52.2, 81.7)
- added Q6: BSS138, Package_TO_SOT_SMD:SOT-23, F.Cu at (52.0, 91.3)
- R6, R8: value 24R -> 56R
- moved R18 7.44 mm to (55.1, 81.9), turned to 90 degrees
- moved R19 4.54 mm to (56.7, 81.9)
- moved R6 3.11 mm to (47.9, 79.1), turned to 0 degrees
- moved D3 3.09 mm to (51.0, 79.1), turned to 180 degrees
- moved D5 3.03 mm to (50.7, 88.7), turned to 180 degrees
- moved R8 2.95 mm to (47.7, 88.7), turned to 0 degrees
- moved R20 2.27 mm to (56.4, 93.1)
- moved R21 0.91 mm to (54.8, 93.1)
Connections:
- Q1 pad 1: Net-(D3-K) -> Net-(Q1-G)
- Q2 pad 3: Net-(D3-K) -> Net-(Q1-G)
- Q3 pad 3: Net-(D5-K) -> Net-(Q3-D)
- Q4 pad 1: Net-(D5-K) -> Net-(Q3-D)
- R5 pad 2: Net-(D3-K) -> Net-(Q1-G)
- R9 pad 2: Net-(D5-K) -> Net-(Q3-D)
Routing:
- net GND: track 28.3 -> 32.7 mm, vias 87 -> 89
- net Net-(Q3-D): track 0.00 -> 4.14 mm
- net Net-(Q1-G): track 0.00 -> 4.14 mm
- net Net-(D5-K): track 5.62 -> 2.77 mm
- net Net-(D3-K): track 5.61 -> 2.78 mm
- net /CH1: track 15.1 -> 17.5 mm

Commit message: .
Parts:
- added TP1: TestPoint, TestPoint:TestPoint_THTPad_D1.0mm_Drill0.5mm, F.Cu at (67.9, 88.9)
- added TP2: TestPoint, TestPoint:TestPoint_THTPad_D1.0mm_Drill0.5mm, F.Cu at (67.9, 90.9)
- added TP3: TestPoint, TestPoint:TestPoint_THTPad_D1.0mm_Drill0.5mm, F.Cu at (67.9, 92.9)
- added TP4: TestPoint, TestPoint:TestPoint_THTPad_D1.0mm_Drill0.5mm, F.Cu at (58.7, 95.1)
- added TP5: TestPoint, TestPoint:TestPoint_THTPad_D1.0mm_Drill0.5mm, F.Cu at (56.1, 90.4)
- added TP6: TestPoint, TestPoint:TestPoint_THTPad_D1.0mm_Drill0.5mm, F.Cu at (57.3, 88.7)
- added TP7: TestPoint, TestPoint:TestPoint_THTPad_D1.0mm_Drill0.5mm, F.Cu at (62.8, 98.1)
- added TP8: TestPoint, TestPoint:TestPoint_THTPad_D1.0mm_Drill0.5mm, F.Cu at (65.0, 98.1)
- added U4: TPV809R-3TR, Package_TO_SOT_SMD:SOT-23-3, F.Cu at (53.3, 86.1)
- added U5: TPV809R-3TR, Package_TO_SOT_SMD:SOT-23-3, F.Cu at (59.4, 80.2)
- moved R8 5.03 mm to (52.8, 88.7), turned to 180 degrees
- moved R6 4.84 mm to (52.8, 79.1), turned to 180 degrees
- moved D3 3.09 mm to (47.9, 79.1), turned to 0 degrees
- moved D5 3.00 mm to (47.7, 88.7), turned to 0 degrees
Connections:
- D3 pad 1: Net-(D3-K) -> GND
- D3 pad 2: Net-(D3-A) -> /CH1_SW
- D5 pad 1: Net-(D5-K) -> GND
- D5 pad 2: Net-(D5-A) -> /CH2_SW
- Q2 pad 1: /CH1 -> /CH1_SW
- Q3 pad 1: /CH2 -> /CH2_SW
- Q5 pad 3: Net-(D3-K) -> /CH1_SW
- Q6 pad 3: Net-(D5-K) -> /CH2_SW
- R6 pad 1: +3.3V -> Net-(U5-RST#)
- R6 pad 2: Net-(D3-A) -> /CH1_SW
- R8 pad 1: +3.3V -> Net-(U4-RST#)
- R8 pad 2: Net-(D5-A) -> /CH2_SW
Routing:
- net /CH2_SW: track 0.00 -> 8.82 mm
- net /CH1_SW: track 0.00 -> 8.49 mm
- net +3.3V: track 42.8 -> 51.1 mm
- net GND: track 32.7 -> 39.8 mm, vias 89 -> 91
- net Net-(U5-RST#): track 0.00 -> 4.92 mm
- net Net-(D3-K): track 2.78 -> 0.00 mm
- net Net-(D5-K): track 2.77 -> 0.00 mm
- net /CH1: track 17.5 -> 14.8 mm, vias 0 -> 1
- net /DI1: track 5.10 -> 7.53 mm
- net Net-(U4-RST#): track 0.00 -> 2.24 mm
- net /CH2: track 11.4 -> 9.49 mm
- net /RST#: track 1.83 -> 3.74 mm
- net Net-(D3-A): track 1.49 -> 0.00 mm
- net Net-(D5-A): track 1.38 -> 0.00 mm
- net /AN0: track 15.8 -> 14.9 mm, vias 2 -> 1
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
Commit message: .
Parts:
- removed R19, R20: 10K, Resistor_SMD:R_0603_1608Metric
- removed U4, U5: TPV809R-3TR, Package_TO_SOT_SMD:SOT-23-3
- added C15: 100n 25V, Capacitor_SMD:C_0603_1608Metric, F.Cu at (55.8, 79.6)
- added C16: 100n 25V, Capacitor_SMD:C_0603_1608Metric, F.Cu at (55.1, 89.5)
- Q5, Q6: value BSS138 -> BVSS84LT1G
- moved D4 23.8 mm to (75.6, 66.4), turned to -90 degrees
- moved R7 22.3 mm to (75.6, 69.5), turned to 90 degrees
- moved TP8 7.97 mm to (57.7, 94.9)
- moved TP7 5.24 mm to (57.7, 96.9)
- moved TP4 2.42 mm to (57.7, 92.9)
- moved TP5 1.68 mm to (57.7, 90.9)
- moved C9 1.30 mm to (72.1, 81.9)
- moved R10 1.30 mm to (72.1, 80.3)
- moved TP6 0.45 mm to (57.7, 88.9)
- moved J5 0.33 mm to (75.7, 88.3)
- moved TP1 0.20 mm to (67.7, 88.9)
- moved TP2 0.20 mm to (67.7, 90.9)
- moved TP3 0.20 mm to (67.7, 92.9)
Connections:
- D3 pad 1: GND -> /CH1_LED
- D3 pad 2: /CH1_SW -> Net-(D3-A)
- D5 pad 1: GND -> /CH2_LED
- D5 pad 2: /CH2_SW -> Net-(D5-A)
- Q2 pad 1: /CH1_SW -> /CH1
- Q3 pad 1: /CH2_SW -> /CH2
- Q5 pad 2: GND -> /CH1_LED
- Q5 pad 3: /CH1_SW -> GND
- Q6 pad 2: GND -> /CH2_LED
- Q6 pad 3: /CH2_SW -> GND
- R6 pad 1: Net-(U5-RST#) -> +3.3V
- R6 pad 2: /CH1_SW -> Net-(D3-A)
- R8 pad 1: Net-(U4-RST#) -> +3.3V
- R8 pad 2: /CH2_SW -> Net-(D5-A)
Routing:
- net /CH2_SW: track 8.82 -> 0.00 mm
- net /CH1_SW: track 8.49 -> 0.00 mm
- net /CH1_LED: track 0.00 -> 6.82 mm
- net /CH2_LED: track 0.00 -> 6.77 mm
- net Net-(U5-RST#): track 4.92 -> 0.00 mm
- net Net-(D5-A): track 0.00 -> 3.42 mm
- net Net-(D3-A): track 0.00 -> 3.21 mm
- net /CH2: track 9.49 -> 12.2 mm
- net /CH1: track 14.8 -> 17.2 mm, vias 1 -> 0
- net Net-(U4-RST#): track 2.24 -> 0.00 mm
- net GND: track 39.8 -> 41.3 mm, vias 91 -> 87
- net +3.3V: track 51.1 -> 52.4 mm
- net Net-(J4-Pin_2): track 3.74 -> 4.76 mm
- net /RST#: track 3.74 -> 4.74 mm
- net /AN0: track 14.9 -> 14.3 mm
Other:
- board text added: "Power LED"
