File: HW/LED_Dimmer/LedDimmer/LedDimmer.kicad_pcb (KiCad board)
At the start: 2 copper layers, 40 x 45 mm, 64 parts, among them J1 Screw_Terminal_01x03, J2 Screw_Terminal_01x02, J3 Screw_Terminal_01x03, J4 Screw_Terminal_01x03, J5 Screw_Terminal_01x03, J6 Screw_Terminal_01x02, Q1 SSM3J133TU, Q2 BSS138, Q3 BSS138, Q4 SSM3J133TU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

Commit message: .
Parts:
- added FID1: Fiducial_05_1, Fiducial:Fiducial_0.5mm_Mask1mm, F.Cu at (44.4, 61.8)
- added FID2: Fiducial_05_1, Fiducial:Fiducial_0.5mm_Mask1mm, F.Cu at (46.2, 101.6)
- added FID3: Fiducial_05_1, Fiducial:Fiducial_0.5mm_Mask1mm, F.Cu at (70.3, 101.9)

Commit message: .
Parts:
- C4, C7: value 4u7 10V -> 10u 50V
- R1: value 100K -> 130K
- R10, R11, R12, R14, R3: value 5K0 -> 5K1
- R6, R8: value 56R -> 24R
Changed lines of the file:
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@@
 		(sheetname "Root")
 		(sheetfile "LedDimmer.kicad_sch")
-		(attr smd dnp)
+		(attr smd)
 		(fp_line
 			(start -0.602064 -1.36)
@@
 			)
 		)
-		(property "Value" "56R"
+		(property "Value" "24R"
 			(at 0 1.43 0)
 			(layer "F.Fab")
@@
 			)
 		)
-		(property "CPN" "BT00002-00560"
+		(property "CPN" "BT00002-00240"
 			(at 0 0 180)
 			(unlocked yes)
@@
 			)
 		)
-		(property "Value" "5K0"
+		(property "Value" "5K1"
 			(at 0 1.43 0)
 			(layer "F.Fab")
@@
 			)
 		)
-		(property "MPN" "R;G;T1;S;P0603;NA"
+		(property "MPN" "R;G;5K1;S;P0603;NA"
 			(at 0 0 180)
 			(unlocked yes)
@@
 			)
 		)
-		(property "CPN" "BT00002-30050"
+		(property "CPN" "BT00002-30051"
 			(at 0 0 180)
 			(unlocked yes)
@@
 			)
 		)
-		(property "Value" "5K0"
+		(property "Value" "5K1"
 			(at 0 1.43 0)
 			(layer "F.Fab")
@@
 			)
 		)
-		(property "MPN" "R;G;T1;S;P0603;NA"
+		(property "MPN" "R;G;5K1;S;P0603;NA"
 			(at 0 0 180)
 			(unlocked yes)
@@
 			)
 		)
-		(property "CPN" "BT00002-30050"
+		(property "CPN" "BT00002-30051"
 			(at 0 0 180)
 			(unlocked yes)
@@
 			)
 		)
-		(property "Value" "100K"
+		(property "Value" "130K"
 			(at 0 1.43 90)
 			(layer "F.Fab")
@@
 			)
 		)
-		(property "CPN" "BT00002-31000"
+		(property "CPN" "BT00002-31300"
 			(at 0 0 90)
 			(unlocked yes)
@@
 		(sheetname "Root")
 		(sheetfile "LedDimmer.kicad_sch")
-		(attr smd)
+		(attr smd dnp)
 		(fp_line
 			(start -5.76 -5.26)
@@
 			)
 		)
-		(property "Value" "4u7 10V"
+		(property "Value" "10u 50V"
 			(at 0 1.43 90)
 			(layer "F.Fab")
@@
 			)
 		)
-		(property "MPN" "C;C;T1;S;P0603;NA"
+		(property "MPN" "C;M;10u;10p;50V;S;0603"
 			(at 0 0 90)
 			(unlocked yes)
@@
 			)
 		)
-		(property "CPN" "BT00010-060047"
+		(property "CPN" "BT00007-060100"
 			(at 0 0 90)
 			(unlocked yes)
@@
 			)
 		)
-		(property "Value" "56R"
+		(property "Value" "24R"
 			(at 0 1.43 0)
 			(layer "F.Fab")
@@
 			)
 		)
-		(property "CPN" "BT00002-00560"
+		(property "CPN" "BT00002-00240"
 			(at 0 0 180)
 			(unlocked yes)
@@
 			)
 		)
-		(property "Value" "5K0"
+		(property "Value" "5K1"
 			(at 0 1.43 0)
 			(layer "F.Fab")
@@
 			)
 		)
-		(property "MPN" "R;G;T1;S;P0603;NA"
+		(property "MPN" "R;G;5K1;S;P0603;NA"
 			(at 0 0 180)
 			(unlocked yes)
@@
 			)
 		)
-		(property "CPN" "BT00002-30050"
+		(property "CPN" "BT00002-30051"
 			(at 0 0 180)
 			(unlocked yes)
@@
 			)
 		)
-		(property "Value" "4u7 10V"
+		(property "Value" "10u 50V"
 			(at 0 1.43 90)
 			(layer "F.Fab")
@@
 			)
 		)
-		(property "MPN" "C;C;T1;S;P0603;NA"
+		(property "MPN" "C;M;10u;10p;50V;S;0603"
 			(at 0 0 -90)
 			(unlocked yes)
@@
 			)
 		)
-		(property "CPN" "BT00010-060047"
+		(property "CPN" "BT00007-060100"
 			(at 0 0 -90)
 			(unlocked yes)
@@
 			)
 		)
-		(property "Value" "5K0"
+		(property "Value" "5K1"
 			(at 0 1.43 0)
 			(layer "F.Fab")
@@
 			)
 		)
-		(property "MPN" "R;G;T1;S;P0603;NA"
+		(property "MPN" "R;G;5K1;S;P0603;NA"
 			(at 0 0 180)
 			(unlocked yes)
@@
 			)
 		)
-		(property "CPN" "BT00002-30050"
+		(property "CPN" "BT00002-30051"
 			(at 0 0 180)
 			(unlocked yes)
@@
 			)
 		)
-		(property "Value" "5K0"
+		(property "Value" "5K1"
 			(at 0 1.43 0)
 			(layer "F.Fab")
@@
 			)
 		)
-		(property "MPN" "R;G;T1;S;P0603;NA"
+		(property "MPN" "R;G;5K1;S;P0603;NA"
 			(at 0 0 180)
 			(unlocked yes)
@@
 			)
 		)
-		(property "CPN" "BT00002-30050"
+		(property "CPN" "BT00002-30051"
 			(at 0 0 180)
 			(unlocked yes)
