File: HW/LED_Dimmer/LedDimmer/LedDimmer.kicad_sch (KiCad schematic)
At the start: 48 parts, among them J1 Screw_Terminal_01x03, J2 Screw_Terminal_01x02, J3 Screw_Terminal_01x03, J4 Screw_Terminal_01x03, J5 Screw_Terminal_01x03, J6 Screw_Terminal_01x02, Q1 SSM3J133TU, Q2 BSS138, Q3 BSS138, Q4 SSM3J133TU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

Commit message: .
Parts:
- removed C1: 22u 100V, Capacitor_SMD:CP_Elec_8x10.5, symbol bt_capacitor:C;E;22u;10p;100V;S;8x10.5
- added C1, C14: 10u 50V, Capacitor_SMD:C_0805_2012Metric, symbol bt_capacitor:C;M;10u;10p;50V;S;0805
- added C12: 4u7 10V, Capacitor_SMD:C_0603_1608Metric, symbol bt_capacitor:C;M;4u7;10p;10V;S;0603
- added C13: 22u 100V, Capacitor_SMD:CP_Elec_8x10.5, symbol bt_capacitor:C;E;22u;10p;100V;S;8x10.5
- added L2: 2.2uH 1.4A, bt_footprints:L_0806_2016Metric, symbol bt_Inductors:L;2.2uH;1.4A;S;0806
- added R15: 0R, Resistor_SMD:R_0603_1608Metric, symbol bt_resistors:R;G;0R;10P0;S;0603
- added R16: 150K, Resistor_SMD:R_0603_1608Metric, symbol bt_resistors:R;G;150K;10P0;S;0603
- added R17: 33K, Resistor_SMD:R_0603_1608Metric, symbol bt_resistors:R;G;33K;10P0;S;0603
- added U3: TPS629203-Q1, Package_TO_SOT_SMD:SOT-583-8, symbol bt_power:TPS629203-Q1
Connections:
- net +3.3V: now also C12.1, L2.2, R16.1, U3.3 (VOS)
- net GND: now also C1.2, C12.2, C13.2, C14.2, R15.2, R17.2
- net VIN: now also C1.1, C13.1, C14.1, U3.6 (VIN), U3.7 (EN)
- new net: R16.2, R17.1, U3.1 (FB)
- new net: L2.1, U3.4 (SW)
- new net: R15.1, U3.8 (MODE)
Other:
- moved on the sheet: D1

Commit message: .
Parts:
- added R18, R19, R20, R21: 10K, Resistor_SMD:R_0603_1608Metric, symbol bt_resistors:R;G;10K;10P0;S;0603
Connections:
- net +3.3V: now also R19.1, R20.1
- net CH1: now also R18.1, R19.2
- net CH2: now also R20.2, R21.1
- net GND: now also U3.5 (GND), R18.2, R21.2
- net RST#: now reaches R14.2, U2.4 (RA3)
- net at U3.8 (MODE): now also R15.1
- no-connect marks 0 -> 1

Commit message: .
Parts:
- added Q5, Q6: BSS138, Package_TO_SOT_SMD:SOT-23, symbol bt_transistor:T;Mn;BSS138;SOT23
- R6, R8: value 24R -> 56R; symbol bt_resistors:R;G;24R;10P0;S;0603 -> bt_resistors:R;G;56R;10P0;S;0603; CPN BT00002-00240 -> BT00002-00560
Connections:
- net CH1: now also Q5.1 (G)
- net CH2: now also Q6.1 (G)
- net GND: now also Q5.2 (S), Q6.2 (S)
- net at Q3.3 (D), Q4.1 (G), R9.2: no longer D5.1 (K)
- net at Q1.1 (G), Q2.3 (D), R5.2: no longer D3.1 (K)
- new net: D3.1 (K), Q5.3 (D)
- new net: D5.1 (K), Q6.3 (D)
Other:
- moved on the sheet: D2, D3, D5, D6, J1, J3, Q1, Q2, Q3, Q4, R18, R19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

Commit message: .
Parts:
- added R22, R23: 0R, Resistor_SMD:R_0603_1608Metric, symbol bt_resistors:R;G;0R;10P0;S;0603
- added TP1, TP2, TP3, TP4, TP5, TP6, TP7, TP8: TestPoint, TestPoint:TestPoint_THTPad_D1.0mm_Drill0.5mm, symbol bt_misc:TestPoint_THD
- added U4, U5: TPV809R-3TR, Package_TO_SOT_SMD:SOT-23-3, symbol bt_power:TPV809R-3TR
Connections:
- net +3.3V: now also TP7.1, U4.3 (VCC), U5.3 (VCC); no longer R6.1, R8.1
- net AN0: now also TP1.1
- net AN1: now also TP2.1
- net CH1: now also R22.1, TP6.1; no longer Q2.1 (G)
- net CH2: now also R23.1, TP5.1; no longer Q3.1 (G)
- net DI1: now also TP3.1
- net GND: now also D3.1 (K), D5.1 (K), TP8.1, U4.1 (GND), U5.1 (GND)
- net RST#: now also TP4.1
- net CH1_SW: now reaches Q5.3 (D)
- net CH1_SW: now also D3.2 (A), Q2.1 (G), R6.2, R22.2; no longer D3.1 (K)
- net CH2_SW: now reaches Q6.3 (D)
- net CH2_SW: now also D5.2 (A), Q3.1 (G), R8.2, R23.2; no longer D5.1 (K)
- new net: R6.1, U5.2 (RST#)
- new net: R8.1, U4.2 (RST#)
Other:
- note added: "Not used and excluded from PCB and BOM"
- moved on the sheet: C12, C13, C8, D3, D5, L2, Q5, Q6, R14, R15, R16, R17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

Commit message: .
Parts:
- removed Q5, Q6: BSS138, Package_TO_SOT_SMD:SOT-23, symbol bt_transistor:T;Mn;BSS138;SOT23
- removed R19, R20: 10K, Resistor_SMD:R_0603_1608Metric, symbol bt_resistors:R;G;10K;10P0;S;0603
- removed R22, R23: 0R, Resistor_SMD:R_0603_1608Metric, symbol bt_resistors:R;G;0R;10P0;S;0603
- removed U4, U5: TPV809R-3TR, Package_TO_SOT_SMD:SOT-23-3, symbol bt_power:TPV809R-3TR
- added C15, C16: 100n 25V, Capacitor_SMD:C_0603_1608Metric, symbol bt_capacitor:C;M;100n;10p;25V;S;0603
- added Q5, Q6: BVSS84LT1G, Package_TO_SOT_SMD:SOT-23, symbol bt_transistor:T;Mp;BVSS84LT1G;SOT23-3
- Q1, Q4: symbol bt_transistor:T;Np;SSM3J133TU;SOT323F -> bt_transistor:T;Mp;SSM3J133TU;SOT323F
Connections:
- net +3.3V: now also R6.1, R8.1, C15.2, C16.2
- net CH1: now also Q2.1 (G), Q5.1 (G)
- net CH2: now also Q3.1 (G), Q6.1 (G)
- net GND: now also C15.1, C16.1, Q5.3 (D), Q6.3 (D); no longer D3.1 (K), D5.1 (K)
- net CH1_SW: no longer names the net of D3.2 (A), R6.2
- net CH1_SW: no longer Q2.1 (G)
- net CH2_SW: no longer names the net of D5.2 (A), R8.2
- net CH2_SW: no longer Q3.1 (G)
- new net CH1_LED: D3.1 (K), Q5.2 (S)
- new net CH2_LED: D5.1 (K), Q6.2 (S)
Other:
- moved on the sheet: D3, D5, R6, R8, TP7
