File: HW/LED_Dimmer/LedDimmer/LedDimmer.kicad_sch (KiCad schematic)
At the start: 74 parts, among them J1 Screw_Terminal_01x03, J2 Screw_Terminal_01x02, J3 Screw_Terminal_01x03, J4 Screw_Terminal_01x03, J5 Screw_Terminal_01x03, J6 Screw_Terminal_01x02, Q1 SSM3J133TU, Q2 BSS138, Q3 BSS138, Q4 SSM3J133TU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

Commit message: .
Parts:
- C12: now in the parts list
- C4, C7: value 4u7 10V -> 10u 50V; symbol bt_capacitor:C;M;4u7;10p;10V;S;0603 -> bt_capacitor:C;M;10u;10p;50V;S;0603; CPN BT00010-060047 -> BT00007-060100; MPN C;C;T1;S;P0603;NA -> C;M;10u;10p;50V;S;0603
- L1: now not fitted
- L3: now fitted
- R1: value 100K -> 130K; symbol bt_resistors:R;G;100K;10P0;S;0603 -> bt_resistors:R;G;130K;10P0;S;0603; CPN BT00002-31000 -> BT00002-31300
- R10, R11, R12, R14, R3: value 5K0 -> 5K1; symbol bt_resistors:R;G;5K0;10P0;S;0603 -> bt_resistors:R;G;5K1;10P0;S;0603; CPN BT00002-30050 -> BT00002-30051; MPN R;G;T1;S;P0603;NA -> R;G;5K1;S;P0603;NA
- R6, R8: value 56R -> 24R; symbol bt_resistors:R;G;56R;10P0;S;0603 -> bt_resistors:R;G;24R;10P0;S;0603; CPN BT00002-00560 -> BT00002-00240
Other:
- note added: "2025-07-11:schamatic updated with mountet values"
- moved on the sheet: C1

Commit message: .
Parts:
- C10, C9: now not fitted
Other:
- note added: "ICSP pins: 4 : VPP 1 : VDD (3.3V) 8 : VSS (GND) 7 : ICSPData 6 : ICSPCLK"
Changed lines of the file:
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@@
 		)
 	)
+	(text "ICSP pins:\n4 : VPP\n1 : VDD (3.3V)\n8 : VSS (GND)\n7 : ICSPData\n6 : ICSPCLK"
+		(exclude_from_sim no)
+		(at 164.592 149.098 0)
+		(effects
+			(font
+				(size 1.27 1.27)
+			)
+			(justify left)
+		)
+	)
 	(text "2025-07-11:schamatic updated with mountet values"
 		(exclude_from_sim no)
@@
 		(in_bom yes)
 		(on_board yes)
-		(dnp no)
+		(dnp yes)
 		(fields_autoplaced yes)
 		(property "Reference" "C9"
@@
 		(in_bom yes)
 		(on_board yes)
-		(dnp no)
+		(dnp yes)
 		(fields_autoplaced yes)
 		(property "Reference" "C10"
